File: kicad/highspeed.kicad_sch (KiCad schematic)
At the start: 44 parts, among them J60 SFP cage 0, J61 SFP cage 1, J62 SFP cage 2, J63 SFP cage 3, Q1 SFP power gate, U17 PCF8574T, X2 125MHz LVDS

Commit message: power input: single USB-C with CH224K PD sink at 9V, Schottky OR-ing, degraded 5V mode; record missing board-ID pins
Parts:
- removed C124: 100nF, Capacitor_SMD:C_0402_1005Metric, symbol Device:C
- removed R40: 4.7k, Resistor_SMD:R_0402_1005Metric, symbol Device:R
- added C150: 100nF, Capacitor_SMD:C_0402_1005Metric, symbol Device:C
- added R29: 100, Resistor_SMD:R_0603_1608Metric, symbol Device:R
- C125: value 4.7uF -> 100nF; footprint Capacitor_SMD:C_0603_1608Metric -> Capacitor_SMD:C_0402_1005Metric
- C126: value 100nF -> 4.7uF; footprint Capacitor_SMD:C_0402_1005Metric -> Capacitor_SMD:C_0603_1608Metric
- C128: value 10uF -> 100nF; footprint Capacitor_SMD:C_0805_2012Metric -> Capacitor_SMD:C_0402_1005Metric
- C129: value 100nF -> 10uF; footprint Capacitor_SMD:C_0402_1005Metric -> Capacitor_SMD:C_0805_2012Metric
- R30: value 100 -> 100k; footprint Resistor_SMD:R_0603_1608Metric -> Resistor_SMD:R_0402_1005Metric
- R31: value 100k -> 4.7k
Connections:
- net +3V3: now also C126.1, R30.1, C150.1; no longer C149.1
- net EN_SFP_N: now also R30.2; no longer R31.2
- net GND: now also C126.2, C129.2, C134.2, C139.2, C144.2, C150.2, R29.2; no longer C128.2, C133.2, C138.2, C143.2, C148.2, R30.2
- net MGTPRXN0: now also C133.2; no longer C132.2
- net MGTPRXN1: now also C138.2; no longer C137.2
- net MGTPRXN2: now also C143.2; no longer C142.2
- net MGTPRXN3: now also C148.2; no longer C147.2
- net MGTPRXP0: now also C132.2; no longer C131.2
- net MGTPRXP1: now also C137.2; no longer C136.2
- net MGTPRXP2: now also C142.2; no longer C141.2
- net MGTPRXP3: now also C147.2; no longer C146.2
- net MGTPTXN0: now also C131.1; no longer C130.1
- net MGTPTXN1: now also C136.1; no longer C135.1
- net MGTPTXN2: now also C141.1; no longer C140.1
- net MGTPTXN3: now also C146.1; no longer C145.1
- net MGTPTXP0: now also C130.1; no longer C129.1
- net MGTPTXP1: now also C135.1; no longer C134.1
- net MGTPTXP2: now also C140.1; no longer C139.1
- net MGTPTXP3: now also C145.1; no longer C144.1
- net MGTREFCLK0N: now also C128.2; no longer C127.2
- net MGTREFCLK0P: now also C127.2; no longer C126.2
- net MGTRREF: now also R29.1; no longer R30.1
- net REFCLK_OSC_N: now also C128.1; no longer C127.1
- net REFCLK_OSC_P: now also C127.1; no longer C126.1
- net SFP0_LOS: now also R35.2; no longer R36.2
- net SFP0_MOD_ABS: now also R33.2; no longer R34.2
- net SFP0_RD_N: now also C133.1; no longer C132.1
- net SFP0_RD_P: now also C132.1; no longer C131.1
- net SFP0_TD_N: now also C131.2; no longer C130.2
- net SFP0_TD_P: now also C130.2; no longer C129.2
- net SFP0_TX_FAULT: now also R34.2; no longer R35.2
- net SFP1_LOS: now also R38.2; no longer R39.2
- net SFP1_MOD_ABS: now also R36.2; no longer R37.2
- net SFP1_RD_N: now also C138.1; no longer C137.1
- net SFP1_RD_P: now also C137.1; no longer C136.1
- net SFP1_TD_N: now also C136.2; no longer C135.2
- net SFP1_TD_P: now also C135.2; no longer C134.2
- net SFP1_TX_FAULT: now also R37.2; no longer R38.2
- net SFP2_RD_N: now also C143.1; no longer C142.1
- net SFP2_RD_P: now also C142.1; no longer C141.1
- net SFP2_TD_N: now also C141.2; no longer C140.2
- net SFP2_TD_P: now also C140.2; no longer C139.2
- net SFP3_RD_N: now also C148.1; no longer C147.1
- net SFP3_RD_P: now also C147.1; no longer C146.1
- net SFP3_TD_N: now also C146.2; no longer C145.2
- net SFP3_TD_P: now also C145.2; no longer C144.2
- net SFP_EXP_INT: now also R39.2
- net SFP_SCL: now also R31.2; no longer R32.2
- net SFP_SDA: now also R32.2; no longer R33.2
- net SFP_VCC: now also C129.1, C134.1, C139.1, C144.1, C149.1; no longer C128.1, C133.1, C138.1, C143.1, C148.1
Other:
- moved on the sheet: C125, C126, C127, C128, C129, C130, C131, C132, C133, C134, C135, C136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

Commit message: supervisor flash: document the role, add BOOTSEL series resistor
Parts:
- removed R29: 100, Resistor_SMD:R_0603_1608Metric, symbol Device:R
- added R40: 4.7k, Resistor_SMD:R_0402_1005Metric, symbol Device:R
- R30: value 100k -> 100; footprint Resistor_SMD:R_0402_1005Metric -> Resistor_SMD:R_0603_1608Metric
- R31: value 4.7k -> 100k
Connections:
- net +3V3: now also R40.1; no longer R30.1
- net EN_SFP_N: now also R31.2; no longer R30.2
- net GND: now also R30.2
- net MGTRREF: now also R30.1
- net SFP0_LOS: now also R36.2; no longer R35.2
- net SFP0_MOD_ABS: now also R34.2; no longer R33.2
- net SFP0_TX_FAULT: now also R35.2; no longer R34.2
- net SFP1_LOS: now also R39.2; no longer R38.2
- net SFP1_MOD_ABS: now also R37.2; no longer R36.2
- net SFP1_TX_FAULT: now also R38.2; no longer R37.2
- net SFP_EXP_INT: now also R40.2; no longer R39.2
- net SFP_SCL: now also R32.2; no longer R31.2
- net SFP_SDA: now also R33.2; no longer R32.2
Other:
- moved on the sheet: R30, R31, R32, R33, R34, R35, R36, R37, R38, R39
Changed lines of the file:
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@@
 	(symbol (lib_id "Device:R") (at 55.88 119.38 0) (unit 1)
 		(exclude_from_sim no) (in_bom yes) (on_board yes) (dnp no)
-		(property "Reference" "R29" (at 55.88 111.76 0) (effects (font (size 1.27 1.27))))
+		(property "Reference" "R30" (at 55.88 111.76 0) (effects (font (size 1.27 1.27))))
 		(property "Value" "100" (at 55.88 127.0 0) (effects (font (size 1.27 1.27))))
 		(property "Footprint" "Resistor_SMD:R_0603_1608Metric" (at 55.88 127.0 0) (effects (font (size 1.27 1.27)) (hide yes)))
-		(instances (project "odin" (path "/c44fb7fe-6133-ad34-68fd-fb66126197ef/e9248ad1-6b14-c545-7edc-53de7184d0bd" (reference "R29") (unit 1))))
+		(instances (project "odin" (path "/c44fb7fe-6133-ad34-68fd-fb66126197ef/e9248ad1-6b14-c545-7edc-53de7184d0bd" (reference "R30") (unit 1))))
 	)
 	(wire (pts (xy 55.88 115.57) (xy 55.88 113.03)) (stroke (width 0) (type default)))
@@
 	(symbol (lib_id "Device:R") (at 250.19 72.39 0) (unit 1)
 		(exclude_from_sim no) (in_bom yes) (on_board yes) (dnp no)
-		(property "Reference" "R30" (at 250.19 64.77 0) (effects (font (size 1.27 1.27))))
+		(property "Reference" "R31" (at 250.19 64.77 0) (effects (font (size 1.27 1.27))))
 		(property "Value" "100k" (at 250.19 80.01 0) (effects (font (size 1.27 1.27))))
 		(property "Footprint" "Resistor_SMD:R_0402_1005Metric" (at 250.19 80.01 0) (effects (font (size 1.27 1.27)) (hide yes)))
-		(instances (project "odin" (path "/c44fb7fe-6133-ad34-68fd-fb66126197ef/e9248ad1-6b14-c545-7edc-53de7184d0bd" (reference "R30") (unit 1))))
+		(instances (project "odin" (path "/c44fb7fe-6133-ad34-68fd-fb66126197ef/e9248ad1-6b14-c545-7edc-53de7184d0bd" (reference "R31") (unit 1))))
 	)
 	(wire (pts (xy 250.19 68.58) (xy 250.19 66.04)) (stroke (width 0) (type default)))
@@
 	(symbol (lib_id "Device:R") (at 55.88 195.58 0) (unit 1)
 		(exclude_from_sim no) (in_bom yes) (on_board yes) (dnp no)
-		(property "Reference" "R31" (at 55.88 187.96 0) (effects (font (size 1.27 1.27))))
+		(property "Reference" "R32" (at 55.88 187.96 0) (effects (font (size 1.27 1.27))))
 		(property "Value" "4.7k" (at 55.88 203.2 0) (effects (font (size 1.27 1.27))))
 		(property "Footprint" "Resistor_SMD:R_0402_1005Metric" (at 55.88 203.2 0) (effects (font (size 1.27 1.27)) (hide yes)))
-		(instances (project "odin" (path "/c44fb7fe-6133-ad34-68fd-fb66126197ef/e9248ad1-6b14-c545-7edc-53de7184d0bd" (reference "R31") (unit 1))))
+		(instances (project "odin" (path "/c44fb7fe-6133-ad34-68fd-fb66126197ef/e9248ad1-6b14-c545-7edc-53de7184d0bd" (reference "R32") (unit 1))))
 	)
 	(wire (pts (xy 55.88 191.77) (xy 55.88 189.23)) (stroke (width 0) (type default)))
@@
 	(symbol (lib_id "Device:R") (at 88.9 195.58 0) (unit 1)
 		(exclude_from_sim no) (in_bom yes) (on_board yes) (dnp no)
-		(property "Reference" "R32" (at 88.9 187.96 0) (effects (font (size 1.27 1.27))))
+		(property "Reference" "R33" (at 88.9 187.96 0) (effects (font (size 1.27 1.27))))
 		(property "Value" "4.7k" (at 88.9 203.2 0) (effects (font (size 1.27 1.27))))
 		(property "Footprint" "Resistor_SMD:R_0402_1005Metric" (at 88.9 203.2 0) (effects (font (size 1.27 1.27)) (hide yes)))
-		(instances (project "odin" (path "/c44fb7fe-6133-ad34-68fd-fb66126197ef/e9248ad1-6b14-c545-7edc-53de7184d0bd" (reference "R32") (unit 1))))
+		(instances (project "odin" (path "/c44fb7fe-6133-ad34-68fd-fb66126197ef/e9248ad1-6b14-c545-7edc-53de7184d0bd" (reference "R33") (unit 1))))
 	)
 	(wire (pts (xy 88.9 191.77) (xy 88.9 189.23)) (stroke (width 0) (type default)))
@@
 	(symbol (lib_id "Device:R") (at 316.23 273.05 0) (unit 1)
 		(exclude_from_sim no) (in_bom yes) (on_board yes) (dnp no)
-		(property "Reference" "R35" (at 316.23 265.43 0) (effects (font (size 1.27 1.27))))
+		(property "Reference" "R36" (at 316.23 265.43 0) (effects (font (size 1.27 1.27))))
 		(property "Value" "4.7k" (at 316.23 280.67 0) (effects (font (size 1.27 1.27))))
 		(property "Footprint" "Resistor_SMD:R_0402_1005Metric" (at 316.23 280.67 0) (effects (font (size 1.27 1.27)) (hide yes)))
-		(instances (project "odin" (path "/c44fb7fe-6133-ad34-68fd-fb66126197ef/e9248ad1-6b14-c545-7edc-53de7184d0bd" (reference "R35") (unit 1))))
+		(instances (project "odin" (path "/c44fb7fe-6133-ad34-68fd-fb66126197ef/e9248ad1-6b14-c545-7edc-53de7184d0bd" (reference "R36") (unit 1))))
 	)
 	(wire (pts (xy 316.23 269.24) (xy 316.23 266.7)) (stroke (width 0) (type default)))
@@
 	(symbol (lib_id "Device:R") (at 349.25 273.05 0) (unit 1)
 		(exclude_from_sim no) (in_bom yes) (on_board yes) (dnp no)
-		(property "Reference" "R33" (at 349.25 265.43 0) (effects (font (size 1.27 1.27))))
+		(property "Reference" "R34" (at 349.25 265.43 0) (effects (font (size 1.27 1.27))))
 		(property "Value" "4.7k" (at 349.25 280.67 0) (effects (font (size 1.27 1.27))))
 		(property "Footprint" "Resistor_SMD:R_0402_1005Metric" (at 349.25 280.67 0) (effects (font (size 1.27 1.27)) (hide yes)))
-		(instances (project "odin" (path "/c44fb7fe-6133-ad34-68fd-fb66126197ef/e9248ad1-6b14-c545-7edc-53de7184d0bd" (reference "R33") (unit 1))))
+		(instances (project "odin" (path "/c44fb7fe-6133-ad34-68fd-fb66126197ef/e9248ad1-6b14-c545-7edc-53de7184d0bd" (reference "R34") (unit 1))))
 	)
 	(wire (pts (xy 349.25 269.24) (xy 349.25 266.7)) (stroke (width 0) (type default)))
@@
 	(symbol (lib_id "Device:R") (at 382.27 273.05 0) (unit 1)
 		(exclude_from_sim no) (in_bom yes) (on_board yes) (dnp no)
-		(property "Reference" "R34" (at 382.27 265.43 0) (effects (font (size 1.27 1.27))))
+		(property "Reference" "R35" (at 382.27 265.43 0) (effects (font (size 1.27 1.27))))
 		(property "Value" "4.7k" (at 382.27 280.67 0) (effects (font (size 1.27 1.27))))
 		(property "Footprint" "Resistor_SMD:R_0402_1005Metric" (at 382.27 280.67 0) (effects (font (size 1.27 1.27)) (hide yes)))
-		(instances (project "odin" (path "/c44fb7fe-6133-ad34-68fd-fb66126197ef/e9248ad1-6b14-c545-7edc-53de7184d0bd" (reference "R34") (unit 1))))
+		(instances (project "odin" (path "/c44fb7fe-6133-ad34-68fd-fb66126197ef/e9248ad1-6b14-c545-7edc-53de7184d0bd" (reference "R35") (unit 1))))
 	)
 	(wire (pts (xy 382.27 269.24) (xy 382.27 266.7)) (stroke (width 0) (type default)))
@@
 	(symbol (lib_id "Device:R") (at 220.98 426.72 0) (unit 1)
 		(exclude_from_sim no) (in_bom yes) (on_board yes) (dnp no)
-		(property "Reference" "R38" (at 220.98 419.1 0) (effects (font (size 1.27 1.27))))
+		(property "Reference" "R39" (at 220.98 419.1 0) (effects (font (size 1.27 1.27))))
 		(property "Value" "4.7k" (at 220.98 434.34 0) (effects (font (size 1.27 1.27))))
 		(property "Footprint" "Resistor_SMD:R_0402_1005Metric" (at 220.98 434.34 0) (effects (font (size 1.27 1.27)) (hide yes)))
-		(instances (project "odin" (path "/c44fb7fe-6133-ad34-68fd-fb66126197ef/e9248ad1-6b14-c545-7edc-53de7184d0bd" (reference "R38") (unit 1))))
+		(instances (project "odin" (path "/c44fb7fe-6133-ad34-68fd-fb66126197ef/e9248ad1-6b14-c545-7edc-53de7184d0bd" (reference "R39") (unit 1))))
 	)
 	(wire (pts (xy 220.98 422.91) (xy 220.98 420.37)) (stroke (width 0) (type default)))
@@
 	(symbol (lib_id "Device:R") (at 254.0 426.72 0) (unit 1)
 		(exclude_from_sim no) (in_bom yes) (on_board yes) (dnp no)
-		(property "Reference" "R36" (at 254.0 419.1 0) (effects (font (size 1.27 1.27))))
+		(property "Reference" "R37" (at 254.0 419.1 0) (effects (font (size 1.27 1.27))))
 		(property "Value" "4.7k" (at 254.0 434.34 0) (effects (font (size 1.27 1.27))))
 		(property "Footprint" "Resistor_SMD:R_0402_1005Metric" (at 254.0 434.34 0) (effects (font (size 1.27 1.27)) (hide yes)))
-		(instances (project "odin" (path "/c44fb7fe-6133-ad34-68fd-fb66126197ef/e9248ad1-6b14-c545-7edc-53de7184d0bd" (reference "R36") (unit 1))))
+		(instances (project "odin" (path "/c44fb7fe-6133-ad34-68fd-fb66126197ef/e9248ad1-6b14-c545-7edc-53de7184d0bd" (reference "R37") (unit 1))))
 	)
 	(wire (pts (xy 254.0 422.91) (xy 254.0 420.37)) (stroke (width 0) (type default)))
@@
 	(symbol (lib_id "Device:R") (at 287.02 426.72 0) (unit 1)
 		(exclude_from_sim no) (in_bom yes) (on_board yes) (dnp no)
-		(property "Reference" "R37" (at 287.02 419.1 0) (effects (font (size 1.27 1.27))))
+		(property "Reference" "R38" (at 287.02 419.1 0) (effects (font (size 1.27 1.27))))
 		(property "Value" "4.7k" (at 287.02 434.34 0) (effects (font (size 1.27 1.27))))
 		(property "Footprint" "Resistor_SMD:R_0402_1005Metric" (at 287.02 434.34 0) (effects (font (size 1.27 1.27)) (hide yes)))
-		(instances (project "odin" (path "/c44fb7fe-6133-ad34-68fd-fb66126197ef/e9248ad1-6b14-c545-7edc-53de7184d0bd" (reference "R37") (unit 1))))
+		(instances (project "odin" (path "/c44fb7fe-6133-ad34-68fd-fb66126197ef/e9248ad1-6b14-c545-7edc-53de7184d0bd" (reference "R38") (unit 1))))
 	)
 	(wire (pts (xy 287.02 422.91) (xy 287.02 420.37)) (stroke (width 0) (type default)))
@@
 	(symbol (lib_id "Device:R") (at 88.9 727.71 0) (unit 1)
 		(exclude_from_sim no) (in_bom yes) (on_board yes) (dnp no)
-		(property "Reference" "R39" (at 88.9 720.09 0) (effects (font (size 1.27 1.27))))
+		(property "Reference" "R40" (at 88.9 720.09 0) (effects (font (size 1.27 1.27))))
 		(property "Value" "4.7k" (at 88.9 735.33 0) (effects (font (size 1.27 1.27))))
 		(property "Footprint" "Resistor_SMD:R_0402_1005Metric" (at 88.9 735.33 0) (effects (font (size 1.27 1.27)) (hide yes)))
-		(instances (project "odin" (path "/c44fb7fe-6133-ad34-68fd-fb66126197ef/e9248ad1-6b14-c545-7edc-53de7184d0bd" (reference "R39") (unit 1))))
+		(instances (project "odin" (path "/c44fb7fe-6133-ad34-68fd-fb66126197ef/e9248ad1-6b14-c545-7edc-53de7184d0bd" (reference "R40") (unit 1))))
 	)
 	(wire (pts (xy 88.9 723.9) (xy 88.9 721.36)) (stroke (width 0) (type default)))

Commit message: audit response: fix 5V-overstressed translators, add USB ESD protection and keying posts, load the PCB, reconcile every stale doc
Parts:
- Q1: symbol Device:Q_PMOS -> Transistor_FET:Q_PMOS_GSD
Connections:
- net +3V3: now also Q1.2 (S); no longer Q1.S
- net EN_SFP_N: now also Q1.1 (G); no longer Q1.G
- net SFP_VCC: now also Q1.3 (D); no longer Q1.D

Commit message: fix 14 package mismatches, assert footprints against ki_fp_filters, rebalance fuses, correct JTAG and PD-voltage claims
Parts:
- U17: footprint Package_SO:SOIC-16_3.9x9.9mm_P1.27mm -> Package_SO:SOIC-16W_7.5x10.3mm_P1.27mm
Changed lines of the file:
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@@
 		(property "Reference" "U17" (at 87.63 648.97 0) (effects (font (size 1.27 1.27))))
 		(property "Value" "PCF8574T" (at 87.63 687.07 0) (effects (font (size 1.27 1.27))))
-		(property "Footprint" "Package_SO:SOIC-16_3.9x9.9mm_P1.27mm" (at 87.63 687.07 0) (effects (font (size 1.27 1.27)) (hide yes)))
+		(property "Footprint" "Package_SO:SOIC-16W_7.5x10.3mm_P1.27mm" (at 87.63 687.07 0) (effects (font (size 1.27 1.27)) (hide yes)))
 		(instances (project "odin" (path "/c44fb7fe-6133-ad34-68fd-fb66126197ef/e9248ad1-6b14-c545-7edc-53de7184d0bd" (reference "U17") (unit 1))))
 	)

Commit message: Update Odin hardware design, imported parts, and documentation
Include EasyEDA symbols, footprints and 3D models; revise FPGA allocation, power and extension buses; add qualification audits and user documentation.

Validation: EasyEDA audit, qualified parts, power budget and Python syntax pass. KiCad ERC reports 1 error and 319 warnings; DRC reports 90 violations, 499 unconnected items and 209 schematic parity issues. This is a work-in-progress design snapshot. Imported vendor assets retain their original formatting.
Parts:
- removed C125, C127, C128, C130, C131, C132, C133, C134, C135, C136, C137, C138, C139, C140, C141, C142, C143, C144, C145, C146, C147, C148, C149, C150: 100nF, Capacitor_SMD:C_0402_1005Metric, symbol Device:C
- removed C126: 4.7uF, Capacitor_SMD:C_0603_1608Metric, symbol Device:C
- removed C129: 10uF, Capacitor_SMD:C_0805_2012Metric, symbol Device:C
- removed J62: SFP cage 2, Connector:Connector_SFP_and_Cage, symbol Interface_Optical:SFP
- removed J63: SFP cage 3, Connector:Connector_SFP_and_Cage, symbol Interface_Optical:SFP
- removed R30: 100, Resistor_SMD:R_0603_1608Metric, symbol Device:R
- removed R31: 100k, Resistor_SMD:R_0402_1005Metric, symbol Device:R
- removed R32, R33, R34: 4.7k, Resistor_SMD:R_0402_1005Metric, symbol Device:R
- added C168, C170, C171, C173, C174, C175, C176, C177, C178, C179, C180, C181, C182, C183: 100nF, Capacitor_SMD:C_0402_1005Metric, symbol Device:C
- added C169: 4.7uF, Capacitor_SMD:C_0603_1608Metric, symbol Device:C
- added C172: 10uF, Capacitor_SMD:C_0805_2012Metric, symbol Device:C
- added R41, R42, R43, R44, R45: 4.7k, Resistor_SMD:R_0402_1005Metric, symbol Device:R
- added SH1, SH2: 2007198-1, EasyEDA:TH_HC-SFP-01L, symbol EasyEDA:2007198-1
- J60: value SFP cage 0 -> SFP 0; footprint Connector:Connector_SFP_and_Cage -> EasyEDA:CONN-SMD_20P-P0.80-S8.20_1888247-1; LCSC (none) -> C305914
- J61: value SFP cage 1 -> SFP 1; footprint Connector:Connector_SFP_and_Cage -> EasyEDA:CONN-SMD_20P-P0.80-S8.20_1888247-1; LCSC (none) -> C305914
- Q1: value SFP power gate -> DMG2305UX-7; footprint Package_TO_SOT_SMD:SOT-23 -> EasyEDA:SOT-23-3_L2.9-W1.3-P1.90-LS2.4-BR; LCSC (none) -> C5261054
- R35: value 4.7k -> 100; footprint Resistor_SMD:R_0402_1005Metric -> Resistor_SMD:R_0603_1608Metric
- R36: value 4.7k -> 100k; LCSC (none) -> C25741
- R37, R38, R39, R40: LCSC (none) -> C25900
- U17: value PCF8574T -> PCF8574T_3,518; footprint Package_SO:SOIC-16W_7.5x10.3mm_P1.27mm -> EasyEDA:SOIC-16_L10.3-W7.5-P1.27-LS10.3-BL; symbol Interface_Expansion:PCF8574T -> EasyEDA:PCF8574T_3,518; LCSC (none) -> C7605; now fitted
- X2: value 125MHz LVDS -> DSC1123CI2-125.0000; footprint Oscillator:Oscillator_SMD_SiTime_SiT9121-6Pin_3.2x2.5mm -> EasyEDA:OSC-SMD_6P-L3.2-W2.5-BL; symbol odin:OSC_DIFF_6P_3225 -> EasyEDA:DSC1123CI2-125.0000; LCSC (none) -> C617173
Connections:
- net SFP3_LOS_NP is gone; now on net EN_SFP_N: U17.12 (P7)
- net +3V3: now also C168.1, C169.1, C183.1, R41.1, R42.1, R43.1, R44.1, R45.1; no longer R35.1
- net EN_SFP_N: now also R36.2
- net GND: now also R35.2, X2.3 (GND), C168.2, C169.2, C172.2, C177.2, C182.2, C183.2, SH1.1, SH1.10, SH1.11, SH1.12, SH1.13, SH1.14, SH1.15, SH1.16, SH1.17, SH1.18, SH1.19, SH1.2, SH1.20, SH1.3, SH1.4, SH1.5, SH1.6, SH1.7, SH1.8, SH1.9, SH2.1, SH2.10, SH2.11, SH2.12, SH2.13, SH2.14, SH2.15, SH2.16, SH2.17, SH2.18, SH2.19, SH2.2, SH2.20, SH2.3, SH2.4, SH2.5, SH2.6, SH2.7, SH2.8, SH2.9; no longer J60.CAGE, J61.CAGE, X2.2 (GND)
- net MGTPRXN0: now also C176.2
- net MGTPRXN1: now also C181.2
- net MGTPRXP0: now also C175.2
- net MGTPRXP1: now also C180.2
- net MGTPTXN0: now also C174.1
- net MGTPTXN1: now also C179.1
- net MGTPTXP0: now also C173.1
- net MGTPTXP1: now also C178.1
- net MGTREFCLK0N: now also C171.2
- net MGTREFCLK0P: now also C170.2
- net MGTRREF: now also R35.1
- net REFCLK_OSC_N: now also X2.5 (~{Output}), C171.1; no longer X2.4 (OUT-)
- net REFCLK_OSC_P: now also X2.4 (Output), C170.1; no longer X2.5 (OUT+)
- net SFP0_LOS: now also R41.2; no longer R36.2
- net SFP0_MOD_ABS: now also R39.2
- net SFP0_RD_N: now also C176.1
- net SFP0_RD_P: now also C175.1
- net SFP0_TD_N: now also C174.2
- net SFP0_TD_P: now also C173.2
- net SFP0_TX_FAULT: now also R40.2; no longer R35.2
- net SFP1_LOS: now also R44.2; no longer R39.2
- net SFP1_MOD_ABS: now also R42.2; no longer R37.2
- net SFP1_RD_N: now also C181.1
- net SFP1_RD_P: now also C180.1
- net SFP1_TD_N: now also C179.2
- net SFP1_TD_P: now also C178.2
- net SFP1_TX_FAULT: now also R43.2; no longer R38.2
- net SFP_EXP_INT: now also R45.2; no longer R40.2
- net SFP_SCL: now also R37.2
- net SFP_SDA: now also R38.2
- net SFP_VCC: now also C172.1, C177.1, C182.1
- net SFP2_LOS_NP: no longer names the net of U17.7 (P3)
- net SFP2_MOD_ABS_NP: no longer names the net of U17.4 (P0)
- net SFP2_TX_DIS_NP: no longer names the net of U17.5 (P1)
- net SFP2_TX_FAULT_NP: no longer names the net of U17.6 (P2)
- net SFP3_MOD_ABS_NP: no longer names the net of U17.9 (P4)
- net SFP3_TX_DIS_NP: no longer names the net of U17.10 (P5)
- net SFP3_TX_FAULT_NP: no longer names the net of U17.11 (P6)
- no-connect marks 1 -> 10
Other:
- note added: "HIGHSPEED — Four serial lanes: SFP cages, reference clock, power gate — HW 0.1.0-proto.1"
- note added: "SFP port 0"
- note added: "SFP port 1"
- note added: "SFP port expander"
- note removed: "HIGHSPEED — Four serial lanes: SFP cages, reference clock, power gate"
- note removed: "SFP cage 0"
- note removed: "SFP cage 1"
- note removed: "SFP cage 2 (not fitted)"
- note removed: "SFP cage 3 (not fitted)"
- note removed: "SFP port expander (not fitted)"
- moved on the sheet: J60, J61, R35, R36, R37, R38, R39, R40
