File: kicad/highspeed.kicad_sch (KiCad schematic)
At the start: 34 parts, among them J60 SFP 0, J61 SFP 1, Q1 DMG2305UX-7, U17 PCF8574T_3,518, X2 DSC1123CI2-125.0000

Commit message: wip
Parts:
- removed C183: 100nF, Capacitor_SMD:C_0402_1005Metric, symbol Device:C
- added C167, C231: 100nF, Capacitor_SMD:C_0402_1005Metric, symbol Device:C
- added D10, D11, D9: F.0603.00025/P2-0603G1TS2-06T-002, EasyEDA:LED0603-RD_GREEN, symbol EasyEDA:F.0603.00025_P2-0603G1TS2-06T-002
- added R100, R101, R102, R99: 4.7k, Resistor_SMD:R_0402_1005Metric, symbol Device:R
- added R103: 10k, Resistor_SMD:R_0402_1005Metric, symbol Device:R
- added R128, R129, R130: 1k, Resistor_SMD:R_0402_1005Metric, symbol Device:R
- added R89: 100 1%, Resistor_SMD:R_0603_1608Metric, symbol Device:R
- added U27: PCA9543APW,118, Package_SO:TSSOP-14_4.4x5mm_P0.65mm, symbol odin:PCA9543APW
- C168: value 100nF -> 4.7uF; footprint Capacitor_SMD:C_0402_1005Metric -> Capacitor_SMD:C_0603_1608Metric; LCSC C1525 -> C277476
- C169: value 4.7uF -> 100nF; footprint Capacitor_SMD:C_0603_1608Metric -> Capacitor_SMD:C_0402_1005Metric; LCSC C277476 -> C1525
- C171: value 100nF -> 10uF; footprint Capacitor_SMD:C_0402_1005Metric -> Capacitor_SMD:C_0805_2012Metric; LCSC C1525 -> C15850
- C172: value 10uF -> 100nF; footprint Capacitor_SMD:C_0805_2012Metric -> Capacitor_SMD:C_0402_1005Metric; LCSC C15850 -> C1525
- R35: value 100 -> 100 1%
- SH1, SH2: value 2007198-1 -> U77A11133001; footprint EasyEDA:TH_HC-SFP-01L -> odin:Amphenol_U77A11133001; symbol EasyEDA:2007198-1 -> odin:U77A11133001; LCSC C573949 -> C5355132
Connections:
- net +3V3: now also C182.1, C167.1, C231.1, R103.1, R128.1, R129.1, R130.1, U27.14 (VDD); no longer C169.1
- net GND: now also C171.2, C176.2, C181.2, C167.2, C231.2, U27.1 (A0), U27.2 (A1), U27.7 (VSS); no longer C169.2, C172.2, C177.2, R35.2
- net MGTPRXN0: now also C175.2; no longer C176.2
- net MGTPRXN1: now also C180.2; no longer C181.2
- net MGTPRXP0: now also C174.2; no longer C175.2
- net MGTPRXP1: now also C179.2; no longer C180.2
- net MGTPTXN0: now also C173.1; no longer C174.1
- net MGTPTXN1: now also C178.1; no longer C179.1
- net MGTPTXP0: now also C172.1; no longer C173.1
- net MGTPTXP1: now also C177.1; no longer C178.1
- net MGTREFCLK0N: now also C170.2; no longer C171.2
- net MGTREFCLK0P: now also C169.2; no longer C170.2
- net REFCLK_OSC_N: now also C170.1; no longer C171.1
- net REFCLK_OSC_P: now also C169.1; no longer C170.1
- net SFP0_RD_N: now also C175.1; no longer C176.1
- net SFP0_RD_P: now also C174.1; no longer C175.1
- net SFP0_TD_N: now also C173.2; no longer C174.2
- net SFP0_TD_P: now also C172.2; no longer C173.2
- net SFP1_RD_N: now also C180.1; no longer C181.1
- net SFP1_RD_P: now also C179.1; no longer C180.1
- net SFP1_TD_N: now also C178.2; no longer C179.2
- net SFP1_TD_P: now also C177.2; no longer C178.2
- net SFP_SCL: now also U27.12 (SCL); no longer J60.5 (MOD_DEF1), J61.5 (MOD_DEF1)
- net SFP_SDA: now also U27.13 (SDA); no longer J60.4 (MOD_DEF2), J61.4 (MOD_DEF2)
- net SFP_VCC: now also C171.1, C176.1, C181.1, R100.1, R101.1, R102.1, R99.1; no longer C172.1, C177.1, C182.1
- net LED_HEARTBEAT_N: now reaches U17.4 (P0)
- net LED_HEARTBEAT_N: now also D9.1 (C)
- net LED_USER1_N: now reaches U17.5 (P1)
- net LED_USER1_N: now also D10.1 (C)
- net LED_USER2_N: now reaches U17.6 (P2)
- net LED_USER2_N: now also D11.1 (C)
- net CORE_1V0_GOOD: now reaches U17.7 (P3)
- new net +1V2_MGT: R35.2, R89.2
- new net LED_HEARTBEAT_A: D9.2 (A), R128.2
- new net LED_USER1_A: D10.2 (A), R129.2
- new net LED_USER2_A: D11.2 (A), R130.2
- new net MGTRREF_213: R89.1
- new net SFP0_SCL: J60.5 (MOD_DEF1), R99.2, U27.6 (SC0)
- new net SFP0_SDA: J60.4 (MOD_DEF2), R100.2, U27.5 (SD0)
- new net SFP1_SCL: J61.5 (MOD_DEF1), R101.2, U27.10 (SC1)
- new net SFP1_SDA: J61.4 (MOD_DEF2), R102.2, U27.9 (SD1)
- new net SFP_MUX_INT_UNUSED: R103.2, U27.4 (~{INT0}), U27.8 (~{INT1})
- new net SUP_RUN: U27.3 (~{RESET})
- no-connect marks 10 -> 7
Other:
- note added: "SFP I2C mux"
- note added: "Unused quad 213 calibration"
- note added: "board status LEDs"
- moved on the sheet: C168, C169, C170, C171, C172, C173, C174, C175, C176, C177, C178, C179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
