File: kicad/highspeed.kicad_sch (KiCad schematic)
At the start: 48 parts, among them J60 SFP 0, J61 SFP 1, Q1 DMG2305UX-7, U17 PCF8574T_3,518, U27 PCA9543APW,118, X2 DSC1123CI2-125.0000

Commit message: Through-hole extension headers, AUX supply rework, and board state before rev A cleanup
J3/J5 become single 2x32 through-hole bodies with IO IO GND rows and a long
grounded key post per zone. Power sheet reworked around the AUX rail.
Decoupling moved off B.Cu. New footprints, 3D models and check scripts.
Parts:
- added C248, C249: 22uF 6.3V, Capacitor_SMD:C_0805_2012Metric, symbol Device:C
- added FB1, FB2: BLM18PG221SN1D 220R@100MHz 1.4A, Inductor_SMD:L_0603_1608Metric, symbol Device:FerriteBead
- added R145: 4.7k, Resistor_SMD:R_0402_1005Metric, symbol Device:R
- J60, J61: symbol Interface_Optical:SFP -> odin:SFP_NoCage
Connections:
- net GND: now also C248.2, C249.2; no longer J60.7 (RATE_SELECT), J61.7 (RATE_SELECT)
- net SFP_VCC: now also FB1.1, FB2.1; no longer C176.1, C181.1, J60.15 (VccR), J60.16 (VccT), J61.15 (VccR), J61.16 (VccT)
- new net SFP0_RATE_SELECT: J60.7 (RATE_SELECT)
- new net SFP0_VCC: C176.1, C248.1, FB1.2, J60.15 (VccR), J60.16 (VccT)
- new net SFP1_RATE_SELECT: J61.7 (RATE_SELECT), R145.2
- new net SFP1_VCC: C181.1, C249.1, FB2.2, J61.15 (VccR), J61.16 (VccT), R145.1
- no-connect marks 7 -> 5
Other:
- moved on the sheet: C172, C173, C174, C175, C176, C177, C178, C179, C180, C181, C182, C231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
