File: kicad/power.kicad_sch (KiCad schematic)
At the start: 77 parts, among them J50 VIN (optional), Q2 VBUS pass, Q3 gate driver, U11 TPS54202DDC, U12 TPS54202DDC, U13 TLV62569DRL, U14 TLV62569DRL, U15 TLV62569DRL, U16 TLV62569DRL, U19 TPS61085PW

Commit message: Update Odin hardware design, imported parts, and documentation
Include EasyEDA symbols, footprints and 3D models; revise FPGA allocation, power and extension buses; add qualification audits and user documentation.

Validation: EasyEDA audit, qualified parts, power budget and Python syntax pass. KiCad ERC reports 1 error and 319 warnings; DRC reports 90 violations, 499 unconnected items and 209 schematic parity issues. This is a work-in-progress design snapshot. Imported vendor assets retain their original formatting.
Parts:
- removed C151, C152, C155, C156, C157, C159, C160, C161, C162, C163, C165, C166, C168, C169, C171, C172: 22uF, Capacitor_SMD:C_0805_2012Metric, symbol Device:C
- removed C153, C176, C177, C178: 10uF, Capacitor_SMD:C_0805_2012Metric, symbol Device:C
- removed C154, C158, C164, C167, C170, C173: 100nF, Capacitor_SMD:C_0402_1005Metric, symbol Device:C
- removed C174: 2.2nF, Capacitor_SMD:C_0402_1005Metric, symbol Device:C
- removed C175: 10nF, Capacitor_SMD:C_0402_1005Metric, symbol Device:C
- removed C179: 4.7uF, Capacitor_SMD:C_0603_1608Metric, symbol Device:C
- removed R41, R44: 100k, Resistor_SMD:R_0603_1608Metric, symbol Device:R
- removed R42: 10k, Resistor_SMD:R_0402_1005Metric, symbol Device:R
- removed R43: 100k, Resistor_SMD:R_0402_1005Metric, symbol Device:R
- removed R45: 13.7k, Resistor_SMD:R_0603_1608Metric, symbol Device:R
- added C184: 100nF 25V, Capacitor_SMD:C_0402_1005Metric, symbol Device:C
- added C185: 2.2nF 25V, Capacitor_SMD:C_0402_1005Metric, symbol Device:C
- added C186, C187: 22uF 25V, Capacitor_SMD:C_0805_2012Metric, symbol Device:C
- added C188, C193, C216, C217: 10uF 25V, Capacitor_SMD:C_0805_2012Metric, symbol Device:C
- added C189, C194, C201, C204, C207, C226, C227, C228, C229, C230, C231: 100nF, Capacitor_SMD:C_0402_1005Metric, symbol Device:C
- added C190, C191, C192, C196, C197, C198, C199, C200, C202, C203, C205, C206, C208, C212, C213: 22uF, Capacitor_SMD:C_0805_2012Metric, symbol Device:C
- added C195: 56pF, Capacitor_SMD:C_0402_1005Metric, symbol Device:C
- added C209, C219, C220, C221, C222: 1uF, Capacitor_SMD:C_0603_1608Metric, symbol Device:C
- added C210: 1nF, Capacitor_SMD:C_0402_1005Metric, symbol Device:C
- added C211: 22pF, Capacitor_SMD:C_0402_1005Metric, symbol Device:C
- added C214: 2.2nF, Capacitor_SMD:C_0402_1005Metric, symbol Device:C
- added C215: 10nF, Capacitor_SMD:C_0402_1005Metric, symbol Device:C
- added C218: 10uF, Capacitor_SMD:C_0805_2012Metric, symbol Device:C
- added C223: 3.3nF 25V, Capacitor_SMD:C_0402_1005Metric, symbol Device:C
- added C224: 1uF 25V, Capacitor_SMD:C_0603_1608Metric, symbol Device:C
- added C225: 4.7uF, Capacitor_SMD:C_0603_1608Metric, symbol Device:C
- added R68: 150k, Resistor_SMD:R_0603_1608Metric, symbol Device:R
- added R69, R72, R81, R83: 100k, Resistor_SMD:R_0603_1608Metric, symbol Device:R
- added R70: 11.5k, Resistor_SMD:R_0603_1608Metric, symbol Device:R
- added R71: 47k, Resistor_SMD:R_0402_1005Metric, symbol Device:R
- added R73: 10k, Resistor_SMD:R_0603_1608Metric, symbol Device:R
- added R74: 1.15k, Resistor_SMD:R_0603_1608Metric, symbol Device:R
- added R75, R76, R77: 2.21k, Resistor_SMD:R_0603_1608Metric, symbol Device:R
- added R78: 121k, Resistor_SMD:R_0603_1608Metric, symbol Device:R
- added R79: 12.1k, Resistor_SMD:R_0603_1608Metric, symbol Device:R
- added R80: 6.65k, Resistor_SMD:R_0603_1608Metric, symbol Device:R
- added R82: 16k, Resistor_SMD:R_0603_1608Metric, symbol Device:R
- added R84: 47k, Resistor_SMD:R_0603_1608Metric, symbol Device:R
- added R85, R86, R87, R88: 1k, Resistor_SMD:R_0603_1608Metric, symbol Device:R
- added U21, U22, U23, U24: TPS22950CDDCR, EasyEDA:SOT-23-6_L2.9-W1.6-P0.95-LS2.8-BL_3, symbol odin:TPS22950CDDC
- added U25: TPS259470LRPWR, Package_DFN_QFN:Texas_RPU0010A_VQFN-HR-10_2x2mm_P0.5mm, symbol odin:TPS259470LRPW
- added U26: TPS259470ARPWR, Package_DFN_QFN:Texas_RPU0010A_VQFN-HR-10_2x2mm_P0.5mm, symbol odin:TPS259470ARPW
- D3, D4, D5: footprint Diode_SMD:D_SMA -> EasyEDA:SMA_L4.3-W2.6-LS5.2-RD; LCSC (none) -> C8678
- J50: value VIN (optional) -> 9-14V POWER IN; footprint Connector_PinHeader_2.54mm:PinHeader_1x02_P2.54mm_Vertical -> EasyEDA:CONN-TH_P5.00_KF301-5.0-2P; symbol Connector_Generic:Conn_01x02 -> EasyEDA:KF301-5.0-2P; LCSC (none) -> C474881
- L2, L8: value 4.7uH -> 10uH SRN6045TA-100M; footprint Inductor_SMD:L_Bourns-SRN4018 -> EasyEDA:IND-SMD_L6.0-W6.0-1; LCSC (none) -> C2046332
- L3: value 4.7uH -> 4.7uH SRN6045TA-4R7M; footprint Inductor_SMD:L_Bourns-SRN4018 -> EasyEDA:IND-SMD_L6.0-W6.0; LCSC (none) -> C2044594
- L4, L5, L6: value 1.5uH -> 2.2uH SRN4018-2R2M; footprint Inductor_SMD:L_Bourns-SRN4018 -> EasyEDA:IND-SMD_L4.0-W4.0_SNR4018; LCSC (none) -> C913207
- L7: value 1.5uH -> 1uH_core FTC201610S1R0MBCA; footprint Inductor_SMD:L_Bourns-SRN4018 -> EasyEDA:IND-SMD_L2.0-W1.6-B; LCSC (none) -> C5832342
- L9: value 1uH -> 1uH VLS252010HBX-1R0M-1; footprint Inductor_SMD:L_Bourns-SRN4018 -> EasyEDA:IND-SMD_L2.5-W2.0-1; LCSC (none) -> C88211
- Q2: value VBUS pass -> DMG2305UX-7; footprint Package_TO_SOT_SMD:SOT-23 -> EasyEDA:SOT-23-3_L2.9-W1.3-P1.90-LS2.4-BR; LCSC (none) -> C5261054
- Q3: value gate driver -> BSS138LT1G; footprint Package_TO_SOT_SMD:SOT-23 -> EasyEDA:SOT-23-3_L2.9-W1.6-P1.90-LS2.8-BR; LCSC (none) -> C82045
- R47: value 100k -> 10k; footprint Resistor_SMD:R_0603_1608Metric -> Resistor_SMD:R_0402_1005Metric
- R48: value 22.1k -> 100k; footprint Resistor_SMD:R_0603_1608Metric -> Resistor_SMD:R_0402_1005Metric; LCSC (none) -> C25741
- R49, R53: value 100k -> 10k
- R50: value 31.6k -> 100k
- R51: value 100k -> 47k
- R52: value 49.9k -> 73.2k
- R54: value 150k -> 1.65k
- R56: value 100k -> 13.7k
- R57: value 100k -> 93.1k
- R58: value 11.5k -> 30.1k
- R59: value 47k -> 100k; footprint Resistor_SMD:R_0402_1005Metric -> Resistor_SMD:R_0603_1608Metric
- R60: value 100k -> 31.6k
- R61: value 33k -> 100k
- R62: value 100k -> 49.9k
- R64, R67: value 1k -> 100k
- R65: value 1k -> 10
- R66: value 1k -> 100k; footprint Resistor_SMD:R_0603_1608Metric -> Resistor_SMD:R_0402_1005Metric; LCSC (none) -> C25741
- U11: value TPS54202DDC -> TPS54202DDCR; footprint Package_TO_SOT_SMD:SOT-23-6 -> EasyEDA:SOT-23-6_L2.9-W1.6-P0.95-LS2.8-BL
- U12: value TPS54202DDC -> AP63300WU-7; footprint Package_TO_SOT_SMD:SOT-23-6 -> EasyEDA:TSOT-23-6_L2.9-W1.6-P0.95-LS2.8-BR; symbol Regulator_Switching:TPS54202DDC -> odin:AP63300WU; LCSC C191884 -> C2158012
- U13, U14, U16: value TLV62569DRL -> TLV62569DRLR; footprint Package_TO_SOT_SMD:SOT-563 -> EasyEDA:SOT-563_L1.6-W1.2-P0.50-LS1.6-BL
- U15: value TLV62569DRL -> SY8047QDC; footprint Package_TO_SOT_SMD:SOT-563 -> EasyEDA:TQFN-16_L3.0-W3.0-P0.50-TL-EP1.6; symbol Regulator_Switching:TLV62569DRL -> EasyEDA:SY8047QDC; LCSC C163217 -> C3018651
- U19: value TPS61085PW -> TPS61085PWR; footprint Package_SO:TSSOP-8_4.4x3mm_P0.65mm -> EasyEDA:TSSOP-8_L4.4-W3.0-P0.65-LS6.4-BL; LCSC (none) -> C13505
Connections:
- net +12V: now also C216.1, C217.1, C224.1, R69.1, R78.1, U25.5 (IN); no longer R57.1
- net +1V0: now also L7.1, C211.1, C212.1, C213.1, R88.1; no longer L6.1, R53.1
- net +1V0_MGT: now also C225.1
- net +1V2_MGT: now also L6.1, R63.1, C205.1, C206.1; no longer L7.1, R55.1
- net +1V8: now also R61.1, C202.1, C203.1, R87.1; no longer R51.1, R66.1
- net +2V5: now also R59.1, C199.1, C200.1, R86.1; no longer R49.1, R65.1
- net +3V3: now also R57.1, R66.1, C195.1, C196.1, C197.1, C198.1, C220.1, R73.1, R85.1, U22.2 (VIN); no longer R47.1, R64.1
- net +5V: now also R55.1, R65.1, U15.11 (PVIN), U15.12 (PVIN), C190.1, C191.1, C192.1, C201.1, C204.1, C207.1, C208.1, C218.1, C219.1, R83.1, U21.2 (VIN); no longer R62.1, U15.3 (VIN)
- net BOOT_3V3: now also C194.1
- net BOOT_5V: now also C189.1
- net COMP_12V: now also R71.1; no longer R59.1
- net COMP_12V_C: now also C214.1, R71.2; no longer R59.2
- net EN_1V0: now also U15.13 (EN); no longer U15.5 (EN)
- net EN_VBUS5: now also R47.1
- net EN_VBUS5_G: now also R47.2, R48.1
- net FB+1V0: now also R67.2, U15.5 (FB), C211.2, R68.1; no longer R53.2, R54.1, U15.1 (FB)
- net FB+1V2_MGT: now also R63.2, R64.1; no longer R55.2, R56.1
- net FB+1V8: now also R61.2, R62.1; no longer R51.2, R52.1
- net FB+2V5: now also R59.2, R60.1; no longer R49.2, R50.1
- net FB_12V: now also R69.2, R70.1; no longer R57.2, R58.1
- net FB_3V3: now also R57.2, R58.1, U12.1 (FB), C195.2; no longer R47.2, R48.1, U12.4 (FB)
- net FB_5V: now also R55.2, R56.1
- net GND: now also R51.2, R53.2, R60.2, R62.2, R64.2, U12.4 (GND), U15.14 (PGND), U15.15 (PGND), U15.17 (EP), U15.6 (AGND), C185.2, C186.2, C187.2, C188.2, C190.2, C191.2, C192.2, C193.2, C196.2, C197.2, C198.2, C199.2, C200.2, C201.2, C202.2, C203.2, C204.2, C205.2, C206.2, C207.2, C208.2, C209.2, C210.2, C212.2, C213.2, C214.2, C215.2, C216.2, C217.2, C218.2, C219.2, C220.2, C221.2, C222.2, C223.2, C224.2, C225.2, C226.2, C227.2, C228.2, C229.2, C230.2, C231.2, R68.2, R70.2, R72.2, R74.2, R75.2, R76.2, R77.2, R79.2, R80.2, R82.2, R84.2, U21.3 (GND), U22.3 (GND), U23.3 (GND), U24.3 (GND), U25.8 (GND), U26.8 (GND); no longer R50.2, R52.2, R61.2, R63.2, U12.1 (GND), U15.2 (GND)
- net MON_1V0: now also C231.1, R88.2; no longer R67.2
- net MON_1V8: now also C230.1, R87.2; no longer R66.2
- net MON_2V5: now also C229.1, R86.2; no longer R65.2
- net MON_3V3: now also C228.1, R85.2; no longer R64.2
- net MON_5V: now also C227.1, R83.2, R84.1; no longer R62.2, R63.1
- net MON_VSYS: now also C226.1, R81.2, R82.1; no longer R60.2, R61.1
- net SS_12V: now also C215.1
- net SW+1V0: now also L7.2, U15.1 (LX), U15.2 (LX); no longer L6.2, U15.4 (SW)
- net SW+1V2_MGT: now also L6.2; no longer L7.2
- net SW_3V3: now also U12.5 (SW), C194.2; no longer U12.2 (SW)
- net SW_5V: now also C189.2
- net VBUS: now also R46.1, R50.1, R52.1, C184.2, C188.1, U26.5 (IN); no longer D3.2 (A)
- net VBUS5_GATE: now also R46.2, R49.2, C184.1; no longer Q3.3 (D)
- net VSYS: now also C186.1, C187.1, C193.1, R81.1; no longer R46.1, R60.1
- removed net EN_3V3_AO: R46.2, U12.5 (EN)
- new net +12V_EXT: U25.6 (OUT)
- new net +3V3_EXT: U22.5 (VOUT)
- new net +5V_EXT: U21.5 (VOUT)
- new net CORE_1V0_GOOD: R66.2, U15.4 (PG)
- new net CORE_1V0_SS: C210.1, U15.9 (SS)
- new net CORE_1V0_SVIN: C209.1, R65.2, U15.10 (SVIN)
- new net EXT12_DVDT: C223.1, U25.7 (dVdt)
- new net EXT12_ILM: R80.1, U25.9 (ILM)
- new net EXT12_OVLO: R78.2, R79.1, U25.2 (OVLO)
- new net EXT_EN: R72.1, U21.1 (ON), U22.1 (ON), U23.1 (ON), U24.1 (ON), U25.1 (EN/UVLO)
- new net EXT_FAULT: R73.2, U21.6 (FLT), U22.6 (FLT), U23.6 (FLT), U24.6 (FLT), U25.4 (FLT), U26.4 (FLT)
- new net U21_ILIM: R74.1, U21.4 (ILIM)
- new net U22_ILIM: R75.1, U22.4 (ILIM)
- new net U23_ILIM: R76.1, U23.4 (ILIM)
- new net U24_ILIM: R77.1, U24.4 (ILIM)
- new net VBUS5_PULL: Q3.3 (D), R49.1
- new net VBUS_DVDT: C185.1, U26.7 (dVdt)
- new net VBUS_ILM: R54.1, U26.9 (ILM)
- new net VBUS_OVLO: R52.2, R53.1, U26.2 (OVLO)
- new net VBUS_SS: D3.2 (A), U26.6 (OUT)
- new net VBUS_UVLO: R50.2, R51.1, U26.1 (EN/UVLO)
- new net VCCIO_1: C221.1, U23.2 (VIN)
- new net VCCIO_1_EXT: U23.5 (VOUT)
- new net VCCIO_2: C222.1, U24.2 (VIN)
- new net VCCIO_2_EXT: U24.5 (VOUT)
- no-connect marks 4 -> 12
Other:
- note added: "POWER — Power tree: 12V input to every rail, with monitoring — HW 0.1.0-proto.1"
- note added: "U12 VSYS to +3V3 (always-on AP63300 reference circuit)"
- note added: "U15 5V to +1V0 (4A FPGA core supply)"
- note added: "U21 +5V to +5V_EXT"
- note added: "U22 +3V3 to +3V3_EXT"
- note added: "U23 VCCIO_1 to VCCIO_1_EXT"
- note added: "U24 VCCIO_2 to VCCIO_2_EXT"
- note added: "U25 +12V to +12V_EXT"
- note added: "extension power protection control"
- note removed: "POWER — Power tree: 12V input to every rail, with monitoring"
- note removed: "U12 VSYS to +3V3 (always on)"
- note removed: "U15 5V to +1V0"
- moved on the sheet: D3, D4, L2, L3, L4, L5, L6, L7, L8, L9, Q2, Q3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

Commit message: wip
Parts:
- removed C231: 100nF, Capacitor_SMD:C_0402_1005Metric, symbol Device:C
- added C183: 100nF 25V, Capacitor_SMD:C_0402_1005Metric, symbol Device:C
- added C232: 10uF 25V, Capacitor_SMD:C_0805_2012Metric, symbol Device:C
- added D8: SMBJ15A-13-F, Diode_SMD:D_SMB, symbol Device:D_Zener
- added R90, R91, R92, R93, R94, R95: 100k, Resistor_SMD:R_0603_1608Metric, symbol Device:R
- C184: value 100nF 25V -> 2.2nF 25V; LCSC C1525 -> (none)
- C185: value 2.2nF 25V -> 22uF 25V; footprint Capacitor_SMD:C_0402_1005Metric -> Capacitor_SMD:C_0805_2012Metric; LCSC (none) -> C86816
- C187: value 22uF 25V -> 10uF 25V; LCSC C86816 -> C15850
- C188, C193: value 10uF 25V -> 100nF; footprint Capacitor_SMD:C_0805_2012Metric -> Capacitor_SMD:C_0402_1005Metric; LCSC C15850 -> C1525
- C189, C201, C204, C207: value 100nF -> 22uF; footprint Capacitor_SMD:C_0402_1005Metric -> Capacitor_SMD:C_0805_2012Metric; LCSC C1525 -> C86816
- C192: value 22uF -> 10uF 25V; LCSC C86816 -> C15850
- C194: value 100nF -> 56pF; LCSC C1525 -> (none)
- C195: value 56pF -> 22uF; footprint Capacitor_SMD:C_0402_1005Metric -> Capacitor_SMD:C_0805_2012Metric; LCSC (none) -> C86816
- C200, C203, C206: value 22uF -> 100nF; footprint Capacitor_SMD:C_0805_2012Metric -> Capacitor_SMD:C_0402_1005Metric; LCSC C86816 -> C1525
- C208: value 22uF -> 1uF; footprint Capacitor_SMD:C_0805_2012Metric -> Capacitor_SMD:C_0603_1608Metric; LCSC C86816 -> C29936
- C209: value 1uF -> 1nF; footprint Capacitor_SMD:C_0603_1608Metric -> Capacitor_SMD:C_0402_1005Metric; LCSC C29936 -> (none)
- C210: value 1nF -> 22pF
- C211: value 22pF -> 22uF; footprint Capacitor_SMD:C_0402_1005Metric -> Capacitor_SMD:C_0805_2012Metric; LCSC (none) -> C86816
- C213: value 22uF -> 2.2nF; footprint Capacitor_SMD:C_0805_2012Metric -> Capacitor_SMD:C_0402_1005Metric; LCSC C86816 -> (none)
- C214: value 2.2nF -> 10nF
- C215: value 10nF -> 10uF 25V; footprint Capacitor_SMD:C_0402_1005Metric -> Capacitor_SMD:C_0805_2012Metric; LCSC (none) -> C15850
- C217: value 10uF 25V -> 10uF
- C218: value 10uF -> 1uF; footprint Capacitor_SMD:C_0805_2012Metric -> Capacitor_SMD:C_0603_1608Metric; LCSC C15850 -> C29936
- C222: value 1uF -> 3.3nF 25V; footprint Capacitor_SMD:C_0603_1608Metric -> Capacitor_SMD:C_0402_1005Metric; LCSC C29936 -> (none)
- C223: value 3.3nF 25V -> 1uF 25V; footprint Capacitor_SMD:C_0402_1005Metric -> Capacitor_SMD:C_0603_1608Metric; LCSC (none) -> C29936
- C224: value 1uF 25V -> 4.7uF; LCSC C29936 -> C277476
- C225: value 4.7uF -> 100nF; footprint Capacitor_SMD:C_0603_1608Metric -> Capacitor_SMD:C_0402_1005Metric; LCSC C277476 -> C1525
- R49: value 10k -> 47k
Connections:
- net +12V: now also C215.1, C223.1; no longer C217.1, C224.1
- net +12V_EXT: now also C232.1
- net +1V0: now also C210.1; no longer C213.1
- net +1V0_MGT: now also C224.1; no longer C225.1
- net +1V2_MGT: now also C204.1; no longer C206.1
- net +1V8: now also C201.1; no longer C203.1
- net +2V5: now also C198.1; no longer C200.1
- net +3V3: now also C194.1, C219.1; no longer C198.1, C220.1
- net +5V: now also C189.1, C200.1, C203.1, C206.1, C217.1; no longer C192.1, C201.1, C204.1, C208.1, C219.1
- net BOOT_3V3: now also C193.1; no longer C194.1
- net BOOT_5V: now also C188.1; no longer C189.1
- net COMP_12V_C: now also C213.1; no longer C214.1
- net CORE_1V0_SS: now also C209.1; no longer C210.1
- net CORE_1V0_SVIN: now also C208.1; no longer C209.1
- net EN_12V: now also R95.1
- net EN_1V0: now also R94.1
- net EN_1V2: now also R93.1
- net EN_1V8: now also R92.1
- net EN_2V5: now also R91.1
- net EN_5V: now also R90.1
- net EXT12_DVDT: now also C222.1; no longer C223.1
- net FB+1V0: now also C210.2; no longer C211.2
- net FB_3V3: now also C194.2; no longer C195.2
- net GND: now also C184.2, C189.2, C195.2, C211.2, C232.2, D8.2 (A), R90.2, R91.2, R92.2, R93.2, R94.2, R95.2; no longer C188.2, C193.2, C210.2
- net MON_1V0: now also C230.1
- net MON_1V8: now also C229.1; no longer C230.1
- net MON_2V5: now also C228.1; no longer C229.1
- net MON_3V3: now also C227.1; no longer C228.1
- net MON_5V: now also C226.1; no longer C227.1
- net MON_VSYS: now also C225.1; no longer C226.1
- net SS_12V: now also C214.1; no longer C215.1
- net SW_3V3: now also C193.2; no longer C194.2
- net SW_5V: now also C188.2; no longer C189.2
- net VBUS: now also C187.1, C183.2; no longer C184.2, C188.1
- net VBUS5_GATE: now also C183.1; no longer C184.1
- net VBUS_DVDT: now also C184.1; no longer C185.1
- net VCCIO_1: now also C220.1; no longer C221.1
- net VCCIO_2: now also C221.1; no longer C222.1
- net VIN_EXT: now also D8.1 (K)
- net VSYS: now also C185.1, C192.1; no longer C187.1, C193.1
Other:
- moved on the sheet: C184, C185, C186, C187, C188, C189, C190, C191, C192, C194, C195, C196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
