File: kicad/power.kicad_sch (KiCad schematic)
At the start: 126 parts, among them J50 9-14V POWER IN, Q2 DMG2305UX-7, Q3 BSS138LT1G, U11 TPS54202DDCR, U12 AP63300WU-7, U13 TLV62569DRLR, U14 TLV62569DRLR, U15 SY8047QDC, U16 TLV62569DRLR, U19 TPS61085PWR, U21 TPS22950CDDCR, U22 TPS22950CDDCR, U23 TPS22950CDDCR, U24 TPS22950CDDCR, U25 TPS259470LRPWR, U26 TPS259470ARPWR

Commit message: Through-hole extension headers, AUX supply rework, and board state before rev A cleanup
J3/J5 become single 2x32 through-hole bodies with IO IO GND rows and a long
grounded key post per zone. Power sheet reworked around the AUX rail.
Decoupling moved off B.Cu. New footprints, 3D models and check scripts.
Parts:
- removed C213: 2.2nF, Capacitor_SMD:C_0402_1005Metric, symbol Device:C
- removed C214: 10nF, Capacitor_SMD:C_0402_1005Metric, symbol Device:C
- removed C215, C216, C232: 10uF 25V, Capacitor_SMD:C_0805_2012Metric, symbol Device:C
- removed C217: 10uF, Capacitor_SMD:C_0805_2012Metric, symbol Device:C
- removed C222: 3.3nF 25V, Capacitor_SMD:C_0402_1005Metric, symbol Device:C
- removed C223: 1uF 25V, Capacitor_SMD:C_0603_1608Metric, symbol Device:C
- removed D5: SS34, EasyEDA:SMA_L4.3-W2.6-LS5.2-RD, symbol Device:D_Schottky
- removed L8: 10uH SRN6045TA-100M, EasyEDA:IND-SMD_L6.0-W6.0-1, symbol Device:L
- removed R69, R95: 100k, Resistor_SMD:R_0603_1608Metric, symbol Device:R
- removed R70: 11.5k, Resistor_SMD:R_0603_1608Metric, symbol Device:R
- removed R71: 47k, Resistor_SMD:R_0402_1005Metric, symbol Device:R
- removed R78: 121k, Resistor_SMD:R_0603_1608Metric, symbol Device:R
- removed R79: 12.1k, Resistor_SMD:R_0603_1608Metric, symbol Device:R
- removed R80: 6.65k, Resistor_SMD:R_0603_1608Metric, symbol Device:R
- removed U19: TPS61085PWR, EasyEDA:TSSOP-8_L4.4-W3.0-P0.65-LS6.4-BL, symbol Regulator_Switching:TPS61085PW
- removed U25: TPS259470LRPWR, Package_DFN_QFN:Texas_RPU0010A_VQFN-HR-10_2x2mm_P0.5mm, symbol odin:TPS259470LRPW
- added C233, C234, C241, C242, C243, C244, C245: 10uF 50V X7R, Capacitor_SMD:C_1210_3225Metric, symbol Device:C
- added C235, C246: 100nF 50V, Capacitor_SMD:C_0603_1608Metric, symbol Device:C
- added C236: 1uF 16V, Capacitor_SMD:C_0603_1608Metric, symbol Device:C
- added C237, C238: 47nF 50V, Capacitor_SMD:C_0603_1608Metric, symbol Device:C
- added C239: 220pF 50V, Capacitor_SMD:C_0603_1608Metric, symbol Device:C
- added C240: 10uF 50V X7R SEPIC, Capacitor_SMD:C_1210_3225Metric, symbol Device:C
- added C247: 100nF, Capacitor_SMD:C_0402_1005Metric, symbol Device:C
- added D12: PMEG060V100EPDZ, EasyEDA:SOT1289_L5.8-W4.4-LS6.5-RD, symbol EasyEDA:PMEG060V100EPDZ
- added D13, D14, D15, D16: 1N4148W, Diode_SMD:D_SOD-123, symbol Device:D
- added J66: AUX SOURCE REG/AUX/RAW, Connector_PinHeader_2.54mm:PinHeader_1x03_P2.54mm_Vertical, symbol Connector_Generic:Conn_01x03
- added J67: AUX VOLTAGE 9/12/15/24; ONE CAP ONLY, Connector_PinHeader_2.54mm:PinHeader_2x04_P2.54mm_Vertical, symbol Connector_Generic:Conn_02x04_Odd_Even
- added J68: AUX IN 9-28V UNREGULATED, EasyEDA:CONN-TH_P5.00_KF301-5.0-2P, symbol EasyEDA:KF301-5.0-2P
- added L10: PSSCAQ1285-4R7MP 4.7uH coupled, odin:L_PROD_PSSCAQ1285, symbol odin:PSSCAQ1285_4R7MP
- added Q5, Q6, Q7, Q8: BSS138LT1G, EasyEDA:SOT-23-3_L2.9-W1.6-P1.90-LS2.8-BR, symbol Transistor_FET:Q_NMOS_GSD
- added R131: 4.99, Resistor_SMD:R_0603_1608Metric, symbol Device:R
- added R132: 49.9k, Resistor_SMD:R_0603_1608Metric, symbol Device:R
- added R133: 62k, Resistor_SMD:R_0603_1608Metric, symbol Device:R
- added R134: 2k, Resistor_SMD:R_0603_1608Metric, symbol Device:R
- added R135: 10k 1%, Resistor_SMD:R_0603_1608Metric, symbol Device:R
- added R136: 80.6k 1%, Resistor_SMD:R_0603_1608Metric, symbol Device:R
- added R137, R138: 30.1k 1%, Resistor_SMD:R_0603_1608Metric, symbol Device:R
- added R139: 90.9k 1%, Resistor_SMD:R_0603_1608Metric, symbol Device:R
- added R140, R141, R142, R143, R144: 100k, Resistor_SMD:R_0402_1005Metric, symbol Device:R
- added U28: LM5157RTER, Package_DFN_QFN:WQFN-16-1EP_3x3mm_P0.5mm_EP1.68x1.68mm_ThermalVias, symbol odin:LM5157RTE
- added U29: 74HC04D,653, Package_SO:SOIC-14_3.9x8.7mm_P1.27mm, symbol odin:74HC04D
- C185, C186: value 22uF 25V -> 10uF 50V; footprint Capacitor_SMD:C_0805_2012Metric -> Capacitor_SMD:C_1210_3225Metric; LCSC C86816 -> C77102
- C192: value 10uF 25V -> 10uF 50V; footprint Capacitor_SMD:C_0805_2012Metric -> Capacitor_SMD:C_1210_3225Metric; LCSC C15850 -> C77102
- D8: value SMBJ15A-13-F -> SMBJ22A; LCSC C135046 -> C151920
- J50: value 9-14V POWER IN -> 9-21V POWER IN
- L2: value 10uH SRN6045TA-100M -> 4.7uH SRN6045TA-4R7M; footprint EasyEDA:IND-SMD_L6.0-W6.0-1 -> EasyEDA:IND-SMD_L6.0-W6.0; LCSC C2046332 -> C2044594
- R56: value 13.7k -> 19.1k
- U11: value TPS54202DDCR -> AP63300WU-7; footprint EasyEDA:SOT-23-6_L2.9-W1.6-P0.95-LS2.8-BL -> EasyEDA:TSOT-23-6_L2.9-W1.6-P0.95-LS2.8-BR; symbol Regulator_Switching:TPS54202DDC -> odin:AP63300WU; LCSC C191884 -> C2158012
Connections:
- net +3V3: now also C247.1, R140.1, R141.1, R142.1, R143.1, U29.14 (VCC)
- net EN_5V: now also U11.2 (EN); no longer U11.5 (EN)
- net FB_5V: now also U11.1 (FB); no longer U11.4 (FB)
- net GND: now also U11.4 (GND), C233.2, C234.2, C235.2, C236.2, C237.2, C238.2, C239.2, C241.2, C242.2, C243.2, C244.2, C245.2, C246.2, C247.2, J67.2 (Pin_2), J67.4 (Pin_4), J67.6 (Pin_6), J67.8 (Pin_8), J68.2, L10.2 (SEC_DOT), R132.2, R133.2, R135.2, R144.2, U28.1 (PGND1), U28.16 (PGND2), U28.17 (EP), U28.7 (AGND), U29.11 (A5), U29.13 (A6), U29.7 (GND); no longer U11.1 (GND)
- net SW_5V: now also U11.5 (SW); no longer U11.2 (SW)
- net VSYS: now also C233.1, C234.1, C235.1, L10.1 (PRI_DOT), U28.3 (BIAS)
- new net AUX_COMP: C239.1, R134.1, U28.8 (COMP)
- new net AUX_COMP_C: C238.1, R134.2
- new net AUX_EN: D13.1 (K), D14.1 (K), D15.1 (K), D16.1 (K), R144.1, U28.6 (UVLO/SYNC/EN)
- new net AUX_FB: Q5.2 (S), Q6.2 (S), Q7.2 (S), Q8.2 (S), R135.1, U28.9 (FB)
- new net AUX_MODE: R133.1, U28.11 (MODE)
- new net AUX_RAIL: J66.2 (Pin_2)
- new net AUX_RAW: J66.3 (Pin_3), J68.1
- new net AUX_REG: C241.1, C242.1, C243.1, C244.1, C245.1, C246.1, D12.3 (K), J66.1 (Pin_1), R136.1
- new net AUX_RT: R132.1, U28.5 (RT)
- new net AUX_SEL_12: J67.3 (Pin_3), R141.2, U29.3 (A2)
- new net AUX_SEL_12_ON: D14.2 (A), Q6.1 (G), U29.4 (Y2)
- new net AUX_SEL_15: J67.5 (Pin_5), R142.2, U29.5 (A3)
- new net AUX_SEL_15_ON: D15.2 (A), Q7.1 (G), U29.6 (Y3)
- new net AUX_SEL_24: J67.7 (Pin_7), R143.2, U29.9 (A4)
- new net AUX_SEL_24_ON: D16.2 (A), Q8.1 (G), U29.8 (Y4)
- new net AUX_SEL_9: J67.1 (Pin_1), R140.2, U29.1 (A1)
- new net AUX_SEL_9_ON: D13.2 (A), Q5.1 (G), U29.2 (Y1)
- new net AUX_SEPIC: C240.2, D12.1 (A), D12.2 (A), L10.4 (SEC)
- new net AUX_SS: C237.1, U28.10 (SS)
- new net AUX_SW: C240.1, L10.3 (PRI), U28.12 (SW1), U28.13 (SW2), U28.14 (SW3)
- new net AUX_TAP_12: Q6.3 (D), R137.2, R138.1
- new net AUX_TAP_15: Q7.3 (D), R138.2, R139.1
- new net AUX_TAP_24: Q8.3 (D), R139.2
- new net AUX_TAP_9: Q5.3 (D), R136.2, R137.1
- new net AUX_VCC: C236.1, R131.2
- new net AUX_VCC_PIN: R131.1, U28.2 (VCC)
- no-connect marks 12 -> 14
Other:
- note added: "AUX lab rail"
- note added: "POWER — Power tree: VSYS input, selectable AUX lab rail and monitoring — HW 0.1.0-proto.1"
- note added: "U11 VSYS to +5V"
- note removed: "POWER — Power tree: 12V input to every rail, with monitoring — HW 0.1.0-proto.1"
- note removed: "U11 12V to 5V"
- note removed: "U19 5V to 12V boost (AUX)"
- note removed: "U25 +12V to +12V_EXT"
- moved on the sheet: C184, C185, C186, C188, C189, C190, C191, C198, C199, C200, C201, C202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

Commit message: Remove the AUX lab rail: J68 feeds AUX_RAIL straight into the ten branch PTCs
Decision D1 of the rev A plan. The LM5157 SEPIC (U28, L10, D12), the
cap-selected 9/12/15/24 V feedback ladder (J67, U29, Q5-Q8, D13-D16) and
the REG/AUX/RAW source selector J66 are gone, 43 parts in all. The AUX
pin of every power row is now fed only from the AUX IN screw terminal
through its slot's 33 V PTC. The SMBJ22A clamp plus a charged 24 V
output could exceed the LM5157 SW pin's 50 V absolute maximum, and the
converter is not needed for a board that configures and runs.

budget.py drops the SEPIC derating math and the surge release hold;
qualified.py, gen_kicad.py, gen_project.py, the connector checker, the
silkscreen labels and the power docs follow. PCB synced with load_pcb.py,
0 of 477 footprints moved; DRC errors 49 -> 18.
Parts:
- removed C233, C234, C241, C242, C243, C244, C245: 10uF 50V X7R, Capacitor_SMD:C_1210_3225Metric, symbol Device:C
- removed C235, C246: 100nF 50V, Capacitor_SMD:C_0603_1608Metric, symbol Device:C
- removed C236: 1uF 16V, Capacitor_SMD:C_0603_1608Metric, symbol Device:C
- removed C237, C238: 47nF 50V, Capacitor_SMD:C_0603_1608Metric, symbol Device:C
- removed C239: 220pF 50V, Capacitor_SMD:C_0603_1608Metric, symbol Device:C
- removed C240: 10uF 50V X7R SEPIC, Capacitor_SMD:C_1210_3225Metric, symbol Device:C
- removed C247: 100nF, Capacitor_SMD:C_0402_1005Metric, symbol Device:C
- removed D12: PMEG060V100EPDZ, EasyEDA:SOT1289_L5.8-W4.4-LS6.5-RD, symbol EasyEDA:PMEG060V100EPDZ
- removed D13, D14, D15, D16: 1N4148W, Diode_SMD:D_SOD-123, symbol Device:D
- removed J66: AUX SOURCE REG/AUX/RAW, Connector_PinHeader_2.54mm:PinHeader_1x03_P2.54mm_Vertical, symbol Connector_Generic:Conn_01x03
- removed J67: AUX VOLTAGE 9/12/15/24; ONE CAP ONLY, Connector_PinHeader_2.54mm:PinHeader_2x04_P2.54mm_Vertical, symbol Connector_Generic:Conn_02x04_Odd_Even
- removed L10: PSSCAQ1285-4R7MP 4.7uH coupled, odin:L_PROD_PSSCAQ1285, symbol odin:PSSCAQ1285_4R7MP
- removed Q5, Q6, Q7, Q8: BSS138LT1G, EasyEDA:SOT-23-3_L2.9-W1.6-P1.90-LS2.8-BR, symbol Transistor_FET:Q_NMOS_GSD
- removed R131: 4.99, Resistor_SMD:R_0603_1608Metric, symbol Device:R
- removed R132: 49.9k, Resistor_SMD:R_0603_1608Metric, symbol Device:R
- removed R133: 62k, Resistor_SMD:R_0603_1608Metric, symbol Device:R
- removed R134: 2k, Resistor_SMD:R_0603_1608Metric, symbol Device:R
- removed R135: 10k 1%, Resistor_SMD:R_0603_1608Metric, symbol Device:R
- removed R136: 80.6k 1%, Resistor_SMD:R_0603_1608Metric, symbol Device:R
- removed R137, R138: 30.1k 1%, Resistor_SMD:R_0603_1608Metric, symbol Device:R
- removed R139: 90.9k 1%, Resistor_SMD:R_0603_1608Metric, symbol Device:R
- removed R140, R141, R142, R143, R144: 100k, Resistor_SMD:R_0402_1005Metric, symbol Device:R
- removed U28: LM5157RTER, Package_DFN_QFN:WQFN-16-1EP_3x3mm_P0.5mm_EP1.68x1.68mm_ThermalVias, symbol odin:LM5157RTE
- removed U29: 74HC04D,653, Package_SO:SOIC-14_3.9x8.7mm_P1.27mm, symbol odin:74HC04D
Connections:
- net AUX_RAW is gone; now on net AUX_RAIL: J68.1
- no-connect marks 14 -> 10
Other:
- note added: "AUX IN"
- note added: "POWER — Power tree: VSYS input, regulators, AUX IN pass-through and monitoring — HW 0.1.0-proto.1"
- note removed: "AUX lab rail"
- note removed: "POWER — Power tree: VSYS input, selectable AUX lab rail and monitoring — HW 0.1.0-proto.1"
- moved on the sheet: C207, C208, C209, C210, C211, C212, C218, C219, C220, C221, C224, C225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

Commit message: Explain the remaining four sheets: power, memory, board controller, slots
Every part and group on the board now has its plain-words purpose, and the
gate enforces it on all six sheets. Net notes can cover a family of nets
by prefix, so regulator feedback, enables and the PSRAM series resistors
read correctly; passives credit their group's IC or connector rather than
a key post; monitor nets are no longer mistaken for supplies; parts that
are not fitted say so. PCB synced with no footprint moved.
Other:
- note added: "A shortcut for plain 5 V USB. A regulator cannot make 5 V out of 5 V, so when the USB source is 5 V the board controller turns Q2 on and USB power goes straight onto the +5V rail. It is off by default and must stay off at 9 V, or 9 V would reach parts rated for 5.5 V; Q3 is the small transistor the controller uses to switch it."
- note added: "A small inductor and capacitor that make +1V0_MGT from +1V0: the same voltage, with the core's switching noise filtered out, for the transceivers' MGTAVCC supply."
- note added: "Lets the board controller measure every supply. Each rail goes to one of its analog inputs (ADC), which read 0-3.3 V. Rails at or below 3.3 V go through a 1 k resistor that protects the pin; VSYS and +5V are higher, so two resistors divide them down first. A 100 nF capacitor on each input steadies the reading. Firmware uses this to check each regulator came up before enabling the next."
- note added: "Optional extra power for extensions that need more than 5 V (motors, LED strips, displays). Whatever you connect here (9-28 V DC) goes, unregulated, to the AUX pin of every extension port through each port's own fuse. The board itself never uses it."
- note added: "Protected switch between +3V3 and the 3.3 V pins of every extension port, limited to about 0.5 A, with reverse blocking. Keeps a faulty extension from taking down the board controller's supply."
- note added: "Protected switch between the board's +5V and the 5 V pins of every extension port. Limits current to about 1 A and blocks current flowing back from an extension. Without it, a shorted extension would pull the whole board's 5 V down."
- note added: "Protected switch for the PIN V supply of slots A-D (the voltage chosen on J19), limited to about 0.5 A, with reverse blocking."
- note added: "Protected switch for the PIN V supply of slots E-H (the voltage chosen on J20), limited to about 0.5 A, with reverse blocking."
- note added: "Shared control for the four protected extension supplies (U21-U24). EXT_EN, from the board controller, turns them all on; the pull-down keeps them off until firmware decides. EXT_FAULT is pulled up and goes low if any of them (or the USB eFuse) detects a fault, so one controller pin hears all of them."
- note added: "Small switching regulator that makes +1V2_MGT from +5V for the FPGA transceivers' MGTAVTT supply. The transceivers are unused in rev A but must stay powered. Enabled by the board controller (EN_1V2)."
- note added: "Small switching regulator that makes +1V8 from +5V for the FPGA's auxiliary supply (VCCAUX) and its ADC. Enabled by the board controller (EN_1V8); the feedback resistors set 1.8 V."
- note added: "Small switching regulator that makes +2V5 from +5V for FPGA bank 16 (network) and the PHY's RGMII pins. Enabled by the board controller (EN_2V5); the feedback resistors set 2.5 V."
- note added: "Switching regulator (buck converter) that makes +5V from VSYS. +5V feeds the 5 V buses, the extension 5 V pins and the four small regulators below. The board controller turns it on (EN_5V); the pull-down keeps it off until then. The two feedback resistors set the output voltage; the inductor and capacitors are its power stage."
- note added: "Switching regulator that makes +3V3 from VSYS. It has no enable: it starts as soon as any power is present, because +3V3 runs the board controller, which then switches everything else on. Also powers the PSRAM, the flashes, the PHY and most logic. The two feedback resistors set 3.3 V; the inductor and capacitors are its power stage."
- note added: "The FPGA core supply: up to 4 A at 1.0 V from +5V, the heaviest rail on the board. Enabled by the board controller (EN_1V0); its power-good output (CORE_1V0_GOOD) is read through the status expander so firmware knows the core is up. The soft-start capacitor makes it ramp slowly; the feedback resistors set 1.0 V."
- note added: "Where power enters. Two inputs feed one internal supply, VSYS: USB-C (5 V, or 9 V when a USB-PD charger agrees) and the J50 screw terminal (9-21 V). A diode on each (D3, D4) lets whichever is higher supply the board and stops one input from back-feeding the other. On the USB side, U26 is an electronic fuse: it ramps the voltage up gently so plugging in does not spark, cuts off above about 10 V or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"
- moved on the sheet: C183, C184, C185, C186, C187, C188, C189, C190, C191, C192, C193, C194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

Commit message: Step 1: the +1V8_IO rail
Parts:
- added C250: 10uF, Capacitor_SMD:C_0805_2012Metric, symbol Device:C
- added C251: 100nF, Capacitor_SMD:C_0402_1005Metric, symbol Device:C
- added FB1: 120R 2A BLM18PG121SN1D, Inductor_SMD:L_0603_1608Metric, symbol Device:FerriteBead
Connections:
- net +1V8: now also FB1.2; no longer C201.1, C202.1, L5.1, R61.1, R87.1
- net GND: now also C250.2, C251.2
- net FB+1V8 renamed FB+1V8_IO
- net SW+1V8 renamed SW+1V8_IO
- new net +1V8_IO: C201.1, C202.1, C250.1, C251.1, FB1.1, L5.1, R61.1, R87.1
Other:
- note added: "Small switching regulator that makes 1.8 V from +5V. Its output node is +1V8_IO: FPGA bank 13 and the 1.8 V memory on it, the 1.8 V position of the J19/J20 jumpers, and, through the bead below, the FPGA's auxiliary supply (VCCAUX) and its ADC as +1V8. Enabled by the board controller (EN_1V8); the feedback resistors set 1.8 V."
- note added: "The split between +1V8_IO and +1V8. VCCAUX and VCCADC are the FPGA's internal supplies (clocking, I/O pre- drivers, the XADC) and should not share copper with switching 1.8 V I/O loads, so they hang off U14's output through one ferrite bead (120 ohm at 100 MHz, 2 A, 50 mohm: 9 mV at the 0.18 A VCCAUX allowance, inside VCCAUX's 1.71 V minimum). The 10 uF and 100 nF sit at U14's output beside its o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"
- note added: "U14 5V to +1V8_IO"
- note added: "VCCAUX filter"
- note removed: "Small switching regulator that makes +1V8 from +5V for the FPGA's auxiliary supply (VCCAUX) and its ADC. Enabled by the board controller (EN_1V8); the feedback resistors set 1.8 V."
- note removed: "U14 5V to +1V8"
- moved on the sheet: C220, C221, C224, L9, R76, R77, U23, U24
