File: kicad/power.kicad_sch (KiCad schematic)
At the start: 111 parts, among them J50 9-21V POWER IN, J68 AUX IN 9-28V UNREGULATED, Q2 DMG2305UX-7, Q3 BSS138LT1G, U11 AP63300WU-7, U12 AP63300WU-7, U13 TLV62569DRLR, U14 TLV62569DRLR, U15 SY8047QDC, U16 TLV62569DRLR, U21 TPS22950CDDCR, U22 TPS22950CDDCR, U23 TPS22950CDDCR, U24 TPS22950CDDCR, U26 TPS259470ARPWR

Commit message: Step 4: SDRAM
Parts:
- removed C250: 10uF, Capacitor_SMD:C_0805_2012Metric, symbol Device:C
- removed C251: 100nF, Capacitor_SMD:C_0402_1005Metric, symbol Device:C
- added C258: 10uF, Capacitor_SMD:C_0805_2012Metric, symbol Device:C
- added C259: 100nF, Capacitor_SMD:C_0402_1005Metric, symbol Device:C
Connections:
- net +1V8_IO: now also C258.1, C259.1
- net GND: now also C258.2, C259.2
Changed lines of the file:
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@@
 	(symbol (lib_id "Device:C") (at 55.88 1071.88 0) (unit 1)
 		(exclude_from_sim no) (in_bom yes) (on_board yes) (dnp no)
-		(property "Reference" "C251" (at 55.88 1064.26 0) (effects (font (size 1.27 1.27))))
+		(property "Reference" "C259" (at 55.88 1064.26 0) (effects (font (size 1.27 1.27))))
 		(property "Value" "100nF" (at 55.88 1079.5 0) (effects (font (size 1.27 1.27))))
 		(property "Footprint" "Capacitor_SMD:C_0402_1005Metric" (at 55.88 1079.5 0) (effects (font (size 1.27 1.27)) (hide yes)))
 		(property "LCSC" "C1525" (at 55.88 1079.5 0) (effects (font (size 1.27 1.27)) (hide yes)))
 		(property "Description" "100nF bypass on +1V8_IO" (at 55.88 1079.5 0) (effects (font (size 1.27 1.27)) (hide yes)))
-		(instances (project "odin" (path "/c44fb7fe-6133-ad34-68fd-fb66126197ef/d8079187-14d6-b109-30bb-e1c878749fb7" (reference "C251") (unit 1))))
+		(instances (project "odin" (path "/c44fb7fe-6133-ad34-68fd-fb66126197ef/d8079187-14d6-b109-30bb-e1c878749fb7" (reference "C259") (unit 1))))
 	)
 	(wire (pts (xy 55.88 1068.07) (xy 55.88 1065.53)) (stroke (width 0) (type default)))
@@
 	(symbol (lib_id "Device:C") (at 88.9 1071.88 0) (unit 1)
 		(exclude_from_sim no) (in_bom yes) (on_board yes) (dnp no)
-		(property "Reference" "C250" (at 88.9 1064.26 0) (effects (font (size 1.27 1.27))))
+		(property "Reference" "C258" (at 88.9 1064.26 0) (effects (font (size 1.27 1.27))))
 		(property "Value" "10uF" (at 88.9 1079.5 0) (effects (font (size 1.27 1.27))))
 		(property "Footprint" "Capacitor_SMD:C_0805_2012Metric" (at 88.9 1079.5 0) (effects (font (size 1.27 1.27)) (hide yes)))
 		(property "LCSC" "C15850" (at 88.9 1079.5 0) (effects (font (size 1.27 1.27)) (hide yes)))
 		(property "Description" "10uF bypass on +1V8_IO" (at 88.9 1079.5 0) (effects (font (size 1.27 1.27)) (hide yes)))
-		(instances (project "odin" (path "/c44fb7fe-6133-ad34-68fd-fb66126197ef/d8079187-14d6-b109-30bb-e1c878749fb7" (reference "C250") (unit 1))))
+		(instances (project "odin" (path "/c44fb7fe-6133-ad34-68fd-fb66126197ef/d8079187-14d6-b109-30bb-e1c878749fb7" (reference "C258") (unit 1))))
 	)
 	(wire (pts (xy 88.9 1068.07) (xy 88.9 1065.53)) (stroke (width 0) (type default)))

Commit message: Step 5: MRAM, optional populate
Parts:
- removed C258: 10uF, Capacitor_SMD:C_0805_2012Metric, symbol Device:C
- added C260: 100nF, Capacitor_SMD:C_0402_1005Metric, symbol Device:C
- C259: value 100nF -> 10uF; footprint Capacitor_SMD:C_0402_1005Metric -> Capacitor_SMD:C_0805_2012Metric; LCSC C1525 -> C15850
Connections:
- net +1V8_IO: now also C260.1
- net GND: now also C260.2
Other:
- moved on the sheet: C259
Changed lines of the file:
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@@
 	(symbol (lib_id "Device:C") (at 55.88 1071.88 0) (unit 1)
 		(exclude_from_sim no) (in_bom yes) (on_board yes) (dnp no)
-		(property "Reference" "C259" (at 55.88 1064.26 0) (effects (font (size 1.27 1.27))))
+		(property "Reference" "C260" (at 55.88 1064.26 0) (effects (font (size 1.27 1.27))))
 		(property "Value" "100nF" (at 55.88 1079.5 0) (effects (font (size 1.27 1.27))))
 		(property "Footprint" "Capacitor_SMD:C_0402_1005Metric" (at 55.88 1079.5 0) (effects (font (size 1.27 1.27)) (hide yes)))
 		(property "LCSC" "C1525" (at 55.88 1079.5 0) (effects (font (size 1.27 1.27)) (hide yes)))
 		(property "Description" "100nF bypass on +1V8_IO" (at 55.88 1079.5 0) (effects (font (size 1.27 1.27)) (hide yes)))
-		(instances (project "odin" (path "/c44fb7fe-6133-ad34-68fd-fb66126197ef/d8079187-14d6-b109-30bb-e1c878749fb7" (reference "C259") (unit 1))))
+		(instances (project "odin" (path "/c44fb7fe-6133-ad34-68fd-fb66126197ef/d8079187-14d6-b109-30bb-e1c878749fb7" (reference "C260") (unit 1))))
 	)
 	(wire (pts (xy 55.88 1068.07) (xy 55.88 1065.53)) (stroke (width 0) (type default)))
@@
 	(symbol (lib_id "Device:C") (at 88.9 1071.88 0) (unit 1)
 		(exclude_from_sim no) (in_bom yes) (on_board yes) (dnp no)
-		(property "Reference" "C258" (at 88.9 1064.26 0) (effects (font (size 1.27 1.27))))
+		(property "Reference" "C259" (at 88.9 1064.26 0) (effects (font (size 1.27 1.27))))
 		(property "Value" "10uF" (at 88.9 1079.5 0) (effects (font (size 1.27 1.27))))
 		(property "Footprint" "Capacitor_SMD:C_0805_2012Metric" (at 88.9 1079.5 0) (effects (font (size 1.27 1.27)) (hide yes)))
 		(property "LCSC" "C15850" (at 88.9 1079.5 0) (effects (font (size 1.27 1.27)) (hide yes)))
 		(property "Description" "10uF bypass on +1V8_IO" (at 88.9 1079.5 0) (effects (font (size 1.27 1.27)) (hide yes)))
-		(instances (project "odin" (path "/c44fb7fe-6133-ad34-68fd-fb66126197ef/d8079187-14d6-b109-30bb-e1c878749fb7" (reference "C258") (unit 1))))
+		(instances (project "odin" (path "/c44fb7fe-6133-ad34-68fd-fb66126197ef/d8079187-14d6-b109-30bb-e1c878749fb7" (reference "C259") (unit 1))))
 	)
 	(wire (pts (xy 88.9 1068.07) (xy 88.9 1065.53)) (stroke (width 0) (type default)))

Commit message: Step 6: microSD socket
Parts:
- removed C259: 10uF, Capacitor_SMD:C_0805_2012Metric, symbol Device:C
- removed C260: 100nF, Capacitor_SMD:C_0402_1005Metric, symbol Device:C
- added C261: 10uF, Capacitor_SMD:C_0805_2012Metric, symbol Device:C
- added C262: 100nF, Capacitor_SMD:C_0402_1005Metric, symbol Device:C
Connections:
- net +1V8_IO: now also C261.1, C262.1
- net GND: now also C261.2, C262.2
Changed lines of the file:
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@@
 	(symbol (lib_id "Device:C") (at 55.88 1071.88 0) (unit 1)
 		(exclude_from_sim no) (in_bom yes) (on_board yes) (dnp no)
-		(property "Reference" "C260" (at 55.88 1064.26 0) (effects (font (size 1.27 1.27))))
+		(property "Reference" "C262" (at 55.88 1064.26 0) (effects (font (size 1.27 1.27))))
 		(property "Value" "100nF" (at 55.88 1079.5 0) (effects (font (size 1.27 1.27))))
 		(property "Footprint" "Capacitor_SMD:C_0402_1005Metric" (at 55.88 1079.5 0) (effects (font (size 1.27 1.27)) (hide yes)))
 		(property "LCSC" "C1525" (at 55.88 1079.5 0) (effects (font (size 1.27 1.27)) (hide yes)))
 		(property "Description" "100nF bypass on +1V8_IO" (at 55.88 1079.5 0) (effects (font (size 1.27 1.27)) (hide yes)))
-		(instances (project "odin" (path "/c44fb7fe-6133-ad34-68fd-fb66126197ef/d8079187-14d6-b109-30bb-e1c878749fb7" (reference "C260") (unit 1))))
+		(instances (project "odin" (path "/c44fb7fe-6133-ad34-68fd-fb66126197ef/d8079187-14d6-b109-30bb-e1c878749fb7" (reference "C262") (unit 1))))
 	)
 	(wire (pts (xy 55.88 1068.07) (xy 55.88 1065.53)) (stroke (width 0) (type default)))
@@
 	(symbol (lib_id "Device:C") (at 88.9 1071.88 0) (unit 1)
 		(exclude_from_sim no) (in_bom yes) (on_board yes) (dnp no)
-		(property "Reference" "C259" (at 88.9 1064.26 0) (effects (font (size 1.27 1.27))))
+		(property "Reference" "C261" (at 88.9 1064.26 0) (effects (font (size 1.27 1.27))))
 		(property "Value" "10uF" (at 88.9 1079.5 0) (effects (font (size 1.27 1.27))))
 		(property "Footprint" "Capacitor_SMD:C_0805_2012Metric" (at 88.9 1079.5 0) (effects (font (size 1.27 1.27)) (hide yes)))
 		(property "LCSC" "C15850" (at 88.9 1079.5 0) (effects (font (size 1.27 1.27)) (hide yes)))
 		(property "Description" "10uF bypass on +1V8_IO" (at 88.9 1079.5 0) (effects (font (size 1.27 1.27)) (hide yes)))
-		(instances (project "odin" (path "/c44fb7fe-6133-ad34-68fd-fb66126197ef/d8079187-14d6-b109-30bb-e1c878749fb7" (reference "C259") (unit 1))))
+		(instances (project "odin" (path "/c44fb7fe-6133-ad34-68fd-fb66126197ef/d8079187-14d6-b109-30bb-e1c878749fb7" (reference "C261") (unit 1))))
 	)
 	(wire (pts (xy 88.9 1068.07) (xy 88.9 1065.53)) (stroke (width 0) (type default)))

Commit message: Power path: U34 mux replaces the Q2 bypass, U11/U14 always on, PD defaults to 5 V, USB series resistors, native controller pins
Parts:
- removed C183: 100nF 25V, Capacitor_SMD:C_0402_1005Metric, symbol Device:C
- removed Q2: DMG2305UX-7, EasyEDA:SOT-23-3_L2.9-W1.3-P1.90-LS2.4-BR, symbol Transistor_FET:Q_PMOS_GSD
- removed Q3: BSS138LT1G, EasyEDA:SOT-23-3_L2.9-W1.6-P1.90-LS2.8-BR, symbol Transistor_FET:Q_NMOS_GSD
- removed R46, R90, R92: 100k, Resistor_SMD:R_0603_1608Metric, symbol Device:R
- removed R47: 10k, Resistor_SMD:R_0402_1005Metric, symbol Device:R
- removed R48: 100k, Resistor_SMD:R_0402_1005Metric, symbol Device:R
- removed R49: 47k, Resistor_SMD:R_0603_1608Metric, symbol Device:R
- added C263: 100nF, Capacitor_SMD:C_0402_1005Metric, symbol Device:C
- added C264: 100nF 25V, Capacitor_SMD:C_0402_1005Metric, symbol Device:C
- added C265, C266: 22uF, Capacitor_SMD:C_0805_2012Metric, symbol Device:C
- added C267: 10uF 50V, Capacitor_SMD:C_1210_3225Metric, symbol Device:C
- added C268, C269, C270: 4.7uF, Capacitor_SMD:C_0603_1608Metric, symbol Device:C
- added R162, R164, R166: 100k, Resistor_SMD:R_0603_1608Metric, symbol Device:R
- added R163: 36.5k, Resistor_SMD:R_0603_1608Metric, symbol Device:R
- added R165: 23.2k, Resistor_SMD:R_0603_1608Metric, symbol Device:R
- added R167: 56.2k, Resistor_SMD:R_0603_1608Metric, symbol Device:R
- added R168: 44.2k, Resistor_SMD:R_0603_1608Metric, symbol Device:R
- added R169: 10k, Resistor_SMD:R_0603_1608Metric, symbol Device:R
- added U34: TPS2121RUXR, Package_DFN_QFN:Texas_VQFN-HR-12_2x2.5mm_P0.5mm, symbol odin:TPS2121RUX
Connections:
- net EN_1V8 is gone; now on net +5V: U14.5 (EN)
- net +1V8: now also R87.1
- net +1V8_IO: no longer R87.1
- net +3V3: now also R166.1, R169.1
- net +5V: now also C265.1, C266.1, C268.1, C269.1, C270.1, U34.1 (OUT), U34.8 (OUT); no longer C189.1, C190.1, C191.1, L2.1, R55.1
- net GND: now also C263.2, C264.2, C265.2, C266.2, C267.2, C268.2, C269.2, C270.2, R163.2, R165.2, R167.2, R168.2, U34.12 (GND), U34.4 (OV2)
- net VBUS: now also C264.1, R162.1, R164.1, U34.7 (IN1)
- net VSYS: now also C267.1
- net EN_5V: no longer names the net of U11.2 (EN)
- new net +5V_BUCK: C189.1, C190.1, C191.1, L2.1, R55.1, U34.2 (IN2)
- new net VBUS5_CP2: R166.2, R167.1, U34.3 (CP2)
- new net VBUS5_ILIM: R168.1, U34.10 (ILIM)
- new net VBUS5_OV1: R164.2, R165.1, U34.5 (OV1)
- new net VBUS5_PR1: R162.2, R163.1, U34.6 (PR1)
- new net VBUS5_SS: C263.1, U34.11 (SS)
- new net VBUS5_ST: R169.2, U34.9 (ST)
- no-connect marks 10 -> 11
Other:
- note added: "Chooses what feeds the +5V rail: USB power straight from the connector, or U11. A regulator cannot make 5 V out of 5 V, so on a plain 5 V USB source the mux passes VBUS to the rail; the moment a USB-PD charger raises VBUS above about 5.6 V, or VBUS is absent, it switches to U11 within microseconds. The choice is set by three resistor dividers, not by firmware, and the chip blocks current flowing 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"
- note added: "Lets the board controller measure every supply. Each rail goes to one of its eight analog inputs (ADC), which read 0-3.3 V. Rails at or below 3.3 V go through a 1 k resistor that protects the pin; VSYS and +5V are higher, so two resistors divide them down first. A 100 nF capacitor on each input steadies the reading. MON_1V8 reads +1V8 itself, the FPGA's VCCAUX behind the bead, so an open bead sho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"
- note added: "Small switching regulator that makes 1.8 V from +5V. Its output node is +1V8_IO: FPGA bank 13 and the 1.8 V memory on it, the 1.8 V position of the J19/J20 jumpers, and, through the bead below, the FPGA's auxiliary supply (VCCAUX) and its ADC as +1V8. Its enable is tied to +5V, so it runs whenever U11 does: the FPGA's 3.3 V banks are never left on an unpowered VCCAUX (DS181 Table 7). The feedback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"
- note added: "Switching regulator (buck converter) that makes +5V from VSYS. It runs whenever power is present (no enable), like U12, so the FPGA's 1.8 V auxiliary supply is never missing while its 3.3 V banks are powered. Its output goes to the +5V rail through U34. +5V feeds the 5 V buses, the extension 5 V pins and the four small regulators below. The two feedback resistors set the output voltage; the induc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"
- note added: "U34 +5V source select"
- note removed: "A shortcut for plain 5 V USB. A regulator cannot make 5 V out of 5 V, so when the USB source is 5 V the board controller turns Q2 on and USB power goes straight onto the +5V rail. It is off by default and must stay off at 9 V, or 9 V would reach parts rated for 5.5 V; Q3 is the small transistor the controller uses to switch it."
- note removed: "Lets the board controller measure every supply. Each rail goes to one of its analog inputs (ADC), which read 0-3.3 V. Rails at or below 3.3 V go through a 1 k resistor that protects the pin; VSYS and +5V are higher, so two resistors divide them down first. A 100 nF capacitor on each input steadies the reading. Firmware uses this to check each regulator came up before enabling the next."
- note removed: "Small switching regulator that makes 1.8 V from +5V. Its output node is +1V8_IO: FPGA bank 13 and the 1.8 V memory on it, the 1.8 V position of the J19/J20 jumpers, and, through the bead below, the FPGA's auxiliary supply (VCCAUX) and its ADC as +1V8. Enabled by the board controller (EN_1V8); the feedback resistors set 1.8 V."
- note removed: "Switching regulator (buck converter) that makes +5V from VSYS. +5V feeds the 5 V buses, the extension 5 V pins and the four small regulators below. The board controller turns it on (EN_5V); the pull-down keeps it off until then. The two feedback resistors set the output voltage; the inductor and capacitors are its power stage."
- note removed: "VBUS pass switch to +5V"
- moved on the sheet: C184, C185, C186, C187, C188, C189, C190, C191, C192, C193, C194, C195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

Commit message: PSRAM power-up states with PUDC_B high; TPS22953 for the jumpered PIN V exports
Parts:
- removed R76, R77: 2.21k, Resistor_SMD:R_0603_1608Metric, symbol Device:R
- added C271, C274, C277, C278: 100nF, Capacitor_SMD:C_0402_1005Metric, symbol Device:C
- added C272, C275: 1nF 50V, Capacitor_SMD:C_0402_1005Metric, symbol Device:C
- added C273, C276: 1uF, Capacitor_SMD:C_0603_1608Metric, symbol Device:C
- added R198, R199: 1k, Resistor_SMD:R_0603_1608Metric, symbol Device:R
- U23, U24: value TPS22950CDDCR -> TPS22953DSQR; footprint EasyEDA:SOT-23-6_L2.9-W1.6-P0.95-LS2.8-BL_3 -> Package_DFN_QFN:Texas_DSQ0010A_WSON-10-1EP_2x2mm_P0.4mm_EP0.9x1.5mm; symbol odin:TPS22950CDDC -> odin:TPS22953DSQ; LCSC C7587833 -> C2680343
Connections:
- net U23_ILIM is gone; now on net EXT_EN: U23.4 (EN)
- net U24_ILIM is gone; now on net EXT_EN: U24.4 (EN)
- net +3V3: now also U23.3 (BIAS), U24.3 (BIAS), C271.1, C274.1
- net EXT_EN: no longer U23.1 (ON), U24.1 (ON)
- net EXT_FAULT: no longer U23.6 (FLT), U24.6 (FLT)
- net GND: now also U23.11 (EP), U23.5 (GND), U24.11 (EP), U24.5 (GND), C271.2, C272.2, C273.2, C274.2, C275.2, C276.2, C277.2, C278.2; no longer U23.3 (GND), U24.3 (GND)
- net VCCIO_1: now also U23.1 (IN), R198.1
- net VCCIO_1_EXT: now also U23.10 (OUT), U23.8 (SNS), U23.9 (OUT), C273.1; no longer U23.5 (VOUT)
- net VCCIO_2: now also U24.1 (IN), R199.1
- net VCCIO_2_EXT: now also U24.10 (OUT), U24.8 (SNS), U24.9 (OUT), C276.1; no longer U24.5 (VOUT)
- new net MON_VCCIO_1: C277.1, R198.2
- new net MON_VCCIO_2: C278.1, R199.2
- new net U23_CT: C272.1, U23.6 (CT)
- new net U24_CT: C275.1, U24.6 (CT)
- no-connect marks 11 -> 13
Other:
- note added: "Switch for the PIN V supply of slots A-D (the voltage chosen on J19). It is biased from +3V3 so it works down to the 1.8 V setting, blocks current flowing back in while off, ramps its output in about 1.5 ms and shuts down when hot. Overload protection is each slot's 500 mA fuse; the switch itself has no current limit."
- note added: "Switch for the PIN V supply of slots E-H (the voltage chosen on J20). It is biased from +3V3 so it works down to the 1.8 V setting, blocks current flowing back in while off, ramps its output in about 1.5 ms and shuts down when hot. Overload protection is each slot's 500 mA fuse; the switch itself has no current limit."
- note removed: "Protected switch for the PIN V supply of slots A-D (the voltage chosen on J19), limited to about 0.5 A, with reverse blocking."
- note removed: "Protected switch for the PIN V supply of slots E-H (the voltage chosen on J20), limited to about 0.5 A, with reverse blocking."
- moved on the sheet: C220, C221, C224, C225, C226, C227, C228, C229, C230, C261, C262, C263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

Commit message: Re-audit corrections, part 1: U34 selects by intent (Q6 hold, Q7 screw input), FCS_B pull-up, TPS22953 PG grounded, IN2 bypass, budget per path with recovery accounting, source policy
Parts:
- added C279: 10uF, Capacitor_SMD:C_0805_2012Metric, symbol Device:C
- added C280: 1uF, Capacitor_SMD:C_0603_1608Metric, symbol Device:C
- added D24: 1N4148W, Diode_SMD:D_SOD-123, symbol Device:D
- added Q6, Q7: BSS138LT1G, EasyEDA:SOT-23-3_L2.9-W1.6-P1.90-LS2.8-BR, symbol Transistor_FET:Q_NMOS_GSD
- added R200: 470k, Resistor_SMD:R_0603_1608Metric, symbol Device:R
- added R201: 100k, Resistor_SMD:R_0603_1608Metric, symbol Device:R
- added R202: 33k, Resistor_SMD:R_0603_1608Metric, symbol Device:R
Connections:
- net +5V_BUCK: now also C280.1
- net GND: now also U23.7 (PG), U24.7 (PG), C279.2, C280.2, Q6.2 (S), Q7.2 (S), R200.2, R202.2
- net VBUS5_PR1: now also Q6.3 (D), Q7.3 (D)
- net VIN_EXT: now also R201.1
- new net EXT_PRESENT: Q7.1 (G), R201.2, R202.1
- new net PD_REQ_9V: D24.2 (A)
- new net SEL_IN2: C279.1, D24.1 (K), Q6.1 (G), R200.1
- no-connect marks 13 -> 11
Other:
- note added: "Q6 mux hold: 9 V request"
- note added: "Q7 mux hold: screw input present"
- moved on the sheet: C265, C266, R163, R165, R167, R168

Commit message: wip
Other:
- note added: "Chooses what feeds the +5V rail: USB power straight from the connector, or U11. A regulator cannot make 5 V out of 5 V, so on a plain 5 V USB source the mux passes VBUS to the rail. It hands the rail to U11 while the board controller asks the charger for 9 V and for a few seconds after (Q6), while the screw input is powered (Q7), and, as a backstop, if VBUS rises above about 5.6 V unasked or goes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"
- note added: "Keeps U34 on U11 around a 9 V negotiation. The controller's 9 V request charges a capacitor through D24 at once and the capacitor drains through its resistor in 2-7 s, so the rail leaves VBUS before the charger moves it and returns only when VBUS is back at 5 V. No voltage threshold can do that within the tolerances involved."
- note added: "Keeps U34 on U11 whenever the screw input carries voltage, so a bench supply on J50 carries the whole board even with a 5 V USB cable plugged in; before, the USB port kept the 5 V load."
- note added: "The FPGA core supply: up to 4 A at 1.0 V from +5V, the heaviest rail on the board. Enabled by the board controller (EN_1V0); its power-good output (CORE_1V0_GOOD) goes to the board controller (GPIO38) so firmware knows the core is up. The soft-start capacitor makes it ramp slowly; the feedback resistors set 1.0 V."
- note removed: "Chooses what feeds the +5V rail: USB power straight from the connector, or U11. A regulator cannot make 5 V out of 5 V, so on a plain 5 V USB source the mux passes VBUS to the rail; the moment a USB-PD charger raises VBUS above about 5.6 V, or VBUS is absent, it switches to U11 within microseconds. The choice is set by three resistor dividers, not by firmware, and the chip blocks current flowing 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"
- note removed: "The FPGA core supply: up to 4 A at 1.0 V from +5V, the heaviest rail on the board. Enabled by the board controller (EN_1V0); its power-good output (CORE_1V0_GOOD) is read through the status expander so firmware knows the core is up. The soft-start capacitor makes it ramp slowly; the feedback resistors set 1.0 V."
- moved on the sheet: C263, C264, C265, C266, C279, C280, D24, Q6, Q7, R162, R163, R164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
