File: kicad/slots.kicad_sch (KiCad schematic)
At the start: 84 parts, among them J10 AUX_SEL_C, J11 SLOT_D, J12 AUX_SEL_D, J13 SLOT_E, J14 AUX_SEL_E, J15 SLOT_F, J16 AUX_SEL_F, J17 SLOT_G, J18 AUX_SEL_G, J19 SLOT_H, J20 AUX_SEL_H, J21 VCCIO1_SEL, J22 VCCIO2_SEL, J3 SLOT_L, J4 AUX_SEL_L, J5 SLOT_A, J6 AUX_SEL_A, J7 SLOT_B, J8 AUX_SEL_B, J9 SLOT_C, U10 SN74AVC8T245PW, U9 SN74AVC8T245PW

Commit message: power input: single USB-C with CH224K PD sink at 9V, Schottky OR-ing, degraded 5V mode; record missing board-ID pins
Parts:
- removed C98: 100nF, Capacitor_SMD:C_0402_1005Metric, symbol Device:C
- added C124: 22uF, Capacitor_SMD:C_0805_2012Metric, symbol Device:C
- C102, C104, C106, C108, C110, C112, C114, C116, C118: value 10uF -> 100nF; footprint Capacitor_SMD:C_0805_2012Metric -> Capacitor_SMD:C_0402_1005Metric
- C103, C105, C107, C109, C111, C113, C115, C117, C119: value 100nF -> 10uF; footprint Capacitor_SMD:C_0402_1005Metric -> Capacitor_SMD:C_0805_2012Metric
- C120: value 22uF -> 100nF; footprint Capacitor_SMD:C_0805_2012Metric -> Capacitor_SMD:C_0402_1005Metric
Connections:
- net +3V3: now also C101.1, C99.1; no longer C100.1
- net +5V: now also C100.1, C102.1; no longer C101.1, C99.1
- net GND: now also C124.2
- net V33_A: now also C106.1; no longer C105.1
- net V33_B: now also C108.1; no longer C107.1
- net V33_C: now also C110.1; no longer C109.1
- net V33_D: now also C112.1; no longer C111.1
- net V33_E: now also C114.1; no longer C113.1
- net V33_F: now also C116.1; no longer C115.1
- net V33_G: now also C118.1; no longer C117.1
- net V33_H: now also C120.1; no longer C119.1
- net V33_L: now also C104.1; no longer C103.1
- net VCCIO_1: now also C122.1; no longer C120.1
- net VCCIO_2: now also C124.1; no longer C122.1
- net VIO_A: now also C105.1; no longer C104.1
- net VIO_B: now also C107.1; no longer C106.1
- net VIO_C: now also C109.1; no longer C108.1
- net VIO_D: now also C111.1; no longer C110.1
- net VIO_E: now also C113.1; no longer C112.1
- net VIO_F: now also C115.1; no longer C114.1
- net VIO_G: now also C117.1; no longer C116.1
- net VIO_H: now also C119.1; no longer C118.1
- net VIO_L: now also C103.1; no longer C102.1
- net +12V renamed VSYS
Other:
- moved on the sheet: C100, C101, C102, C103, C104, C105, C106, C107, C108, C109, C110, C111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

Commit message: assume 5V for function, PD only for headroom: boost 12V AUX from the 5V rail
Connections:
- net VSYS renamed +12V

Commit message: audit response: fix 5V-overstressed translators, add USB ESD protection and keying posts, load the PCB, reconcile every stale doc
Parts:
- added MK65: key A, Connector_PinHeader_2.54mm:PinHeader_1x01_P2.54mm_Vertical, symbol Connector_Generic:Conn_01x01
- added MK66: key B, Connector_PinHeader_2.54mm:PinHeader_1x01_P2.54mm_Vertical, symbol Connector_Generic:Conn_01x01
- added MK67: key C, Connector_PinHeader_2.54mm:PinHeader_1x01_P2.54mm_Vertical, symbol Connector_Generic:Conn_01x01
- added MK68: key D, Connector_PinHeader_2.54mm:PinHeader_1x01_P2.54mm_Vertical, symbol Connector_Generic:Conn_01x01
- added MK69: key E, Connector_PinHeader_2.54mm:PinHeader_1x01_P2.54mm_Vertical, symbol Connector_Generic:Conn_01x01
- added MK70: key F, Connector_PinHeader_2.54mm:PinHeader_1x01_P2.54mm_Vertical, symbol Connector_Generic:Conn_01x01
- added MK71: key G, Connector_PinHeader_2.54mm:PinHeader_1x01_P2.54mm_Vertical, symbol Connector_Generic:Conn_01x01
- added MK72: key H, Connector_PinHeader_2.54mm:PinHeader_1x01_P2.54mm_Vertical, symbol Connector_Generic:Conn_01x01
- added MK76: key L, Connector_PinHeader_2.54mm:PinHeader_1x01_P2.54mm_Vertical, symbol Connector_Generic:Conn_01x01
- U10, U9: value SN74AVC8T245PW -> SN74LXC8T245PW; symbol Logic_LevelTranslator:SN74AVC8T245PW -> odin:SN74LXC8T245PW
Connections:
- net GND: now also MK65.1 (Pin_1), MK66.1 (Pin_1), MK67.1 (Pin_1), MK68.1 (Pin_1), MK69.1 (Pin_1), MK70.1 (Pin_1), MK71.1 (Pin_1), MK72.1 (Pin_1), MK76.1 (Pin_1)
Other:
- moved on the sheet: C107, C108, C111, C112, C115, C116, C119, C120, F10, F11, F12, F17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

Commit message: fix 14 package mismatches, assert footprints against ki_fp_filters, rebalance fuses, correct JTAG and PD-voltage claims
Parts:
- F1, F13, F17, F21, F25, F29, F33, F5, F9: footprint Resistor_SMD:R_0603_1608Metric -> Fuse:Fuse_1206_3216Metric
- F10, F14, F18, F2, F22, F26, F30, F34, F6: value 1A -> 500mA; footprint Resistor_SMD:R_0603_1608Metric -> Fuse:Fuse_1206_3216Metric
- F11, F15, F19, F23, F27, F3, F31, F35, F7: value 500mA -> 300mA; footprint Resistor_SMD:R_0603_1608Metric -> Fuse:Fuse_1206_3216Metric
- F12, F16, F20, F24, F28, F32, F36, F4, F8: value 500mA -> 200mA; footprint Resistor_SMD:R_0603_1608Metric -> Fuse:Fuse_1206_3216Metric
Other:
- moved on the sheet: F10, F12, F14, F16, F18, F2, F20, F22, F24, F26, F28, F30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

Commit message: Update Odin hardware design, imported parts, and documentation
Include EasyEDA symbols, footprints and 3D models; revise FPGA allocation, power and extension buses; add qualification audits and user documentation.

Validation: EasyEDA audit, qualified parts, power budget and Python syntax pass. KiCad ERC reports 1 error and 319 warnings; DRC reports 90 violations, 499 unconnected items and 209 schematic parity issues. This is a work-in-progress design snapshot. Imported vendor assets retain their original formatting.
Parts:
- removed C100, C101, C102, C104, C106, C108, C110, C112, C114, C116, C118, C120, C99: 100nF, Capacitor_SMD:C_0402_1005Metric, symbol Device:C
- removed C103, C105, C107, C109, C111, C113, C115, C117, C119: 10uF, Capacitor_SMD:C_0805_2012Metric, symbol Device:C
- removed C121, C122, C123, C124: 22uF, Capacitor_SMD:C_0805_2012Metric, symbol Device:C
- removed J22: VCCIO2_SEL, Connector_PinHeader_2.54mm:PinHeader_2x03_P2.54mm_Vertical, symbol Connector_Generic:Conn_02x03_Odd_Even
- removed J9: SLOT_C, Connector_PinHeader_2.54mm:PinHeader_2x08_P2.54mm_Vertical_SMD, symbol Connector_Generic:Conn_02x08_Odd_Even
- added C140, C141, C142, C143, C145, C147, C149, C151, C153, C155, C157, C159, C161, C163: 100nF, Capacitor_SMD:C_0402_1005Metric, symbol Device:C
- added C144, C146, C148, C150, C152, C154, C156, C158, C160, C162: 10uF, Capacitor_SMD:C_0805_2012Metric, symbol Device:C
- added C164, C165, C166, C167: 22uF, Capacitor_SMD:C_0805_2012Metric, symbol Device:C
- added F37, F38: 500mA, EasyEDA:F1206, symbol Device:Polyfuse
- added F39: 300mA, EasyEDA:F1206, symbol Device:Polyfuse
- added F40: 200mA, EasyEDA:F1206, symbol Device:Polyfuse
- added J53, J54, J55, J56: ZX-PM2.54-1-16PY, EasyEDA:HDR-TH_16P-P2.54-V-F-1, symbol EasyEDA:ZX-PM2.54-1-16PY
- added J57, J58: 2.54-1*8P, EasyEDA:HDR-TH_8P-P2.54-V-F, symbol EasyEDA:Header-Female-2.54_1x8
- added MK77: PH2.54-1X1P-H25, EasyEDA:HDR-TH_1P-P2.54-V-M, symbol EasyEDA:PH2.54-1X1P-H25
- F1, F10, F13, F14, F17, F18, F2, F21, F22, F25, F26, F29, F30, F33, F34, F5, F6, F9: footprint Fuse:Fuse_1206_3216Metric -> EasyEDA:F1206; LCSC (none) -> C269115
- F11, F15, F19, F23, F27, F3, F31, F35, F7: footprint Fuse:Fuse_1206_3216Metric -> EasyEDA:F1206; LCSC (none) -> C22378340
- F12, F16, F20, F24, F28, F32, F36, F4, F8: footprint Fuse:Fuse_1206_3216Metric -> EasyEDA:F1206; LCSC (none) -> C269111
- J10: value AUX_SEL_C -> 2.54-2*3P; footprint Connector_PinHeader_2.54mm:PinHeader_2x03_P2.54mm_Vertical -> EasyEDA:HDR-TH_6P-P2.54-V-M-R2-C3-S2.54-1; symbol Connector_Generic:Conn_02x03_Odd_Even -> EasyEDA:Header-Male-2.54_2x3; LCSC (none) -> C65114
- J11: value SLOT_D -> 2.54-2*3P; footprint Connector_PinHeader_2.54mm:PinHeader_2x08_P2.54mm_Vertical_SMD -> EasyEDA:HDR-TH_6P-P2.54-V-M-R2-C3-S2.54-1; symbol Connector_Generic:Conn_02x08_Odd_Even -> EasyEDA:Header-Male-2.54_2x3; LCSC (none) -> C65114
- J12: value AUX_SEL_D -> 2.54-2*3P; footprint Connector_PinHeader_2.54mm:PinHeader_2x03_P2.54mm_Vertical -> EasyEDA:HDR-TH_6P-P2.54-V-M-R2-C3-S2.54-1; symbol Connector_Generic:Conn_02x03_Odd_Even -> EasyEDA:Header-Male-2.54_2x3; LCSC (none) -> C65114
- J13: value SLOT_E -> 2.54-2*3P; footprint Connector_PinHeader_2.54mm:PinHeader_2x08_P2.54mm_Vertical_SMD -> EasyEDA:HDR-TH_6P-P2.54-V-M-R2-C3-S2.54-1; symbol Connector_Generic:Conn_02x08_Odd_Even -> EasyEDA:Header-Male-2.54_2x3; LCSC (none) -> C65114
- J14: value AUX_SEL_E -> 2.54-2*3P; footprint Connector_PinHeader_2.54mm:PinHeader_2x03_P2.54mm_Vertical -> EasyEDA:HDR-TH_6P-P2.54-V-M-R2-C3-S2.54-1; symbol Connector_Generic:Conn_02x03_Odd_Even -> EasyEDA:Header-Male-2.54_2x3; LCSC (none) -> C65114
- J15: value SLOT_F -> 2.54-2*3P; footprint Connector_PinHeader_2.54mm:PinHeader_2x08_P2.54mm_Vertical_SMD -> EasyEDA:HDR-TH_6P-P2.54-V-M-R2-C3-S2.54-1; symbol Connector_Generic:Conn_02x08_Odd_Even -> EasyEDA:Header-Male-2.54_2x3; LCSC (none) -> C65114
- J16: value AUX_SEL_F -> 2.54-2*3P; footprint Connector_PinHeader_2.54mm:PinHeader_2x03_P2.54mm_Vertical -> EasyEDA:HDR-TH_6P-P2.54-V-M-R2-C3-S2.54-1; symbol Connector_Generic:Conn_02x03_Odd_Even -> EasyEDA:Header-Male-2.54_2x3; LCSC (none) -> C65114
- J17: value SLOT_G -> 2.54-2*3P; footprint Connector_PinHeader_2.54mm:PinHeader_2x08_P2.54mm_Vertical_SMD -> EasyEDA:HDR-TH_6P-P2.54-V-M-R2-C3-S2.54-1; symbol Connector_Generic:Conn_02x08_Odd_Even -> EasyEDA:Header-Male-2.54_2x3; LCSC (none) -> C65114
- J18: value AUX_SEL_G -> 2.54-2*3P; footprint Connector_PinHeader_2.54mm:PinHeader_2x03_P2.54mm_Vertical -> EasyEDA:HDR-TH_6P-P2.54-V-M-R2-C3-S2.54-1; symbol Connector_Generic:Conn_02x03_Odd_Even -> EasyEDA:Header-Male-2.54_2x3; LCSC (none) -> C65114
- J19: value SLOT_H -> 2.54-2*3P; footprint Connector_PinHeader_2.54mm:PinHeader_2x08_P2.54mm_Vertical_SMD -> EasyEDA:HDR-TH_6P-P2.54-V-M-R2-C3-S2.54-1; symbol Connector_Generic:Conn_02x08_Odd_Even -> EasyEDA:Header-Male-2.54_2x3; LCSC (none) -> C65114
- J20: value AUX_SEL_H -> 2.54-2*3P; footprint Connector_PinHeader_2.54mm:PinHeader_2x03_P2.54mm_Vertical -> EasyEDA:HDR-TH_6P-P2.54-V-M-R2-C3-S2.54-1; symbol Connector_Generic:Conn_02x03_Odd_Even -> EasyEDA:Header-Male-2.54_2x3; LCSC (none) -> C65114
- J21: value VCCIO1_SEL -> 2.54-2*3P; footprint Connector_PinHeader_2.54mm:PinHeader_2x03_P2.54mm_Vertical -> EasyEDA:HDR-TH_6P-P2.54-V-M-R2-C3-S2.54-1; symbol Connector_Generic:Conn_02x03_Odd_Even -> EasyEDA:Header-Male-2.54_2x3; LCSC (none) -> C65114
- J3: value SLOT_L -> PM254-2-16-S-8.5; footprint Connector_PinHeader_2.54mm:PinHeader_2x08_P2.54mm_Vertical_SMD -> EasyEDA:HDR-SMD_32P-P2.54-V-F-R2-C16-LS7.1; symbol Connector_Generic:Conn_02x08_Odd_Even -> EasyEDA:PM254-2-16-S-8.5; LCSC (none) -> C3975161
- J4: value AUX_SEL_L -> PM254-2-16-S-8.5; footprint Connector_PinHeader_2.54mm:PinHeader_2x03_P2.54mm_Vertical -> EasyEDA:HDR-SMD_32P-P2.54-V-F-R2-C16-LS7.1; symbol Connector_Generic:Conn_02x03_Odd_Even -> EasyEDA:PM254-2-16-S-8.5; LCSC (none) -> C3975161
- J5: value SLOT_A -> PM254-2-16-S-8.5; footprint Connector_PinHeader_2.54mm:PinHeader_2x08_P2.54mm_Vertical_SMD -> EasyEDA:HDR-SMD_32P-P2.54-V-F-R2-C16-LS7.1; symbol Connector_Generic:Conn_02x08_Odd_Even -> EasyEDA:PM254-2-16-S-8.5; LCSC (none) -> C3975161
- J6: value AUX_SEL_A -> PM254-2-16-S-8.5; footprint Connector_PinHeader_2.54mm:PinHeader_2x03_P2.54mm_Vertical -> EasyEDA:HDR-SMD_32P-P2.54-V-F-R2-C16-LS7.1; symbol Connector_Generic:Conn_02x03_Odd_Even -> EasyEDA:PM254-2-16-S-8.5; LCSC (none) -> C3975161
- J7: value SLOT_B -> PM254-2-08-S-8.5; footprint Connector_PinHeader_2.54mm:PinHeader_2x08_P2.54mm_Vertical_SMD -> EasyEDA:HDR-SMD_16P-P2.54-V-F-R2-C8-LS7.1; symbol Connector_Generic:Conn_02x08_Odd_Even -> EasyEDA:PM254-2-08-S-8.5; LCSC (none) -> C3975153
- J8: value AUX_SEL_B -> PM254-2-08-S-8.5; footprint Connector_PinHeader_2.54mm:PinHeader_2x03_P2.54mm_Vertical -> EasyEDA:HDR-SMD_16P-P2.54-V-F-R2-C8-LS7.1; symbol Connector_Generic:Conn_02x03_Odd_Even -> EasyEDA:PM254-2-08-S-8.5; LCSC (none) -> C3975153
- MK65: value key A -> PH2.54-1X1P-H25; footprint Connector_PinHeader_2.54mm:PinHeader_1x01_P2.54mm_Vertical -> EasyEDA:HDR-TH_1P-P2.54-V-M; symbol Connector_Generic:Conn_01x01 -> EasyEDA:PH2.54-1X1P-H25; LCSC (none) -> C42431799
- MK66: value key B -> PH2.54-1X1P-H25; footprint Connector_PinHeader_2.54mm:PinHeader_1x01_P2.54mm_Vertical -> EasyEDA:HDR-TH_1P-P2.54-V-M; symbol Connector_Generic:Conn_01x01 -> EasyEDA:PH2.54-1X1P-H25; LCSC (none) -> C42431799
- MK67: value key C -> PH2.54-1X1P-H25; footprint Connector_PinHeader_2.54mm:PinHeader_1x01_P2.54mm_Vertical -> EasyEDA:HDR-TH_1P-P2.54-V-M; symbol Connector_Generic:Conn_01x01 -> EasyEDA:PH2.54-1X1P-H25; LCSC (none) -> C42431799
- MK68: value key D -> PH2.54-1X1P-H25; footprint Connector_PinHeader_2.54mm:PinHeader_1x01_P2.54mm_Vertical -> EasyEDA:HDR-TH_1P-P2.54-V-M; symbol Connector_Generic:Conn_01x01 -> EasyEDA:PH2.54-1X1P-H25; LCSC (none) -> C42431799
- MK69: value key E -> PH2.54-1X1P-H25; footprint Connector_PinHeader_2.54mm:PinHeader_1x01_P2.54mm_Vertical -> EasyEDA:HDR-TH_1P-P2.54-V-M; symbol Connector_Generic:Conn_01x01 -> EasyEDA:PH2.54-1X1P-H25; LCSC (none) -> C42431799
- MK70: value key F -> PH2.54-1X1P-H25; footprint Connector_PinHeader_2.54mm:PinHeader_1x01_P2.54mm_Vertical -> EasyEDA:HDR-TH_1P-P2.54-V-M; symbol Connector_Generic:Conn_01x01 -> EasyEDA:PH2.54-1X1P-H25; LCSC (none) -> C42431799
- MK71: value key G -> PH2.54-1X1P-H25; footprint Connector_PinHeader_2.54mm:PinHeader_1x01_P2.54mm_Vertical -> EasyEDA:HDR-TH_1P-P2.54-V-M; symbol Connector_Generic:Conn_01x01 -> EasyEDA:PH2.54-1X1P-H25; LCSC (none) -> C42431799
- MK72: value key H -> PH2.54-1X1P-H25; footprint Connector_PinHeader_2.54mm:PinHeader_1x01_P2.54mm_Vertical -> EasyEDA:HDR-TH_1P-P2.54-V-M; symbol Connector_Generic:Conn_01x01 -> EasyEDA:PH2.54-1X1P-H25; LCSC (none) -> C42431799
- MK76: value key L -> PH2.54-1X1P-H25; footprint Connector_PinHeader_2.54mm:PinHeader_1x01_P2.54mm_Vertical -> EasyEDA:HDR-TH_1P-P2.54-V-M; symbol Connector_Generic:Conn_01x01 -> EasyEDA:PH2.54-1X1P-H25; LCSC (none) -> C42431799
- U10, U9: value SN74LXC8T245PW -> SN74LXC8T245PWR; footprint Package_SO:TSSOP-24_4.4x7.8mm_P0.65mm -> EasyEDA:TSSOP-24_L7.8-W4.4-P0.65-LS6.4-BL_1; LCSC (none) -> C4363995
Connections:
- net SLOTA_P2_N is gone; now on net GND: J5.8
- net SLOTA_P2_P is gone; now on net GND: J5.7
- net SLOTB_P3_N is gone; now on net GND: J7.10
- net SLOTB_P3_P is gone; now on net GND: J7.9
- net SLOTB_P4_N is gone; now on net GND: J7.12
- net SLOTB_P4_P is gone; now on net GND: J7.11
- net SLOTD_P0_P is gone; now on net +12V_EXT: J11.1
- net SLOTD_P1_N is gone; now on net SLOT_A_POWER_SELECTED: J11.4
- net SLOTE_P0_P is gone; now on net +12V_EXT: J13.1
- net SLOTE_P1_N is gone; now on net SLOT_C_POWER_SELECTED: J13.4
- net SLOTE_P1_P is gone; now on net +5V_EXT: J13.3
- net SLOTF_P0_P is gone; now on net +12V_EXT: J15.1
- net SLOTF_P1_N is gone; now on net SLOT_E_POWER_SELECTED: J15.4
- net SLOTF_P1_P is gone; now on net +5V_EXT: J15.3
- net SLOTG_P0_P is gone; now on net +12V_EXT: J17.1
- net SLOTG_P1_N is gone; now on net SLOT_G_POWER_SELECTED: J17.4
- net SLOTG_P1_P is gone; now on net +5V_EXT: J17.3
- net SLOTH_P0_N is gone; now on net VCCIO_1: J19.2
- net SLOTH_P0_P is gone; now on net +3V3: J19.1
- net SLOTH_P1_N is gone; now on net VCCIO_1: J19.4
- net SLOTH_P1_P is gone; now on net +2V5: J19.3
- net +1V8: now also J19.5, J20.5; no longer J21.5 (Pin_5)
- net +2V5: now also J20.3; no longer J21.3 (Pin_3)
- net +3V3: now also J20.1, C140.1, C142.1; no longer F1.1, F11.1, F15.1, F19.1, F23.1, F27.1, F3.1, F31.1, F35.1, F7.1, J10.5 (Pin_5), J12.5 (Pin_5)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
- net +5V: now also C141.1, C143.1; no longer F10.1, F14.1, F18.1, F2.1, F22.1, F26.1, F30.1, F34.1, F6.1, J10.3 (Pin_3), J12.3 (Pin_3), J14.3 (Pin_3)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
- net GND: now also J3.15, J3.16, J3.17, J3.18, J3.25, J3.26, J3.7, J3.8, J4.15, J4.16, J4.17, J4.18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; no longer J11.5 (Pin_5), J11.6 (Pin_6), J13.5 (Pin_5), J13.6 (Pin_6), J15.5 (Pin_5), J15.6 (Pin_6), J17.5 (Pin_5), J17.6 (Pin_6), J19.5 (Pin_5), J19.6 (Pin_6), J3.5 (Pin_5), J3.6 (Pin_6)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
- net VCCIO_1: now also J19.6, C164.1, C165.1; no longer F13.1, F17.1, F5.1, F9.1, J21.2 (Pin_2), J21.4 (Pin_4), J21.6 (Pin_6)
- net VCCIO_2: now also J20.2, J20.4, J20.6, C166.1, C167.1; no longer F21.1, F25.1, F29.1, F33.1
- net BUS5V1_IO7: now reaches U10.10 (A8)
- net BUS5V1_PIN7: now reaches U10.14 (B8)
- net BUS5V1_PIN7: now also J8.8
- net BUS5V1_PIN6: now reaches U10.15 (B7)
- net BUS5V1_PIN6: now also J8.7
- net BUS5V1_PIN5: now reaches U10.16 (B6)
- net BUS5V1_PIN5: now also J8.6
- net BUS5V1_PIN4: now reaches U10.17 (B5)
- net BUS5V1_PIN4: now also J8.5
- net BUS5V1_PIN3: now reaches U10.18 (B4)
- net BUS5V1_PIN3: now also J8.4
- net BUS5V1_PIN2: now reaches U10.19 (B3)
- net BUS5V1_PIN2: now also J8.3
- net BUS5V1_IO2: now reaches U10.5 (A3)
- net BUS5V1_IO3: now reaches U10.6 (A4)
- net BUS5V1_IO4: now reaches U10.7 (A5)
- net BUS5V1_IO5: now reaches U10.8 (A6)
- net BUS5V1_IO6: now reaches U10.9 (A7)
- net +12V renamed +12V_EXT
- net +12V_EXT: now also J21.1; no longer J20.1 (Pin_1), J4.1 (Pin_1), J6.1 (Pin_1), J8.1 (Pin_1)
- removed net AUXSEL_A: F8.1, J6.2 (Pin_2), J6.4 (Pin_4), J6.6 (Pin_6)
- removed net AUXSEL_B: F12.1, J8.2 (Pin_2), J8.4 (Pin_4), J8.6 (Pin_6)
- net AUXSEL_C renamed SLOT_L_POWER_SELECTED
- net SLOT_L_POWER_SELECTED: now also F4.1; no longer F16.1
- net AUXSEL_D renamed SLOT_B_POWER_SELECTED
- net SLOT_B_POWER_SELECTED: now also F16.1; no longer F20.1
- net AUXSEL_E renamed SLOT_D_POWER_SELECTED
- net AUXSEL_F renamed SLOT_F_POWER_SELECTED
- net SLOT_F_POWER_SELECTED: now also F32.1; no longer F28.1
- net AUXSEL_G renamed SLOT_H_POWER_SELECTED
- net SLOT_H_POWER_SELECTED: now also F40.1; no longer F32.1
- removed net AUXSEL_H: F36.1, J20.2 (Pin_2), J20.4 (Pin_4), J20.6 (Pin_6)
- removed net AUXSEL_L: F4.1, J4.2 (Pin_2), J4.4 (Pin_4), J4.6 (Pin_6)
- net AUX_A renamed SLOT_M_POWER
- net SLOT_M_POWER: now also J58.8; no longer J5.16 (Pin_16)
- net AUX_B renamed SLOT_A_POWER
- net SLOT_A_POWER: now also J53.8; no longer J7.16 (Pin_16)
- net AUX_C renamed SLOT_B_POWER
- net SLOT_B_POWER: now also J53.16
- net AUX_D renamed SLOT_C_POWER
- net SLOT_C_POWER: now also J54.8; no longer J11.16 (Pin_16)
- net AUX_E renamed SLOT_D_POWER
- net SLOT_D_POWER: now also J54.16; no longer J13.16 (Pin_16)
- net AUX_F renamed SLOT_E_POWER
- net SLOT_E_POWER: now also J55.8; no longer J15.16 (Pin_16)
- net AUX_G renamed SLOT_F_POWER
- net SLOT_F_POWER: now also J55.16; no longer J17.16 (Pin_16)
- net AUX_H renamed SLOT_G_POWER
- net SLOT_G_POWER: now also J56.8; no longer J19.16 (Pin_16)
- net AUX_L renamed SLOT_L_POWER
- net SLOT_L_POWER: now also J57.8; no longer J3.16 (Pin_16)
- net SLOTA_P0_N renamed SLOTE_IO2
- net SLOTA_P0_P renamed SLOTE_IO0
- net SLOTA_P1_N renamed SLOTE_IO6
- net SLOTA_P1_P renamed SLOTE_IO4
- net SLOTA_P3_N renamed SLOTF_IO2
- net SLOTA_P3_P renamed SLOTF_IO0
- net SLOTA_P4_N renamed SLOTF_IO6
- net SLOTA_P4_P renamed SLOTF_IO4
- net SLOTB_P0_N renamed BUS5V0_PIN1
- net BUS5V0_PIN1: now also U9.20 (B2)
- net SLOTB_P0_P renamed BUS5V0_PIN0
- net BUS5V0_PIN0: now also U9.21 (B1)
- net SLOTB_P1_N renamed BUS5V0_PIN3
- net BUS5V0_PIN3: now also U9.18 (B4)
- net SLOTB_P1_P renamed BUS5V0_PIN2
- net BUS5V0_PIN2: now also U9.19 (B3)
- net SLOTB_P2_N renamed BUS5V0_PIN7
- net BUS5V0_PIN7: now also U9.14 (B8)
- net SLOTB_P2_P renamed BUS5V0_PIN6
- net BUS5V0_PIN6: now also U9.15 (B7)
- net SLOTD_P0_N renamed SLOT_A_POWER_SELECTED
- net SLOT_A_POWER_SELECTED: now also F12.1, J11.6
- net SLOTD_P1_P renamed +5V_EXT
- net +5V_EXT: now also F10.1, F14.1, F18.1, F2.1, F22.1, F26.1, F30.1, F34.1, F6.1, J10.3, J12.3, J14.3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
- removed net SLOTD_P2_N: J11.8 (Pin_8)
- removed net SLOTD_P2_P: J11.7 (Pin_7)
- removed net SLOTD_P3_N: J11.10 (Pin_10)
- removed net SLOTD_P3_P: J11.9 (Pin_9)
- removed net SLOTD_P4_N: J11.12 (Pin_12)
- removed net SLOTD_P4_P: J11.11 (Pin_11)
- net SLOTE_P0_N renamed SLOT_C_POWER_SELECTED
- net SLOT_C_POWER_SELECTED: now also F20.1, J13.6
- removed net SLOTE_P2_N: J13.8 (Pin_8)
- removed net SLOTE_P2_P: J13.7 (Pin_7)
- removed net SLOTE_P3_N: J13.10 (Pin_10)
- removed net SLOTE_P3_P: J13.9 (Pin_9)
- removed net SLOTE_P4_N: J13.12 (Pin_12)
- removed net SLOTE_P4_P: J13.11 (Pin_11)
- net SLOTF_P0_N renamed SLOT_E_POWER_SELECTED
- net SLOT_E_POWER_SELECTED: now also F28.1, J15.6
- removed net SLOTF_P2_N: J15.8 (Pin_8)
- removed net SLOTF_P2_P: J15.7 (Pin_7)
- removed net SLOTF_P3_N: J15.10 (Pin_10)
- removed net SLOTF_P3_P: J15.9 (Pin_9)
- removed net SLOTF_P4_N: J15.12 (Pin_12)
- removed net SLOTF_P4_P: J15.11 (Pin_11)
- net SLOTG_P0_N renamed SLOT_G_POWER_SELECTED
- net SLOT_G_POWER_SELECTED: now also F36.1, J17.6
- removed net SLOTG_P2_N: J17.8 (Pin_8)
- removed net SLOTG_P2_P: J17.7 (Pin_7)
- removed net SLOTG_P3_N: J17.10 (Pin_10)
- removed net SLOTG_P3_P: J17.9 (Pin_9)
- removed net SLOTG_P4_N: J17.12 (Pin_12)
- removed net SLOTG_P4_P: J17.11 (Pin_11)
- removed net SLOTH_P2_N: J19.8 (Pin_8)
- removed net SLOTH_P2_P: J19.7 (Pin_7)
- removed net SLOTH_P3_N: J19.10 (Pin_10)
- removed net SLOTH_P3_P: J19.9 (Pin_9)
- removed net SLOTH_P4_N: J19.12 (Pin_12)
- removed net SLOTH_P4_P: J19.11 (Pin_11)
- net SLOTL_DIR0 renamed BUS5V0_DIR
- net SLOTL_DIR1 renamed BUS5V1_DIR
- net SLOTL_IO0 renamed SLOTA_IO0
- net SLOTA_IO0: no longer U9.21 (B1)
- net SLOTL_IO1 renamed SLOTA_IO2
- net SLOTA_IO2: no longer U9.20 (B2)
- net SLOTL_IO2 renamed SLOTA_IO4
- net SLOTA_IO4: no longer U9.19 (B3)
- net SLOTL_IO3 renamed SLOTA_IO6
- net SLOTA_IO6: no longer U9.18 (B4)
- net SLOTL_IO4 renamed BUS5V0_PIN4
- net BUS5V0_PIN4: now also J7.5; no longer J3.7 (Pin_7)
- net SLOTL_IO5 renamed BUS5V0_PIN5
- net BUS5V0_PIN5: now also J7.6; no longer J3.8 (Pin_8)
- net SLOTL_IO6 renamed SLOTB_IO0
- net SLOTB_IO0: no longer U9.15 (B7)
- net SLOTL_IO7 renamed SLOTB_IO2
- net SLOTB_IO2: no longer U9.14 (B8)
- net SLOTL_IO8 renamed BUS5V1_PIN0
- net BUS5V1_PIN0: now also J8.1; no longer J3.11 (Pin_11)
- net SLOTL_IO9 renamed BUS5V1_PIN1
- net BUS5V1_PIN1: now also J8.2; no longer J3.12 (Pin_12)
- net SLOTL_P0_N renamed BUS5V0_IO1
- net SLOTL_P0_P renamed BUS5V0_IO0
- net SLOTL_P1_N renamed BUS5V0_IO3
- net SLOTL_P1_P renamed BUS5V0_IO2
- net SLOTL_P2_N renamed BUS5V0_IO5
- net SLOTL_P2_P renamed BUS5V0_IO4
- net SLOTL_P3_N renamed BUS5V0_IO7
- net SLOTL_P3_P renamed BUS5V0_IO6
- net SLOTL_P4_N renamed BUS5V1_IO1
- net SLOTL_P4_P renamed BUS5V1_IO0
- net V33_A renamed SLOTF_IO10
- net SLOTF_IO10: no longer F7.2
- net V33_B renamed SLOT_A_3V3
- net SLOT_A_3V3: now also C149.1, J53.4; no longer J7.14 (Pin_14)
- net V33_C renamed SLOT_B_3V3
- net SLOT_B_3V3: now also C151.1, J53.12
- net V33_D renamed SLOT_C_3V3
- net SLOT_C_3V3: now also C153.1, J54.4; no longer J11.14 (Pin_14)
- net V33_E renamed SLOT_D_3V3
- net SLOT_D_3V3: now also C155.1, J54.12; no longer J13.14 (Pin_14)
- net V33_F renamed SLOT_E_3V3
- net SLOT_E_3V3: now also C157.1, J55.4; no longer J15.14 (Pin_14)
- net V33_G renamed SLOT_F_3V3
- net SLOT_F_3V3: now also C159.1, J55.12; no longer J17.14 (Pin_14)
- net V33_H renamed SLOT_G_3V3
- net SLOT_G_3V3: now also C161.1, J56.4; no longer J19.14 (Pin_14)
- net V33_L renamed SLOTB_IO10
- net SLOTB_IO10: no longer F3.2
- net V5_A renamed SLOT_M_5V
- net SLOT_M_5V: now also J58.6; no longer J5.15 (Pin_15)
- net V5_B renamed SLOT_A_5V
- net SLOT_A_5V: now also J53.6; no longer J7.15 (Pin_15)
- net V5_C renamed SLOT_B_5V
- net SLOT_B_5V: now also J53.14
- net V5_D renamed SLOT_C_5V
- net SLOT_C_5V: now also J54.6; no longer J11.15 (Pin_15)
- net V5_E renamed SLOT_D_5V
- net SLOT_D_5V: now also J54.14; no longer J13.15 (Pin_15)
- net V5_F renamed SLOT_E_5V
- net SLOT_E_5V: now also J55.6; no longer J15.15 (Pin_15)
- net V5_G renamed SLOT_F_5V
- net SLOT_F_5V: now also J55.14; no longer J17.15 (Pin_15)
- net V5_H renamed SLOT_G_5V
- net V5_L renamed SLOT_L_5V
- net VIO_A renamed SLOTF_IO8
- net VIO_B renamed SLOT_A_PIN_VOLTAGE
- net VIO_C renamed SLOT_B_PIN_VOLTAGE
- net VIO_D renamed SLOT_C_PIN_VOLTAGE
- net VIO_E renamed SLOT_D_PIN_VOLTAGE
- net VIO_F renamed SLOT_E_PIN_VOLTAGE
- net VIO_G renamed SLOT_F_PIN_VOLTAGE
- net VIO_H renamed SLOT_G_PIN_VOLTAGE
- net VIO_L renamed SLOTB_IO8
- new net +3V3_EXT: F1.1, F11.1, F15.1, F19.1, F23.1, F27.1, F3.1, F31.1, F35.1, F39.1, F5.1, F7.1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
- new net SLOTA_IO1: J3.32
- new net SLOTA_IO10: J3.6
- new net SLOTA_IO11: J3.27
- new net SLOTA_IO3: J3.31
- new net SLOTA_IO5: J3.30
- new net SLOTA_IO7: J3.29
- new net SLOTA_IO8: J3.5
- new net SLOTA_IO9: J3.28
- new net SLOTB_IO1: J3.24
- new net SLOTB_IO11: J3.19
- new net SLOTB_IO3: J3.23
- new net SLOTB_IO4: J3.11
- new net SLOTB_IO5: J3.22
- new net SLOTB_IO6: J3.12
- new net SLOTB_IO7: J3.21
- new net SLOTB_IO9: J3.20
- new net SLOTC_IO0: J4.1
- new net SLOTC_IO1: J4.32
- new net SLOTC_IO10: J4.6
- new net SLOTC_IO11: J4.27
- new net SLOTC_IO2: J4.2
- new net SLOTC_IO3: J4.31
- new net SLOTC_IO4: J4.3
- new net SLOTC_IO5: J4.30
- new net SLOTC_IO6: J4.4
- new net SLOTC_IO7: J4.29
- new net SLOTC_IO8: J4.5
- new net SLOTC_IO9: J4.28
- new net SLOTD_IO0: J4.9
- new net SLOTD_IO1: J4.24
- new net SLOTD_IO10: J4.14
- new net SLOTD_IO11: J4.19
- new net SLOTD_IO2: J4.10
- new net SLOTD_IO3: J4.23
- new net SLOTD_IO4: J4.11
- new net SLOTD_IO5: J4.22
- new net SLOTD_IO6: J4.12
- new net SLOTD_IO7: J4.21
- new net SLOTD_IO8: J4.13
- new net SLOTD_IO9: J4.20
- new net SLOTE_IO1: J5.32
- new net SLOTE_IO10: J5.6
- new net SLOTE_IO11: J5.27
- new net SLOTE_IO3: J5.31
- new net SLOTE_IO5: J5.30
- new net SLOTE_IO7: J5.29
- new net SLOTE_IO8: J5.5
- new net SLOTE_IO9: J5.28
- new net SLOTF_IO1: J5.24
- new net SLOTF_IO11: J5.19
- new net SLOTF_IO3: J5.23
- new net SLOTF_IO5: J5.22
- new net SLOTF_IO7: J5.21
- new net SLOTF_IO9: J5.20
- new net SLOTG_IO0: J6.1
- new net SLOTG_IO1: J6.32
- new net SLOTG_IO10: J6.6
- new net SLOTG_IO11: J6.27
- new net SLOTG_IO2: J6.2
- new net SLOTG_IO3: J6.31
- new net SLOTG_IO4: J6.3
- new net SLOTG_IO5: J6.30
- new net SLOTG_IO6: J6.4
- new net SLOTG_IO7: J6.29
- new net SLOTG_IO8: J6.5
- new net SLOTG_IO9: J6.28
- new net SLOTH_IO0: J6.9
- new net SLOTH_IO1: J6.24
- new net SLOTH_IO10: J6.14
- new net SLOTH_IO11: J6.19
- new net SLOTH_IO2: J6.10
- new net SLOTH_IO3: J6.23
- new net SLOTH_IO4: J6.11
- new net SLOTH_IO5: J6.22
- new net SLOTH_IO6: J6.12
- new net SLOTH_IO7: J6.21
- new net SLOTH_IO8: J6.13
- new net SLOTH_IO9: J6.20
- new net SLOT_H_3V3: C163.1, F39.2, J56.12
- new net SLOT_H_5V: F38.2, J56.14
- new net SLOT_H_PIN_VOLTAGE: C162.1, F37.2, J56.10
- new net SLOT_H_POWER: F40.2, J56.16
- new net SLOT_L_3V3: C145.1, F3.2, J57.4
- new net SLOT_L_PIN_VOLTAGE: C144.1, F1.2, J57.2
- new net SLOT_M_3V3: C147.1, F7.2, J58.4
- new net SLOT_M_PIN_VOLTAGE: C146.1, F5.2, J58.2
- new net SLOT_M_POWER_SELECTED: F8.1, J21.2, J21.4, J21.6
- new net VCCIO_1_EXT: F13.1, F17.1, F21.1, F9.1
- new net VCCIO_2_EXT: F25.1, F29.1, F33.1, F37.1
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Other:
- note added: "5V BUS 0 converter"
- note added: "5V BUS 1 converter"
- note added: "SHIELD HEADER AB"
- note added: "SHIELD HEADER CD"
- note added: "SHIELD HEADER EF"
- note added: "SHIELD HEADER GH"
- note added: "SLOT A branches"
- note added: "SLOT B branches"
- note added: "SLOT C branches"
- note added: "SLOT D branches"
- note added: "SLOT E branches"
- note added: "SLOT F branches"
- note added: "SLOT G branches"
- note added: "SLOT H branches"
- note added: "SLOT L branches"
- note added: "SLOT M branches"
- note added: "SLOTS — Ten extension ports, rail selection, fusing, level shifting — HW 0.1.0-proto.1"
- note removed: "SLOT A"
- note removed: "SLOT B"
- note removed: "SLOT C"
- note removed: "SLOT D"
- note removed: "SLOT E"
- note removed: "SLOT F"
- note removed: "SLOT G"
- note removed: "SLOT H"
- note removed: "SLOT L"
- note removed: "SLOTS — Nine extension slots, rail selection, fusing, level shifting"
- note removed: "slot L level shifter 0"
- note removed: "slot L level shifter 1"
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
Commit message: wip
Parts:
- removed C167: 22uF, Capacitor_SMD:C_0805_2012Metric, symbol Device:C
- added C139: 100nF, Capacitor_SMD:C_0402_1005Metric, symbol Device:C
- added R96, R97: 10k, Resistor_SMD:R_0603_1608Metric, symbol Device:R
- C143, C145, C147, C149, C151, C153, C155, C157, C159, C161: value 100nF -> 10uF; footprint Capacitor_SMD:C_0402_1005Metric -> Capacitor_SMD:C_0805_2012Metric; LCSC C1525 -> C15850
- C144, C146, C148, C150, C152, C154, C156, C158, C160, C162: value 10uF -> 100nF; footprint Capacitor_SMD:C_0805_2012Metric -> Capacitor_SMD:C_0402_1005Metric; LCSC C15850 -> C1525
- C163: value 100nF -> 22uF; footprint Capacitor_SMD:C_0402_1005Metric -> Capacitor_SMD:C_0805_2012Metric; LCSC C1525 -> C86816
Connections:
- net +3V3: now also C141.1, C139.1, R96.1, R97.1; no longer C140.1, C142.1
- net +5V: now also C140.1, C142.1; no longer C141.1, C143.1
- net GND: now also C139.2; no longer U10.22 (~{OE}), U9.22 (~{OE})
- net SLOT_A_3V3: now also C148.1; no longer C149.1
- net SLOT_A_PIN_VOLTAGE: now also C147.1; no longer C148.1
- net SLOT_B_3V3: now also C150.1; no longer C151.1
- net SLOT_B_PIN_VOLTAGE: now also C149.1; no longer C150.1
- net SLOT_C_3V3: now also C152.1; no longer C153.1
- net SLOT_C_PIN_VOLTAGE: now also C151.1; no longer C152.1
- net SLOT_D_3V3: now also C154.1; no longer C155.1
- net SLOT_D_PIN_VOLTAGE: now also C153.1; no longer C154.1
- net SLOT_E_3V3: now also C156.1; no longer C157.1
- net SLOT_E_PIN_VOLTAGE: now also C155.1; no longer C156.1
- net SLOT_F_3V3: now also C158.1; no longer C159.1
- net SLOT_F_PIN_VOLTAGE: now also C157.1; no longer C158.1
- net SLOT_G_3V3: now also C160.1; no longer C161.1
- net SLOT_G_PIN_VOLTAGE: now also C159.1; no longer C160.1
- net SLOT_H_3V3: now also C162.1; no longer C163.1
- net SLOT_H_PIN_VOLTAGE: now also C161.1; no longer C162.1
- net SLOT_L_3V3: now also C144.1; no longer C145.1
- net SLOT_L_PIN_VOLTAGE: now also C143.1; no longer C144.1
- net SLOT_M_3V3: now also C146.1; no longer C147.1
- net SLOT_M_PIN_VOLTAGE: now also C145.1; no longer C146.1
- net VCCIO_1: now also C163.1; no longer C165.1
- net VCCIO_2: now also C165.1
- new net BUS5V0_OE_N: R96.2, U9.22 (~{OE})
- new net BUS5V1_OE_N: R97.2, U10.22 (~{OE})
Other:
- moved on the sheet: C140, C141, C142, C143, C144, C145, C146, C147, C148, C149, C150, C151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

Commit message: Through-hole extension headers, AUX supply rework, and board state before rev A cleanup
J3/J5 become single 2x32 through-hole bodies with IO IO GND rows and a long
grounded key post per zone. Power sheet reworked around the AUX rail.
Decoupling moved off B.Cu. New footprints, 3D models and check scripts.
Parts:
- removed J10, J11, J12, J13, J14, J15, J16, J17, J18, J21: 2.54-2*3P, EasyEDA:HDR-TH_6P-P2.54-V-M-R2-C3-S2.54-1, symbol EasyEDA:Header-Male-2.54_2x3
- removed J4, J6: PM254-2-16-S-8.5, EasyEDA:HDR-SMD_32P-P2.54-V-F-R2-C16-LS7.1, symbol EasyEDA:PM254-2-16-S-8.5
- added J62, J63, J64, J65: XFCN PM254V-11-07-H85, EasyEDA:HDR-TH_7P-P2.54-V-F, symbol EasyEDA:PM254V-11-07-H85
- F12, F16, F20, F24, F28, F32, F36, F4, F40, F8: value 200mA -> 1.1A 33V; footprint EasyEDA:F1206 -> odin:Fuse_TECHFUSE_SMD2018; LCSC C269111 -> C70150
- J3, J5: value PM254-2-16-S-8.5 -> WingTAT 2044-2X32G00SA; footprint EasyEDA:HDR-SMD_32P-P2.54-V-F-R2-C16-LS7.1 -> EasyEDA:HDR-TH_64P-P2.54-V-F-R2-C32-S2.54-1; symbol EasyEDA:PM254-2-16-S-8.5 -> EasyEDA:2044-2X32G00SA; LCSC C3975161 -> C49569844
- J53, J54, J55, J56: value ZX-PM2.54-1-16PY -> XFCN PM254V-11-07-H85; footprint EasyEDA:HDR-TH_16P-P2.54-V-F-1 -> EasyEDA:HDR-TH_7P-P2.54-V-F; symbol EasyEDA:ZX-PM2.54-1-16PY -> EasyEDA:PM254V-11-07-H85; LCSC C7499334 -> C2832270
- J57, J58: value 2.54-1*8P -> XFCN PM254V-11-07-H85; footprint EasyEDA:HDR-TH_8P-P2.54-V-F -> EasyEDA:HDR-TH_7P-P2.54-V-F; symbol EasyEDA:Header-Female-2.54_1x8 -> EasyEDA:PM254V-11-07-H85; LCSC C27438 -> C2832270
- J7, J8: value PM254-2-08-S-8.5 -> PM254-2-08-Z-8.5; footprint EasyEDA:HDR-SMD_16P-P2.54-V-F-R2-C8-LS7.1 -> EasyEDA:HDR-TH_16P-P2.54-V-F-R2-C8-S2.54; symbol EasyEDA:PM254-2-08-S-8.5 -> EasyEDA:PM254-2-08-Z-8.5; LCSC C3975153 -> C2897409
- MK65, MK66, MK67, MK68, MK69, MK70, MK71, MK72, MK76, MK77: value PH2.54-1X1P-H25 -> BOOMELE 2.54-1x40P-21mm; cut to 1P; hand/wave soldered; footprint EasyEDA:HDR-TH_1P-P2.54-V-M -> EasyEDA:HDR-TH_1P-P2.54-V-M-21MM-C51353; symbol EasyEDA:PH2.54-1X1P-H25 -> Connector_Generic:Conn_01x01; LCSC C42431799 -> C51353
Connections:
- net SLOT_B_POWER_SELECTED is gone; now on net AUX_RAIL: F16.1
- net SLOT_C_POWER_SELECTED is gone; now on net AUX_RAIL: F20.1
- net SLOT_D_POWER_SELECTED is gone; now on net AUX_RAIL: F24.1
- net SLOT_E_POWER_SELECTED is gone; now on net AUX_RAIL: F28.1
- net SLOT_F_POWER_SELECTED is gone; now on net AUX_RAIL: F32.1
- net SLOT_G_POWER_SELECTED is gone; now on net AUX_RAIL: F36.1
- net SLOT_H_POWER_SELECTED is gone; now on net AUX_RAIL: F40.1
- net SLOT_L_POWER_SELECTED is gone; now on net AUX_RAIL: F4.1
- net SLOT_M_POWER_SELECTED is gone; now on net AUX_RAIL: F8.1
- net BUS5V0_PIN4: now also J7.7; no longer J7.5
- net BUS5V0_PIN5: now also J7.8; no longer J7.6
- net BUS5V0_PIN6: now also J7.9; no longer J7.7
- net BUS5V0_PIN7: now also J7.10; no longer J7.8
- net BUS5V1_PIN4: now also J8.7; no longer J8.5
- net BUS5V1_PIN5: now also J8.8; no longer J8.6
- net BUS5V1_PIN6: now also J8.9; no longer J8.7
- net BUS5V1_PIN7: now also J8.10; no longer J8.8
- net GND: now also J3.11, J3.12, J3.21, J3.22, J3.27, J3.28, J3.37, J3.38, J3.43, J3.44, J3.5, J3.53, J3.54, J3.59, J3.6, J3.60, J5.11, J5.12, J5.21, J5.22, J5.27, J5.28, J5.37, J5.38, J5.43, J5.44, J5.5, J5.53, J5.54, J5.59, J5.6, J5.60, J53.2, J53.4, J53.6, J54.2, J54.4, J54.6, J55.2, J55.4, J55.6, J56.2, J56.4, J56.6, J57.2, J57.4, J57.6, J58.2, J58.4, J58.6, J7.5, J7.6, J8.5, J8.6, J62.2, J62.4, J62.6, J63.2, J63.4, J63.6, J64.2, J64.4, J64.6, J65.2, J65.4, J65.6; no longer J3.15, J3.16, J3.17, J3.18, J3.25, J3.26, J3.7, J3.8, J5.15, J5.16, J5.17, J5.18, J5.25, J5.26, J5.7, J5.8, J53.1, J53.11, J53.13, J53.15, J53.3, J53.5, J53.7, J53.9, J54.1, J54.11, J54.13, J54.15, J54.3, J54.5, J54.7, J54.9, J55.1, J55.11, J55.13, J55.15, J55.3, J55.5, J55.7, J55.9, J56.1, J56.11, J56.13, J56.15, J56.3, J56.5, J56.7, J56.9, J57.1, J57.3, J57.5, J57.7, J58.1, J58.3, J58.5, J58.7, J7.10, J7.13, J7.14, J7.15, J7.16, J7.9, J8.10, J8.13, J8.14, J8.15, J8.16, J8.9
- net SLOTA_IO1: now also J3.2; no longer J3.32
- net SLOTA_IO10: now also J3.15; no longer J3.6
- net SLOTA_IO11: now also J3.16; no longer J3.27
- net SLOTA_IO2: now also J3.3; no longer J3.2
- net SLOTA_IO3: now also J3.4; no longer J3.31
- net SLOTA_IO4: now also J3.7; no longer J3.3
- net SLOTA_IO5: now also J3.8; no longer J3.30
- net SLOTA_IO6: now also J3.9; no longer J3.4
- net SLOTA_IO7: now also J3.10; no longer J3.29
- net SLOTA_IO8: now also J3.13; no longer J3.5
- net SLOTA_IO9: now also J3.14; no longer J3.28
- net SLOTB_IO0: now also J3.17; no longer J3.9
- net SLOTB_IO1: now also J3.18; no longer J3.24
- net SLOTB_IO10: now also J3.31; no longer J3.14
- net SLOTB_IO11: now also J3.32; no longer J3.19
- net SLOTB_IO2: now also J3.19; no longer J3.10
- net SLOTB_IO3: now also J3.20; no longer J3.23
- net SLOTB_IO4: now also J3.23; no longer J3.11
- net SLOTB_IO5: now also J3.24; no longer J3.22
- net SLOTB_IO6: now also J3.25; no longer J3.12
- net SLOTB_IO7: now also J3.26; no longer J3.21
- net SLOTB_IO8: now also J3.29; no longer J3.13
- net SLOTB_IO9: now also J3.30; no longer J3.20
- net SLOTC_IO0: now also J3.33
- net SLOTC_IO1: now also J3.34
- net SLOTC_IO10: now also J3.47
- net SLOTC_IO11: now also J3.48
- net SLOTC_IO2: now also J3.35
- net SLOTC_IO3: now also J3.36
- net SLOTC_IO4: now also J3.39
- net SLOTC_IO5: now also J3.40
- net SLOTC_IO6: now also J3.41
- net SLOTC_IO7: now also J3.42
- net SLOTC_IO8: now also J3.45
- net SLOTC_IO9: now also J3.46
- net SLOTD_IO0: now also J3.49
- net SLOTD_IO1: now also J3.50
- net SLOTD_IO10: now also J3.63
- net SLOTD_IO11: now also J3.64
- net SLOTD_IO2: now also J3.51
- net SLOTD_IO3: now also J3.52
- net SLOTD_IO4: now also J3.55
- net SLOTD_IO5: now also J3.56
- net SLOTD_IO6: now also J3.57
- net SLOTD_IO7: now also J3.58
- net SLOTD_IO8: now also J3.61
- net SLOTD_IO9: now also J3.62
- net SLOTE_IO0: now also J5.64; no longer J5.1
- net SLOTE_IO1: now also J5.63; no longer J5.32
- net SLOTE_IO10: now also J5.50; no longer J5.6
- net SLOTE_IO11: now also J5.49; no longer J5.27
- net SLOTE_IO2: now also J5.62; no longer J5.2
- net SLOTE_IO3: now also J5.61; no longer J5.31
- net SLOTE_IO4: now also J5.58; no longer J5.3
- net SLOTE_IO5: now also J5.57; no longer J5.30
- net SLOTE_IO6: now also J5.56; no longer J5.4
- net SLOTE_IO7: now also J5.55; no longer J5.29
- net SLOTE_IO8: now also J5.52; no longer J5.5
- net SLOTE_IO9: now also J5.51; no longer J5.28
- net SLOTF_IO0: now also J5.48; no longer J5.9
- net SLOTF_IO1: now also J5.47; no longer J5.24
- net SLOTF_IO10: now also J5.34; no longer J5.14
- net SLOTF_IO11: now also J5.33; no longer J5.19
- net SLOTF_IO2: now also J5.46; no longer J5.10
- net SLOTF_IO3: now also J5.45; no longer J5.23
- net SLOTF_IO4: now also J5.42; no longer J5.11
- net SLOTF_IO5: now also J5.41; no longer J5.22
- net SLOTF_IO6: now also J5.40; no longer J5.12
- net SLOTF_IO7: now also J5.39; no longer J5.21
- net SLOTF_IO8: now also J5.36; no longer J5.13
- net SLOTF_IO9: now also J5.35; no longer J5.20
- net SLOTG_IO0: now also J5.32
- net SLOTG_IO1: now also J5.31
- net SLOTG_IO10: now also J5.18
- net SLOTG_IO11: now also J5.17
- net SLOTG_IO2: now also J5.30
- net SLOTG_IO3: now also J5.29
- net SLOTG_IO4: now also J5.26
- net SLOTG_IO5: now also J5.25
- net SLOTG_IO6: now also J5.24
- net SLOTG_IO7: now also J5.23
- net SLOTG_IO8: now also J5.20
- net SLOTG_IO9: now also J5.19
- net SLOTH_IO0: now also J5.16
- net SLOTH_IO1: now also J5.15
- net SLOTH_IO10: now also J5.2
- net SLOTH_IO11: now also J5.1
- net SLOTH_IO2: now also J5.14
- net SLOTH_IO3: now also J5.13
- net SLOTH_IO4: now also J5.10
- net SLOTH_IO5: now also J5.9
- net SLOTH_IO6: now also J5.8
- net SLOTH_IO7: now also J5.7
- net SLOTH_IO8: now also J5.4
- net SLOTH_IO9: now also J5.3
- net SLOT_A_3V3: now also J53.3; no longer J53.4
- net SLOT_A_5V: now also J53.5; no longer J53.6
- net SLOT_A_PIN_VOLTAGE: now also J53.1; no longer J53.2
- net SLOT_B_3V3: now also J62.3; no longer J53.12
- net SLOT_B_5V: now also J62.5; no longer J53.14
- net SLOT_B_PIN_VOLTAGE: now also J62.1; no longer J53.10
- net SLOT_C_3V3: now also J54.3; no longer J54.4
- net SLOT_C_5V: now also J54.5; no longer J54.6
- net SLOT_C_PIN_VOLTAGE: now also J54.1; no longer J54.2
- net SLOT_D_3V3: now also J63.3; no longer J54.12
- net SLOT_D_5V: now also J63.5; no longer J54.14
- net SLOT_D_PIN_VOLTAGE: now also J63.1; no longer J54.10
- net SLOT_E_3V3: now also J55.3; no longer J55.4
- net SLOT_E_5V: now also J55.5; no longer J55.6
- net SLOT_E_PIN_VOLTAGE: now also J55.1; no longer J55.2
- net SLOT_F_3V3: now also J64.3; no longer J55.12
- net SLOT_F_5V: now also J64.5; no longer J55.14
- net SLOT_F_PIN_VOLTAGE: now also J64.1; no longer J55.10
- net SLOT_G_3V3: now also J56.3; no longer J56.4
- net SLOT_G_5V: now also J56.5; no longer J56.6
- net SLOT_G_PIN_VOLTAGE: now also J56.1; no longer J56.2
- net SLOT_H_3V3: now also J65.3; no longer J56.12
- net SLOT_H_5V: now also J65.5; no longer J56.14
- net SLOT_H_PIN_VOLTAGE: now also J65.1; no longer J56.10
- net SLOT_L_3V3: now also J57.3; no longer J57.4
- net SLOT_L_5V: now also J57.5; no longer J57.6
- net SLOT_L_PIN_VOLTAGE: now also J57.1; no longer J57.2
- net SLOT_M_3V3: now also J58.3; no longer J58.4
- net SLOT_M_5V: now also J58.5; no longer J58.6
- net SLOT_M_PIN_VOLTAGE: now also J58.1; no longer J58.2
- net SLOT_A_POWER renamed SLOT_A_AUX
- net SLOT_A_AUX: now also J53.7; no longer J53.8
- net SLOT_A_POWER_SELECTED renamed AUX_RAIL
- net SLOT_B_POWER renamed SLOT_B_AUX
- net SLOT_B_AUX: now also J62.7; no longer J53.16
- net SLOT_C_POWER renamed SLOT_C_AUX
- net SLOT_C_AUX: now also J54.7; no longer J54.8
- net SLOT_D_POWER renamed SLOT_D_AUX
- net SLOT_D_AUX: now also J63.7; no longer J54.16
- net SLOT_E_POWER renamed SLOT_E_AUX
- net SLOT_E_AUX: now also J55.7; no longer J55.8
- net SLOT_F_POWER renamed SLOT_F_AUX
- net SLOT_F_AUX: now also J64.7; no longer J55.16
- net SLOT_G_POWER renamed SLOT_G_AUX
- net SLOT_G_AUX: now also J56.7; no longer J56.8
- net SLOT_H_POWER renamed SLOT_H_AUX
- net SLOT_H_AUX: now also J65.7; no longer J56.16
- net SLOT_L_POWER renamed SLOT_L_AUX
- net SLOT_L_AUX: now also J57.7; no longer J57.8
- net SLOT_M_POWER renamed SLOT_M_AUX
- net SLOT_M_AUX: now also J58.7; no longer J58.8
- no-connect marks 0 -> 8
Other:
- note added: "SHIELD HEADER ABCD"
- note added: "SHIELD HEADER EFGH"
- note added: "SHIELD HEADER L"
- note added: "SHIELD HEADER M"
- note added: "SLOTS — Ten keyed extension ports, branch fusing and level shifting — HW 0.1.0-proto.1"
- note removed: "SHIELD HEADER AB"
- note removed: "SHIELD HEADER CD"
- note removed: "SHIELD HEADER EF"
- note removed: "SHIELD HEADER GH"
- note removed: "SLOTS — Ten extension ports, rail selection, fusing, level shifting — HW 0.1.0-proto.1"
- moved on the sheet: C143, C144, C145, C146, C147, C148, C149, C150, C151, C152, C153, C154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
