File: kicad/memory.kicad_sch (KiCad schematic)
At the start: 10 parts, among them U2 APS1604M-3SQR-SN, U3 APS1604M-3SQR-SN, U4 APS1604M-3SQR-SN, U5 APS1604M-3SQR-SN, U6 W25Q256JVEIQ

Commit message: fix 14 package mismatches, assert footprints against ki_fp_filters, rebalance fuses, correct JTAG and PD-voltage claims
Parts:
- U2, U3, U4, U5: footprint Package_SO:SOIC-8_5.3x5.3mm_P1.27mm -> Package_SO:SOIC-8_3.9x4.9mm_P1.27mm
- U6: footprint Package_SO:SOIC-8_5.3x5.3mm_P1.27mm -> Package_SON:WSON-8-1EP_8x6mm_P1.27mm_EP3.4x4.3mm
Changed lines of the file:
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@@
 		(property "Reference" "U2" (at 87.63 67.31 0) (effects (font (size 1.27 1.27))))
 		(property "Value" "APS1604M-3SQR-SN" (at 87.63 100.33 0) (effects (font (size 1.27 1.27))))
-		(property "Footprint" "Package_SO:SOIC-8_5.3x5.3mm_P1.27mm" (at 87.63 100.33 0) (effects (font (size 1.27 1.27)) (hide yes)))
+		(property "Footprint" "Package_SO:SOIC-8_3.9x4.9mm_P1.27mm" (at 87.63 100.33 0) (effects (font (size 1.27 1.27)) (hide yes)))
 		(property "LCSC" "C18214056" (at 87.63 100.33 0) (effects (font (size 1.27 1.27)) (hide yes)))
 		(instances (project "odin" (path "/c44fb7fe-6133-ad34-68fd-fb66126197ef/97100407-f2fb-0487-90af-0c60df3be2db" (reference "U2") (unit 1))))
@@
 		(property "Reference" "U3" (at 213.36 67.31 0) (effects (font (size 1.27 1.27))))
 		(property "Value" "APS1604M-3SQR-SN" (at 213.36 100.33 0) (effects (font (size 1.27 1.27))))
-		(property "Footprint" "Package_SO:SOIC-8_5.3x5.3mm_P1.27mm" (at 213.36 100.33 0) (effects (font (size 1.27 1.27)) (hide yes)))
+		(property "Footprint" "Package_SO:SOIC-8_3.9x4.9mm_P1.27mm" (at 213.36 100.33 0) (effects (font (size 1.27 1.27)) (hide yes)))
 		(property "LCSC" "C18214056" (at 213.36 100.33 0) (effects (font (size 1.27 1.27)) (hide yes)))
 		(instances (project "odin" (path "/c44fb7fe-6133-ad34-68fd-fb66126197ef/97100407-f2fb-0487-90af-0c60df3be2db" (reference "U3") (unit 1))))
@@
 		(property "Reference" "U4" (at 87.63 210.82 0) (effects (font (size 1.27 1.27))))
 		(property "Value" "APS1604M-3SQR-SN" (at 87.63 243.84 0) (effects (font (size 1.27 1.27))))
-		(property "Footprint" "Package_SO:SOIC-8_5.3x5.3mm_P1.27mm" (at 87.63 243.84 0) (effects (font (size 1.27 1.27)) (hide yes)))
+		(property "Footprint" "Package_SO:SOIC-8_3.9x4.9mm_P1.27mm" (at 87.63 243.84 0) (effects (font (size 1.27 1.27)) (hide yes)))
 		(property "LCSC" "C18214056" (at 87.63 243.84 0) (effects (font (size 1.27 1.27)) (hide yes)))
 		(instances (project "odin" (path "/c44fb7fe-6133-ad34-68fd-fb66126197ef/97100407-f2fb-0487-90af-0c60df3be2db" (reference "U4") (unit 1))))
@@
 		(property "Reference" "U5" (at 213.36 210.82 0) (effects (font (size 1.27 1.27))))
 		(property "Value" "APS1604M-3SQR-SN" (at 213.36 243.84 0) (effects (font (size 1.27 1.27))))
-		(property "Footprint" "Package_SO:SOIC-8_5.3x5.3mm_P1.27mm" (at 213.36 243.84 0) (effects (font (size 1.27 1.27)) (hide yes)))
+		(property "Footprint" "Package_SO:SOIC-8_3.9x4.9mm_P1.27mm" (at 213.36 243.84 0) (effects (font (size 1.27 1.27)) (hide yes)))
 		(property "LCSC" "C18214056" (at 213.36 243.84 0) (effects (font (size 1.27 1.27)) (hide yes)))
 		(instances (project "odin" (path "/c44fb7fe-6133-ad34-68fd-fb66126197ef/97100407-f2fb-0487-90af-0c60df3be2db" (reference "U5") (unit 1))))
@@
 		(property "Reference" "U6" (at 95.25 353.06 0) (effects (font (size 1.27 1.27))))
 		(property "Value" "W25Q256JVEIQ" (at 95.25 370.84 0) (effects (font (size 1.27 1.27))))
-		(property "Footprint" "Package_SO:SOIC-8_5.3x5.3mm_P1.27mm" (at 95.25 370.84 0) (effects (font (size 1.27 1.27)) (hide yes)))
+		(property "Footprint" "Package_SON:WSON-8-1EP_8x6mm_P1.27mm_EP3.4x4.3mm" (at 95.25 370.84 0) (effects (font (size 1.27 1.27)) (hide yes)))
 		(property "LCSC" "C97522" (at 95.25 370.84 0) (effects (font (size 1.27 1.27)) (hide yes)))
 		(instances (project "odin" (path "/c44fb7fe-6133-ad34-68fd-fb66126197ef/97100407-f2fb-0487-90af-0c60df3be2db" (reference "U6") (unit 1))))

Commit message: Update Odin hardware design, imported parts, and documentation
Include EasyEDA symbols, footprints and 3D models; revise FPGA allocation, power and extension buses; add qualification audits and user documentation.

Validation: EasyEDA audit, qualified parts, power budget and Python syntax pass. KiCad ERC reports 1 error and 319 warnings; DRC reports 90 violations, 499 unconnected items and 209 schematic parity issues. This is a work-in-progress design snapshot. Imported vendor assets retain their original formatting.
Parts:
- removed C75, C76, C77, C78, C79: 100nF, Capacitor_SMD:C_0402_1005Metric, symbol Device:C
- added C112, C113, C114, C115, C116: 100nF, Capacitor_SMD:C_0402_1005Metric, symbol Device:C
- U2, U3, U4, U5: footprint Package_SO:SOIC-8_3.9x4.9mm_P1.27mm -> EasyEDA:SOIC-8_L4.9-W3.9-P1.27-LS6.0-BL
- U6: footprint Package_SON:WSON-8-1EP_8x6mm_P1.27mm_EP3.4x4.3mm -> EasyEDA:WSON-8_L8.0-W6.10-P1.27-BL-EP
Connections:
- net +3V3: now also C112.1, C113.1, C114.1, C115.1, C116.1
- net GND: now also U6.9 (EP), C112.2, C113.2, C114.2, C115.2, C116.2
Other:
- note added: "MEMORY — PSRAM x4 (independent buses) and configuration flash — HW 0.1.0-proto.1"
- note removed: "MEMORY — PSRAM x4 (independent buses) and configuration flash"

Commit message: wip
Parts:
- removed C116: 100nF, Capacitor_SMD:C_0402_1005Metric, symbol Device:C
- added C111: 100nF, Capacitor_SMD:C_0402_1005Metric, symbol Device:C
- added R104, R105, R106, R107, R108, R109, R110, R111, R112, R113, R114, R115, R116, R117, R118, R119, R120, R121, R122, R123, R124, R125, R126, R127: 33, Resistor_SMD:R_0402_1005Metric, symbol Device:R
Connections:
- net +3V3: now also C111.1
- net GND: now also C111.2
- net PSRAM0_CE_B: now also R105.1; no longer U2.1 (~{CE})
- net PSRAM0_IO0: now also R106.1; no longer U2.5 (SI/SIO0)
- net PSRAM0_IO1: now also R107.1; no longer U2.2 (SO/SIO1)
- net PSRAM0_IO2: now also R108.1; no longer U2.3 (SIO2)
- net PSRAM0_IO3: now also R109.1; no longer U2.7 (SIO3)
- net PSRAM0_SCK: now also R104.1; no longer U2.6 (SCLK)
- net PSRAM1_CE_B: now also R111.1; no longer U3.1 (~{CE})
- net PSRAM1_IO0: now also R112.1; no longer U3.5 (SI/SIO0)
- net PSRAM1_IO1: now also R113.1; no longer U3.2 (SO/SIO1)
- net PSRAM1_IO2: now also R114.1; no longer U3.3 (SIO2)
- net PSRAM1_IO3: now also R115.1; no longer U3.7 (SIO3)
- net PSRAM1_SCK: now also R110.1; no longer U3.6 (SCLK)
- net PSRAM2_CE_B: now also R117.1; no longer U4.1 (~{CE})
- net PSRAM2_IO0: now also R118.1; no longer U4.5 (SI/SIO0)
- net PSRAM2_IO1: now also R119.1; no longer U4.2 (SO/SIO1)
- net PSRAM2_IO2: now also R120.1; no longer U4.3 (SIO2)
- net PSRAM2_IO3: now also R121.1; no longer U4.7 (SIO3)
- net PSRAM2_SCK: now also R116.1; no longer U4.6 (SCLK)
- net PSRAM3_CE_B: now also R123.1; no longer U5.1 (~{CE})
- net PSRAM3_IO0: now also R124.1; no longer U5.5 (SI/SIO0)
- net PSRAM3_IO1: now also R125.1; no longer U5.2 (SO/SIO1)
- net PSRAM3_IO2: now also R126.1; no longer U5.3 (SIO2)
- net PSRAM3_IO3: now also R127.1; no longer U5.7 (SIO3)
- net PSRAM3_SCK: now also R122.1; no longer U5.6 (SCLK)
- new net PSRAM0_CE_B_MEM: R105.2, U2.1 (~{CE})
- new net PSRAM0_IO0_MEM: R106.2, U2.5 (SI/SIO0)
- new net PSRAM0_IO1_MEM: R107.2, U2.2 (SO/SIO1)
- new net PSRAM0_IO2_MEM: R108.2, U2.3 (SIO2)
- new net PSRAM0_IO3_MEM: R109.2, U2.7 (SIO3)
- new net PSRAM0_SCK_MEM: R104.2, U2.6 (SCLK)
- new net PSRAM1_CE_B_MEM: R111.2, U3.1 (~{CE})
- new net PSRAM1_IO0_MEM: R112.2, U3.5 (SI/SIO0)
- new net PSRAM1_IO1_MEM: R113.2, U3.2 (SO/SIO1)
- new net PSRAM1_IO2_MEM: R114.2, U3.3 (SIO2)
- new net PSRAM1_IO3_MEM: R115.2, U3.7 (SIO3)
- new net PSRAM1_SCK_MEM: R110.2, U3.6 (SCLK)
- new net PSRAM2_CE_B_MEM: R117.2, U4.1 (~{CE})
- new net PSRAM2_IO0_MEM: R118.2, U4.5 (SI/SIO0)
- new net PSRAM2_IO1_MEM: R119.2, U4.2 (SO/SIO1)
- new net PSRAM2_IO2_MEM: R120.2, U4.3 (SIO2)
- new net PSRAM2_IO3_MEM: R121.2, U4.7 (SIO3)
- new net PSRAM2_SCK_MEM: R116.2, U4.6 (SCLK)
- new net PSRAM3_CE_B_MEM: R123.2, U5.1 (~{CE})
- new net PSRAM3_IO0_MEM: R124.2, U5.5 (SI/SIO0)
- new net PSRAM3_IO1_MEM: R125.2, U5.2 (SO/SIO1)
- new net PSRAM3_IO2_MEM: R126.2, U5.3 (SIO2)
- new net PSRAM3_IO3_MEM: R127.2, U5.7 (SIO3)
- new net PSRAM3_SCK_MEM: R122.2, U5.6 (SCLK)
Other:
- note added: "PSRAM0 series termination"
- note added: "PSRAM1 series termination"
- note added: "PSRAM2 series termination"
- note added: "PSRAM3 series termination"
- moved on the sheet: C112, C113, C115, U4, U5, U6
