File: kicad/memory.kicad_sch (KiCad schematic)
At the start: 34 parts, among them U2 APS1604M-3SQR-SN, U3 APS1604M-3SQR-SN, U4 APS1604M-3SQR-SN, U5 APS1604M-3SQR-SN, U6 W25Q256JVEIQ

Commit message: Explain the remaining four sheets: power, memory, board controller, slots
Every part and group on the board now has its plain-words purpose, and the
gate enforces it on all six sheets. Net notes can cover a family of nets
by prefix, so regulator feedback, enables and the PSRAM series resistors
read correctly; passives credit their group's IC or connector rather than
a key post; monitor nets are no longer mistaken for supplies; parts that
are not fitted say so. PCB synced with no footprint moved.
Other:
- note added: "One 33 ohm resistor per PSRAM0 line, placed next to the FPGA: they soften the fast signal edges so they do not ring along the trace. Values can be tuned after measurement (ref/psram.md)."
- note added: "One 33 ohm resistor per PSRAM1 line, next to the FPGA, to damp ringing."
- note added: "One 33 ohm resistor per PSRAM2 line, next to the FPGA, to damp ringing."
- note added: "One 33 ohm resistor per PSRAM3 line, next to the FPGA, to damp ringing."
- note added: "The FPGA's non-volatile memory. At power-on the FPGA reads its design (bitstream) from this 32 MB flash by itself (master SPI, set by the mode straps). The board controller can rewrite it through the series resistors on the Board Controller sheet, and spare space can hold user data or software for a soft CPU."
- note added: "Working-memory chip 0: 2 MB of fast RAM for the FPGA design, on its own four-bit (QSPI) bus to bank 14. The four chips are independent, so a design can use them in parallel. Notes: ref/psram.md."
- note added: "Working-memory chip 1: 2 MB of RAM on its own QSPI bus to bank 14."
- note added: "Working-memory chip 2: 2 MB of RAM on its own QSPI bus to bank 14."
- note added: "Working-memory chip 3: 2 MB of RAM on its own QSPI bus to bank 14."
- moved on the sheet: C111, C112, C113, C114, C115, R104, R105, R106, R107, R108, R109, R110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

Commit message: Step 2: bank 13 to 1.8V and the PSRAM move
SN74LXC8T245 datasheet SCES916A (rev. March 2023), section 6.3
Recommended Operating Conditions, page 5: VCCA 1.08 V to 5.5 V, so the
A side runs from +1V8_IO. Table 5-1 (page 3) states the same range on
the VCCA pin. Copy in ref/datasheets/sn74lxc8t245.pdf.

APS6404L-SQN-SN: datasheet rev 4.0, Table 9 page 26 (VDD 1.62 to 1.98 V,
ICC 7 mA), section 4.1 page 5 (SOP-8L(150): D 4.90, E1 3.90, E 6.00 BSC,
e 1.27 BSC), which the fitted SOIC-8_L4.9-W3.9-P1.27-LS6.0-BL matches.
Copy in ref/datasheets/aps6404l-sqn.pdf. The symbol for C5360304 is
imported into easyeda/EasyEDA.kicad_sym pointing at that footprint, and
load_pcb.py now refreshes the LCSC field on every sync.
Parts:
- U2, U3, U4, U5: value APS1604M-3SQR-SN -> APS6404L-SQN-SN; symbol Memory_RAM:APS1604M-3SQRx-SN -> Memory_RAM:APS6404L-SQRx-SN; LCSC C18214056 -> C5360304
Connections:
- net +3V3: no longer C111.1, C112.1, C113.1, C114.1, U2.8 (VDD), U3.8 (VDD), U4.8 (VDD), U5.8 (VDD)
- new net +1V8_IO: C111.1, C112.1, C113.1, C114.1, U2.8 (VDD), U3.8 (VDD), U4.8 (VDD), U5.8 (VDD)
Other:
- note added: "Working-memory chip 0: 8 MB of fast RAM for the FPGA design, on its own four-bit (QSPI) bus to bank 13 at 1.8 V. The four chips are independent, so a design can use them in parallel. Notes: ref/psram.md."
- note added: "Working-memory chip 1: 8 MB of RAM on its own QSPI bus to bank 13, at 1.8 V."
- note added: "Working-memory chip 2: 8 MB of RAM on its own QSPI bus to bank 13, at 1.8 V."
- note added: "Working-memory chip 3: 8 MB of RAM on its own QSPI bus to bank 13, at 1.8 V."
- note removed: "Working-memory chip 0: 2 MB of fast RAM for the FPGA design, on its own four-bit (QSPI) bus to bank 14. The four chips are independent, so a design can use them in parallel. Notes: ref/psram.md."
- note removed: "Working-memory chip 1: 2 MB of RAM on its own QSPI bus to bank 14."
- note removed: "Working-memory chip 2: 2 MB of RAM on its own QSPI bus to bank 14."
- note removed: "Working-memory chip 3: 2 MB of RAM on its own QSPI bus to bank 14."

Commit message: Step 4: SDRAM
Parts:
- added C250, C251, C252, C253, C254, C255, C256: 100nF, Capacitor_SMD:C_0402_1005Metric, symbol Device:C
- added C257: 10uF, Capacitor_SMD:C_0805_2012Metric, symbol Device:C
- added R151: 22, Resistor_SMD:R_0402_1005Metric, symbol Device:R
- added R152, R153: 10k, Resistor_SMD:R_0603_1608Metric, symbol Device:R
- added U32: W9825G6KH-6, Package_SO:TSOP-II-54_22.2x10.16mm_P0.8mm, symbol odin:W9825G6KH
Connections:
- net +3V3: now also C250.1, C251.1, C252.1, C253.1, C254.1, C255.1, C256.1, C257.1, R152.1, U32.1 (VDD), U32.14 (VDD), U32.27 (VDD), U32.3 (VDDQ), U32.43 (VDDQ), U32.49 (VDDQ), U32.9 (VDDQ)
- net GND: now also C250.2, C251.2, C252.2, C253.2, C254.2, C255.2, C256.2, C257.2, R153.2, U32.12 (VSSQ), U32.28 (VSS), U32.41 (VSS), U32.46 (VSSQ), U32.52 (VSSQ), U32.54 (VSS), U32.6 (VSSQ)
- new net SDRAM_A0: U32.23 (A0)
- new net SDRAM_A1: U32.24 (A1)
- new net SDRAM_A10: U32.22 (A10)
- new net SDRAM_A11: U32.35 (A11)
- new net SDRAM_A12: U32.36 (A12)
- new net SDRAM_A2: U32.25 (A2)
- new net SDRAM_A3: U32.26 (A3)
- new net SDRAM_A4: U32.29 (A4)
- new net SDRAM_A5: U32.30 (A5)
- new net SDRAM_A6: U32.31 (A6)
- new net SDRAM_A7: U32.32 (A7)
- new net SDRAM_A8: U32.33 (A8)
- new net SDRAM_A9: U32.34 (A9)
- new net SDRAM_BA0: U32.20 (BS0)
- new net SDRAM_BA1: U32.21 (BS1)
- new net SDRAM_CAS_N: U32.17 (~{CAS})
- new net SDRAM_CKE: R153.1, U32.37 (CKE)
- new net SDRAM_CLK: R151.1
- new net SDRAM_CLK_MEM: R151.2, U32.38 (CLK)
- new net SDRAM_CS_N: R152.2, U32.19 (~{CS})
- new net SDRAM_DQ0: U32.2 (DQ0)
- new net SDRAM_DQ1: U32.4 (DQ1)
- new net SDRAM_DQ10: U32.45 (DQ10)
- new net SDRAM_DQ11: U32.47 (DQ11)
- new net SDRAM_DQ12: U32.48 (DQ12)
- new net SDRAM_DQ13: U32.50 (DQ13)
- new net SDRAM_DQ14: U32.51 (DQ14)
- new net SDRAM_DQ15: U32.53 (DQ15)
- new net SDRAM_DQ2: U32.5 (DQ2)
- new net SDRAM_DQ3: U32.7 (DQ3)
- new net SDRAM_DQ4: U32.8 (DQ4)
- new net SDRAM_DQ5: U32.10 (DQ5)
- new net SDRAM_DQ6: U32.11 (DQ6)
- new net SDRAM_DQ7: U32.13 (DQ7)
- new net SDRAM_DQ8: U32.42 (DQ8)
- new net SDRAM_DQ9: U32.44 (DQ9)
- new net SDRAM_LDQM: U32.15 (LDQM)
- new net SDRAM_RAS_N: U32.18 (~{RAS})
- new net SDRAM_UDQM: U32.39 (UDQM)
- new net SDRAM_WE_N: U32.16 (~{WE})
- no-connect marks 0 -> 1
Other:
- note added: "A 32 MB SDR SDRAM (Winbond W9825G6KH-6, 16 bits wide, up to 166 MHz) for designs that outgrow the PSRAMs: a framebuffer, a soft CPU's main memory, a capture buffer. Its data and control lines come from bank 35 and its address lines from bank 14, both at 3.3 V. One 100 nF per VDD/VDDQ pin pair (seven, datasheet pins 1, 14, 27 and 3, 9, 43, 49) and a 10 uF bulk; a 22 ohm series resistor at the FPGA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"
- note added: "MEMORY — PSRAM x4 (independent buses, 1.8 V), SDRAM and configuration flash — HW 0.1.0-proto.1"
- note added: "SDRAM"
- note removed: "MEMORY — PSRAM x4 (independent buses) and configuration flash — HW 0.1.0-proto.1"
- moved on the sheet: R116, R117, R118, R119, R120, R121, R122, R123, R124, R125, R126, R127
