File: kicad/memory.kicad_sch (KiCad schematic)
At the start: 46 parts, among them U2 APS6404L-SQN-SN, U3 APS6404L-SQN-SN, U32 W9825G6KH-6, U4 APS6404L-SQN-SN, U5 APS6404L-SQN-SN, U6 W25Q256JVEIQ

Commit message: Step 5: MRAM, optional populate
Parts:
- added C258: 100nF, Capacitor_SMD:C_0402_1005Metric, symbol Device:C
- added R154, R155, R156: 10k, Resistor_SMD:R_0603_1608Metric, symbol Device:R
- added U33: MR25H10CDF, odin:DFN-8_L5.0-W6.0-P1.27-EP2.0-2VIA, symbol EasyEDA:MR25H10CDF
Connections:
- net +3V3: now also C258.1, R154.1, R155.1, R156.1, U33.8 (VDD)
- net GND: now also C258.2, U33.4 (VSS), U33.9 (EP)
- new net MRAM_CS: R154.2, U33.1 (~{CS})
- new net MRAM_HOLD: R156.2, U33.7 (~{HOLD})
- new net MRAM_SCK: U33.6 (SCK)
- new net MRAM_SI: U33.5 (SI)
- new net MRAM_SO: U33.2 (SO)
- new net MRAM_WP: R155.2, U33.3 (~{WP})
Other:
- note added: "A 128 KB non-volatile SPI memory (Everspin MR25H10CDF) that keeps its contents without power and has no write wear: settings, logs, a boot menu, a save file. Not fitted by default; a build that wants it fits U33 and these four passives together. CS is pulled up so the chip stays deselected while power comes up (datasheet section 4); WP and HOLD are pulled up and not connected to the FPGA, so writ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"
- note added: "MEMORY — PSRAM x4 (independent buses, 1.8 V), SDRAM, MRAM option and configuration flash — HW 0.1.0-proto.1"
- note added: "MRAM (populate option)"
- note removed: "MEMORY — PSRAM x4 (independent buses, 1.8 V), SDRAM and configuration flash — HW 0.1.0-proto.1"

Commit message: Step 6: microSD socket
Parts:
- added C259: 100nF, Capacitor_SMD:C_0402_1005Metric, symbol Device:C
- added C260: 10uF, Capacitor_SMD:C_0805_2012Metric, symbol Device:C
- added J74: microSD, EasyEDA:TF-SMD_TF-01A, symbol EasyEDA:TF-01A_C91145
- added R157, R158, R159, R160, R161: 10k, Resistor_SMD:R_0603_1608Metric, symbol Device:R
Connections:
- net +3V3: now also C259.1, C260.1, J74.4 (VDD), R157.1, R158.1, R159.1, R160.1, R161.1
- net GND: now also C259.2, C260.2, J74.10 (GND), J74.11 (GND), J74.12 (GND), J74.13 (GND), J74.6 (VSS)
- new net SD_CD: J74.9 (CD)
- new net SD_CS: J74.2 (CDDAT3(CS)), R157.2
- new net SD_DAT1: J74.8 (DAT1(RSV)), R160.2
- new net SD_DAT2: J74.1 (DAT2(RSV)), R161.2
- new net SD_MISO: J74.7 (DAT0(D0)), R159.2
- new net SD_MOSI: J74.3 (CMD(DI)), R158.2
- new net SD_SCK: J74.5 (CLK(SCLK))
Other:
- note added: "A push-push microSD socket (Hroparts TF-01A) wired for SPI mode: chip select on DAT3, data in on CMD, data out on DAT0, clock on CLK, five bank 14 lines at 3.3 V including the card-detect switch. The 10k pull-ups hold CS, the two data lines and the two unused DAT lines high, as the SD specification asks for SPI mode; the 100 nF and 10 uF feed the card's supply at the socket; the shell is grounded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"
- note added: "MEMORY — PSRAM x4 (independent buses, 1.8 V), SDRAM, MRAM option, microSD and configuration flash — HW 0.1.0-proto.1"
- note added: "microSD socket"
- note removed: "MEMORY — PSRAM x4 (independent buses, 1.8 V), SDRAM, MRAM option and configuration flash — HW 0.1.0-proto.1"
- moved on the sheet: C113, C114, C115, C250, C251, C252, C253, C254, C255, C256, C257, C258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

Commit message: MRAM fitted on every board
Parts:
- C258, R154, R155, R156, U33: now fitted
Other:
- note added: "A 128 KB non-volatile SPI memory (Everspin MR25H10CDF) that keeps its contents without power and has no write wear: settings, logs, a boot menu, a save file. CS is pulled up so the chip stays deselected while power comes up (datasheet section 4); WP and HOLD are pulled up and not connected to the FPGA, so writes are allowed and transfers never pause. The exposed pad is ground only, with two vias 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"
- note added: "MEMORY — PSRAM x4 (independent buses, 1.8 V), SDRAM, MRAM, microSD and configuration flash — HW 0.1.0-proto.1"
- note added: "MRAM"
- note removed: "A 128 KB non-volatile SPI memory (Everspin MR25H10CDF) that keeps its contents without power and has no write wear: settings, logs, a boot menu, a save file. Not fitted by default; a build that wants it fits U33 and these four passives together. CS is pulled up so the chip stays deselected while power comes up (datasheet section 4); WP and HOLD are pulled up and not connected to the FPGA, so writ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"
- note removed: "MEMORY — PSRAM x4 (independent buses, 1.8 V), SDRAM, MRAM option, microSD and configuration flash — HW 0.1.0-proto.1"
- note removed: "MRAM (populate option)"

Commit message: microSD locating pegs are plain holes
Parts:
- J74: footprint EasyEDA:TF-SMD_TF-01A -> EasyEDA:TF-SMD_TF-01A-NPTH
Changed lines of the file:
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@@
 		(property "Reference" "J74" (at 275.59 739.14 0) (effects (font (size 1.27 1.27))))
 		(property "Value" "microSD" (at 275.59 782.32 0) (effects (font (size 1.27 1.27))))
-		(property "Footprint" "EasyEDA:TF-SMD_TF-01A" (at 275.59 782.32 0) (effects (font (size 1.27 1.27)) (hide yes)))
+		(property "Footprint" "EasyEDA:TF-SMD_TF-01A-NPTH" (at 275.59 782.32 0) (effects (font (size 1.27 1.27)) (hide yes)))
 		(property "LCSC" "C91145" (at 275.59 782.32 0) (effects (font (size 1.27 1.27)) (hide yes)))
 		(property "Description" "microSD socket: Hroparts TF-01A push-push microSD socket, SPI mode to FPGA bank 14 at 3.3 V; card detect on the switch." (at 275.59 782.32 0) (effects (font (size 1.27 1.27)) (hide yes)))

Commit message: PSRAM power-up states with PUDC_B high; TPS22953 for the jumpered PIN V exports
Parts:
- added R174, R175, R176, R177, R178, R179, R180, R181, R182, R183, R184, R185, R186, R187, R188, R189, R190, R191, R192, R193, R194, R195, R196, R197: 10k, Resistor_SMD:R_0603_1608Metric, symbol Device:R
Connections:
- net +1V8_IO: now also R174.1, R180.1, R186.1, R192.1
- net GND: now also R175.2, R176.2, R177.2, R178.2, R179.2, R181.2, R182.2, R183.2, R184.2, R185.2, R187.2, R188.2, R189.2, R190.2, R191.2, R193.2, R194.2, R195.2, R196.2, R197.2
- net PSRAM0_CE_B_MEM: now also R174.2
- net PSRAM0_IO0_MEM: now also R176.1
- net PSRAM0_IO1_MEM: now also R177.1
- net PSRAM0_IO2_MEM: now also R178.1
- net PSRAM0_IO3_MEM: now also R179.1
- net PSRAM0_SCK_MEM: now also R175.1
- net PSRAM1_CE_B_MEM: now also R180.2
- net PSRAM1_IO0_MEM: now also R182.1
- net PSRAM1_IO1_MEM: now also R183.1
- net PSRAM1_IO2_MEM: now also R184.1
- net PSRAM1_IO3_MEM: now also R185.1
- net PSRAM1_SCK_MEM: now also R181.1
- net PSRAM2_CE_B_MEM: now also R186.2
- net PSRAM2_IO0_MEM: now also R188.1
- net PSRAM2_IO1_MEM: now also R189.1
- net PSRAM2_IO2_MEM: now also R190.1
- net PSRAM2_IO3_MEM: now also R191.1
- net PSRAM2_SCK_MEM: now also R187.1
- net PSRAM3_CE_B_MEM: now also R192.2
- net PSRAM3_IO0_MEM: now also R194.1
- net PSRAM3_IO1_MEM: now also R195.1
- net PSRAM3_IO2_MEM: now also R196.1
- net PSRAM3_IO3_MEM: now also R197.1
- net PSRAM3_SCK_MEM: now also R193.1
Other:
- note added: "PSRAM0 power-up state"
- note added: "PSRAM1 power-up state"
- note added: "PSRAM2 power-up state"
- note added: "PSRAM3 power-up state"
- note added: "Six 10k resistors at the PSRAM0 pins: CE# pulled up to its own supply, clock and the four data lines pulled down. The chip requires these levels from the first moment of its supply ramp until 150 us after it, and an unconfigured FPGA leaves its pins floating, so resistors, not the FPGA, guarantee them (APS6404L section 8, findings 39)."
- note added: "Six 10k resistors at the PSRAM1 pins: CE# up, clock and data down, from power-up (APS6404L section 8)."
- note added: "Six 10k resistors at the PSRAM2 pins: CE# up, clock and data down, from power-up (APS6404L section 8)."
- note added: "Six 10k resistors at the PSRAM3 pins: CE# up, clock and data down, from power-up (APS6404L section 8)."
- moved on the sheet: C250, C251, C252, C253, C254, C255, C256, C257, C258, C259, C260, J74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

Commit message: Tools: honest gate verdicts, source-side island ownership, key posts at their rows, J1 pads clear of the holes, budget checks for capacitance, inductors and sources
Other:
- note added: "The 22 ohm resistor in the SDRAM clock line. It sits at the FPGA ball that drives the clock, so it damps the edge at its source; it is in U1's island, not the SDRAM's (findings 44)."
- note added: "U1 PSRAM0 series termination"
- note added: "U1 PSRAM1 series termination"
- note added: "U1 PSRAM2 series termination"
- note added: "U1 PSRAM3 series termination"
- note added: "U1 SDRAM clock source"
- note removed: "PSRAM0 series termination"
- note removed: "PSRAM1 series termination"
- note removed: "PSRAM2 series termination"
- note removed: "PSRAM3 series termination"
- moved on the sheet: C258, C259, C260, J74, R151, R154, R155, R156, R157, R158, R159, R160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
