File: kicad/odin.kicad_sch (KiCad schematic)
At the start: 1 part, among them U1 XC7A50T-2CSG325I

Commit message: kicad: full 289-part project - PSRAM x4, RP2350B supervisor, 9 slots, power tree, 4-layer board
Parts:
- added C1, C10, C100, C101, C103, C105, C107, C109, C11, C111, C113, C115, C117, C119, C12, C127, C13, C133, C136, C139, C14, C142, C145, C15, C16, C17, C18, C19, C2, C20, C21, C22, C23, C24, C25, C26, C27, C28, C29, C3, C30, C31, C32, C33, C34, C35, C36, C37, C38, C39, C4, C40, C41, C42, C43, C44, C45, C46, C47, C48, C49, C5, C50, C51, C52, C53, C54, C55, C56, C57, C58, C59, C6, C60, C7, C75, C76, C77, C78, C79, C8, C80, C81, C82, C83, C84, C85, C86, C87, C88, C89, C9, C90, C91, C96, C97, C98, C99: 100nF, Capacitor_SMD:C_0402_1005Metric, symbol Device:C
- added C102, C104, C106, C108, C110, C112, C114, C116, C118, C126, C93: 10uF, Capacitor_SMD:C_0805_2012Metric, symbol Device:C
- added C120, C121, C122, C123, C124, C125, C128, C129, C130, C131, C132, C134, C135, C137, C138, C140, C141, C143, C144: 22uF, Capacitor_SMD:C_0805_2012Metric, symbol Device:C
- added C146, C61, C62, C63, C64, C65, C66, C67, C68, C69, C70, C71, C72, C73, C74, C92: 4.7uF, Capacitor_SMD:C_0603_1608Metric, symbol Device:C
- added C94, C95: 15pF, Capacitor_SMD:C_0402_1005Metric, symbol Device:C
- added D1: green, LED_SMD:LED_0603_1608Metric, symbol Device:LED
- added D2: SS34, Diode_SMD:D_SMA, symbol Device:D_Schottky
- added F1, F11, F12, F13, F15, F16, F17, F19, F20, F21, F23, F24, F25, F27, F28, F29, F3, F31, F32, F33, F35, F36, F4, F5, F7, F8, F9: 500mA, Resistor_SMD:R_0603_1608Metric, symbol Device:Polyfuse
- added F10, F14, F18, F2, F22, F26, F30, F34, F6: 1A, Resistor_SMD:R_0603_1608Metric, symbol Device:Polyfuse
- added J1: USB-C, Connector_USB:USB_C_Receptacle_HCTL_HC-TYPE-C-16P-01A, symbol Connector:USB_C_Receptacle_USB2.0_16P
- added J10: AUX_SEL_C, Connector_PinHeader_2.54mm:PinHeader_2x03_P2.54mm_Vertical, symbol Connector_Generic:Conn_02x03_Odd_Even
- added J11: SLOT_D, Connector_PinHeader_2.54mm:PinHeader_2x08_P2.54mm_Vertical_SMD, symbol Connector_Generic:Conn_02x08_Odd_Even
- added J12: AUX_SEL_D, Connector_PinHeader_2.54mm:PinHeader_2x03_P2.54mm_Vertical, symbol Connector_Generic:Conn_02x03_Odd_Even
- added J13: SLOT_E, Connector_PinHeader_2.54mm:PinHeader_2x08_P2.54mm_Vertical_SMD, symbol Connector_Generic:Conn_02x08_Odd_Even
- added J14: AUX_SEL_E, Connector_PinHeader_2.54mm:PinHeader_2x03_P2.54mm_Vertical, symbol Connector_Generic:Conn_02x03_Odd_Even
- added J15: SLOT_F, Connector_PinHeader_2.54mm:PinHeader_2x08_P2.54mm_Vertical_SMD, symbol Connector_Generic:Conn_02x08_Odd_Even
- added J16: AUX_SEL_F, Connector_PinHeader_2.54mm:PinHeader_2x03_P2.54mm_Vertical, symbol Connector_Generic:Conn_02x03_Odd_Even
- added J17: SLOT_G, Connector_PinHeader_2.54mm:PinHeader_2x08_P2.54mm_Vertical_SMD, symbol Connector_Generic:Conn_02x08_Odd_Even
- added J18: AUX_SEL_G, Connector_PinHeader_2.54mm:PinHeader_2x03_P2.54mm_Vertical, symbol Connector_Generic:Conn_02x03_Odd_Even
- added J19: SLOT_H, Connector_PinHeader_2.54mm:PinHeader_2x08_P2.54mm_Vertical_SMD, symbol Connector_Generic:Conn_02x08_Odd_Even
- added J2: JTAG, Connector_PinHeader_2.54mm:PinHeader_2x05_P2.54mm_Vertical, symbol Connector_Generic:Conn_02x05_Odd_Even
- added J20: AUX_SEL_H, Connector_PinHeader_2.54mm:PinHeader_2x03_P2.54mm_Vertical, symbol Connector_Generic:Conn_02x03_Odd_Even
- added J21: VCCIO1_SEL, Connector_PinHeader_2.54mm:PinHeader_2x03_P2.54mm_Vertical, symbol Connector_Generic:Conn_02x03_Odd_Even
- added J22: VCCIO2_SEL, Connector_PinHeader_2.54mm:PinHeader_2x03_P2.54mm_Vertical, symbol Connector_Generic:Conn_02x03_Odd_Even
- added J3: SLOT_L, Connector_PinHeader_2.54mm:PinHeader_2x08_P2.54mm_Vertical_SMD, symbol Connector_Generic:Conn_02x08_Odd_Even
- added J4: AUX_SEL_L, Connector_PinHeader_2.54mm:PinHeader_2x03_P2.54mm_Vertical, symbol Connector_Generic:Conn_02x03_Odd_Even
- added J5: SLOT_A, Connector_PinHeader_2.54mm:PinHeader_2x08_P2.54mm_Vertical_SMD, symbol Connector_Generic:Conn_02x08_Odd_Even
- added J50: VIN 12V, Connector_PinHeader_2.54mm:PinHeader_1x02_P2.54mm_Vertical, symbol Connector_Generic:Conn_01x02
- added J51: SUP_SWD, Connector_PinHeader_2.54mm:PinHeader_1x03_P2.54mm_Vertical, symbol Connector_Generic:Conn_01x03
- added J6: AUX_SEL_A, Connector_PinHeader_2.54mm:PinHeader_2x03_P2.54mm_Vertical, symbol Connector_Generic:Conn_02x03_Odd_Even
- added J7: SLOT_B, Connector_PinHeader_2.54mm:PinHeader_2x08_P2.54mm_Vertical_SMD, symbol Connector_Generic:Conn_02x08_Odd_Even
- added J8: AUX_SEL_B, Connector_PinHeader_2.54mm:PinHeader_2x03_P2.54mm_Vertical, symbol Connector_Generic:Conn_02x03_Odd_Even
- added J9: SLOT_C, Connector_PinHeader_2.54mm:PinHeader_2x08_P2.54mm_Vertical_SMD, symbol Connector_Generic:Conn_02x08_Odd_Even
- added L1: 3.3uH, Inductor_SMD:L_Bourns-SRN4018, symbol Device:L
- added L2: 4.7uH, Inductor_SMD:L_Bourns-SRN4018, symbol Device:L
- added L3, L4, L5, L6, L7: 1.5uH, Inductor_SMD:L_Bourns-SRN4018, symbol Device:L
- added L8: 1uH, Inductor_SMD:L_Bourns-SRN4018, symbol Device:L
- added R1, R2, R3, R4, R5, R6: 4.7k, Resistor_SMD:R_0402_1005Metric, symbol Device:R
- added R10, R9: 5.1k, Resistor_SMD:R_0402_1005Metric, symbol Device:R
- added R11, R12, R13, R14, R15, R16, R17, R18, R19, R20, R21, R22, R23, R24, R25, R26, R27, R28, R29: 33, Resistor_SMD:R_0402_1005Metric, symbol Device:R
- added R30, R32, R34, R36, R38, R40, R42, R44, R45: 100k, Resistor_SMD:R_0603_1608Metric, symbol Device:R
- added R31: 16.2k, Resistor_SMD:R_0603_1608Metric, symbol Device:R
- added R33: 33.2k, Resistor_SMD:R_0603_1608Metric, symbol Device:R
- added R35: 49.9k, Resistor_SMD:R_0603_1608Metric, symbol Device:R
- added R37: 80.6k, Resistor_SMD:R_0603_1608Metric, symbol Device:R
- added R39: 200k, Resistor_SMD:R_0603_1608Metric, symbol Device:R
- added R41: 150k, Resistor_SMD:R_0603_1608Metric, symbol Device:R
- added R43: 33k, Resistor_SMD:R_0603_1608Metric, symbol Device:R
- added R46, R47, R48, R49, R50, R51: 1k, Resistor_SMD:R_0603_1608Metric, symbol Device:R
- added R52, R53, R54, R55: 10k, Resistor_SMD:R_0402_1005Metric, symbol Device:R
- added R7: 330, Resistor_SMD:R_0402_1005Metric, symbol Device:R
- added R8: 1k, Resistor_SMD:R_0402_1005Metric, symbol Device:R
- added SW1: BOOTSEL, Button_Switch_SMD:SW_SPST_B3U-1000P, symbol Switch:SW_Push
- added U10, U9: SN74AVC8T245PW, Package_SO:TSSOP-24_4.4x7.8mm_P0.65mm, symbol Logic_LevelTranslator:SN74AVC8T245PW
- added U11: TPS54202DDC, Package_TO_SOT_SMD:SOT-23-6, symbol Regulator_Switching:TPS54202DDC
- added U12, U13, U14, U15, U16: TLV62569DRL, Package_TO_SOT_SMD:SOT-23-6, symbol Regulator_Switching:TLV62569DRL
- added U2, U3, U4, U5: APS1604M-3SQR-SN, Package_SO:SOIC-8_5.3x5.3mm_P1.27mm, symbol Memory_RAM:APS1604M-3SQRx-SN
- added U6: W25Q256JVEIQ, Package_SO:SOIC-8_5.3x5.3mm_P1.27mm, symbol odin:W25Q256JVEIQ
- added U7: RP2350B, Package_DFN_QFN:QFN-80-1EP_10x10mm_P0.4mm_EP3.4x3.4mm_ThermalVias, symbol MCU_RaspberryPi:RP2350B
- added U8: W25Q32JVZP, Package_SON:Winbond_USON-8-1EP_3x2mm_P0.5mm_EP0.2x1.6mm, symbol Memory_Flash:W25Q32JVZP
- added Y1: 12MHz, Crystal:Crystal_SMD_3225-4Pin_3.2x2.5mm, symbol Device:Crystal_GND24
Connections:
- net +1V0: now also C11.1, C12.1, C13.1, C14.1, C140.1, C141.1, C15.1, C16.1, C17.1, C18.1, C19.1, C20.1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
- net +1V0_MGT: now also C146.1, C32.1, C33.1, C34.1, C35.1, C73.1, L8.2
- net +1V2_MGT: now also C143.1, C144.1, C36.1, C37.1, C38.1, C39.1, C40.1, C74.1, L7.2, R40.1, R50.1
- net +1V8: now also C1.1, C10.1, C137.1, C138.1, C2.1, C6.1, C65.1, C66.1, C7.1, C8.1, C9.1, J21.5 (Pin_5)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
- net +3V3: now also C100.1, C131.1, C132.1, C3.1, C4.1, C41.1, C42.1, C43.1, C44.1, C45.1, C46.1, C47.1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
- net CFG_CCLK: now also R18.2, U6.6 (CLK)
- net CFG_DONE: now also R17.2, R7.1
- net CFG_INIT_B: now also R16.2, R5.1
- net CFG_M0: now also R1.1
- net CFG_M1: now also R2.1
- net CFG_M2: now also R3.1
- net CFG_PROG_B: now also R15.2, R4.1
- net DBG_TCK: now also R24.2
- net DBG_TDI: now also R26.2
- net DBG_TDO: now also R27.2
- net DBG_TMS: now also R25.2
- net FLASH_CS_B: now also R19.2, U6.1 (~{CS})
- net FLASH_D0_MOSI: now also R20.2, U6.5 (DI/IO0)
- net FLASH_D1_MISO: now also R21.2, U6.2 (DO/IO1)
- net FLASH_D2_WP: now also R22.2, U6.3 (~{WP}/IO2)
- net FLASH_D3_HOLD: now also R23.2, U6.7 (~{HOLD}/IO3)
- net GND: now also C1.2, C10.2, C100.2, C101.2, C102.2, C103.2, C104.2, C105.2, C106.2, C107.2, C108.2, C109.2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
- net JTAG_TCK: now also J2.5 (Pin_5), R11.2
- net JTAG_TDI: now also J2.9 (Pin_9), R13.2
- net JTAG_TDO: now also J2.7 (Pin_7), R14.2
- net JTAG_TMS: now also J2.3 (Pin_3), R12.2
- net PSRAM0_CE_B: now also U2.1 (~{CE})
- net PSRAM0_IO0: now also U2.5 (SI/SIO0)
- net PSRAM0_IO1: now also U2.2 (SO/SIO1)
- net PSRAM0_IO2: now also U2.3 (SIO2)
- net PSRAM0_IO3: now also U2.7 (SIO3)
- net PSRAM0_SCK: now also U2.6 (SCLK)
- net PSRAM1_CE_B: now also U3.1 (~{CE})
- net PSRAM1_IO0: now also U3.5 (SI/SIO0)
- net PSRAM1_IO1: now also U3.2 (SO/SIO1)
- net PSRAM1_IO2: now also U3.3 (SIO2)
- net PSRAM1_IO3: now also U3.7 (SIO3)
- net PSRAM1_SCK: now also U3.6 (SCLK)
- net PSRAM2_CE_B: now also U4.1 (~{CE})
- net PSRAM2_IO0: now also U4.5 (SI/SIO0)
- net PSRAM2_IO1: now also U4.2 (SO/SIO1)
- net PSRAM2_IO2: now also U4.3 (SIO2)
- net PSRAM2_IO3: now also U4.7 (SIO3)
- net PSRAM2_SCK: now also U4.6 (SCLK)
- net PSRAM3_CE_B: now also U5.1 (~{CE})
- net PSRAM3_IO0: now also U5.5 (SI/SIO0)
- net PSRAM3_IO1: now also U5.2 (SO/SIO1)
- net PSRAM3_IO2: now also U5.3 (SIO2)
- net PSRAM3_IO3: now also U5.7 (SIO3)
- net PSRAM3_SCK: now also U5.6 (SCLK)
- net PUDC_B: now also R6.1
- net SB_UART_RX: now also R28.2
- net SB_UART_TX: now also R29.2
- net SLOTA_P0_N: now also J5.2 (Pin_2)
- net SLOTA_P0_P: now also J5.1 (Pin_1)
- net SLOTA_P1_N: now also J5.4 (Pin_4)
- net SLOTA_P1_P: now also J5.3 (Pin_3)
- net SLOTA_P2_N: now also J5.8 (Pin_8)
- net SLOTA_P2_P: now also J5.7 (Pin_7)
- net SLOTA_P3_N: now also J5.10 (Pin_10)
- net SLOTA_P3_P: now also J5.9 (Pin_9)
- net SLOTA_P4_N: now also J5.12 (Pin_12)
- net SLOTA_P4_P: now also J5.11 (Pin_11)
- net SLOTB_P0_N: now also J7.2 (Pin_2)
- net SLOTB_P0_P: now also J7.1 (Pin_1)
- net SLOTB_P1_N: now also J7.4 (Pin_4)
- net SLOTB_P1_P: now also J7.3 (Pin_3)
- net SLOTB_P2_N: now also J7.8 (Pin_8)
- net SLOTB_P2_P: now also J7.7 (Pin_7)
- net SLOTB_P3_N: now also J7.10 (Pin_10)
- net SLOTB_P3_P: now also J7.9 (Pin_9)
- net SLOTB_P4_N: now also J7.12 (Pin_12)
- net SLOTB_P4_P: now also J7.11 (Pin_11)
- net SLOTC_P0_N: now also J9.2 (Pin_2)
- net SLOTC_P0_P: now also J9.1 (Pin_1)
- net SLOTC_P1_N: now also J9.4 (Pin_4)
- net SLOTC_P1_P: now also J9.3 (Pin_3)
- net SLOTC_P2_N: now also J9.8 (Pin_8)
- net SLOTC_P2_P: now also J9.7 (Pin_7)
- net SLOTC_P3_N: now also J9.10 (Pin_10)
- net SLOTC_P3_P: now also J9.9 (Pin_9)
- net SLOTC_P4_N: now also J9.12 (Pin_12)
- net SLOTC_P4_P: now also J9.11 (Pin_11)
- net SLOTD_P0_N: now also J11.2 (Pin_2)
- net SLOTD_P0_P: now also J11.1 (Pin_1)
- net SLOTD_P1_N: now also J11.4 (Pin_4)
- net SLOTD_P1_P: now also J11.3 (Pin_3)
- net SLOTD_P2_N: now also J11.8 (Pin_8)
- net SLOTD_P2_P: now also J11.7 (Pin_7)
- net SLOTD_P3_N: now also J11.10 (Pin_10)
- net SLOTD_P3_P: now also J11.9 (Pin_9)
- net SLOTD_P4_N: now also J11.12 (Pin_12)
- net SLOTD_P4_P: now also J11.11 (Pin_11)
- net SLOTE_P0_N: now also J13.2 (Pin_2)
- net SLOTE_P0_P: now also J13.1 (Pin_1)
- net SLOTE_P1_N: now also J13.4 (Pin_4)
- net SLOTE_P1_P: now also J13.3 (Pin_3)
- net SLOTE_P2_N: now also J13.8 (Pin_8)
- net SLOTE_P2_P: now also J13.7 (Pin_7)
- net SLOTE_P3_N: now also J13.10 (Pin_10)
- net SLOTE_P3_P: now also J13.9 (Pin_9)
- net SLOTE_P4_N: now also J13.12 (Pin_12)
- net SLOTE_P4_P: now also J13.11 (Pin_11)
- net SLOTF_P0_N: now also J15.2 (Pin_2)
- net SLOTF_P0_P: now also J15.1 (Pin_1)
- net SLOTF_P1_N: now also J15.4 (Pin_4)
- net SLOTF_P1_P: now also J15.3 (Pin_3)
- net SLOTF_P2_N: now also J15.8 (Pin_8)
- net SLOTF_P2_P: now also J15.7 (Pin_7)
- net SLOTF_P3_N: now also J15.10 (Pin_10)
- net SLOTF_P3_P: now also J15.9 (Pin_9)
- net SLOTF_P4_N: now also J15.12 (Pin_12)
- net SLOTF_P4_P: now also J15.11 (Pin_11)
- net SLOTG_P0_N: now also J17.2 (Pin_2)
- net SLOTG_P0_P: now also J17.1 (Pin_1)
- net SLOTG_P1_N: now also J17.4 (Pin_4)
- net SLOTG_P1_P: now also J17.3 (Pin_3)
- net SLOTG_P2_N: now also J17.8 (Pin_8)
- net SLOTG_P2_P: now also J17.7 (Pin_7)
- net SLOTG_P3_N: now also J17.10 (Pin_10)
- net SLOTG_P3_P: now also J17.9 (Pin_9)
- net SLOTG_P4_N: now also J17.12 (Pin_12)
- net SLOTG_P4_P: now also J17.11 (Pin_11)
- net SLOTH_P0_N: now also J19.2 (Pin_2)
- net SLOTH_P0_P: now also J19.1 (Pin_1)
- net SLOTH_P1_N: now also J19.4 (Pin_4)
- net SLOTH_P1_P: now also J19.3 (Pin_3)
- new net +12V: C124.1, C125.1, J10.1 (Pin_1), J12.1 (Pin_1), J14.1 (Pin_1), J16.1 (Pin_1), J18.1 (Pin_1), J20.1 (Pin_1), J4.1 (Pin_1), J50.1 (Pin_1), J6.1 (Pin_1), J8.1 (Pin_1)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
- new net +1V1: C88.1, C89.1, C90.1, C91.1, C92.1, L1.2, U7.10 (DVDD), U7.32 (DVDD), U7.51 (DVDD), U7.65 (VREG_FB)
- new net +2V5: C134.1, C135.1, J21.3 (Pin_3), J22.3 (Pin_3), L4.2, R34.1, R47.1
- new net +5V: C101.1, C128.1, C129.1, C130.1, C133.1, C136.1, C139.1, C142.1, C145.1, C99.1, D2.1 (K), F10.1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
- new net AUXSEL_A: F8.1, J6.2 (Pin_2), J6.4 (Pin_4), J6.6 (Pin_6)
- new net AUXSEL_B: F12.1, J8.2 (Pin_2), J8.4 (Pin_4), J8.6 (Pin_6)
- new net AUXSEL_C: F16.1, J10.2 (Pin_2), J10.4 (Pin_4), J10.6 (Pin_6)
- new net AUXSEL_D: F20.1, J12.2 (Pin_2), J12.4 (Pin_4), J12.6 (Pin_6)
- new net AUXSEL_E: F24.1, J14.2 (Pin_2), J14.4 (Pin_4), J14.6 (Pin_6)
- new net AUXSEL_F: F28.1, J16.2 (Pin_2), J16.4 (Pin_4), J16.6 (Pin_6)
- new net AUXSEL_G: F32.1, J18.2 (Pin_2), J18.4 (Pin_4), J18.6 (Pin_6)
- new net AUXSEL_H: F36.1, J20.2 (Pin_2), J20.4 (Pin_4), J20.6 (Pin_6)
- new net AUXSEL_L: F4.1, J4.2 (Pin_2), J4.4 (Pin_4), J4.6 (Pin_6)
- new net AUX_A: F8.2, J5.16 (Pin_16)
- new net AUX_B: F12.2, J7.16 (Pin_16)
- new net AUX_C: F16.2, J9.16 (Pin_16)
- new net AUX_D: F20.2, J11.16 (Pin_16)
- new net AUX_E: F24.2, J13.16 (Pin_16)
- new net AUX_F: F28.2, J15.16 (Pin_16)
- new net AUX_G: F32.2, J17.16 (Pin_16)
- new net AUX_H: F36.2, J19.16 (Pin_16)
- new net AUX_L: F4.2, J3.16 (Pin_16)
- new net BOARDID_0: R52.1, U7.28 (GPIO27)
- new net BOARDID_1: R53.1, U7.36 (GPIO28)
- new net BOARDID_2: R54.1, U7.37 (GPIO29)
- new net BOARDID_3: R55.1, U7.38 (GPIO30)
- new net BOOT_5V: C127.1, U11.6 (BOOT)
- new net DONE_LED_A: D1.2 (A), R7.2
- new net EN_1V0: U15.5 (EN), U7.25 (GPIO24)
- new net EN_1V2: U16.5 (EN), U7.26 (GPIO25)
- new net EN_1V8: U14.5 (EN), U7.23 (GPIO23)
- new net EN_2V5: U13.5 (EN), U7.22 (GPIO22)
- new net EN_3V3: U12.5 (EN), U7.21 (GPIO21)
- new net EN_5V: U11.5 (EN), U7.27 (GPIO26)
- new net FB+1V0: R38.2, R39.1, U15.1 (FB)
- new net FB+1V2_MGT: R40.2, R41.1, U16.1 (FB)
- new net FB+1V8: R36.2, R37.1, U14.1 (FB)
- new net FB+2V5: R34.2, R35.1, U13.1 (FB)
- new net FB+3V3: R32.2, R33.1, U12.1 (FB)
- new net FB_5V: R30.2, R31.1, U11.4 (FB)
- new net MON_12V: R42.2, R43.1, U7.49 (GPIO40/ADC0)
- new net MON_1V0: R49.2, U7.56 (GPIO45/ADC5)
- new net MON_1V2: R50.2, U7.57 (GPIO46/ADC6)
- new net MON_1V8: R48.2, U7.55 (GPIO44/ADC4)
- new net MON_2V5: R47.2, U7.54 (GPIO43/ADC3)
- new net MON_3V3: R46.2, U7.53 (GPIO42/ADC2)
- new net MON_5V: R44.2, R45.1, U7.52 (GPIO41/ADC1)
- new net MON_VCCIO1: R51.2, U7.58 (GPIO47/ADC7)
- new net SLOTL_IO0: J3.1 (Pin_1), U9.21 (B1)
- new net SLOTL_IO1: J3.2 (Pin_2), U9.20 (B2)
- new net SLOTL_IO2: J3.3 (Pin_3), U9.19 (B3)
- new net SLOTL_IO3: J3.4 (Pin_4), U9.18 (B4)
- new net SLOTL_IO4: J3.7 (Pin_7), U9.17 (B5)
- new net SLOTL_IO5: J3.8 (Pin_8), U9.16 (B6)
- new net SLOTL_IO6: J3.9 (Pin_9), U9.15 (B7)
- new net SLOTL_IO7: J3.10 (Pin_10), U9.14 (B8)
- new net SLOTL_IO8: J3.11 (Pin_11), U10.21 (B1)
- new net SLOTL_IO9: J3.12 (Pin_12), U10.20 (B2)
- new net SUPF_CLK: U7.71 (QSPI_SCLK), U8.6 (CLK)
- new net SUPF_CS: SW1.1, U7.75 (~{QSPI_SS}), U8.1 (~{CS})
- new net SUPF_D0: U7.72 (QSPI_SD0), U8.5 (DI/IO_{0})
- new net SUPF_D1: U7.74 (QSPI_SD1), U8.2 (DO/IO_{1})
- new net SUPF_D2: U7.73 (QSPI_SD2), U8.3 (~{WP}/IO_{2})
- new net SUPF_D3: U7.70 (QSPI_SD3), U8.7 (~{HOLD}/~{RESET}/IO_{3})
- new net SUP_CCLK: R18.1, U7.4 (GPIO7)
- new net SUP_DBG_TCK: R24.1, U7.14 (GPIO15)
- new net SUP_DBG_TDI: R26.1, U7.17 (GPIO17)
- new net SUP_DBG_TDO: R27.1, U7.18 (GPIO18)
- new net SUP_DBG_TMS: R25.1, U7.16 (GPIO16)
- new net SUP_DONE: R17.1, U7.3 (GPIO6)
- new net SUP_FCS_B: R19.1, U7.7 (GPIO9)
- new net SUP_FD0: R20.1, U7.8 (GPIO10)
- new net SUP_FD1: R21.1, U7.9 (GPIO11)
- new net SUP_FD2: R22.1, U7.11 (GPIO12)
- new net SUP_FD3: R23.1, U7.12 (GPIO13)
- new net SUP_INIT_B: R16.1, U7.2 (GPIO5)
- new net SUP_JTAG_TCK: R11.1, U7.77 (GPIO0)
- new net SUP_JTAG_TDI: R13.1, U7.79 (GPIO2)
- new net SUP_JTAG_TDO: R14.1, U7.80 (GPIO3)
- new net SUP_JTAG_TMS: R12.1, U7.78 (GPIO1)
- new net SUP_LX: L1.1, U7.63 (VREG_LX)
- new net SUP_PROG_B: R15.1, U7.1 (GPIO4)
- new net SUP_RUN: C96.1, R8.1, U7.35 (RUN)
- new net SUP_SWCLK: J51.1 (Pin_1), U7.33 (SWCLK)
- new net SUP_SWDIO: J51.3 (Pin_3), U7.34 (SWDIO)
- new net SUP_UART_RX: R29.1, U7.20 (GPIO20)
- new net SUP_UART_TX: R28.1, U7.19 (GPIO19)
- new net SUP_XIN: C94.1, U7.30 (XIN), Y1.1
- new net SUP_XOUT: C95.1, U7.31 (XOUT), Y1.3
- new net SW+1V0: L6.1, U15.4 (SW)
- new net SW+1V2_MGT: L7.1, U16.4 (SW)
- new net SW+1V8: L5.1, U14.4 (SW)
- new net SW+2V5: L4.1, U13.4 (SW)
- new net SW+3V3: L3.1, U12.4 (SW)
- new net SW_5V: C127.2, L2.1, U11.2 (SW)
- new net USB_CC1: J1.A5 (CC1), R9.1
- new net USB_CC2: J1.B5 (CC2), R10.1
- new net USB_DM: J1.A7 (D-), J1.B7 (D-), U7.66 (USB_DM)
- new net USB_DP: J1.A6 (D+), J1.B6 (D+), U7.67 (USB_DP)
- new net V33_A: C105.1, F7.2, J5.14 (Pin_14)
- new net V33_B: C107.1, F11.2, J7.14 (Pin_14)
- new net V33_C: C109.1, F15.2, J9.14 (Pin_14)
- new net V33_D: C111.1, F19.2, J11.14 (Pin_14)
- new net V33_E: C113.1, F23.2, J13.14 (Pin_14)
- new net V33_F: C115.1, F27.2, J15.14 (Pin_14)
- new net V33_G: C117.1, F31.2, J17.14 (Pin_14)
- new net V33_H: C119.1, F35.2, J19.14 (Pin_14)
- new net V33_L: C103.1, F3.2, J3.14 (Pin_14)
- new net V5_A: F6.2, J5.15 (Pin_15)
- new net V5_B: F10.2, J7.15 (Pin_15)
- new net V5_C: F14.2, J9.15 (Pin_15)
- new net V5_D: F18.2, J11.15 (Pin_15)
- new net V5_E: F22.2, J13.15 (Pin_15)
- new net V5_F: F26.2, J15.15 (Pin_15)
- new net V5_G: F30.2, J17.15 (Pin_15)
- new net V5_H: F34.2, J19.15 (Pin_15)
- new net V5_L: F2.2, J3.15 (Pin_15)
- new net VBUS: C126.1, D2.2 (A), J1.A4 (VBUS), J1.A9 (VBUS), J1.B4 (VBUS), J1.B9 (VBUS)
- new net VIO_A: C104.1, F5.2, J5.13 (Pin_13)
- new net VIO_B: C106.1, F9.2, J7.13 (Pin_13)
- new net VIO_C: C108.1, F13.2, J9.13 (Pin_13)
- new net VIO_D: C110.1, F17.2, J11.13 (Pin_13)
- new net VIO_E: C112.1, F21.2, J13.13 (Pin_13)
- new net VIO_F: C114.1, F25.2, J15.13 (Pin_13)
- new net VIO_G: C116.1, F29.2, J17.13 (Pin_13)
- new net VIO_H: C118.1, F33.2, J19.13 (Pin_13)
- new net VIO_L: C102.1, F1.2, J3.13 (Pin_13)
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Other:
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
Commit message: fix: all six feedback dividers were wrong; now computed from E96 and verified against Vref
Parts:
- R31: value 16.2k -> 13.7k
- R33: value 33.2k -> 22.1k
- R35: value 49.9k -> 31.6k
- R37: value 80.6k -> 49.9k
- R39: value 200k -> 150k
- R41: value 150k -> 100k
Changed lines of the file:
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@@
 		(exclude_from_sim no) (in_bom yes) (on_board yes) (dnp no)
 		(property "Reference" "R31" (at 1007.11 1459.52 0) (effects (font (size 1.27 1.27))))
-		(property "Value" "16.2k" (at 1007.11 1459.52 0) (effects (font (size 1.27 1.27))))
+		(property "Value" "13.7k" (at 1007.11 1459.52 0) (effects (font (size 1.27 1.27))))
 		(property "Footprint" "Resistor_SMD:R_0603_1608Metric" (at 1007.11 1459.52 0) (effects (font (size 1.27 1.27)) (hide yes)))
 		(instances (project "odin" (path "/c44fb7fe-6133-ad34-68fd-fb66126197ef" (reference "R31") (unit 1))))
@@
 		(exclude_from_sim no) (in_bom yes) (on_board yes) (dnp no)
 		(property "Reference" "R33" (at 594.36 1520.48 0) (effects (font (size 1.27 1.27))))
-		(property "Value" "33.2k" (at 594.36 1520.48 0) (effects (font (size 1.27 1.27))))
+		(property "Value" "22.1k" (at 594.36 1520.48 0) (effects (font (size 1.27 1.27))))
 		(property "Footprint" "Resistor_SMD:R_0603_1608Metric" (at 594.36 1520.48 0) (effects (font (size 1.27 1.27)) (hide yes)))
 		(instances (project "odin" (path "/c44fb7fe-6133-ad34-68fd-fb66126197ef" (reference "R33") (unit 1))))
@@
 		(exclude_from_sim no) (in_bom yes) (on_board yes) (dnp no)
 		(property "Reference" "R35" (at 110.49 1581.44 0) (effects (font (size 1.27 1.27))))
-		(property "Value" "49.9k" (at 110.49 1581.44 0) (effects (font (size 1.27 1.27))))
+		(property "Value" "31.6k" (at 110.49 1581.44 0) (effects (font (size 1.27 1.27))))
 		(property "Footprint" "Resistor_SMD:R_0603_1608Metric" (at 110.49 1581.44 0) (effects (font (size 1.27 1.27)) (hide yes)))
 		(instances (project "odin" (path "/c44fb7fe-6133-ad34-68fd-fb66126197ef" (reference "R35") (unit 1))))
@@
 		(exclude_from_sim no) (in_bom yes) (on_board yes) (dnp no)
 		(property "Reference" "R37" (at 671.83 1581.44 0) (effects (font (size 1.27 1.27))))
-		(property "Value" "80.6k" (at 671.83 1581.44 0) (effects (font (size 1.27 1.27))))
+		(property "Value" "49.9k" (at 671.83 1581.44 0) (effects (font (size 1.27 1.27))))
 		(property "Footprint" "Resistor_SMD:R_0603_1608Metric" (at 671.83 1581.44 0) (effects (font (size 1.27 1.27)) (hide yes)))
 		(instances (project "odin" (path "/c44fb7fe-6133-ad34-68fd-fb66126197ef" (reference "R37") (unit 1))))
@@
 		(exclude_from_sim no) (in_bom yes) (on_board yes) (dnp no)
 		(property "Reference" "R39" (at 189.23 1642.4 0) (effects (font (size 1.27 1.27))))
-		(property "Value" "200k" (at 189.23 1642.4 0) (effects (font (size 1.27 1.27))))
+		(property "Value" "150k" (at 189.23 1642.4 0) (effects (font (size 1.27 1.27))))
 		(property "Footprint" "Resistor_SMD:R_0603_1608Metric" (at 189.23 1642.4 0) (effects (font (size 1.27 1.27)) (hide yes)))
 		(instances (project "odin" (path "/c44fb7fe-6133-ad34-68fd-fb66126197ef" (reference "R39") (unit 1))))
@@
 		(exclude_from_sim no) (in_bom yes) (on_board yes) (dnp no)
 		(property "Reference" "R41" (at 750.57 1642.4 0) (effects (font (size 1.27 1.27))))
-		(property "Value" "150k" (at 750.57 1642.4 0) (effects (font (size 1.27 1.27))))
+		(property "Value" "100k" (at 750.57 1642.4 0) (effects (font (size 1.27 1.27))))
 		(property "Footprint" "Resistor_SMD:R_0603_1608Metric" (at 750.57 1642.4 0) (effects (font (size 1.27 1.27)) (hide yes)))
 		(instances (project "odin" (path "/c44fb7fe-6133-ad34-68fd-fb66126197ef" (reference "R41") (unit 1))))

Commit message: wire the four fast lanes: 2 populated SFP cages + 2 reserved, 125MHz refclk, supervisor-gated power, self-describing over I2C
Parts:
- added C147, C148, C149, C153, C159, C162, C165, C168, C171: 100nF, Capacitor_SMD:C_0402_1005Metric, symbol Device:C
- added C150, C151, C154, C155, C156, C157, C158, C160, C161, C163, C164, C166, C167, C169, C170: 22uF, Capacitor_SMD:C_0805_2012Metric, symbol Device:C
- added C152: 10uF, Capacitor_SMD:C_0805_2012Metric, symbol Device:C
- added C172: 4.7uF, Capacitor_SMD:C_0603_1608Metric, symbol Device:C
- added J60: SFP cage 0, Connector:Connector_SFP_and_Cage, symbol Interface_Optical:SFP
- added J61: SFP cage 1, Connector:Connector_SFP_and_Cage, symbol Interface_Optical:SFP
- added J62: SFP cage 2, Connector:Connector_SFP_and_Cage, symbol Interface_Optical:SFP
- added J63: SFP cage 3, Connector:Connector_SFP_and_Cage, symbol Interface_Optical:SFP
- added Q1: SFP power gate, Package_TO_SOT_SMD:SOT-23, symbol Device:Q_PMOS
- added R56: 100k, Resistor_SMD:R_0603_1608Metric, symbol Device:R
- added R57, R58, R59, R60, R61: 1k, Resistor_SMD:R_0603_1608Metric, symbol Device:R
- added R62, R63, R64, R65: 10k, Resistor_SMD:R_0402_1005Metric, symbol Device:R
- added U17: PCF8574T, Package_SO:SOIC-16_3.9x9.9mm_P1.27mm, symbol Interface_Expansion:PCF8574T
- added X2: 125MHz LVDS, Oscillator:Oscillator_SMD_SiTime_SiT9121-6Pin_3.2x2.5mm, symbol odin:OSC_DIFF_6P_3225
- C124, C129, C130, C131, C132, C134, C135, C137, C138, C140, C141, C143, C144: value 22uF -> 100nF; footprint Capacitor_SMD:C_0805_2012Metric -> Capacitor_SMD:C_0402_1005Metric
- C125: value 22uF -> 4.7uF; footprint Capacitor_SMD:C_0805_2012Metric -> Capacitor_SMD:C_0603_1608Metric
- C126: value 10uF -> 100nF; footprint Capacitor_SMD:C_0805_2012Metric -> Capacitor_SMD:C_0402_1005Metric
- C128: value 22uF -> 10uF
- C146: value 4.7uF -> 100nF; footprint Capacitor_SMD:C_0603_1608Metric -> Capacitor_SMD:C_0402_1005Metric
- R30: value 100k -> 100
- R31: value 13.7k -> 100k; footprint Resistor_SMD:R_0603_1608Metric -> Resistor_SMD:R_0402_1005Metric
- R32, R34, R36, R38, R40: value 100k -> 4.7k; footprint Resistor_SMD:R_0603_1608Metric -> Resistor_SMD:R_0402_1005Metric
- R33: value 22.1k -> 4.7k; footprint Resistor_SMD:R_0603_1608Metric -> Resistor_SMD:R_0402_1005Metric
- R35: value 31.6k -> 4.7k; footprint Resistor_SMD:R_0603_1608Metric -> Resistor_SMD:R_0402_1005Metric
- R37: value 49.9k -> 4.7k; footprint Resistor_SMD:R_0603_1608Metric -> Resistor_SMD:R_0402_1005Metric
- R39: value 150k -> 4.7k; footprint Resistor_SMD:R_0603_1608Metric -> Resistor_SMD:R_0402_1005Metric
- R42: value 100k -> 13.7k
- R43: value 33k -> 100k
- R44: value 100k -> 22.1k
- R46: value 1k -> 31.6k
- R47, R49, R51: value 1k -> 100k
- R48: value 1k -> 49.9k
- R50: value 1k -> 150k
- R52, R53, R55: value 10k -> 100k; footprint Resistor_SMD:R_0402_1005Metric -> Resistor_SMD:R_0603_1608Metric
- R54: value 10k -> 33k; footprint Resistor_SMD:R_0402_1005Metric -> Resistor_SMD:R_0603_1608Metric
Connections:
- net +12V: now also R53.1, C150.1, C151.1; no longer C124.1, C125.1, R42.1
- net +1V0: now also C166.1, C167.1, R60.1; no longer C140.1, C141.1, R38.1
- net +1V0_MGT: now also C172.1; no longer C146.1
- net +1V2_MGT: now also R51.1, C169.1, C170.1, R61.1; no longer C143.1, C144.1, R40.1, R50.1
- net +1V8: now also R47.1, C163.1, C164.1, R59.1; no longer C137.1, C138.1, R36.1, R48.1
- net +2V5: now also R45.1, C160.1, C161.1, R58.1; no longer C134.1, C135.1, R34.1, R47.1
- net +3V3: now also C124.1, C125.1, R31.2, R32.2, R33.2, R34.2, R35.2, R36.2, R37.2, R38.2, R39.2, R40.2, R43.1, C149.1, C157.1, C158.1, Q1.S, R57.1, U17.16 (VDD), U17.3 (A2), X2.1 (OE), X2.6 (VDD); no longer C131.1, C132.1, R32.1, R46.1
- net +5V: now also R41.1, R55.1, C154.1, C155.1, C156.1, C159.1, C162.1, C165.1, C168.1, C171.1; no longer C128.1, C129.1, C130.1, C133.1, C136.1, C139.1, C142.1, C145.1, R30.1, R44.1
- net BOARDID_0: now also R62.1; no longer R52.1
- net BOARDID_1: now also R63.1; no longer R53.1
- net BOARDID_2: now also R64.1; no longer R54.1
- net BOARDID_3: now also R65.1; no longer R55.1
- net BOOT_5V: now also C153.1; no longer C127.1
- net FB+1V0: now also R49.2, R50.1; no longer R38.2, R39.1
- net FB+1V2_MGT: now also R51.2, R52.1; no longer R40.2, R41.1
- net FB+1V8: now also R47.2, R48.1; no longer R36.2, R37.1
- net FB+2V5: now also R45.2, R46.1; no longer R34.2, R35.1
- net FB+3V3: now also R43.2, R44.1; no longer R32.2, R33.1
- net FB_5V: now also R41.2, R42.1; no longer R30.2, R31.1
- net GND: now also R30.2, R42.2, R44.2, R46.2, R48.2, R50.2, C148.2, C149.2, C150.2, C151.2, C152.2, C154.2, C155.2, C156.2, C157.2, C158.2, C159.2, C160.2, C161.2, C162.2, C163.2, C164.2, C165.2, C166.2, C167.2, C168.2, C169.2, C170.2, C171.2, C172.2, J60.1 (VeeT), J60.10 (VeeR), J60.11 (VeeR), J60.14 (VeeR), J60.17 (VeeT), J60.20 (VeeT), J60.7 (RATE_SELECT), J60.9 (VeeR), J60.CAGE, J61.1 (VeeT), J61.10 (VeeR), J61.11 (VeeR), J61.14 (VeeR), J61.17 (VeeT), J61.20 (VeeT), J61.7 (RATE_SELECT), J61.9 (VeeR), J61.CAGE, J62.1 (VeeT), J62.10 (VeeR), J62.11 (VeeR), J62.14 (VeeR), J62.17 (VeeT), J62.20 (VeeT), J62.7 (RATE_SELECT), J62.9 (VeeR), J62.CAGE, J63.1 (VeeT), J63.10 (VeeR), J63.11 (VeeR), J63.14 (VeeR), J63.17 (VeeT), J63.20 (VeeT), J63.7 (RATE_SELECT), J63.9 (VeeR), J63.CAGE, R56.2, R62.2, R63.2, R64.2, R65.2, U17.1 (A0), U17.2 (A1), U17.8 (GND), X2.2 (GND); no longer C126.2, C129.2, C130.2, C131.2, C132.2, C134.2, C135.2, C136.2, C137.2, C139.2, C140.2, C141.2, C142.2, C144.2, C145.2, C146.2, R31.2, R33.2, R35.2, R37.2, R39.2, R41.2, R43.2, R45.2, R53.2, R55.2
- net MGTPRXN0: now also C132.2
- net MGTPRXN1: now also C137.2
- net MGTPRXN2: now also C142.2
- net MGTPRXN3: now also C147.2
- net MGTPRXP0: now also C131.2
- net MGTPRXP1: now also C136.2
- net MGTPRXP2: now also C141.2
- net MGTPRXP3: now also C146.2
- net MGTPTXN0: now also C130.1
- net MGTPTXN1: now also C135.1
- net MGTPTXN2: now also C140.1
- net MGTPTXN3: now also C145.1
- net MGTPTXP0: now also C129.1
- net MGTPTXP1: now also C134.1
- net MGTPTXP2: now also C139.1
- net MGTPTXP3: now also C144.1
- net MGTREFCLK0N: now also C127.2
- net MGTREFCLK0P: now also C126.2
- net MGTRREF: now also R30.1
- net MON_12V: now also R53.2, R54.1; no longer R42.2, R43.1
- net MON_1V0: now also R60.2; no longer R49.2
- net MON_1V2: now also R61.2; no longer R50.2
- net MON_1V8: now also R59.2; no longer R48.2
- net MON_2V5: now also R58.2; no longer R47.2
- net MON_3V3: now also R57.2; no longer R46.2
- net MON_5V: now also R55.2, R56.1; no longer R44.2, R45.1
- net SW_5V: now also C153.2; no longer C127.2
- net VBUS: now also C152.1; no longer C126.1
- net VCCIO_1: no longer R51.1
- net SFP_SCL: now reaches U7.13 (GPIO14)
- net SFP_SCL: now also R32.1, J60.5 (MOD_DEF1), J61.5 (MOD_DEF1), J62.5 (MOD_DEF1), J63.5 (MOD_DEF1), U17.14 (SCL)
- net SFP_SDA: now reaches U7.39 (GPIO31)
- net SFP_SDA: now also R33.1, J60.4 (MOD_DEF2), J61.4 (MOD_DEF2), J62.4 (MOD_DEF2), J63.4 (MOD_DEF2), U17.15 (SDA)
- net SFP0_MOD_ABS: now reaches U7.40 (GPIO32)
- net SFP0_MOD_ABS: now also R34.1, J60.6 (MOD_DEF0)
- net SFP0_TX_DIS: now reaches U7.42 (GPIO33)
- net SFP0_TX_DIS: now also J60.3 (TX_DISABLE)
- net SFP0_TX_FAULT: now reaches U7.43 (GPIO34)
- net SFP0_TX_FAULT: now also R35.1, J60.2 (TX_FAULT)
- net SFP0_LOS: now reaches U7.44 (GPIO35)
- net SFP0_LOS: now also R36.1, J60.8 (RX_LOS)
- net SFP1_MOD_ABS: now reaches U7.45 (GPIO36)
- net SFP1_MOD_ABS: now also R37.1, J61.6 (MOD_DEF0)
- net SFP1_TX_DIS: now reaches U7.46 (GPIO37)
- net SFP1_TX_DIS: now also J61.3 (TX_DISABLE)
- net SFP1_TX_FAULT: now reaches U7.47 (GPIO38)
- net SFP1_TX_FAULT: now also R38.1, J61.2 (TX_FAULT)
- net SFP1_LOS: now reaches U7.48 (GPIO39)
- net SFP1_LOS: now also R39.1, J61.8 (RX_LOS)
- net MON_VCCIO1 renamed EN_SFP_N
- net EN_SFP_N: now also R31.1, Q1.G; no longer R51.2
- new net REFCLK_OSC_N: C127.1, X2.4 (OUT-)
- new net REFCLK_OSC_P: C126.1, X2.5 (OUT+)
- new net SFP0_RD_N: C132.1, J60.12 (RD-)
- new net SFP0_RD_P: C131.1, J60.13 (RD+)
- new net SFP0_TD_N: C130.2, J60.19 (TD-)
- new net SFP0_TD_P: C129.2, J60.18 (TD+)
- new net SFP1_RD_N: C137.1, J61.12 (RD-)
- new net SFP1_RD_P: C136.1, J61.13 (RD+)
- new net SFP1_TD_N: C135.2, J61.19 (TD-)
- new net SFP1_TD_P: C134.2, J61.18 (TD+)
- new net SFP2_LOS_NP: J62.8 (RX_LOS), U17.7 (P3)
- new net SFP2_MOD_ABS_NP: J62.6 (MOD_DEF0), U17.4 (P0)
- new net SFP2_RD_N: C142.1, J62.12 (RD-)
- new net SFP2_RD_P: C141.1, J62.13 (RD+)
- new net SFP2_TD_N: C140.2, J62.19 (TD-)
- new net SFP2_TD_P: C139.2, J62.18 (TD+)
- new net SFP2_TX_DIS_NP: J62.3 (TX_DISABLE), U17.5 (P1)
- new net SFP2_TX_FAULT_NP: J62.2 (TX_FAULT), U17.6 (P2)
- new net SFP3_LOS_NP: J63.8 (RX_LOS), U17.12 (P7)
- new net SFP3_MOD_ABS_NP: J63.6 (MOD_DEF0), U17.9 (P4)
- new net SFP3_RD_N: C147.1, J63.12 (RD-)
- new net SFP3_RD_P: C146.1, J63.13 (RD+)
- new net SFP3_TD_N: C145.2, J63.19 (TD-)
- new net SFP3_TD_P: C144.2, J63.18 (TD+)
- new net SFP3_TX_DIS_NP: J63.3 (TX_DISABLE), U17.10 (P5)
- new net SFP3_TX_FAULT_NP: J63.2 (TX_FAULT), U17.11 (P6)
- new net SFP_EXP_INT: R40.1, U17.13 (~{INT})
- new net SFP_VCC: C128.1, C133.1, C138.1, C143.1, C148.1, J60.15 (VccR), J60.16 (VccT), J61.15 (VccR), J61.16 (VccT), J62.15 (VccR), J62.16 (VccT), J63.15 (VccR), J63.16 (VccT), Q1.D
- no-connect marks 52 -> 43
Other:
- moved on the sheet: C124, C125, C126, C127, C128, C129, C130, C131, C132, C133, C134, C135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

Commit message: schematic is now six grouped pages with power symbols, not a cloud of parts
Parts:
- removed C1, C10, C100, C101, C103, C105, C107, C109, C11, C111, C113, C115, C117, C119, C12, C124, C126, C127, C129, C13, C130, C131, C132, C133, C134, C135, C136, C137, C138, C139, C14, C140, C141, C142, C143, C144, C145, C146, C147, C148, C149, C15, C153, C159, C16, C162, C165, C168, C17, C171, C18, C19, C2, C20, C21, C22, C23, C24, C25, C26, C27, C28, C29, C3, C30, C31, C32, C33, C34, C35, C36, C37, C38, C39, C4, C40, C41, C42, C43, C44, C45, C46, C47, C48, C49, C5, C50, C51, C52, C53, C54, C55, C56, C57, C58, C59, C6, C60, C7, C75, C76, C77, C78, C79, C8, C80, C81, C82, C83, C84, C85, C86, C87, C88, C89, C9, C90, C91, C96, C97, C98, C99: 100nF, Capacitor_SMD:C_0402_1005Metric, symbol Device:C
- removed C102, C104, C106, C108, C110, C112, C114, C116, C118, C128, C152, C93: 10uF, Capacitor_SMD:C_0805_2012Metric, symbol Device:C
- removed C120, C121, C122, C123, C150, C151, C154, C155, C156, C157, C158, C160, C161, C163, C164, C166, C167, C169, C170: 22uF, Capacitor_SMD:C_0805_2012Metric, symbol Device:C
- removed C125, C172, C61, C62, C63, C64, C65, C66, C67, C68, C69, C70, C71, C72, C73, C74, C92: 4.7uF, Capacitor_SMD:C_0603_1608Metric, symbol Device:C
- removed C94, C95: 15pF, Capacitor_SMD:C_0402_1005Metric, symbol Device:C
- removed D1: green, LED_SMD:LED_0603_1608Metric, symbol Device:LED
- removed D2: SS34, Diode_SMD:D_SMA, symbol Device:D_Schottky
- removed F1, F11, F12, F13, F15, F16, F17, F19, F20, F21, F23, F24, F25, F27, F28, F29, F3, F31, F32, F33, F35, F36, F4, F5, F7, F8, F9: 500mA, Resistor_SMD:R_0603_1608Metric, symbol Device:Polyfuse
- removed F10, F14, F18, F2, F22, F26, F30, F34, F6: 1A, Resistor_SMD:R_0603_1608Metric, symbol Device:Polyfuse
- removed J1: USB-C, Connector_USB:USB_C_Receptacle_HCTL_HC-TYPE-C-16P-01A, symbol Connector:USB_C_Receptacle_USB2.0_16P
- removed J10: AUX_SEL_C, Connector_PinHeader_2.54mm:PinHeader_2x03_P2.54mm_Vertical, symbol Connector_Generic:Conn_02x03_Odd_Even
- removed J11: SLOT_D, Connector_PinHeader_2.54mm:PinHeader_2x08_P2.54mm_Vertical_SMD, symbol Connector_Generic:Conn_02x08_Odd_Even
- removed J12: AUX_SEL_D, Connector_PinHeader_2.54mm:PinHeader_2x03_P2.54mm_Vertical, symbol Connector_Generic:Conn_02x03_Odd_Even
- removed J13: SLOT_E, Connector_PinHeader_2.54mm:PinHeader_2x08_P2.54mm_Vertical_SMD, symbol Connector_Generic:Conn_02x08_Odd_Even
- removed J14: AUX_SEL_E, Connector_PinHeader_2.54mm:PinHeader_2x03_P2.54mm_Vertical, symbol Connector_Generic:Conn_02x03_Odd_Even
- removed J15: SLOT_F, Connector_PinHeader_2.54mm:PinHeader_2x08_P2.54mm_Vertical_SMD, symbol Connector_Generic:Conn_02x08_Odd_Even
- removed J16: AUX_SEL_F, Connector_PinHeader_2.54mm:PinHeader_2x03_P2.54mm_Vertical, symbol Connector_Generic:Conn_02x03_Odd_Even
- removed J17: SLOT_G, Connector_PinHeader_2.54mm:PinHeader_2x08_P2.54mm_Vertical_SMD, symbol Connector_Generic:Conn_02x08_Odd_Even
- removed J18: AUX_SEL_G, Connector_PinHeader_2.54mm:PinHeader_2x03_P2.54mm_Vertical, symbol Connector_Generic:Conn_02x03_Odd_Even
- removed J19: SLOT_H, Connector_PinHeader_2.54mm:PinHeader_2x08_P2.54mm_Vertical_SMD, symbol Connector_Generic:Conn_02x08_Odd_Even
- removed J2: JTAG, Connector_PinHeader_2.54mm:PinHeader_2x05_P2.54mm_Vertical, symbol Connector_Generic:Conn_02x05_Odd_Even
- removed J20: AUX_SEL_H, Connector_PinHeader_2.54mm:PinHeader_2x03_P2.54mm_Vertical, symbol Connector_Generic:Conn_02x03_Odd_Even
- removed J21: VCCIO1_SEL, Connector_PinHeader_2.54mm:PinHeader_2x03_P2.54mm_Vertical, symbol Connector_Generic:Conn_02x03_Odd_Even
- removed J22: VCCIO2_SEL, Connector_PinHeader_2.54mm:PinHeader_2x03_P2.54mm_Vertical, symbol Connector_Generic:Conn_02x03_Odd_Even
- removed J3: SLOT_L, Connector_PinHeader_2.54mm:PinHeader_2x08_P2.54mm_Vertical_SMD, symbol Connector_Generic:Conn_02x08_Odd_Even
- removed J4: AUX_SEL_L, Connector_PinHeader_2.54mm:PinHeader_2x03_P2.54mm_Vertical, symbol Connector_Generic:Conn_02x03_Odd_Even
- removed J5: SLOT_A, Connector_PinHeader_2.54mm:PinHeader_2x08_P2.54mm_Vertical_SMD, symbol Connector_Generic:Conn_02x08_Odd_Even
- removed J50: VIN 12V, Connector_PinHeader_2.54mm:PinHeader_1x02_P2.54mm_Vertical, symbol Connector_Generic:Conn_01x02
- removed J51: SUP_SWD, Connector_PinHeader_2.54mm:PinHeader_1x03_P2.54mm_Vertical, symbol Connector_Generic:Conn_01x03
- removed J6: AUX_SEL_A, Connector_PinHeader_2.54mm:PinHeader_2x03_P2.54mm_Vertical, symbol Connector_Generic:Conn_02x03_Odd_Even
- removed J60: SFP cage 0, Connector:Connector_SFP_and_Cage, symbol Interface_Optical:SFP
- removed J61: SFP cage 1, Connector:Connector_SFP_and_Cage, symbol Interface_Optical:SFP
- removed J62: SFP cage 2, Connector:Connector_SFP_and_Cage, symbol Interface_Optical:SFP
- removed J63: SFP cage 3, Connector:Connector_SFP_and_Cage, symbol Interface_Optical:SFP
- removed J7: SLOT_B, Connector_PinHeader_2.54mm:PinHeader_2x08_P2.54mm_Vertical_SMD, symbol Connector_Generic:Conn_02x08_Odd_Even
- removed J8: AUX_SEL_B, Connector_PinHeader_2.54mm:PinHeader_2x03_P2.54mm_Vertical, symbol Connector_Generic:Conn_02x03_Odd_Even
- removed J9: SLOT_C, Connector_PinHeader_2.54mm:PinHeader_2x08_P2.54mm_Vertical_SMD, symbol Connector_Generic:Conn_02x08_Odd_Even
- removed L1: 3.3uH, Inductor_SMD:L_Bourns-SRN4018, symbol Device:L
- removed L2: 4.7uH, Inductor_SMD:L_Bourns-SRN4018, symbol Device:L
- removed L3, L4, L5, L6, L7: 1.5uH, Inductor_SMD:L_Bourns-SRN4018, symbol Device:L
- removed L8: 1uH, Inductor_SMD:L_Bourns-SRN4018, symbol Device:L
- removed Q1: SFP power gate, Package_TO_SOT_SMD:SOT-23, symbol Device:Q_PMOS
- removed R1, R2, R3, R32, R33, R34, R35, R36, R37, R38, R39, R4, R40, R5, R6: 4.7k, Resistor_SMD:R_0402_1005Metric, symbol Device:R
- removed R10, R9: 5.1k, Resistor_SMD:R_0402_1005Metric, symbol Device:R
- removed R11, R12, R13, R14, R15, R16, R17, R18, R19, R20, R21, R22, R23, R24, R25, R26, R27, R28, R29: 33, Resistor_SMD:R_0402_1005Metric, symbol Device:R
- removed R30: 100, Resistor_SMD:R_0603_1608Metric, symbol Device:R
- removed R31: 100k, Resistor_SMD:R_0402_1005Metric, symbol Device:R
- removed R41, R43, R45, R47, R49, R51, R52, R53, R55, R56: 100k, Resistor_SMD:R_0603_1608Metric, symbol Device:R
- removed R42: 13.7k, Resistor_SMD:R_0603_1608Metric, symbol Device:R
- removed R44: 22.1k, Resistor_SMD:R_0603_1608Metric, symbol Device:R
- removed R46: 31.6k, Resistor_SMD:R_0603_1608Metric, symbol Device:R
- removed R48: 49.9k, Resistor_SMD:R_0603_1608Metric, symbol Device:R
- removed R50: 150k, Resistor_SMD:R_0603_1608Metric, symbol Device:R
- removed R54: 33k, Resistor_SMD:R_0603_1608Metric, symbol Device:R
- removed R57, R58, R59, R60, R61: 1k, Resistor_SMD:R_0603_1608Metric, symbol Device:R
- removed R62, R63, R64, R65: 10k, Resistor_SMD:R_0402_1005Metric, symbol Device:R
- removed R7: 330, Resistor_SMD:R_0402_1005Metric, symbol Device:R
- removed R8: 1k, Resistor_SMD:R_0402_1005Metric, symbol Device:R
- removed SW1: BOOTSEL, Button_Switch_SMD:SW_SPST_B3U-1000P, symbol Switch:SW_Push
- removed U1: XC7A50T-2CSG325I, odin:BGA-324_15x15mm_Layout18x18_P0.8mm, symbol odin:XC7A50T-2CSG325I
- removed U10, U9: SN74AVC8T245PW, Package_SO:TSSOP-24_4.4x7.8mm_P0.65mm, symbol Logic_LevelTranslator:SN74AVC8T245PW
- removed U11: TPS54202DDC, Package_TO_SOT_SMD:SOT-23-6, symbol Regulator_Switching:TPS54202DDC
- removed U12, U13, U14, U15, U16: TLV62569DRL, Package_TO_SOT_SMD:SOT-23-6, symbol Regulator_Switching:TLV62569DRL
- removed U17: PCF8574T, Package_SO:SOIC-16_3.9x9.9mm_P1.27mm, symbol Interface_Expansion:PCF8574T
- removed U2, U3, U4, U5: APS1604M-3SQR-SN, Package_SO:SOIC-8_5.3x5.3mm_P1.27mm, symbol Memory_RAM:APS1604M-3SQRx-SN
- removed U6: W25Q256JVEIQ, Package_SO:SOIC-8_5.3x5.3mm_P1.27mm, symbol odin:W25Q256JVEIQ
- removed U7: RP2350B, Package_DFN_QFN:QFN-80-1EP_10x10mm_P0.4mm_EP3.4x3.4mm_ThermalVias, symbol MCU_RaspberryPi:RP2350B
- removed U8: W25Q32JVZP, Package_SON:Winbond_USON-8-1EP_3x2mm_P0.5mm_EP0.2x1.6mm, symbol Memory_Flash:W25Q32JVZP
- removed X2: 125MHz LVDS, Oscillator:Oscillator_SMD_SiTime_SiT9121-6Pin_3.2x2.5mm, symbol odin:OSC_DIFF_6P_3225
- removed Y1: 12MHz, Crystal:Crystal_SMD_3225-4Pin_3.2x2.5mm, symbol Device:Crystal_GND24
Connections:
- no-connect marks 43 -> 0
Other:
- added sheet FPGA (fpga.kicad_sch)
- added sheet HighSpeed (highspeed.kicad_sch)
- added sheet Memory (memory.kicad_sch)
- added sheet Power (power.kicad_sch)
- added sheet Slots (slots.kicad_sch)
- added sheet Supervisor (supervisor.kicad_sch)
- note added: "Artix-7 dev board. Every page is generated — see kicad/README.md"
- note added: "FPGA, decoupling and configuration straps"
- note added: "Four serial lanes: SFP cages, reference clock, power gate"
- note added: "Nine extension slots, rail selection, fusing, level shifting"
- note added: "ODIN"
- note added: "PSRAM x4 (independent buses) and configuration flash"
- note added: "Power tree: 12V input to every rail, with monitoring"
- note added: "RP2350B supervisor, USB-C, flash, and the links to the FPGA"
