File: kicad/fpga.kicad_sch (KiCad schematic)
At the start: 106 parts, among them Q4 BSS138LT1G, U1 XC7A100T-2FGG676I

Commit message: Give the fabric a clock: 50 MHz oscillator on a bank 14 MRCC ball
Preparing the constraints file showed that nothing clocked the FPGA fabric:
X2 only ever fed the GTP reference input, Y1 belongs to the RP2350 and the
PHY's receive clock exists only with a link up. X4, a YXC OT322550MJBA4SL
50 MHz CMOS oscillator, now drives SYS_CLK into bank 14 on an MRCC P ball,
allocated before the PSRAM pairs so it reaches the bank's MMCMs; the
allocator check verifies the placement. Tri-state pin tied high, 100 nF
bypass, 33 ohm at the source.

floorplan.md is rewritten for the rev A board: three jacks on the top
edge, the network strip, the oscillator next to U1 and the UG483
decoupling placement rule.
Parts:
- added C246: 100nF, Capacitor_SMD:C_0402_1005Metric, symbol Device:C
- added R147: 33, Resistor_SMD:R_0402_1005Metric, symbol Device:R
- added X4: 50MHz CMOS, EasyEDA:OSC-SMD_4P-L3.2-W2.5-BL, symbol EasyEDA:OT322550MJBA4SL
Connections:
- net +3V3: now also C246.1, X4.1 (Tri-state), X4.4 (VDD)
- net DBG_TCK: now also U1.N21 (IO_L13P_T2_MRCC_14); no longer U1.M21 (IO_L12P_T1_MRCC_14)
- net DBG_TDI: now also U1.M20 (IO_L8P_T1_D11_14); no longer U1.N21 (IO_L13P_T2_MRCC_14)
- net DBG_TDO: now also U1.L20 (IO_L8N_T1_D12_14); no longer U1.N22 (IO_L13N_T2_MRCC_14)
- net DBG_TMS: now also U1.N22 (IO_L13N_T2_MRCC_14); no longer U1.M22 (IO_L12N_T1_MRCC_14)
- net GND: now also C246.2, X4.2 (GND)
- net SB_UART_RX: now also U1.P20 (IO_L14P_T2_SRCC_14); no longer U1.M20 (IO_L8P_T1_D11_14)
- net SB_UART_TX: now also U1.P21 (IO_L14N_T2_SRCC_14); no longer U1.L20 (IO_L8N_T1_D12_14)
- new net SYS_CLK: R147.2, U1.M21 (IO_L12P_T1_MRCC_14)
- new net SYS_CLK_OSC: R147.1, X4.3 (OUTPUT)
- no-connect marks 240 -> 239
Other:
- note added: "system clock"
Changed lines of the file:
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@@
 	(rectangle (start 410.21 988.06) (end 494.03 1043.94) (stroke (width 0.15) (type dash)) (fill (type none)))
 	(text "GTP calibration" (at 412.75 991.87 0) (effects (font (size 2.2 2.2) (thickness 0.3)) (justify left)))
+	(rectangle (start 506.73 988.06) (end 646.43 1043.94) (stroke (width 0.15) (type dash)) (fill (type none)))
+	(text "system clock" (at 509.27 991.87 0) (effects (font (size 2.2 2.2) (thickness 0.3)) (justify left)))
 	(symbol (lib_id "odin:XC7A100T-2FGG676I") (at 114.3 85.09 0) (unit 1)
 		(exclude_from_sim no) (in_bom yes) (on_board yes) (dnp no)
@@
 	(global_label "PSRAM0_IO3" (shape passive) (at 373.38 76.2 0) (fields_autoplaced yes) (effects (font (size 1.27 1.27)) (justify right)))
 	(wire (pts (xy 375.92 78.74) (xy 373.38 78.74)) (stroke (width 0) (type default)))
-	(global_label "SB_UART_TX" (shape passive) (at 373.38 78.74 0) (fields_autoplaced yes) (effects (font (size 1.27 1.27)) (justify right)))
+	(global_label "DBG_TDO" (shape passive) (at 373.38 78.74 0) (fields_autoplaced yes) (effects (font (size 1.27 1.27)) (justify right)))
 	(wire (pts (xy 375.92 81.28) (xy 373.38 81.28)) (stroke (width 0) (type default)))
 	(symbol (lib_id "power:+3V3") (at 373.38 81.28 90) (unit 1)
@@
 	(no_connect (at 375.92 93.98))
 	(wire (pts (xy 375.92 96.52) (xy 373.38 96.52)) (stroke (width 0) (type default)))
-	(global_label "SB_UART_RX" (shape passive) (at 373.38 96.52 0) (fields_autoplaced yes) (effects (font (size 1.27 1.27)) (justify right)))
+	(global_label "DBG_TDI" (shape passive) (at 373.38 96.52 0) (fields_autoplaced yes) (effects (font (size 1.27 1.27)) (justify right)))
 	(wire (pts (xy 375.92 99.06) (xy 373.38 99.06)) (stroke (width 0) (type default)))
-	(global_label "DBG_TCK" (shape passive) (at 373.38 99.06 0) (fields_autoplaced yes) (effects (font (size 1.27 1.27)) (justify right)))
-	(wire (pts (xy 375.92 101.6) (xy 373.38 101.6)) (stroke (width 0) (type default)))
-	(global_label "DBG_TMS" (shape passive) (at 373.38 101.6 0) (fields_autoplaced yes) (effects (font (size 1.27 1.27)) (justify right)))
+	(global_label "SYS_CLK" (shape passive) (at 373.38 99.06 0) (fields_autoplaced yes) (effects (font (size 1.27 1.27)) (justify right)))
+	(no_connect (at 375.92 101.6))
 	(wire (pts (xy 375.92 104.14) (xy 373.38 104.14)) (stroke (width 0) (type default)))
 	(global_label "PSRAM1_IO2" (shape passive) (at 373.38 104.14 0) (fields_autoplaced yes) (effects (font (size 1.27 1.27)) (justify right)))
@@
 	(no_connect (at 375.92 124.46))
 	(wire (pts (xy 375.92 127.0) (xy 373.38 127.0)) (stroke (width 0) (type default)))
-	(global_label "DBG_TDI" (shape passive) (at 373.38 127.0 0) (fields_autoplaced yes) (effects (font (size 1.27 1.27)) (justify right)))
+	(global_label "DBG_TCK" (shape passive) (at 373.38 127.0 0) (fields_autoplaced yes) (effects (font (size 1.27 1.27)) (justify right)))
 	(wire (pts (xy 375.92 129.54) (xy 373.38 129.54)) (stroke (width 0) (type default)))
-	(global_label "DBG_TDO" (shape passive) (at 373.38 129.54 0) (fields_autoplaced yes) (effects (font (size 1.27 1.27)) (justify right)))
+	(global_label "DBG_TMS" (shape passive) (at 373.38 129.54 0) (fields_autoplaced yes) (effects (font (size 1.27 1.27)) (justify right)))
 	(wire (pts (xy 375.92 132.08) (xy 373.38 132.08)) (stroke (width 0) (type default)))
 	(global_label "PSRAM2_IO0" (shape passive) (at 373.38 132.08 0) (fields_autoplaced yes) (effects (font (size 1.27 1.27)) (justify right)))
@@
 	(global_label "FLASH_CS_B" (shape passive) (at 452.12 78.74 180) (fields_autoplaced yes) (effects (font (size 1.27 1.27)) (justify left)))
 	(no_connect (at 449.58 81.28))
-	(no_connect (at 449.58 83.82))
-	(no_connect (at 449.58 86.36))
+	(wire (pts (xy 449.58 83.82) (xy 452.12 83.82)) (stroke (width 0) (type default)))
+	(global_label "SB_UART_RX" (shape passive) (at 452.12 83.82 180) (fields_autoplaced yes) (effects (font (size 1.27 1.27)) (justify left)))
+	(wire (pts (xy 449.58 86.36) (xy 452.12 86.36)) (stroke (width 0) (type default)))
+	(global_label "SB_UART_TX" (shape passive) (at 452.12 86.36 180) (fields_autoplaced yes) (effects (font (size 1.27 1.27)) (justify left)))
 	(wire (pts (xy 449.58 88.9) (xy 452.12 88.9)) (stroke (width 0) (type default)))
 	(symbol (lib_id "power:+3V3") (at 452.12 88.9 270) (unit 1)
@@
 		(instances (project "odin" (path "/c44fb7fe-6133-ad34-68fd-fb66126197ef/8cec9eb4-56b4-e78b-2213-febb3af15411" (reference "#PWR0434") (unit 1))))
 	)
+	(symbol (lib_id "Device:C") (at 532.13 1019.81 0) (unit 1)
+		(exclude_from_sim no) (in_bom yes) (on_board yes) (dnp no)
+		(property "Reference" "C246" (at 532.13 1012.19 0) (effects (font (size 1.27 1.27))))
+		(property "Value" "100nF" (at 532.13 1027.43 0) (effects (font (size 1.27 1.27))))
+		(property "Footprint" "Capacitor_SMD:C_0402_1005Metric" (at 532.13 1027.43 0) (effects (font (size 1.27 1.27)) (hide yes)))
+		(property "LCSC" "C1525" (at 532.13 1027.43 0) (effects (font (size 1.27 1.27)) (hide yes)))
+		(instances (project "odin" (path "/c44fb7fe-6133-ad34-68fd-fb66126197ef/8cec9eb4-56b4-e78b-2213-febb3af15411" (reference "C246") (unit 1))))
+	)
+	(wire (pts (xy 532.13 1016.0) (xy 532.13 1013.46)) (stroke (width 0) (type default)))
+	(symbol (lib_id "power:+3V3") (at 532.13 1013.46 0) (unit 1)
+		(exclude_from_sim no) (in_bom no) (on_board yes) (dnp no)
+		(property "Reference" "#PWR0435" (at 532.13 1013.46 0) (effects (font (size 1.27 1.27)) (hide yes)))
+		(property "Value" "+3V3" (at 532.13 1009.65 0) (effects (font (size 1.27 1.27))))
+		(instances (project "odin" (path "/c44fb7fe-6133-ad34-68fd-fb66126197ef/8cec9eb4-56b4-e78b-2213-febb3af15411" (reference "#PWR0435") (unit 1))))
+	)
+	(wire (pts (xy 532.13 1023.62) (xy 532.13 1026.16)) (stroke (width 0) (type default)))
+	(symbol (lib_id "power:GND") (at 532.13 1026.16 0) (unit 1)
+		(exclude_from_sim no) (in_bom no) (on_board yes) (dnp no)
+		(property "Reference" "#PWR0436" (at 532.13 1026.16 0) (effects (font (size 1.27 1.27)) (hide yes)))
+		(property "Value" "GND" (at 532.13 1029.97 0) (effects (font (size 1.27 1.27))))
+		(instances (project "odin" (path "/c44fb7fe-6133-ad34-68fd-fb66126197ef/8cec9eb4-56b4-e78b-2213-febb3af15411" (reference "#PWR0436") (unit 1))))
+	)
+	(symbol (lib_id "Device:R") (at 565.15 1019.81 0) (unit 1)
+		(exclude_from_sim no) (in_bom yes) (on_board yes) (dnp no)
+		(property "Reference" "R147" (at 565.15 1012.19 0) (effects (font (size 1.27 1.27))))
+		(property "Value" "33" (at 565.15 1027.43 0) (effects (font (size 1.27 1.27))))
+		(property "Footprint" "Resistor_SMD:R_0402_1005Metric" (at 565.15 1027.43 0) (effects (font (size 1.27 1.27)) (hide yes)))
+		(property "LCSC" "C25105" (at 565.15 1027.43 0) (effects (font (size 1.27 1.27)) (hide yes)))
+		(instances (project "odin" (path "/c44fb7fe-6133-ad34-68fd-fb66126197ef/8cec9eb4-56b4-e78b-2213-febb3af15411" (reference "R147") (unit 1))))
+	)
+	(wire (pts (xy 565.15 1016.0) (xy 565.15 1013.46)) (stroke (width 0) (type default)))
+	(global_label "SYS_CLK_OSC" (shape passive) (at 565.15 1013.46 270) (fields_autoplaced yes) (effects (font (size 1.27 1.27)) (justify left)))
+	(wire (pts (xy 565.15 1023.62) (xy 565.15 1026.16)) (stroke (width 0) (type default)))
+	(global_label "SYS_CLK" (shape passive) (at 565.15 1026.16 90) (fields_autoplaced yes) (effects (font (size 1.27 1.27)) (justify right)))
+	(symbol (lib_id "EasyEDA:OT322550MJBA4SL") (at 609.6 1018.54 0) (unit 1)
+		(exclude_from_sim no) (in_bom yes) (on_board yes) (dnp no)
+		(property "Reference" "X4" (at 609.6 1012.19 0) (effects (font (size 1.27 1.27))))
+		(property "Value" "50MHz CMOS" (at 609.6 1024.89 0) (effects (font (size 1.27 1.27))))
+		(property "Footprint" "EasyEDA:OSC-SMD_4P-L3.2-W2.5-BL" (at 609.6 1024.89 0) (effects (font (size 1.27 1.27)) (hide yes)))
+		(property "LCSC" "C717684" (at 609.6 1024.89 0) (effects (font (size 1.27 1.27)) (hide yes)))
+		(instances (project "odin" (path "/c44fb7fe-6133-ad34-68fd-fb66126197ef/8cec9eb4-56b4-e78b-2213-febb3af15411" (reference "X4") (unit 1))))
+	)
+	(wire (pts (xy 598.17 1016.0) (xy 595.63 1016.0)) (stroke (width 0) (type default)))
+	(symbol (lib_id "power:+3V3") (at 595.63 1016.0 90) (unit 1)
+		(exclude_from_sim no) (in_bom no) (on_board yes) (dnp no)
+		(property "Reference" "#PWR0437" (at 595.63 1016.0 0) (effects (font (size 1.27 1.27)) (hide yes)))
+		(property "Value" "+3V3" (at 591.82 1016.0 0) (effects (font (size 1.27 1.27))))
+		(instances (project "odin" (path "/c44fb7fe-6133-ad34-68fd-fb66126197ef/8cec9eb4-56b4-e78b-2213-febb3af15411" (reference "#PWR0437") (unit 1))))
+	)
+	(wire (pts (xy 598.17 1021.08) (xy 595.63 1021.08)) (stroke (width 0) (type default)))
+	(symbol (lib_id "power:GND") (at 595.63 1021.08 90) (unit 1)
+		(exclude_from_sim no) (in_bom no) (on_board yes) (dnp no)
+		(property "Reference" "#PWR0438" (at 595.63 1021.08 0) (effects (font (size 1.27 1.27)) (hide yes)))
+		(property "Value" "GND" (at 591.82 1021.08 0) (effects (font (size 1.27 1.27))))
+		(instances (project "odin" (path "/c44fb7fe-6133-ad34-68fd-fb66126197ef/8cec9eb4-56b4-e78b-2213-febb3af15411" (reference "#PWR0438") (unit 1))))
+	)
+	(wire (pts (xy 621.03 1021.08) (xy 623.57 1021.08)) (stroke (width 0) (type default)))
+	(global_label "SYS_CLK_OSC" (shape passive) (at 623.57 1021.08 180) (fields_autoplaced yes) (effects (font (size 1.27 1.27)) (justify left)))
+	(wire (pts (xy 621.03 1016.0) (xy 623.57 1016.0)) (stroke (width 0) (type default)))
+	(symbol (lib_id "power:+3V3") (at 623.57 1016.0 270) (unit 1)
+		(exclude_from_sim no) (in_bom no) (on_board yes) (dnp no)
+		(property "Reference" "#PWR0439" (at 623.57 1016.0 0) (effects (font (size 1.27 1.27)) (hide yes)))
+		(property "Value" "+3V3" (at 627.38 1016.0 0) (effects (font (size 1.27 1.27))))
+		(instances (project "odin" (path "/c44fb7fe-6133-ad34-68fd-fb66126197ef/8cec9eb4-56b4-e78b-2213-febb3af15411" (reference "#PWR0439") (unit 1))))
+	)
 )

Commit message: Explain every part: role text in the schematic, the PCB and a parts guide
tools/roles.py says what each part is for: a paragraph per schematic group,
a line per active part, notes on nets such as straps, and derived lines for
resistors and capacitors (bypass, pull-up, series, and the part they serve).
gen_project.py puts the text in each symbol's Description and a paragraph
inside every group box; load_pcb.py copies it into each footprint's
Description field; tools/roles.py --write renders ref/parts-guide.md.
gate.py fails on an unexplained part on a covered sheet or a stale guide.
The FPGA and Network sheets are written; the other four follow.
Other:
- note added: "Bulk capacitor shared by every FPGA I/O bank powered from +2V5: UG483 Table 2-2 note 3 asks one 47 uF per group of up to four banks on one voltage. See ref/decoupling.md."
- note added: "Bulk capacitor shared by every FPGA I/O bank powered from +3V3: UG483 Table 2-2 note 3 asks one 47 uF per group of up to four banks on one voltage. See ref/decoupling.md."
- note added: "Bulk capacitor shared by every FPGA I/O bank powered from VCCIO_1: UG483 Table 2-2 note 3 asks one 47 uF per group of up to four banks on one voltage. See ref/decoupling.md."
- note added: "Bulk capacitor shared by every FPGA I/O bank powered from VCCIO_2: UG483 Table 2-2 note 3 asks one 47 uF per group of up to four banks on one voltage. See ref/decoupling.md."
- note added: "Decoupling for +1V0_MGT (+1V0_MGT), which powers the unused but powered transceivers (MGTAVCC); the MGT supplies are UG482's, not in UG483 Table 2-2: one 100 nF per ball plus 4.7 uF. Placement rule: ref/decoupling.md."
- note added: "Decoupling for +1V2_MGT (+1V2_MGT), which powers the unused but powered transceivers (MGTAVTT); the MGT supplies are UG482's, not in UG483 Table 2-2: one 100 nF per ball plus 4.7 uF. Placement rule: ref/decoupling.md."
- note added: "Decoupling for FPGA I/O bank 13's supply (VCCO): 2 x 4.7 uF and 4 x 0.47 uF, UG483 Table 2-2. They keep the bank's supply steady while its outputs switch. Placement rule: ref/decoupling.md."
- note added: "Decoupling for FPGA I/O bank 14's supply (VCCO): 2 x 4.7 uF and 4 x 0.47 uF, UG483 Table 2-2. They keep the bank's supply steady while its outputs switch. Placement rule: ref/decoupling.md."
- note added: "Decoupling for FPGA I/O bank 15's supply (VCCO): 2 x 4.7 uF and 4 x 0.47 uF, UG483 Table 2-2. They keep the bank's supply steady while its outputs switch. Placement rule: ref/decoupling.md."
- note added: "Decoupling for FPGA I/O bank 16's supply (VCCO): 2 x 4.7 uF and 4 x 0.47 uF, UG483 Table 2-2. They keep the bank's supply steady while its outputs switch. Placement rule: ref/decoupling.md."
- note added: "Decoupling for FPGA I/O bank 34's supply (VCCO): 2 x 4.7 uF and 4 x 0.47 uF, UG483 Table 2-2. They keep the bank's supply steady while its outputs switch. Placement rule: ref/decoupling.md."
- note added: "Decoupling for FPGA I/O bank 35's supply (VCCO): 2 x 4.7 uF and 4 x 0.47 uF, UG483 Table 2-2. They keep the bank's supply steady while its outputs switch. Placement rule: ref/decoupling.md."
- note added: "Decoupling for VCCADC (+1V8), which powers the FPGA's on-chip ADC (XADC); not in UG483 Table 2-2; one 100 nF bypass. Placement rule: ref/decoupling.md."
- note added: "Decoupling for VCCAUX (+1V8), which powers the FPGA auxiliary circuits (clocking, I/O pre-drivers); quantities from UG483 Table 2-2, row FGG676 / XC7A100T. Placement rule: ref/decoupling.md."
- note added: "Decoupling for VCCBRAM (+1V0), which powers the FPGA block RAM; quantities from UG483 Table 2-2, row FGG676 / XC7A100T. Placement rule: ref/decoupling.md."
- note added: "Decoupling for VCCINT (+1V0), which powers the FPGA core logic; quantities from UG483 Table 2-2, row FGG676 / XC7A100T. Placement rule: ref/decoupling.md."
- note added: "Decoupling for VCCO_0 (+3V3), which powers configuration bank 0; quantities from UG483 Table 2-2, row FGG676 / XC7A100T. Placement rule: ref/decoupling.md."
- note added: "How the FPGA loads its design at power-on. M[2:0] = 001 selects master SPI: the FPGA clocks its bitstream out of the W25Q256 flash (U6) by itself. The mode straps are 1 k, the most UG470 v1.17 Table 2-4 allows. PROGRAM_B and INIT_B are pulled up so the board controller can restart configuration; PUDC_B is strapped low so I/O pull-ups stay on while the FPGA configures, which holds outputs such as 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"
- note added: "The FPGA is the board: every user design (a NEORV32 RISC-V core, a video pipeline, a protocol bridge) runs here. Its six user I/O banks are dedicated by job: bank 13 drives the two 5 V buses and the PHY reset/interrupt, bank 14 the PSRAM, the configuration flash, the board-controller sideband and the 50 MHz clock, banks 15 and 34 the direct extension slots A-D and E-H at a jumper-selected voltage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"
- note added: "The FPGA's own clock. X4 runs at 50 MHz from power-on and enters bank 14 on a clock-capable (MRCC) ball, so it can feed an MMCM and make any frequency the design needs. Without it nothing in the fabric would run until a network link came up."
- note added: "The XC7A100T has two quads of multi-gigabit transceivers (GTP). Rev A uses none of them, but UG482 Tables 5-5 and 5-6 still want their supplies powered, their receive inputs grounded and one 100 ohm 1 % calibration resistor per quad to MGTAVTT. These two resistors are that."
- moved on the sheet: C246, C301, C302, C303, C304, C305, C306, C307, C308, C309, C310, C311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
