File: kicad/fpga.kicad_sch (KiCad schematic)
At the start: 110 parts, among them Q4 BSS138LT1G, U1 XC7A100T-2FGG676I, X4 50MHz CMOS

Commit message: PSRAM power-up states with PUDC_B high; TPS22953 for the jumpered PIN V exports
Connections:
- net +3V3: now also R6.1
- net GND: no longer R6.2
- net PUDC_B: now also R6.2; no longer R6.1
Other:
- note added: "How the FPGA loads its design at power-on. M[2:0] = 001 selects master SPI: the FPGA clocks its bitstream out of the W25Q256 flash (U6) by itself. The mode straps are 1 k, the most UG470 v1.17 Table 2-4 allows. PROGRAM_B and INIT_B are pulled up so the board controller can restart configuration; PUDC_B is strapped high so the FPGA adds no pull-ups while it configures: every line that needs a leve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"
- note removed: "How the FPGA loads its design at power-on. M[2:0] = 001 selects master SPI: the FPGA clocks its bitstream out of the W25Q256 flash (U6) by itself. The mode straps are 1 k, the most UG470 v1.17 Table 2-4 allows. PROGRAM_B and INIT_B are pulled up so the board controller can restart configuration; PUDC_B is strapped low so I/O pull-ups stay on while the FPGA configures, which holds outputs such as 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"
- moved on the sheet: D1, Q4, R1, R2, R3, R4, R5, R6, R7, R98
