File: kicad/network.kicad_sch (KiCad schematic)
At the start: 39 parts, among them J70 ETH, J71 LINK P, J72 LINK Q, U30 RTL8211FD-CG, X3 25MHz 12pF

Commit message: Explain every part: role text in the schematic, the PCB and a parts guide
tools/roles.py says what each part is for: a paragraph per schematic group,
a line per active part, notes on nets such as straps, and derived lines for
resistors and capacitors (bypass, pull-up, series, and the part they serve).
gen_project.py puts the text in each symbol's Description and a paragraph
inside every group box; load_pcb.py copies it into each footprint's
Description field; tools/roles.py --write renders ref/parts-guide.md.
gate.py fails on an unexplained part on a covered sheet or a stale guide.
The FPGA and Network sheets are written; the other four follow.
Other:
- note added: "A board-to-board link port, not Ethernet. Four LVDS pairs from FPGA bank 16 go straight to an RJ45 so two boards can be cabled with shielded twisted pair: a clock and a data pair out, a clock and a data pair in. Cable LINK P of one board to LINK Q of the other, and power both boards before plugging in (ref/link-ports.md). The two arrays clamp ESD at the jack."
- note added: "Resistors that configure U30 at reset and drive its LEDs. During reset the PHY reads the level on several output pins as configuration: PHY address 1, PLL kept running, 2 ns clock delays on both RGMII directions (so the FPGA needs none), and an external 2.5 V I/O supply (RTL8211F Tables 10 and 11). The same LED pins later drive the jack's LEDs, whose polarity follows the strap (section 7.9, Figur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"
- note added: "The 25 MHz crystal U30 needs as its reference (RTL8211F Table 56: 25 MHz, +/-50 ppm all in). The two capacitors set the crystal's load; the 0 ohm resistor is a placeholder to limit crystal drive if measurement shows it needs it."
- note added: "The Ethernet connector, with the 1000Base-T transformers and two LEDs built into the jack. The transformers isolate the cable from the board; the capacitor returns their centre taps to ground (ref/network.md)."
- note added: "The second link port, wired as the mirror of LINK P so a straight cable from a P to a Q connects outputs to inputs. Same rules: STP cable, power both boards first (ref/link-ports.md)."
- note added: "U30 is the Ethernet PHY: it turns the FPGA's RGMII bus (four data bits each way plus clock and control, 2.5 V, bank 16) into 1000Base-T signals on the ETH jack's four twisted pairs. The FPGA still needs a MAC; the PHY handles the line, link negotiation and the analog side. It runs from +3V3, takes its RGMII pad supply from +2V5 and makes its own 1.0 V core supply with an internal LDO (the FD vari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"
- moved on the sheet: C232, C233, C234, C235, C236, C237, C238, C239, C240, C241, C242, C243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
