File: kicad/odin.kicad_pcb (KiCad board)
At the start: 8 copper layers, 100 x 100 mm, 544 parts, among them J1 USB-C, J19 2.54-2*3P, J2 FPGA JTAG, J20 2.54-2*3P, J3 WingTAT 2044-2X32G00SA, J5 WingTAT 2044-2X32G00SA, J50 9-21V POWER IN, J51 CTRL SWD, J52 PZ254V-11-02P, J53 XFCN PM254V-11-07-H85, J54 XFCN PM254V-11-07-H85, J55 XFCN PM254V-11-07-H85, J56 XFCN PM254V-11-07-H85, J57 XFCN PM254V-11-07-H85, J58 XFCN PM254V-11-07-H85, J62 XFCN PM254V-11-07-H85, J63 XFCN PM254V-11-07-H85, J64 XFCN PM254V-11-07-H85, J65 XFCN PM254V-11-07-H85, J68 AUX IN 9-28V UNREGULATED, J7 PM254-2-08-Z-8.5, J70 ETH, J71 LINK P, J72 LINK Q, J73 HDMI OUT, J74 microSD, J8 PM254-2-08-Z-8.5, Q3 BSS138LT1G, Q4 BSS138LT1G, SW1 CTRL BOOT, U1 XC7A100T-2FGG676I, U10 SN74LXC8T245PWR, U11 AP63300WU-7, U12 AP63300WU-7, U13 TLV62569DRLR, U14 TLV62569DRLR, U15 SY8047QDC, U16 TLV62569DRLR, U17 PCF8574T_3,518, U18 CH224K, U2 APS6404L-SQN-SN, U20 SN74CB3Q3384APWR, U21 TPS22950CDDCR, U22 TPS22950CDDCR, U23 TPS22953DSQR, U24 TPS22953DSQR, U26 TPS259470ARPWR, U3 APS6404L-SQN-SN, U30 RTL8211FD-CG, U31 TPD12S016PWR, U32 W9825G6KH-6, U33 MR25H10CDF, U34 TPS2121RUXR, U4 APS6404L-SQN-SN, U5 APS6404L-SQN-SN, U6 W25Q256JVEIQ, U7 RP2350B, U8 W25Q32JVZP, U9 SN74LXC8T245PWR, X3 25MHz 12pF, X4 50MHz CMOS, Y1 12MHz ABM8-272-T3

Commit message: Island Q3: the 9 V request switch with the CFG1 pull-up and its gate pull-down
Parts:
- moved R172 441.1 mm to (438.9, 60.1), turned to 180 degrees
- moved R173 431.5 mm to (432.5, 59.2), turned to 180 degrees
- moved Q3 390.9 mm to (435.7, 60.1)
Other:
- board text added: "9 V request switch generic, 3 parts, 2026-10-29"
- board text removed: "9 V request switch pass switch driver generic, 2 parts, 2026-10-28"
Changed lines of the file:
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@@
 	(footprint "Resistor_SMD:R_0402_1005Metric"
 		(layer "F.Cu")
-		(at 52.5 272.746231)
+		(at 438.92 60.11 180)
 		(descr "10k resistor from PD_CFG1 to PD_VDD, for U18 (USB-PD negotiator): CH224K request: high (pull-up) = 5 V, pulled low by Q3 = 9 V; CH224K's internal regulator output")
 		(tags "resistor")
 		(property "Reference" "R172"
-			(at 0 -1.17 0)
+			(at 0 -1.17 180)
 			(layer "F.Fab")
 			(effects
@@
 		)
 		(property "Value" "10k"
-			(at 0 1.17 0)
+			(at 0 1.17 180)
 			(layer "F.Fab")
 			(effects
@@
 		)
 		(property "Datasheet" ""
-			(at 0 0 0)
+			(at 0 0 180)
 			(layer "F.Fab")
 			(hide yes)
@@
 		)
 		(property "Description" "10k resistor from PD_CFG1 to PD_VDD, for U18 (USB-PD negotiator): CH224K request: high (pull-up) = 5 V, pulled low by Q3 = 9 V; CH224K's internal regulator output"
-			(at 0 0 0)
+			(at 0 0 180)
 			(layer "F.Fab")
 			(hide yes)
@@
 		)
 		(fp_text user "${REFERENCE}"
-			(at 0 0 0)
+			(at 0 0 180)
 			(layer "F.Fab")
 			(effects
@@
 		)
 		(pad "1" smd roundrect
-			(at -0.51 0)
+			(at -0.51 0 180)
 			(size 0.54 0.64)
 			(layers "F.Cu" "F.Mask" "F.Paste")
@@
 		)
 		(pad "2" smd roundrect
-			(at 0.51 0)
+			(at 0.51 0 180)
 			(size 0.54 0.64)
 			(layers "F.Cu" "F.Mask" "F.Paste")
@@
 	(footprint "EasyEDA:SOT-23-3_L2.9-W1.6-P1.90-LS2.8-BR"
 		(layer "F.Cu")
-		(at 825.39 90.39 180)
+		(at 435.69 60.11 180)
 		(descr "9 V request switch: Small N-MOSFET the board controller (PD_REQ_9V) uses to pull the CH224K's CFG1 low and ask the charger for 9 V. Off: 5 V.")
 		(property "Reference" "Q3"
@@
 	(footprint "Resistor_SMD:R_0402_1005Metric"
 		(layer "F.Cu")
-		(at 57.5 272.746231)
+		(at 432.46 59.16 180)
 		(descr "100k resistor from PD_REQ_9V to GND, for U7 (board controller): Q3's gate; off (5 V) unless the board controller drives it high")
 		(tags "resistor")
 		(property "Reference" "R173"
-			(at 0 -1.17 0)
+			(at 0 -1.17 180)
 			(layer "F.Fab")
 			(effects
@@
 		)
 		(property "Value" "100k"
-			(at 0 1.17 0)
+			(at 0 1.17 180)
 			(layer "F.Fab")
 			(effects
@@
 		)
 		(property "Datasheet" ""
-			(at 0 0 0)
+			(at 0 0 180)
 			(layer "F.Fab")
 			(hide yes)
@@
 		)
 		(property "Description" "100k resistor from PD_REQ_9V to GND, for U7 (board controller): Q3's gate; off (5 V) unless the board controller drives it high"
-			(at 0 0 0)
+			(at 0 0 180)
 			(layer "F.Fab")
 			(hide yes)
@@
 		)
 		(property "LCSC Part" "C25741"
-			(at 0 0 0)
+			(at 0 0 180)
 			(layer "F.SilkS")
 			(hide yes)
@@
 		)
 		(fp_text user "${REFERENCE}"
-			(at 0 0 0)
+			(at 0 0 180)
 			(layer "F.Fab")
 			(effects
@@
 		)
 		(pad "1" smd roundrect
-			(at -0.51 0)
+			(at -0.51 0 180)
 			(size 0.54 0.64)
 			(layers "F.Cu" "F.Mask" "F.Paste")
@@
 		)
 		(pad "2" smd roundrect
-			(at 0.51 0)
+			(at 0.51 0 180)
 			(size 0.54 0.64)
 			(layers "F.Cu" "F.Mask" "F.Paste")
@@
 	)
 	(gr_rect
-		(start 822.115 87.405)
-		(end 832.095 93.375)
-		(stroke
-			(width 0.15)
-			(type dash)
-		)
-		(fill no)
-		(layer "Cmts.User")
-	)
-	(gr_rect
-		(start 822.115 79.325)
-		(end 832.095 87.405)
-		(stroke
-			(width 0.15)
-			(type solid)
-		)
-		(fill no)
-		(layer "Cmts.User")
-	)
-	(gr_text "island Q3"
-		(at 822.515 80.925 0)
-		(layer "Cmts.User")
-		(effects
-			(font
-				(size 1.2 1.2)
-				(thickness 0.18)
-			)
-			(justify left bottom)
-		)
-	)
-	(gr_text "9 V request\nswitch\npass switch\ndriver generic,\n2 parts,\n2026-10-28"
-		(at 822.515 81.225 0)
-		(layer "Cmts.User")
-		(effects
-			(font
-				(size 0.7 0.7)
-				(thickness 0.105)
-			)
-			(justify left top)
-		)
-	)
-	(group "island Q3"
-		(members
-			"4167d21f-f2b8-4a02-b2d1-caf4fe36532f"
-			"22e163f5-c6dc-4f5f-97c5-6f08034f2674"
-			"75332a15-bedf-496d-83a9-018aa8b792b3"
-			"b931b3e5-c83f-4550-952b-86f09f505e3b"
-			"6f54abb6-7223-446e-82ec-789b94915d7d"
-		)
-	)
-	(gr_rect
 		(start 847.155 156.305)
 		(end 859.175 162.395)
@@
 		)
 	)
+	(gr_rect
+		(start 430.005 57.125)
+		(end 441.375 63.095)
+		(stroke
+			(width 0.15)
+			(type dash)
+		)
+		(fill no)
+		(layer "Cmts.User")
+	)
+	(gr_rect
+		(start 430.005 51.005)
+		(end 441.375 57.125)
+		(stroke
+			(width 0.15)
+			(type solid)
+		)
+		(fill no)
+		(layer "Cmts.User")
+	)
+	(gr_text "island Q3"
+		(at 430.405 52.605 0)
+		(layer "Cmts.User")
+		(effects
+			(font
+				(size 1.2 1.2)
+				(thickness 0.18)
+			)
+			(justify left bottom)
+		)
+	)
+	(gr_text "9 V request\nswitch\ngeneric, 3 parts,\n2026-10-29"
+		(at 430.405 52.905 0)
+		(layer "Cmts.User")
+		(effects
+			(font
+				(size 0.7 0.7)
+				(thickness 0.105)
+			)
+			(justify left top)
+		)
+	)
+	(group "island Q3"
+		(members
+			"6db8634c-5bc6-47a7-ab00-3bac21d77857"
+			"8f838063-e30f-48f0-b2e7-9acd2a3226fa"
+			"b29e7c7e-d26a-4034-ad35-67e8bdaa27c0"
+			"efbbc4e3-a836-455b-a814-5f20018a24ca"
+			"6f54abb6-7223-446e-82ec-789b94915d7d"
+			"06677c63-6067-4f33-8c12-7f2b2df42b47"
+			"97c89a65-0a9f-4de6-9bb4-ec0c850b1bf4"
+		)
+	)

Commit message: Island U11 extended: the 10 uF input capacitor
Parts:
- moved C267 425.3 mm to (440.8, 72.3), turned to 180 degrees
- moved C189 304.1 mm to (440.6, 75.4)
- moved C190 304.1 mm to (448.0, 75.4)
- moved R56 304.1 mm to (443.5, 81.1)
- moved C188 304.1 mm to (440.8, 80.8)
- moved C191 304.1 mm to (444.6, 75.4)
- moved R55 304.1 mm to (443.7, 78.4)
- moved U11 304.1 mm to (440.8, 78.4)
- moved L2 304.1 mm to (435.1, 78.4)
Other:
- board text added: "5 V regulator, always on AP63300, 9 parts, 2026-10-29"
- board text removed: "5 V regulator, always on 5 V regulator AP63300, 9 parts, 2026-10-28"
Changed lines of the file:
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@@
 	(footprint "EasyEDA:IND-SMD_L6.0-W6.0"
 		(layer "F.Cu")
-		(at 738.92 66.5)
+		(at 435.1 78.39)
 		(descr "4.7uH SRN6045TA-4R7M inductor between +5V_BUCK and SW_5V, for U11 (5 V regulator, always on): regulator switching node")
 		(property "Reference" "L2"
@@
 	(footprint "Capacitor_SMD:C_0402_1005Metric"
 		(layer "F.Cu")
-		(at 744.62 68.96 180)
+		(at 440.8 80.85 180)
 		(descr "100nF capacitor between BOOT_5V and SW_5V, for U11 (5 V regulator, always on): bootstrap capacitor for the regulator's high-side switch; regulator switching node")
 		(tags "capacitor")
@@
 	(footprint "Capacitor_SMD:C_1210_3225Metric"
 		(layer "F.Cu")
-		(at 56.725 254.921231)
+		(at 440.8 72.28 180)
 		(descr "10uF 50V bypass on VSYS, for U11 (5 V regulator, always on)")
 		(tags "capacitor")
 		(property "Reference" "C267"
-			(at 0 -2.3 0)
+			(at 0 -2.3 180)
 			(layer "F.Fab")
 			(effects
@@
 		)
 		(property "Value" "10uF 50V"
-			(at 0 2.3 0)
+			(at 0 2.3 180)
 			(layer "F.Fab")
 			(effects
@@
 		)
 		(property "Datasheet" ""
-			(at 0 0 0)
+			(at 0 0 180)
 			(layer "F.Fab")
 			(hide yes)
@@
 		)
 		(property "Description" "10uF 50V bypass on VSYS, for U11 (5 V regulator, always on)"
-			(at 0 0 0)
+			(at 0 0 180)
 			(layer "F.Fab")
 			(hide yes)
@@
 		)
 		(property "LCSC Part" "C77102"
-			(at 0 0 0)
+			(at 0 0 180)
 			(layer "F.SilkS")
 			(hide yes)
@@
 		)
 		(fp_text user "${REFERENCE}"
-			(at 0 0 0)
+			(at 0 0 180)
 			(layer "F.Fab")
 			(effects
@@
 		)
 		(pad "1" smd roundrect
-			(at -1.475 0)
+			(at -1.475 0 180)
 			(size 1.15 2.7)
 			(layers "F.Cu" "F.Mask" "F.Paste")
@@
 		)
 		(pad "2" smd roundrect
-			(at 1.475 0)
+			(at 1.475 0 180)
 			(size 1.15 2.7)
 			(layers "F.Cu" "F.Mask" "F.Paste")
@@
 	(footprint "Capacitor_SMD:C_0805_2012Metric"
 		(layer "F.Cu")
-		(at 744.47 63.52)
+		(at 440.65 75.41)
 		(descr "22uF bypass on +5V_BUCK, for U11 (5 V regulator, always on)")
 		(tags "capacitor")
@@
 	(footprint "EasyEDA:TSOT-23-6_L2.9-W1.6-P0.95-LS2.8-BR"
 		(layer "F.Cu")
-		(at 744.62 66.5)
+		(at 440.8 78.39)
 		(descr "5 V regulator, always on: Diodes AP63300, 3 A switching regulator: VSYS to +5V_BUCK, then U34 to +5V. Starts by itself.")
 		(property "Reference" "U11"
@@
 	(footprint "Capacitor_SMD:C_0805_2012Metric"
 		(layer "F.Cu")
-		(at 748.37 63.52)
+		(at 444.55 75.41)
 		(descr "22uF bypass on +5V_BUCK, for U11 (5 V regulator, always on)")
 		(tags "capacitor")
@@
 	(footprint "Capacitor_SMD:C_0805_2012Metric"
 		(layer "F.Cu")
-		(at 751.82 63.52)
+		(at 448 75.41)
 		(descr "22uF bypass on +5V_BUCK, for U11 (5 V regulator, always on)")
 		(tags "capacitor")
@@
 	(footprint "Resistor_SMD:R_0603_1608Metric"
 		(layer "F.Cu")
-		(at 747.32 69.23 180)
+		(at 443.5 81.12 180)
 		(descr "19.1k resistor from FB_5V to GND, for U11 (5 V regulator, always on): feedback divider, sets the regulator's output voltage")
 		(tags "resistor")
@@
 	(footprint "Resistor_SMD:R_0603_1608Metric"
 		(layer "F.Cu")
-		(at 747.48 66.5 -90)
+		(at 443.66 78.39 -90)
 		(descr "100k series resistor between +5V_BUCK and FB_5V, for U11 (5 V regulator, always on): feedback divider, sets the regulator's output voltage")
 		(tags "resistor")
@@
 	)
 	(gr_rect
-		(start 733.82 61.015)
-		(end 755.045 71.485)
-		(stroke
-			(width 0.15)
-			(type dash)
-		)
-		(fill no)
-		(layer "Cmts.User")
-	)
-	(gr_rect
-		(start 733.82 55.875)
-		(end 755.045 61.015)
-		(stroke
-			(width 0.15)
-			(type solid)
-		)
-		(fill no)
-		(layer "Cmts.User")
-	)
-	(gr_text "island U11"
-		(at 734.22 57.475 0)
-		(layer "Cmts.User")
-		(effects
-			(font
-				(size 1.2 1.2)
-				(thickness 0.18)
-			)
-			(justify left bottom)
-		)
-	)
-	(gr_text "5 V regulator, always on\n5 V regulator AP63300, 9 parts,\n2026-10-28"
-		(at 734.22 57.775 0)
-		(layer "Cmts.User")
-		(effects
-			(font
-				(size 0.7 0.7)
-				(thickness 0.105)
-			)
-			(justify left top)
-		)
-	)
-	(group "island U11"
-		(members
-			"77ff33e9-d0c7-43df-b581-da03843e02d3"
-			"fc1bc73a-dbe1-4948-8b94-541047426757"
-			"15b6fb5e-0940-4167-906f-caca7152807b"
-			"e1e63836-1570-4fdc-9c79-6511d2383280"
-			"7d81e816-b447-4041-957a-fc84308de6e4"
-			"0300b92e-2901-4150-9c23-b5a4c67f4b40"
-			"47b24bf6-6244-40e9-9091-9b278e9327c8"
-			"a683adfd-5974-4cd1-b47c-6da53214b68e"
-			"8b8a52e4-8d2c-4afb-aa9b-2b5d38a76054"
-			"02bd4d60-d15b-4cd8-916c-e68a7a5f13c9"
-			"e60e3c57-1730-4b09-9b07-bb8d55b6eeb8"
-			"d6edac5b-e0c1-4c5d-9536-9146de7be84c"
-		)
-	)
-	(gr_rect
 		(start 757.795 52.755)
 		(end 770.115 66.535)
@@
 		)
 	)
+	(gr_rect
+		(start 430 69.155)
+		(end 451.225 83.375)
+		(stroke
+			(width 0.15)
+			(type dash)
+		)
+		(fill no)
+		(layer "Cmts.User")
+	)
+	(gr_rect
+		(start 430 64.995)
+		(end 451.225 69.155)
+		(stroke
+			(width 0.15)
+			(type solid)
+		)
+		(fill no)
+		(layer "Cmts.User")
+	)
+	(gr_text "island U11"
+		(at 430.4 66.595 0)
+		(layer "Cmts.User")
+		(effects
+			(font
+				(size 1.2 1.2)
+				(thickness 0.18)
+			)
+			(justify left bottom)
+		)
+	)
+	(gr_text "5 V regulator, always on\nAP63300, 9 parts, 2026-10-29"
+		(at 430.4 66.895 0)
+		(layer "Cmts.User")
+		(effects
+			(font
+				(size 0.7 0.7)
+				(thickness 0.105)
+			)
+			(justify left top)
+		)
+	)
+	(group "island U11"
+		(members
+			"320afcc0-5ffe-48c3-9faa-c9e86795672e"
+			"a90a3fc3-1913-4771-8bb9-d070a8ad08c4"
+			"2031ffef-9e68-402c-8066-de0ff45aa42d"
+			"9439d63c-d1bd-4aba-8018-14aa69c689c8"
+			"7d81e816-b447-4041-957a-fc84308de6e4"
+			"0300b92e-2901-4150-9c23-b5a4c67f4b40"
+			"47b24bf6-6244-40e9-9091-9b278e9327c8"
+			"a683adfd-5974-4cd1-b47c-6da53214b68e"
+			"8b8a52e4-8d2c-4afb-aa9b-2b5d38a76054"
+			"171a6cc4-8cc3-467a-bb6c-fec80149283c"
+			"02bd4d60-d15b-4cd8-916c-e68a7a5f13c9"
+			"e60e3c57-1730-4b09-9b07-bb8d55b6eeb8"
+			"d6edac5b-e0c1-4c5d-9536-9146de7be84c"
+		)
+	)

Commit message: Island U13 extended: the 4.7 uF input capacitor
Parts:
- moved C268 408.9 mm to (441.3, 97.6), turned to -90 degrees
- moved C198 335.4 mm to (433.2, 97.4)
- moved C199 335.4 mm to (433.2, 99.7)
- moved L4 335.4 mm to (436.3, 93.9)
- moved R60 335.4 mm to (436.3, 101.9)
- moved R91 335.4 mm to (439.3, 94.6)
- moved U13 335.4 mm to (436.3, 97.6)
- moved C200 335.4 mm to (438.1, 97.6)
- moved R59 335.4 mm to (436.6, 99.9)
Other:
- board text added: "2.5 V regulator TLV62569, 9 parts, 2026-10-29"
- board text removed: "2.5 V regulator TLV62569, 8 parts, 2026-10-28"
Changed lines of the file:
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@@
 	(footprint "Capacitor_SMD:C_0805_2012Metric"
 		(layer "F.Cu")
-		(at 760.2 172.25 180)
+		(at 433.22 97.38 180)
 		(descr "22uF bypass on +2V5, for U13 (2.5 V regulator)")
 		(tags "capacitor")
@@
 	(footprint "Capacitor_SMD:C_0805_2012Metric"
 		(layer "F.Cu")
-		(at 760.2 174.55 180)
+		(at 433.22 99.68 180)
 		(descr "22uF bypass on +2V5, for U13 (2.5 V regulator)")
 		(tags "capacitor")
@@
 	(footprint "Capacitor_SMD:C_0402_1005Metric"
 		(layer "F.Cu")
-		(at 765.06 172.5 -90)
+		(at 438.08 97.63 -90)
 		(descr "100nF bypass on +5V, for U13 (2.5 V regulator)")
 		(tags "capacitor")
@@
 	(footprint "Resistor_SMD:R_0603_1608Metric"
 		(layer "F.Cu")
-		(at 763.25 176.76)
+		(at 436.27 101.89)
 		(descr "31.6k resistor from FB+2V5 to GND, for U13 (2.5 V regulator): feedback divider, sets the regulator's output voltage")
 		(tags "resistor")
@@
 	(footprint "EasyEDA:IND-SMD_L4.0-W4.0_SNR4018"
 		(layer "F.Cu")
-		(at 763.25 168.76 -90)
+		(at 436.27 93.89 -90)
 		(descr "2.2uH SRN4018-2R2M inductor between +2V5 and SW+2V5, for U13 (2.5 V regulator): regulator switching node")
 		(property "Reference" "L4"
@@
 	(footprint "EasyEDA:SOT-563_L1.6-W1.2-P0.50-LS1.6-BL"
 		(layer "F.Cu")
-		(at 763.25 172.5)
+		(at 436.27 97.63)
 		(descr "2.5 V regulator: TI TLV62569, 2 A switching regulator: +5V to +2V5.")
 		(property "Reference" "U13"
@@
 	(footprint "Resistor_SMD:R_0603_1608Metric"
 		(layer "F.Cu")
-		(at 763.55 174.75 180)
+		(at 436.57 99.88 180)
 		(descr "100k resistor from FB+2V5 to +2V5, for U13 (2.5 V regulator): feedback divider, sets the regulator's output voltage")
 		(tags "resistor")
@@
 	(footprint "Capacitor_SMD:C_0603_1608Metric"
 		(layer "F.Cu")
-		(at 63.555 254.296231)
+		(at 441.28 97.63 -90)
 		(descr "4.7uF bypass on +5V, for U13 (2.5 V regulator)")
 		(tags "capacitor")
 		(property "Reference" "C268"
-			(at 0 -1.43 0)
+			(at 0 -1.43 270)
 			(layer "F.Fab")
 			(effects
@@
 		)
 		(property "Value" "4.7uF"
-			(at 0 1.43 0)
+			(at 0 1.43 270)
 			(layer "F.Fab")
 			(effects
@@
 		)
 		(property "Datasheet" ""
-			(at 0 0 0)
+			(at 0 0 270)
 			(layer "F.Fab")
 			(hide yes)
@@
 		)
 		(property "Description" "4.7uF bypass on +5V, for U13 (2.5 V regulator)"
-			(at 0 0 0)
+			(at 0 0 270)
 			(layer "F.Fab")
 			(hide yes)
@@
 		)
 		(property "LCSC Part" "C277476"
-			(at 0 0 0)
+			(at 0 0 270)
 			(layer "F.SilkS")
 			(hide yes)
@@
 		)
 		(fp_text user "${REFERENCE}"
-			(at 0 0 0)
+			(at 0 0 270)
 			(layer "F.Fab")
 			(effects
@@
 		)
 		(pad "1" smd roundrect
-			(at -0.775 0)
+			(at -0.775 0 270)
 			(size 0.9 0.95)
 			(layers "F.Cu" "F.Mask" "F.Paste")
@@
 		)
 		(pad "2" smd roundrect
-			(at 0.775 0)
+			(at 0.775 0 270)
 			(size 0.9 0.95)
 			(layers "F.Cu" "F.Mask" "F.Paste")
@@
 	(footprint "Resistor_SMD:R_0603_1608Metric"
 		(layer "F.Cu")
-		(at 766.25 169.5 90)
+		(at 439.27 94.63 90)
 		(descr "100k pull-down on EN_2V5, for U7 (board controller): keeps the regulator off until the board controller enables it")
 		(tags "resistor")
@@
 	)
 	(gr_rect
-		(start 756.975 165.01)
-		(end 768.505 179.015)
-		(stroke
-			(width 0.15)
-			(type dash)
-		)
-		(fill no)
-		(layer "Cmts.User")
-	)
-	(gr_rect
-		(start 756.975 159.87)
-		(end 768.505 165.01)
-		(stroke
-			(width 0.15)
-			(type solid)
-		)
-		(fill no)
-		(layer "Cmts.User")
-	)
-	(gr_text "island U13"
-		(at 757.375 161.47 0)
-		(layer "Cmts.User")
-		(effects
-			(font
-				(size 1.2 1.2)
-				(thickness 0.18)
-			)
-			(justify left bottom)
-		)
-	)
-	(gr_text "2.5 V regulator\nTLV62569, 8 parts,\n2026-10-28"
-		(at 757.375 161.77 0)
-		(layer "Cmts.User")
-		(effects
-			(font
-				(size 0.7 0.7)
-				(thickness 0.105)
-			)
-			(justify left top)
-		)
-	)
-	(group "island U13"
-		(members
-			"b6b0a615-9e1d-4952-b0be-48a850f9bb0b"
-			"8bd45acc-f8e7-4368-b85d-5e29d826261a"
-			"6b29b62a-30ae-41ea-82d3-c41f851dde41"
-			"a8b18a00-bce7-471c-8832-c25f3648f47b"
-			"b37c7b10-e8ff-4e53-949d-2f72ec9fc3d6"
-			"08348b48-d6ef-47ea-b841-61e06e7f39f0"
-			"219e62ee-73f8-4a08-b77d-90547f89d37e"
-			"57221796-1b05-4fba-8462-ff18f253ed6d"
-			"925090ba-b620-407c-831d-7e7777c49897"
-			"cd2301e4-cb4c-43f9-bc2b-d4bf17629c76"
-			"582d39f3-7ee3-4316-81e0-d71b51cae9ec"
-			"f557c550-ca8d-4ebd-b559-fa7b50cb79d9"
-		)
-	)
-	(gr_rect
 		(start 695.145 52.115)
 		(end 716.22 66.335)
@@
 		)
 	)
+	(gr_rect
+		(start 429.995 90.14)
+		(end 443.535 104.145)
+		(stroke
+			(width 0.15)
+			(type dash)
+		)
+		(fill no)
+		(layer "Cmts.User")
+	)
+	(gr_rect
+		(start 429.995 85)
+		(end 443.535 90.14)
+		(stroke
+			(width 0.15)
+			(type solid)
+		)
+		(fill no)
+		(layer "Cmts.User")
+	)
+	(gr_text "island U13"
+		(at 430.395 86.6 0)
+		(layer "Cmts.User")
+		(effects
+			(font
+				(size 1.2 1.2)
+				(thickness 0.18)
+			)
+			(justify left bottom)
+		)
+	)
+	(gr_text "2.5 V regulator\nTLV62569, 9 parts,\n2026-10-29"
+		(at 430.395 86.9 0)
+		(layer "Cmts.User")
+		(effects
+			(font
+				(size 0.7 0.7)
+				(thickness 0.105)
+			)
+			(justify left top)
+		)
+	)
+	(group "island U13"
+		(members
+			"0136ca49-bf21-40a5-93b0-d4f6f32814d2"
+			"0b5c8ed1-8a53-4712-ac8e-93fe6c8874db"
+			"29d8ef41-7870-4423-a2bb-45db0c44972b"
+			"f159fe56-361a-4c1f-97bc-85f7c93ead6a"
+			"b37c7b10-e8ff-4e53-949d-2f72ec9fc3d6"
+			"08348b48-d6ef-47ea-b841-61e06e7f39f0"
+			"219e62ee-73f8-4a08-b77d-90547f89d37e"
+			"57221796-1b05-4fba-8462-ff18f253ed6d"
+			"f2a2eb73-899c-4bf5-a46c-a727fe43b944"
+			"925090ba-b620-407c-831d-7e7777c49897"
+			"cd2301e4-cb4c-43f9-bc2b-d4bf17629c76"
+			"582d39f3-7ee3-4316-81e0-d71b51cae9ec"
+			"f557c550-ca8d-4ebd-b559-fa7b50cb79d9"
+		)
+	)
