File: kicad/odin.kicad_pcb (KiCad board)
At the start: 8 copper layers, 100 x 100 mm, 544 parts, among them J1 USB-C, J19 2.54-2*3P, J2 FPGA JTAG, J20 2.54-2*3P, J3 WingTAT 2044-2X32G00SA, J5 WingTAT 2044-2X32G00SA, J50 9-21V POWER IN, J51 CTRL SWD, J52 PZ254V-11-02P, J53 XFCN PM254V-11-07-H85, J54 XFCN PM254V-11-07-H85, J55 XFCN PM254V-11-07-H85, J56 XFCN PM254V-11-07-H85, J57 XFCN PM254V-11-07-H85, J58 XFCN PM254V-11-07-H85, J62 XFCN PM254V-11-07-H85, J63 XFCN PM254V-11-07-H85, J64 XFCN PM254V-11-07-H85, J65 XFCN PM254V-11-07-H85, J68 AUX IN 9-28V UNREGULATED, J7 PM254-2-08-Z-8.5, J70 ETH, J71 LINK P, J72 LINK Q, J73 HDMI OUT, J74 microSD, J8 PM254-2-08-Z-8.5, Q3 BSS138LT1G, Q4 BSS138LT1G, SW1 CTRL BOOT, U1 XC7A100T-2FGG676I, U10 SN74LXC8T245PWR, U11 AP63300WU-7, U12 AP63300WU-7, U13 TLV62569DRLR, U14 TLV62569DRLR, U15 SY8047QDC, U16 TLV62569DRLR, U17 PCF8574T_3,518, U18 CH224K, U2 APS6404L-SQN-SN, U20 SN74CB3Q3384APWR, U21 TPS22950CDDCR, U22 TPS22950CDDCR, U23 TPS22953DSQR, U24 TPS22953DSQR, U26 TPS259470ARPWR, U3 APS6404L-SQN-SN, U30 RTL8211FD-CG, U31 TPD12S016PWR, U32 W9825G6KH-6, U33 MR25H10CDF, U34 TPS2121RUXR, U4 APS6404L-SQN-SN, U5 APS6404L-SQN-SN, U6 W25Q256JVEIQ, U7 RP2350B, U8 W25Q32JVZP, U9 SN74LXC8T245PWR, X3 25MHz 12pF, X4 50MHz CMOS, Y1 12MHz ABM8-272-T3

Commit message: Island U14 extended: the 4.7 uF input capacitor
Parts:
- moved C269 390.1 mm to (436.5, 122.0), turned to 180 degrees
- moved C201 347.0 mm to (434.5, 115.3)
- moved C202 347.0 mm to (436.8, 115.3)
- moved C203 347.0 mm to (436.5, 120.2)
- moved L5 347.0 mm to (440.3, 118.4)
- moved R61 347.0 mm to (434.3, 118.7)
- moved R62 347.0 mm to (432.3, 118.4)
- moved U14 347.0 mm to (436.5, 118.4)
Other:
- board text added: "1.8 V regulator, always on TLV62569, 8 parts, 2026-10-29"
- board text removed: "1.8 V regulator, always on 1.8 V regulator TLV62569, 8 parts, 2026-10-28"
Changed lines of the file:
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@@
 	(footprint "Capacitor_SMD:C_0603_1608Metric"
 		(layer "F.Cu")
-		(at 69.565 254.296231)
+		(at 436.52 121.95 180)
 		(descr "4.7uF bypass on +5V, for U14 (1.8 V regulator, always on)")
 		(tags "capacitor")
 		(property "Reference" "C269"
-			(at 0 -1.43 0)
+			(at 0 -1.43 180)
 			(layer "F.Fab")
 			(effects
@@
 		)
 		(property "Value" "4.7uF"
-			(at 0 1.43 0)
+			(at 0 1.43 180)
 			(layer "F.Fab")
 			(effects
@@
 		)
 		(property "Datasheet" ""
-			(at 0 0 0)
+			(at 0 0 180)
 			(layer "F.Fab")
 			(hide yes)
@@
 		)
 		(property "Description" "4.7uF bypass on +5V, for U14 (1.8 V regulator, always on)"
-			(at 0 0 0)
+			(at 0 0 180)
 			(layer "F.Fab")
 			(hide yes)
@@
 		)
 		(property "LCSC Part" "C277476"
-			(at 0 0 0)
+			(at 0 0 180)
 			(layer "F.SilkS")
 			(hide yes)
@@
 		)
 		(fp_text user "${REFERENCE}"
-			(at 0 0 0)
+			(at 0 0 180)
 			(layer "F.Fab")
 			(effects
@@
 		)
 		(pad "1" smd roundrect
-			(at -0.775 0)
+			(at -0.775 0 180)
 			(size 0.9 0.95)
 			(layers "F.Cu" "F.Mask" "F.Paste")
@@
 		)
 		(pad "2" smd roundrect
-			(at 0.775 0)
+			(at 0.775 0 180)
 			(size 0.9 0.95)
 			(layers "F.Cu" "F.Mask" "F.Paste")
@@
 	(footprint "Resistor_SMD:R_0603_1608Metric"
 		(layer "F.Cu")
-		(at 777.92 87.54 -90)
+		(at 432.26 118.4 -90)
 		(descr "49.9k resistor from FB+1V8_IO to GND, for U14 (1.8 V regulator, always on): feedback divider, sets the regulator's output voltage")
 		(tags "resistor")
@@
 	(footprint "Capacitor_SMD:C_0402_1005Metric"
 		(layer "F.Cu")
-		(at 782.18 89.35 180)
+		(at 436.52 120.21 180)
 		(descr "100nF bypass on +5V, for U14 (1.8 V regulator, always on)")
 		(tags "capacitor")
@@
 	(footprint "EasyEDA:IND-SMD_L4.0-W4.0_SNR4018"
 		(layer "F.Cu")
-		(at 785.92 87.54 180)
+		(at 440.26 118.4 180)
 		(descr "2.2uH SRN4018-2R2M inductor between +1V8_IO and SW+1V8_IO, for U14 (1.8 V regulator, always on): regulator switching node")
 		(property "Reference" "L5"
@@
 	(footprint "Capacitor_SMD:C_0805_2012Metric"
 		(layer "F.Cu")
-		(at 782.43 84.49 90)
+		(at 436.77 115.35 90)
 		(descr "22uF bypass on +1V8_IO, for U14 (1.8 V regulator, always on)")
 		(tags "capacitor")
@@
 	(footprint "EasyEDA:SOT-563_L1.6-W1.2-P0.50-LS1.6-BL"
 		(layer "F.Cu")
-		(at 782.18 87.54 -90)
+		(at 436.52 118.4 -90)
 		(descr "1.8 V regulator, always on: TI TLV62569, 2 A switching regulator: +5V to +1V8_IO (bank 13, the 1.8 V memory) and, through FB1, +1V8 (VCCAUX, VCCADC). Enable tied to +5V.")
 		(property "Reference" "U14"
@@
 	(footprint "Resistor_SMD:R_0603_1608Metric"
 		(layer "F.Cu")
-		(at 779.93 87.84 90)
+		(at 434.27 118.7 90)
 		(descr "100k resistor from FB+1V8_IO to +1V8_IO, for U14 (1.8 V regulator, always on): feedback divider, sets the regulator's output voltage")
 		(tags "resistor")
@@
 	(footprint "Capacitor_SMD:C_0805_2012Metric"
 		(layer "F.Cu")
-		(at 780.13 84.49 90)
+		(at 434.47 115.35 90)
 		(descr "22uF bypass on +1V8_IO, for U14 (1.8 V regulator, always on)")
 		(tags "capacitor")
@@
 	)
 	(gr_rect
-		(start 775.665 81.265)
-		(end 789.67 91.335)
-		(stroke
-			(width 0.15)
-			(type dash)
-		)
-		(fill no)
-		(layer "Cmts.User")
-	)
-	(gr_rect
-		(start 775.665 74.165)
-		(end 789.67 81.265)
-		(stroke
-			(width 0.15)
-			(type solid)
-		)
-		(fill no)
-		(layer "Cmts.User")
-	)
-	(gr_text "island U14"
-		(at 776.065 75.765 0)
-		(layer "Cmts.User")
-		(effects
-			(font
-				(size 1.2 1.2)
-				(thickness 0.18)
-			)
-			(justify left bottom)
-		)
-	)
-	(gr_text "1.8 V regulator,\nalways on\n1.8 V regulator\nTLV62569, 8 parts,\n2026-10-28"
-		(at 776.065 76.065 0)
-		(layer "Cmts.User")
-		(effects
-			(font
-				(size 0.7 0.7)
-				(thickness 0.105)
-			)
-			(justify left top)
-		)
-	)
-	(group "island U14"
-		(members
-			"6a07ae00-706a-4219-93dd-1fec190cf255"
-			"63ba5a5f-7753-4702-b9da-3cbf58bf48ca"
-			"605c2f6f-14f0-4eb8-920f-aa596339bf69"
-			"25f0e123-b52b-403a-bda1-f9320308f37c"
-			"e9abddf8-9a6a-4882-b3d0-9a85aad20cdd"
-			"f058002e-a3b0-44e8-a322-d0452b14f0ad"
-			"bff78157-9261-4cda-8ab5-c3c58185e64b"
-			"5de2f7d2-4f6e-4a37-bdd3-4c680c1c12db"
-			"85cc78a3-424e-4237-b733-a5215797f1be"
-			"ee7acb1d-c22a-47cf-98ae-d0dae494d640"
-			"540c6eb6-cc5a-4827-8ff4-278616277863"
-		)
-	)
-	(gr_rect
 		(start 695.145 52.115)
 		(end 716.22 66.335)
@@
 		)
 	)
+	(gr_rect
+		(start 430.005 112.125)
+		(end 444.01 124.205)
+		(stroke
+			(width 0.15)
+			(type dash)
+		)
+		(fill no)
+		(layer "Cmts.User")
+	)
+	(gr_rect
+		(start 430.005 106.005)
+		(end 444.01 112.125)
+		(stroke
+			(width 0.15)
+			(type solid)
+		)
+		(fill no)
+		(layer "Cmts.User")
+	)
+	(gr_text "island U14"
+		(at 430.405 107.605 0)
+		(layer "Cmts.User")
+		(effects
+			(font
+				(size 1.2 1.2)
+				(thickness 0.18)
+			)
+			(justify left bottom)
+		)
+	)
+	(gr_text "1.8 V regulator,\nalways on\nTLV62569, 8 parts,\n2026-10-29"
+		(at 430.405 107.905 0)
+		(layer "Cmts.User")
+		(effects
+			(font
+				(size 0.7 0.7)
+				(thickness 0.105)
+			)
+			(justify left top)
+		)
+	)
+	(group "island U14"
+		(members
+			"78b83d2d-f574-46ff-80fa-209bbe5eda67"
+			"41c4d4a2-3586-4c0c-ac40-af28f2f70dc0"
+			"3912e848-cd43-47fa-9a6d-1a5ecb7411aa"
+			"d16efd7e-08db-4699-b051-372d326f0a44"
+			"e9abddf8-9a6a-4882-b3d0-9a85aad20cdd"
+			"f058002e-a3b0-44e8-a322-d0452b14f0ad"
+			"bff78157-9261-4cda-8ab5-c3c58185e64b"
+			"5de2f7d2-4f6e-4a37-bdd3-4c680c1c12db"
+			"0f71c881-1d17-4c5b-8bfc-633c4a7c0ed4"
+			"85cc78a3-424e-4237-b733-a5215797f1be"
+			"ee7acb1d-c22a-47cf-98ae-d0dae494d640"
+			"540c6eb6-cc5a-4827-8ff4-278616277863"
+		)
+	)

Commit message: Island U16 extended: the 4.7 uF input capacitor
Parts:
- moved C270 377.6 mm to (436.5, 143.4), turned to 180 degrees
- moved C204 315.6 mm to (435.4, 135.3)
- moved C206 315.6 mm to (436.5, 140.2)
- moved L6 315.6 mm to (440.3, 138.4)
- moved R63 315.6 mm to (434.3, 138.7)
- moved R64 315.6 mm to (432.3, 138.7)
- moved R93 315.6 mm to (439.5, 141.4)
- moved U16 315.6 mm to (436.5, 138.4)
- moved C205 315.6 mm to (433.2, 135.3)
Other:
- board text added: "1.2 V transceiver regulator TLV62569, 9 parts, 2026-10-29"
- board text removed: "1.2 V transceiver regulator TLV62569, 8 parts, 2026-10-28"
Changed lines of the file:
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@@
 	(footprint "Capacitor_SMD:C_0805_2012Metric"
 		(layer "F.Cu")
-		(at 746.61 83.03 90)
+		(at 435.37 135.35 90)
 		(descr "22uF bypass on +1V2_MGT, for U16 (1.2 V transceiver regulator)")
 		(tags "capacitor")
@@
 	(footprint "EasyEDA:IND-SMD_L4.0-W4.0_SNR4018"
 		(layer "F.Cu")
-		(at 751.5 86.08 180)
+		(at 440.26 138.4 180)
 		(descr "2.2uH SRN4018-2R2M inductor between +1V2_MGT and SW+1V2_MGT, for U16 (1.2 V transceiver regulator): regulator switching node")
 		(property "Reference" "L6"
@@
 	(footprint "Capacitor_SMD:C_0805_2012Metric"
 		(layer "F.Cu")
-		(at 744.41 83.03 90)
+		(at 433.17 135.35 90)
 		(descr "22uF bypass on +1V2_MGT, for U16 (1.2 V transceiver regulator)")
 		(tags "capacitor")
@@
 	(footprint "Capacitor_SMD:C_0402_1005Metric"
 		(layer "F.Cu")
-		(at 747.76 87.89 180)
+		(at 436.52 140.21 180)
 		(descr "100nF bypass on +5V, for U16 (1.2 V transceiver regulator)")
 		(tags "capacitor")
@@
 	(footprint "Resistor_SMD:R_0603_1608Metric"
 		(layer "F.Cu")
-		(at 745.51 86.38 90)
+		(at 434.27 138.7 90)
 		(descr "100k resistor from FB+1V2_MGT to +1V2_MGT, for U16 (1.2 V transceiver regulator): feedback divider, sets the regulator's output voltage")
 		(tags "resistor")
@@
 	(footprint "Resistor_SMD:R_0603_1608Metric"
 		(layer "F.Cu")
-		(at 743.5 86.38 -90)
+		(at 432.26 138.7 -90)
 		(descr "100k resistor from FB+1V2_MGT to GND, for U16 (1.2 V transceiver regulator): feedback divider, sets the regulator's output voltage")
 		(tags "resistor")
@@
 	(footprint "Resistor_SMD:R_0603_1608Metric"
 		(layer "F.Cu")
-		(at 750.76 89.08)
+		(at 439.52 141.4)
 		(descr "100k pull-down on EN_1V2, for U7 (board controller): keeps the regulator off until the board controller enables it")
 		(tags "resistor")
@@
 	(footprint "Capacitor_SMD:C_0603_1608Metric"
 		(layer "F.Cu")
-		(at 75.575 254.296231)
+		(at 436.52 143.41 180)
 		(descr "4.7uF bypass on +5V, for U16 (1.2 V transceiver regulator)")
 		(tags "capacitor")
 		(property "Reference" "C270"
-			(at 0 -1.43 0)
+			(at 0 -1.43 180)
 			(layer "F.Fab")
 			(effects
@@
 		)
 		(property "Value" "4.7uF"
-			(at 0 1.43 0)
+			(at 0 1.43 180)
 			(layer "F.Fab")
 			(effects
@@
 		)
 		(property "Datasheet" ""
-			(at 0 0 0)
+			(at 0 0 180)
 			(layer "F.Fab")
 			(hide yes)
@@
 		)
 		(property "Description" "4.7uF bypass on +5V, for U16 (1.2 V transceiver regulator)"
-			(at 0 0 0)
+			(at 0 0 180)
 			(layer "F.Fab")
 			(hide yes)
@@
 		)
 		(property "LCSC Part" "C277476"
-			(at 0 0 0)
+			(at 0 0 180)
 			(layer "F.SilkS")
 			(hide yes)
@@
 		)
 		(fp_text user "${REFERENCE}"
-			(at 0 0 0)
+			(at 0 0 180)
 			(layer "F.Fab")
 			(effects
@@
 		)
 		(pad "1" smd roundrect
-			(at -0.775 0)
+			(at -0.775 0 180)
 			(size 0.9 0.95)
 			(layers "F.Cu" "F.Mask" "F.Paste")
@@
 		)
 		(pad "2" smd roundrect
-			(at 0.775 0)
+			(at 0.775 0 180)
 			(size 0.9 0.95)
 			(layers "F.Cu" "F.Mask" "F.Paste")
@@
 	(footprint "EasyEDA:SOT-563_L1.6-W1.2-P0.50-LS1.6-BL"
 		(layer "F.Cu")
-		(at 747.76 86.08 -90)
+		(at 436.52 138.4 -90)
 		(descr "1.2 V transceiver regulator: TI TLV62569, 2 A switching regulator: +5V to +1V2_MGT.")
 		(property "Reference" "U16"
@@
 	)
 	(gr_rect
-		(start 741.245 79.805)
-		(end 755.25 91.335)
-		(stroke
-			(width 0.15)
-			(type dash)
-		)
-		(fill no)
-		(layer "Cmts.User")
-	)
-	(gr_rect
-		(start 741.245 73.685)
-		(end 755.25 79.805)
-		(stroke
-			(width 0.15)
-			(type solid)
-		)
-		(fill no)
-		(layer "Cmts.User")
-	)
-	(gr_text "island U16"
-		(at 741.645 75.285 0)
-		(layer "Cmts.User")
-		(effects
-			(font
-				(size 1.2 1.2)
-				(thickness 0.18)
-			)
-			(justify left bottom)
-		)
-	)
-	(gr_text "1.2 V transceiver\nregulator\nTLV62569, 8 parts,\n2026-10-28"
-		(at 741.645 75.585 0)
-		(layer "Cmts.User")
-		(effects
-			(font
-				(size 0.7 0.7)
-				(thickness 0.105)
-			)
-			(justify left top)
-		)
-	)
-	(group "island U16"
-		(members
-			"69c71feb-6d36-4b9d-bebc-f05d86853d66"
-			"03369172-4a63-4bad-90c2-f1aff0f2087f"
-			"aa86688f-7f1b-4b5f-8d8f-30c0eb0932fe"
-			"43d2114b-a3ec-41ea-a187-18d37e0cba36"
-			"e2638f01-5ffb-478b-abe5-67696db0102d"
-			"1757b1c4-491c-48fb-809d-62eb3fef5cf5"
-			"195068e3-d978-40d0-b212-fb291953da9d"
-			"1aa9984c-545e-4178-904b-73bb1198bbc6"
-			"17fa6aba-c039-4e54-804e-99aa4caa5e85"
-			"2d6653bf-98f5-4a80-8440-6ab0204267d4"
-			"6cb09fb7-6628-4ada-aac5-e9f1e7d09939"
-			"8ac29be4-aed6-4af1-a5c5-4fb25bb1324f"
-		)
-	)
-	(gr_rect
 		(start 757.25 73.995)
 		(end 773.665 91.335)
@@
 		)
 	)
+	(gr_rect
+		(start 430.005 132.125)
+		(end 444.01 145.665)
+		(stroke
+			(width 0.15)
+			(type dash)
+		)
+		(fill no)
+		(layer "Cmts.User")
+	)
+	(gr_rect
+		(start 430.005 126.005)
+		(end 444.01 132.125)
+		(stroke
+			(width 0.15)
+			(type solid)
+		)
+		(fill no)
+		(layer "Cmts.User")
+	)
+	(gr_text "island U16"
+		(at 430.405 127.605 0)
+		(layer "Cmts.User")
+		(effects
+			(font
+				(size 1.2 1.2)
+				(thickness 0.18)
+			)
+			(justify left bottom)
+		)
+	)
+	(gr_text "1.2 V transceiver\nregulator\nTLV62569, 9 parts,\n2026-10-29"
+		(at 430.405 127.905 0)
+		(layer "Cmts.User")
+		(effects
+			(font
+				(size 0.7 0.7)
+				(thickness 0.105)
+			)
+			(justify left top)
+		)
+	)
+	(group "island U16"
+		(members
+			"d5505a49-32d0-42df-9cc1-eb2f1381bf72"
+			"5699eacb-d91b-4211-94bf-8a61f547d337"
+			"001b4532-74e9-4262-8062-95564de24358"
+			"359d232a-5831-4343-bf16-aa230deb9d9e"
+			"e2638f01-5ffb-478b-abe5-67696db0102d"
+			"1757b1c4-491c-48fb-809d-62eb3fef5cf5"
+			"195068e3-d978-40d0-b212-fb291953da9d"
+			"1aa9984c-545e-4178-904b-73bb1198bbc6"
+			"a650f6ee-41af-43cf-9670-55d989d2fdce"
+			"17fa6aba-c039-4e54-804e-99aa4caa5e85"
+			"2d6653bf-98f5-4a80-8440-6ab0204267d4"
+			"6cb09fb7-6628-4ada-aac5-e9f1e7d09939"
+			"8ac29be4-aed6-4af1-a5c5-4fb25bb1324f"
+		)
+	)

Commit message: Island U7 extended: USB series resistors and the two PIN V monitors
Parts:
- moved C277 422.4 mm to (458.6, 164.8)
- moved C278 418.6 mm to (458.6, 161.7)
- moved R170 418.3 mm to (443.5, 153.6), turned to -90 degrees
- moved R171 414.7 mm to (444.8, 153.6), turned to -90 degrees
- moved R198 412.5 mm to (459.2, 166.3), turned to 180 degrees
- moved R199 407.7 mm to (459.2, 163.3), turned to 180 degrees
- moved C116 363.6 mm to (435.8, 164.3)
- moved C120 363.6 mm to (435.8, 168.3)
- moved C129 363.6 mm to (435.8, 166.3)
- moved C125 363.6 mm to (441.9, 173.2)
- moved C127 363.6 mm to (443.1, 173.2)
- moved C130 363.6 mm to (445.1, 160.0)
- moved C131 363.6 mm to (445.5, 158.0)
- moved L1 363.6 mm to (445.5, 155.9)
- moved R10 363.6 mm to (449.2, 177.1)
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Other:
- board text added: "board controller RP2350, 50 parts, 2026-10-29"
- board text removed: "board controller RP2350, 46 parts, 2026-10-28 + Y1, U8"
