File: kicad/odin.kicad_pcb (KiCad board)
At the start: 8 copper layers, 100 x 100 mm, 544 parts, among them J1 USB-C, J19 2.54-2*3P, J2 FPGA JTAG, J20 2.54-2*3P, J3 WingTAT 2044-2X32G00SA, J5 WingTAT 2044-2X32G00SA, J50 9-21V POWER IN, J51 CTRL SWD, J52 PZ254V-11-02P, J53 XFCN PM254V-11-07-H85, J54 XFCN PM254V-11-07-H85, J55 XFCN PM254V-11-07-H85, J56 XFCN PM254V-11-07-H85, J57 XFCN PM254V-11-07-H85, J58 XFCN PM254V-11-07-H85, J62 XFCN PM254V-11-07-H85, J63 XFCN PM254V-11-07-H85, J64 XFCN PM254V-11-07-H85, J65 XFCN PM254V-11-07-H85, J68 AUX IN 9-28V UNREGULATED, J7 PM254-2-08-Z-8.5, J70 ETH, J71 LINK P, J72 LINK Q, J73 HDMI OUT, J74 microSD, J8 PM254-2-08-Z-8.5, Q3 BSS138LT1G, Q4 BSS138LT1G, SW1 CTRL BOOT, U1 XC7A100T-2FGG676I, U10 SN74LXC8T245PWR, U11 AP63300WU-7, U12 AP63300WU-7, U13 TLV62569DRLR, U14 TLV62569DRLR, U15 SY8047QDC, U16 TLV62569DRLR, U17 PCF8574T_3,518, U18 CH224K, U2 APS6404L-SQN-SN, U20 SN74CB3Q3384APWR, U21 TPS22950CDDCR, U22 TPS22950CDDCR, U23 TPS22953DSQR, U24 TPS22953DSQR, U26 TPS259470ARPWR, U3 APS6404L-SQN-SN, U30 RTL8211FD-CG, U31 TPD12S016PWR, U32 W9825G6KH-6, U33 MR25H10CDF, U34 TPS2121RUXR, U4 APS6404L-SQN-SN, U5 APS6404L-SQN-SN, U6 W25Q256JVEIQ, U7 RP2350B, U8 W25Q32JVZP, U9 SN74LXC8T245PWR, X3 25MHz 12pF, X4 50MHz CMOS, Y1 12MHz ABM8-272-T3

Commit message: Island U2 extended: PSRAM0 power-up resistors
Parts:
- moved R176 425.0 mm to (444.3, 192.0)
- moved R177 412.0 mm to (438.9, 200.1), turned to -90 degrees
- moved R178 407.9 mm to (440.8, 200.1), turned to -90 degrees
- moved R179 403.2 mm to (438.9, 189.1), turned to 90 degrees
- moved R175 381.0 mm to (440.8, 189.1), turned to 90 degrees
- moved R174 377.6 mm to (433.0, 197.2)
- moved U2 277.1 mm to (439.9, 194.6)
- moved C111 277.1 mm to (435.9, 192.0)
Other:
- board text added: "PSRAM 0 generic, 8 parts, 2026-10-29"
- board text removed: "PSRAM 0 generic, 8 parts, 2026-10-28"
Changed lines of the file:
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@@
 	(footprint "Resistor_SMD:R_0603_1608Metric"
 		(layer "F.Cu")
-		(at 45.025 299.001231)
+		(at 440.76 200.14 -90)
 		(descr "10k pull-down on PSRAM0_IO2_MEM, for U2 (PSRAM 0): holds the line low from power-up until the FPGA drives it (APS6404L section 8)")
 		(tags "resistor")
 		(property "Reference" "R178"
-			(at 0 -1.43 0)
+			(at 0 -1.43 270)
 			(layer "F.Fab")
 			(effects
@@
 		)
 		(property "Value" "10k"
-			(at 0 1.43 0)
+			(at 0 1.43 270)
 			(layer "F.Fab")
 			(effects
@@
 		)
 		(property "Datasheet" ""
-			(at 0 0 0)
+			(at 0 0 270)
 			(layer "F.Fab")
 			(hide yes)
@@
 		)
 		(property "Description" "10k pull-down on PSRAM0_IO2_MEM, for U2 (PSRAM 0): holds the line low from power-up until the FPGA drives it (APS6404L section 8)"
-			(at 0 0 0)
+			(at 0 0 270)
 			(layer "F.Fab")
 			(hide yes)
@@
 		)
 		(fp_text user "${REFERENCE}"
-			(at 0 0 0)
+			(at 0 0 270)
 			(layer "F.Fab")
 			(effects
@@
 		)
 		(pad "1" smd roundrect
-			(at -0.825 0)
+			(at -0.825 0 270)
 			(size 0.8 0.95)
 			(layers "F.Cu" "F.Mask" "F.Paste")
@@
 		)
 		(pad "2" smd roundrect
-			(at 0.825 0)
+			(at 0.825 0 270)
 			(size 0.8 0.95)
 			(layers "F.Cu" "F.Mask" "F.Paste")
@@
 	(footprint "Resistor_SMD:R_0603_1608Metric"
 		(layer "F.Cu")
-		(at 63.005 272.746231)
+		(at 433 197.24)
 		(descr "10k pull-up of PSRAM0_CE_B_MEM to +1V8_IO, for U2 (PSRAM 0): CE# high and tracking VDD from power-up until the FPGA drives it (APS6404L section 8)")
 		(tags "resistor")
@@
 	(footprint "Resistor_SMD:R_0603_1608Metric"
 		(layer "F.Cu")
-		(at 33.005 299.001231)
+		(at 444.33 192.04)
 		(descr "10k pull-down on PSRAM0_IO0_MEM, for U2 (PSRAM 0): holds the line low from power-up until the FPGA drives it (APS6404L section 8)")
 		(tags "resistor")
@@
 	(footprint "EasyEDA:SOIC-8_L4.9-W3.9-P1.27-LS6.0-BL"
 		(layer "F.Cu")
-		(at 707.47 122.88)
+		(at 439.85 194.64)
 		(descr "PSRAM 0: AP Memory APS6404L-SQN, 64 Mbit (8 MB) QSPI pseudo-static RAM, 1.8 V, on bank 13.")
 		(property "Reference" "U2"
@@
 	(footprint "Resistor_SMD:R_0603_1608Metric"
 		(layer "F.Cu")
-		(at 51.035 299.001231)
+		(at 438.94 189.14 90)
 		(descr "10k pull-down on PSRAM0_IO3_MEM, for U2 (PSRAM 0): holds the line low from power-up until the FPGA drives it (APS6404L section 8)")
 		(tags "resistor")
 		(property "Reference" "R179"
-			(at 0 -1.43 0)
+			(at 0 -1.43 90)
 			(layer "F.Fab")
 			(effects
@@
 		)
 		(property "Value" "10k"
-			(at 0 1.43 0)
+			(at 0 1.43 90)
 			(layer "F.Fab")
 			(effects
@@
 		)
 		(property "Datasheet" ""
-			(at 0 0 0)
+			(at 0 0 90)
 			(layer "F.Fab")
 			(hide yes)
@@
 		)
 		(property "Description" "10k pull-down on PSRAM0_IO3_MEM, for U2 (PSRAM 0): holds the line low from power-up until the FPGA drives it (APS6404L section 8)"
-			(at 0 0 0)
+			(at 0 0 90)
 			(layer "F.Fab")
 			(hide yes)
@@
 		)
 		(fp_text user "${REFERENCE}"
-			(at 0 0 0)
+			(at 0 0 90)
 			(layer "F.Fab")
 			(effects
@@
 		)
 		(pad "1" smd roundrect
-			(at -0.825 0)
+			(at -0.825 0 90)
 			(size 0.8 0.95)
 			(layers "F.Cu" "F.Mask" "F.Paste")
@@
 		)
 		(pad "2" smd roundrect
-			(at 0.825 0)
+			(at 0.825 0 90)
 			(size 0.8 0.95)
 			(layers "F.Cu" "F.Mask" "F.Paste")
@@
 	(footprint "Resistor_SMD:R_0603_1608Metric"
 		(layer "F.Cu")
-		(at 69.015 272.746231)
+		(at 440.76 189.14 90)
 		(descr "10k pull-down on PSRAM0_SCK_MEM, for U2 (PSRAM 0): holds the line low from power-up until the FPGA drives it (APS6404L section 8)")
 		(tags "resistor")
 		(property "Reference" "R175"
-			(at 0 -1.43 0)
+			(at 0 -1.43 90)
 			(layer "F.Fab")
 			(effects
@@
 		)
 		(property "Value" "10k"
-			(at 0 1.43 0)
+			(at 0 1.43 90)
 			(layer "F.Fab")
 			(effects
@@
 		)
 		(property "Datasheet" ""
-			(at 0 0 0)
+			(at 0 0 90)
 			(layer "F.Fab")
 			(hide yes)
@@
 		)
 		(property "Description" "10k pull-down on PSRAM0_SCK_MEM, for U2 (PSRAM 0): holds the line low from power-up until the FPGA drives it (APS6404L section 8)"
-			(at 0 0 0)
+			(at 0 0 90)
 			(layer "F.Fab")
 			(hide yes)
@@
 		)
 		(fp_text user "${REFERENCE}"
-			(at 0 0 0)
+			(at 0 0 90)
 			(layer "F.Fab")
 			(effects
@@
 		)
 		(pad "1" smd roundrect
-			(at -0.825 0)
+			(at -0.825 0 90)
 			(size 0.8 0.95)
 			(layers "F.Cu" "F.Mask" "F.Paste")
@@
 		)
 		(pad "2" smd roundrect
-			(at 0.825 0)
+			(at 0.825 0 90)
 			(size 0.8 0.95)
 			(layers "F.Cu" "F.Mask" "F.Paste")
@@
 	(footprint "Resistor_SMD:R_0603_1608Metric"
 		(layer "F.Cu")
-		(at 39.015 299.001231)
+		(at 438.94 200.14 -90)
 		(descr "10k pull-down on PSRAM0_IO1_MEM, for U2 (PSRAM 0): holds the line low from power-up until the FPGA drives it (APS6404L section 8)")
 		(tags "resistor")
 		(property "Reference" "R177"
-			(at 0 -1.43 0)
+			(at 0 -1.43 270)
 			(layer "F.Fab")
 			(effects
@@
 		)
 		(property "Value" "10k"
-			(at 0 1.43 0)
+			(at 0 1.43 270)
 			(layer "F.Fab")
 			(effects
@@
 		)
 		(property "Datasheet" ""
-			(at 0 0 0)
+			(at 0 0 270)
 			(layer "F.Fab")
 			(hide yes)
@@
 		)
 		(property "Description" "10k pull-down on PSRAM0_IO1_MEM, for U2 (PSRAM 0): holds the line low from power-up until the FPGA drives it (APS6404L section 8)"
-			(at 0 0 0)
+			(at 0 0 270)
 			(layer "F.Fab")
 			(hide yes)
@@
 		)
 		(fp_text user "${REFERENCE}"
-			(at 0 0 0)
+			(at 0 0 270)
 			(layer "F.Fab")
 			(effects
@@
 		)
 		(pad "1" smd roundrect
-			(at -0.825 0)
+			(at -0.825 0 270)
 			(size 0.8 0.95)
 			(layers "F.Cu" "F.Mask" "F.Paste")
@@
 		)
 		(pad "2" smd roundrect
-			(at 0.825 0)
+			(at 0.825 0 270)
 			(size 0.8 0.95)
 			(layers "F.Cu" "F.Mask" "F.Paste")
@@
 	(footprint "Capacitor_SMD:C_0402_1005Metric"
 		(layer "F.Cu")
-		(at 703.56 120.28 180)
+		(at 435.94 192.04 180)
 		(descr "100nF bypass on +1V8_IO, for U2 (PSRAM 0)")
 		(tags "capacitor")
@@
 	)
 	(gr_rect
-		(start 701.125 115.475)
-		(end 713.855 130.295)
-		(stroke
-			(width 0.15)
-			(type dash)
-		)
-		(fill no)
-		(layer "Cmts.User")
-	)
-	(gr_rect
-		(start 701.125 110.335)
-		(end 713.855 115.475)
-		(stroke
-			(width 0.15)
-			(type solid)
-		)
-		(fill no)
-		(layer "Cmts.User")
-	)
-	(gr_text "island U2"
-		(at 701.525 111.935 0)
-		(layer "Cmts.User")
-		(effects
-			(font
-				(size 1.2 1.2)
-				(thickness 0.18)
-			)
-			(justify left bottom)
-		)
-	)
-	(gr_text "PSRAM 0\ngeneric, 8 parts,\n2026-10-28"
-		(at 701.525 112.235 0)
-		(layer "Cmts.User")
-		(effects
-			(font
-				(size 0.7 0.7)
-				(thickness 0.105)
-			)
-			(justify left top)
-		)
-	)
-	(group "island U2"
-		(members
-			"7aeaa9e5-4ad7-44d5-abf1-25c66b28ecd8"
-			"0e40387f-02d1-4d98-bf45-6b179dd8551a"
-			"150a3f17-1254-4195-8693-b3a535932668"
-			"164c5676-dd64-4efa-bc62-45e015bb5764"
-			"8e91f2a8-03e6-4c16-8f2f-6fe9fcac1738"
-			"f390e4ec-6974-43ef-9d13-d0c9888c8cea"
-			"ed64047a-1952-4ae7-ae8f-99b21441dc64"
-			"cad638fb-3869-41ef-aef5-645b41def464"
-			"a332ec8f-a074-4149-8ed9-874b8be45f14"
-			"a1b9d306-d00c-407d-8d4e-8e7ecca4a895"
-			"1bbc5ed2-bc6d-43ee-98a3-1cc6d89e2bf7"
-			"c48850c6-8f91-49de-99e9-35aaf12d6671"
-		)
-	)
-	(gr_rect
 		(start 731.925 97.495)
 		(end 788.075 157.865)
@@
 		)
 	)
+	(gr_rect
+		(start 429.995 186.135)
+		(end 447.335 203.145)
+		(stroke
+			(width 0.15)
+			(type dash)
+		)
+		(fill no)
+		(layer "Cmts.User")
+	)
+	(gr_rect
+		(start 429.995 180.995)
+		(end 447.335 186.135)
+		(stroke
+			(width 0.15)
+			(type solid)
+		)
+		(fill no)
+		(layer "Cmts.User")
+	)
+	(gr_text "island U2"
+		(at 430.395 182.595 0)
+		(layer "Cmts.User")
+		(effects
+			(font
+				(size 1.2 1.2)
+				(thickness 0.18)
+			)
+			(justify left bottom)
+		)
+	)
+	(gr_text "PSRAM 0\ngeneric, 8 parts,\n2026-10-29"
+		(at 430.395 182.895 0)
+		(layer "Cmts.User")
+		(effects
+			(font
+				(size 0.7 0.7)
+				(thickness 0.105)
+			)
+			(justify left top)
+		)
+	)
+	(group "island U2"
+		(members
+			"168fbd61-14f8-42cb-b73d-a4238791c0cc"
+			"28834dcb-98de-4ab4-b1d0-be2156829cc1"
+			"ef4b8281-d75d-4a78-b40f-35b2eae7f079"
+			"93d4eec5-ebf2-479b-b253-e7b0a530aae1"
+			"8e91f2a8-03e6-4c16-8f2f-6fe9fcac1738"
+			"f390e4ec-6974-43ef-9d13-d0c9888c8cea"
+			"54a818f8-24a9-4e40-9d68-aa9f67fd80a8"
+			"c46139b1-3b6f-454c-a48f-9270b3315529"
+			"59b88d46-6679-48ff-bae8-959618f865c6"
+			"e0c023ee-14ac-4127-b7a2-7768ec8c585d"
+			"3660f2c9-b7f4-47bd-80c0-d37c57ade2e1"
+			"98ed041d-d67b-41e6-9ee7-152f4c22d483"
+		)
+	)

Commit message: Island U3 extended: PSRAM1 power-up resistors
Parts:
- moved R181 387.3 mm to (440.8, 213.1), turned to 90 degrees
- moved R182 384.3 mm to (444.3, 216.1)
- moved R180 383.9 mm to (433.0, 221.2)
- moved R183 371.5 mm to (438.9, 224.2), turned to -90 degrees
- moved R184 367.4 mm to (440.8, 224.2), turned to -90 degrees
- moved R185 362.2 mm to (438.9, 213.1), turned to 90 degrees
- moved U3 291.4 mm to (439.9, 218.7)
- moved C112 291.4 mm to (435.9, 216.1)
Other:
- board text added: "PSRAM 1 generic, 8 parts, 2026-10-29"
- board text removed: "PSRAM 1 generic, 8 parts, 2026-10-28"
Changed lines of the file:
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@@
 	(footprint "Resistor_SMD:R_0603_1608Metric"
 		(layer "F.Cu")
-		(at 87.095 299.001231)
+		(at 438.94 213.14 90)
 		(descr "10k pull-down on PSRAM1_IO3_MEM, for U3 (PSRAM 1): holds the line low from power-up until the FPGA drives it (APS6404L section 8)")
 		(tags "resistor")
 		(property "Reference" "R185"
-			(at 0 -1.43 0)
+			(at 0 -1.43 90)
 			(layer "F.Fab")
 			(effects
@@
 		)
 		(property "Value" "10k"
-			(at 0 1.43 0)
+			(at 0 1.43 90)
 			(layer "F.Fab")
 			(effects
@@
 		)
 		(property "Datasheet" ""
-			(at 0 0 0)
+			(at 0 0 90)
 			(layer "F.Fab")
 			(hide yes)
@@
 		)
 		(property "Description" "10k pull-down on PSRAM1_IO3_MEM, for U3 (PSRAM 1): holds the line low from power-up until the FPGA drives it (APS6404L section 8)"
-			(at 0 0 0)
+			(at 0 0 90)
 			(layer "F.Fab")
 			(hide yes)
@@
 		)
 		(fp_text user "${REFERENCE}"
-			(at 0 0 0)
+			(at 0 0 90)
 			(layer "F.Fab")
 			(effects
@@
 		)
 		(pad "1" smd roundrect
-			(at -0.825 0)
+			(at -0.825 0 90)
 			(size 0.8 0.95)
 			(layers "F.Cu" "F.Mask" "F.Paste")
@@
 		)
 		(pad "2" smd roundrect
-			(at 0.825 0)
+			(at 0.825 0 90)
 			(size 0.8 0.95)
 			(layers "F.Cu" "F.Mask" "F.Paste")
@@
 	(footprint "Resistor_SMD:R_0603_1608Metric"
 		(layer "F.Cu")
-		(at 57.044999 299.001231)
+		(at 433 221.25)
 		(descr "10k pull-up of PSRAM1_CE_B_MEM to +1V8_IO, for U3 (PSRAM 1): CE# high and tracking VDD from power-up until the FPGA drives it (APS6404L section 8)")
 		(tags "resistor")
@@
 	(footprint "Resistor_SMD:R_0603_1608Metric"
 		(layer "F.Cu")
-		(at 63.054999 299.001231)
+		(at 440.76 213.14 90)
 		(descr "10k pull-down on PSRAM1_SCK_MEM, for U3 (PSRAM 1): holds the line low from power-up until the FPGA drives it (APS6404L section 8)")
 		(tags "resistor")
 		(property "Reference" "R181"
-			(at 0 -1.43 0)
+			(at 0 -1.43 90)
 			(layer "F.Fab")
 			(effects
@@
 		)
 		(property "Value" "10k"
-			(at 0 1.43 0)
+			(at 0 1.43 90)
 			(layer "F.Fab")
 			(effects
@@
 		)
 		(property "Datasheet" ""
-			(at 0 0 0)
+			(at 0 0 90)
 			(layer "F.Fab")
 			(hide yes)
@@
 		)
 		(property "Description" "10k pull-down on PSRAM1_SCK_MEM, for U3 (PSRAM 1): holds the line low from power-up until the FPGA drives it (APS6404L section 8)"
-			(at 0 0 0)
+			(at 0 0 90)
 			(layer "F.Fab")
 			(hide yes)
@@
 		)
 		(fp_text user "${REFERENCE}"
-			(at 0 0 0)
+			(at 0 0 90)
 			(layer "F.Fab")
 			(effects
@@
 		)
 		(pad "1" smd roundrect
-			(at -0.825 0)
+			(at -0.825 0 90)
 			(size 0.8 0.95)
 			(layers "F.Cu" "F.Mask" "F.Paste")
@@
 		)
 		(pad "2" smd roundrect
-			(at 0.825 0)
+			(at 0.825 0 90)
 			(size 0.8 0.95)
 			(layers "F.Cu" "F.Mask" "F.Paste")
@@
 	(footprint "EasyEDA:SOIC-8_L4.9-W3.9-P1.27-LS6.0-BL"
 		(layer "F.Cu")
-		(at 723.21 150.75)
+		(at 439.85 218.65)
 		(descr "PSRAM 1: AP Memory APS6404L-SQN, 8 MB QSPI RAM, 1.8 V, on bank 13.")
 		(property "Reference" "U3"
@@
 	(footprint "Capacitor_SMD:C_0402_1005Metric"
 		(layer "F.Cu")
-		(at 719.3 148.15 180)
+		(at 435.94 216.05 180)
 		(descr "100nF bypass on +1V8_IO, for U3 (PSRAM 1)")
 		(tags "capacitor")
@@
 	(footprint "Resistor_SMD:R_0603_1608Metric"
 		(layer "F.Cu")
-		(at 69.064999 299.001231)
+		(at 444.33 216.05)
 		(descr "10k pull-down on PSRAM1_IO0_MEM, for U3 (PSRAM 1): holds the line low from power-up until the FPGA drives it (APS6404L section 8)")
 		(tags "resistor")
@@
 	(footprint "Resistor_SMD:R_0603_1608Metric"
 		(layer "F.Cu")
-		(at 75.074999 299.001231)
+		(at 438.94 224.16 -90)
 		(descr "10k pull-down on PSRAM1_IO1_MEM, for U3 (PSRAM 1): holds the line low from power-up until the FPGA drives it (APS6404L section 8)")
 		(tags "resistor")
 		(property "Reference" "R183"
-			(at 0 -1.43 0)
+			(at 0 -1.43 270)
 			(layer "F.Fab")
 			(effects
@@
 		)
 		(property "Value" "10k"
-			(at 0 1.43 0)
+			(at 0 1.43 270)
 			(layer "F.Fab")
 			(effects
@@
 		)
 		(property "Datasheet" ""
-			(at 0 0 0)
+			(at 0 0 270)
 			(layer "F.Fab")
 			(hide yes)
@@
 		)
 		(property "Description" "10k pull-down on PSRAM1_IO1_MEM, for U3 (PSRAM 1): holds the line low from power-up until the FPGA drives it (APS6404L section 8)"
-			(at 0 0 0)
+			(at 0 0 270)
 			(layer "F.Fab")
 			(hide yes)
@@
 		)
 		(fp_text user "${REFERENCE}"
-			(at 0 0 0)
+			(at 0 0 270)
 			(layer "F.Fab")
 			(effects
@@
 		)
 		(pad "1" smd roundrect
-			(at -0.825 0)
+			(at -0.825 0 270)
 			(size 0.8 0.95)
 			(layers "F.Cu" "F.Mask" "F.Paste")
@@
 		)
 		(pad "2" smd roundrect
-			(at 0.825 0)
+			(at 0.825 0 270)
 			(size 0.8 0.95)
 			(layers "F.Cu" "F.Mask" "F.Paste")
@@
 	(footprint "Resistor_SMD:R_0603_1608Metric"
 		(layer "F.Cu")
-		(at 81.085 299.001231)
+		(at 440.76 224.16 -90)
 		(descr "10k pull-down on PSRAM1_IO2_MEM, for U3 (PSRAM 1): holds the line low from power-up until the FPGA drives it (APS6404L section 8)")
 		(tags "resistor")
 		(property "Reference" "R184"
-			(at 0 -1.43 0)
+			(at 0 -1.43 270)
 			(layer "F.Fab")
 			(effects
@@
 		)
 		(property "Value" "10k"
-			(at 0 1.43 0)
+			(at 0 1.43 270)
 			(layer "F.Fab")
 			(effects
@@
 		)
 		(property "Datasheet" ""
-			(at 0 0 0)
+			(at 0 0 270)
 			(layer "F.Fab")
 			(hide yes)
@@
 		)
 		(property "Description" "10k pull-down on PSRAM1_IO2_MEM, for U3 (PSRAM 1): holds the line low from power-up until the FPGA drives it (APS6404L section 8)"
-			(at 0 0 0)
+			(at 0 0 270)
 			(layer "F.Fab")
 			(hide yes)
@@
 		)
 		(fp_text user "${REFERENCE}"
-			(at 0 0 0)
+			(at 0 0 270)
 			(layer "F.Fab")
 			(effects
@@
 		)
 		(pad "1" smd roundrect
-			(at -0.825 0)
+			(at -0.825 0 270)
 			(size 0.8 0.95)
 			(layers "F.Cu" "F.Mask" "F.Paste")
@@
 		)
 		(pad "2" smd roundrect
-			(at 0.825 0)
+			(at 0.825 0 270)
 			(size 0.8 0.95)
 			(layers "F.Cu" "F.Mask" "F.Paste")
@@
 	)
 	(gr_rect
-		(start 716.865 143.335)
-		(end 729.595 158.165)
-		(stroke
-			(width 0.15)
-			(type dash)
-		)
-		(fill no)
-		(layer "Cmts.User")
-	)
-	(gr_rect
-		(start 716.865 138.195)
-		(end 729.595 143.335)
-		(stroke
-			(width 0.15)
-			(type solid)
-		)
-		(fill no)
-		(layer "Cmts.User")
-	)
-	(gr_text "island U3"
-		(at 717.265 139.795 0)
-		(layer "Cmts.User")
-		(effects
-			(font
-				(size 1.2 1.2)
-				(thickness 0.18)
-			)
-			(justify left bottom)
-		)
-	)
-	(gr_text "PSRAM 1\ngeneric, 8 parts,\n2026-10-28"
-		(at 717.265 140.095 0)
-		(layer "Cmts.User")
-		(effects
-			(font
-				(size 0.7 0.7)
-				(thickness 0.105)
-			)
-			(justify left top)
-		)
-	)
-	(group "island U3"
-		(members
-			"36b7b90c-3f9f-4271-91cd-469930f67028"
-			"f34b5ab2-83f0-41f2-b2ec-b4a3d8f81485"
-			"1719d0c2-1c45-4131-8c61-3c825a5a43b4"
-			"097e3d42-8ebc-40a1-8d10-345748b154df"
-			"45079f01-7912-47e5-9fb7-05cfe9238e77"
-			"45d712a4-5bab-40b0-9f7e-698dca3316dd"
-			"a8324be9-6967-4661-83e7-14d3dffaa36d"
-			"fdda04d7-8382-41a8-9ee9-784c9bd3229c"
-			"0fbd1e91-08c2-4eee-85ae-7ad9becd5010"
-			"e8789f12-d404-48b0-9d5a-a6381383d8b6"
-			"acff2393-1176-4757-9604-301f4ef8d73a"
-			"2a63769c-15d3-43d1-9719-71121cb0231f"
-		)
-	)
-	(gr_rect
 		(start 731.925 97.495)
 		(end 788.075 157.865)
@@
 		)
 	)
+	(gr_rect
+		(start 429.995 210.135)
+		(end 447.335 227.165)
+		(stroke
+			(width 0.15)
+			(type dash)
+		)
+		(fill no)
+		(layer "Cmts.User")
+	)
+	(gr_rect
+		(start 429.995 204.995)
+		(end 447.335 210.135)
+		(stroke
+			(width 0.15)
+			(type solid)
+		)
+		(fill no)
+		(layer "Cmts.User")
+	)
+	(gr_text "island U3"
+		(at 430.395 206.595 0)
+		(layer "Cmts.User")
+		(effects
+			(font
+				(size 1.2 1.2)
+				(thickness 0.18)
+			)
+			(justify left bottom)
+		)
+	)
+	(gr_text "PSRAM 1\ngeneric, 8 parts,\n2026-10-29"
+		(at 430.395 206.895 0)
+		(layer "Cmts.User")
+		(effects
+			(font
+				(size 0.7 0.7)
+				(thickness 0.105)
+			)
+			(justify left top)
+		)
+	)
+	(group "island U3"
+		(members
+			"8d906fbd-5f3d-42cc-97ae-8efe25c9eae6"
+			"7f16676c-7da7-4a9d-bbab-adfb8189b9fa"
+			"99b7319c-2876-4b05-ae32-60378f79eb42"
+			"a6f036fc-8542-40fe-a7ae-503c81bbd6ba"
+			"45079f01-7912-47e5-9fb7-05cfe9238e77"
+			"45d712a4-5bab-40b0-9f7e-698dca3316dd"
+			"3963bedc-d6b4-452c-8e42-194fd4a54a6a"
+			"3e310abd-6037-44fe-bc02-14b608ba415c"
+			"a7c4c890-a11d-41a4-93c3-24f7cb6adeb3"
+			"d18447b6-6d37-44c4-bb1b-05d4ff8e1ce2"
+			"f03525fe-d514-47e0-a114-be8752d58b1b"
+			"09c3b006-ad6f-42da-aad1-ce0a29abbb9d"
+		)
+	)
