File: kicad/odin.kicad_pcb (KiCad board)
At the start: 8 copper layers, 100 x 100 mm, 544 parts, among them J1 USB-C, J19 2.54-2*3P, J2 FPGA JTAG, J20 2.54-2*3P, J3 WingTAT 2044-2X32G00SA, J5 WingTAT 2044-2X32G00SA, J50 9-21V POWER IN, J51 CTRL SWD, J52 PZ254V-11-02P, J53 XFCN PM254V-11-07-H85, J54 XFCN PM254V-11-07-H85, J55 XFCN PM254V-11-07-H85, J56 XFCN PM254V-11-07-H85, J57 XFCN PM254V-11-07-H85, J58 XFCN PM254V-11-07-H85, J62 XFCN PM254V-11-07-H85, J63 XFCN PM254V-11-07-H85, J64 XFCN PM254V-11-07-H85, J65 XFCN PM254V-11-07-H85, J68 AUX IN 9-28V UNREGULATED, J7 PM254-2-08-Z-8.5, J70 ETH, J71 LINK P, J72 LINK Q, J73 HDMI OUT, J74 microSD, J8 PM254-2-08-Z-8.5, Q3 BSS138LT1G, Q4 BSS138LT1G, SW1 CTRL BOOT, U1 XC7A100T-2FGG676I, U10 SN74LXC8T245PWR, U11 AP63300WU-7, U12 AP63300WU-7, U13 TLV62569DRLR, U14 TLV62569DRLR, U15 SY8047QDC, U16 TLV62569DRLR, U17 PCF8574T_3,518, U18 CH224K, U2 APS6404L-SQN-SN, U20 SN74CB3Q3384APWR, U21 TPS22950CDDCR, U22 TPS22950CDDCR, U23 TPS22953DSQR, U24 TPS22953DSQR, U26 TPS259470ARPWR, U3 APS6404L-SQN-SN, U30 RTL8211FD-CG, U31 TPD12S016PWR, U32 W9825G6KH-6, U33 MR25H10CDF, U34 TPS2121RUXR, U4 APS6404L-SQN-SN, U5 APS6404L-SQN-SN, U6 W25Q256JVEIQ, U7 RP2350B, U8 W25Q32JVZP, U9 SN74LXC8T245PWR, X3 25MHz 12pF, X4 50MHz CMOS, Y1 12MHz ABM8-272-T3

Commit message: Island U4 extended: PSRAM2 power-up resistors
Parts:
- moved R187 347.2 mm to (440.8, 237.1), turned to 90 degrees
- moved R188 344.3 mm to (444.3, 240.0)
- moved R186 344.1 mm to (433.0, 245.2)
- moved R189 331.7 mm to (438.9, 248.2), turned to -90 degrees
- moved C113 328.5 mm to (435.9, 240.0)
- moved U4 328.5 mm to (439.9, 242.6)
- moved R190 327.6 mm to (440.8, 248.2), turned to -90 degrees
- moved R191 321.8 mm to (438.9, 237.1), turned to 90 degrees
Other:
- board text added: "PSRAM 2 generic, 8 parts, 2026-10-29"
- board text removed: "PSRAM 2 generic, 8 parts, 2026-10-28"
Changed lines of the file:
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@@
 	(footprint "EasyEDA:SOIC-8_L4.9-W3.9-P1.27-LS6.0-BL"
 		(layer "F.Cu")
-		(at 725.31 80.15)
+		(at 439.85 242.64)
 		(descr "PSRAM 2: AP Memory APS6404L-SQN, 8 MB QSPI RAM, 1.8 V, on bank 13.")
 		(property "Reference" "U4"
@@
 	(footprint "Resistor_SMD:R_0603_1608Metric"
 		(layer "F.Cu")
-		(at 123.155 299.001231)
+		(at 438.94 237.14 90)
 		(descr "10k pull-down on PSRAM2_IO3_MEM, for U4 (PSRAM 2): holds the line low from power-up until the FPGA drives it (APS6404L section 8)")
 		(tags "resistor")
 		(property "Reference" "R191"
-			(at 0 -1.43 0)
+			(at 0 -1.43 90)
 			(layer "F.Fab")
 			(effects
@@
 		)
 		(property "Value" "10k"
-			(at 0 1.43 0)
+			(at 0 1.43 90)
 			(layer "F.Fab")
 			(effects
@@
 		)
 		(property "Datasheet" ""
-			(at 0 0 0)
+			(at 0 0 90)
 			(layer "F.Fab")
 			(hide yes)
@@
 		)
 		(property "Description" "10k pull-down on PSRAM2_IO3_MEM, for U4 (PSRAM 2): holds the line low from power-up until the FPGA drives it (APS6404L section 8)"
-			(at 0 0 0)
+			(at 0 0 90)
 			(layer "F.Fab")
 			(hide yes)
@@
 		)
 		(fp_text user "${REFERENCE}"
-			(at 0 0 0)
+			(at 0 0 90)
 			(layer "F.Fab")
 			(effects
@@
 		)
 		(pad "1" smd roundrect
-			(at -0.825 0)
+			(at -0.825 0 90)
 			(size 0.8 0.95)
 			(layers "F.Cu" "F.Mask" "F.Paste")
@@
 		)
 		(pad "2" smd roundrect
-			(at 0.825 0)
+			(at 0.825 0 90)
 			(size 0.8 0.95)
 			(layers "F.Cu" "F.Mask" "F.Paste")
@@
 	(footprint "Resistor_SMD:R_0603_1608Metric"
 		(layer "F.Cu")
-		(at 99.115 299.001231)
+		(at 440.75 237.14 90)
 		(descr "10k pull-down on PSRAM2_SCK_MEM, for U4 (PSRAM 2): holds the line low from power-up until the FPGA drives it (APS6404L section 8)")
 		(tags "resistor")
 		(property "Reference" "R187"
-			(at 0 -1.43 0)
+			(at 0 -1.43 90)
 			(layer "F.Fab")
 			(effects
@@
 		)
 		(property "Value" "10k"
-			(at 0 1.43 0)
+			(at 0 1.43 90)
 			(layer "F.Fab")
 			(effects
@@
 		)
 		(property "Datasheet" ""
-			(at 0 0 0)
+			(at 0 0 90)
 			(layer "F.Fab")
 			(hide yes)
@@
 		)
 		(property "Description" "10k pull-down on PSRAM2_SCK_MEM, for U4 (PSRAM 2): holds the line low from power-up until the FPGA drives it (APS6404L section 8)"
-			(at 0 0 0)
+			(at 0 0 90)
 			(layer "F.Fab")
 			(hide yes)
@@
 		)
 		(fp_text user "${REFERENCE}"
-			(at 0 0 0)
+			(at 0 0 90)
 			(layer "F.Fab")
 			(effects
@@
 		)
 		(pad "1" smd roundrect
-			(at -0.825 0)
+			(at -0.825 0 90)
 			(size 0.8 0.95)
 			(layers "F.Cu" "F.Mask" "F.Paste")
@@
 		)
 		(pad "2" smd roundrect
-			(at 0.825 0)
+			(at 0.825 0 90)
 			(size 0.8 0.95)
 			(layers "F.Cu" "F.Mask" "F.Paste")
@@
 	(footprint "Resistor_SMD:R_0603_1608Metric"
 		(layer "F.Cu")
-		(at 111.135 299.001231)
+		(at 438.94 248.15 -90)
 		(descr "10k pull-down on PSRAM2_IO1_MEM, for U4 (PSRAM 2): holds the line low from power-up until the FPGA drives it (APS6404L section 8)")
 		(tags "resistor")
 		(property "Reference" "R189"
-			(at 0 -1.43 0)
+			(at 0 -1.43 270)
 			(layer "F.Fab")
 			(effects
@@
 		)
 		(property "Value" "10k"
-			(at 0 1.43 0)
+			(at 0 1.43 270)
 			(layer "F.Fab")
 			(effects
@@
 		)
 		(property "Datasheet" ""
-			(at 0 0 0)
+			(at 0 0 270)
 			(layer "F.Fab")
 			(hide yes)
@@
 		)
 		(property "Description" "10k pull-down on PSRAM2_IO1_MEM, for U4 (PSRAM 2): holds the line low from power-up until the FPGA drives it (APS6404L section 8)"
-			(at 0 0 0)
+			(at 0 0 270)
 			(layer "F.Fab")
 			(hide yes)
@@
 		)
 		(fp_text user "${REFERENCE}"
-			(at 0 0 0)
+			(at 0 0 270)
 			(layer "F.Fab")
 			(effects
@@
 		)
 		(pad "1" smd roundrect
-			(at -0.825 0)
+			(at -0.825 0 270)
 			(size 0.8 0.95)
 			(layers "F.Cu" "F.Mask" "F.Paste")
@@
 		)
 		(pad "2" smd roundrect
-			(at 0.825 0)
+			(at 0.825 0 270)
 			(size 0.8 0.95)
 			(layers "F.Cu" "F.Mask" "F.Paste")
@@
 	(footprint "Resistor_SMD:R_0603_1608Metric"
 		(layer "F.Cu")
-		(at 93.105 299.001231)
+		(at 433 245.24)
 		(descr "10k pull-up of PSRAM2_CE_B_MEM to +1V8_IO, for U4 (PSRAM 2): CE# high and tracking VDD from power-up until the FPGA drives it (APS6404L section 8)")
 		(tags "resistor")
@@
 	(footprint "Resistor_SMD:R_0603_1608Metric"
 		(layer "F.Cu")
-		(at 117.145 299.001231)
+		(at 440.75 248.15 -90)
 		(descr "10k pull-down on PSRAM2_IO2_MEM, for U4 (PSRAM 2): holds the line low from power-up until the FPGA drives it (APS6404L section 8)")
 		(tags "resistor")
 		(property "Reference" "R190"
-			(at 0 -1.43 0)
+			(at 0 -1.43 270)
 			(layer "F.Fab")
 			(effects
@@
 		)
 		(property "Value" "10k"
-			(at 0 1.43 0)
+			(at 0 1.43 270)
 			(layer "F.Fab")
 			(effects
@@
 		)
 		(property "Datasheet" ""
-			(at 0 0 0)
+			(at 0 0 270)
 			(layer "F.Fab")
 			(hide yes)
@@
 		)
 		(property "Description" "10k pull-down on PSRAM2_IO2_MEM, for U4 (PSRAM 2): holds the line low from power-up until the FPGA drives it (APS6404L section 8)"
-			(at 0 0 0)
+			(at 0 0 270)
 			(layer "F.Fab")
 			(hide yes)
@@
 		)
 		(fp_text user "${REFERENCE}"
-			(at 0 0 0)
+			(at 0 0 270)
 			(layer "F.Fab")
 			(effects
@@
 		)
 		(pad "1" smd roundrect
-			(at -0.825 0)
+			(at -0.825 0 270)
 			(size 0.8 0.95)
 			(layers "F.Cu" "F.Mask" "F.Paste")
@@
 		)
 		(pad "2" smd roundrect
-			(at 0.825 0)
+			(at 0.825 0 270)
 			(size 0.8 0.95)
 			(layers "F.Cu" "F.Mask" "F.Paste")
@@
 	(footprint "Capacitor_SMD:C_0402_1005Metric"
 		(layer "F.Cu")
-		(at 721.4 77.55 180)
+		(at 435.94 240.04 180)
 		(descr "100nF bypass on +1V8_IO, for U4 (PSRAM 2)")
 		(tags "capacitor")
@@
 	(footprint "Resistor_SMD:R_0603_1608Metric"
 		(layer "F.Cu")
-		(at 105.125 299.001231)
+		(at 444.33 240.04)
 		(descr "10k pull-down on PSRAM2_IO0_MEM, for U4 (PSRAM 2): holds the line low from power-up until the FPGA drives it (APS6404L section 8)")
 		(tags "resistor")
@@
 	)
 	(gr_rect
-		(start 718.965 72.745)
-		(end 731.695 87.565)
-		(stroke
-			(width 0.15)
-			(type dash)
-		)
-		(fill no)
-		(layer "Cmts.User")
-	)
-	(gr_rect
-		(start 718.965 67.605)
-		(end 731.695 72.745)
-		(stroke
-			(width 0.15)
-			(type solid)
-		)
-		(fill no)
-		(layer "Cmts.User")
-	)
-	(gr_text "island U4"
-		(at 719.365 69.205 0)
-		(layer "Cmts.User")
-		(effects
-			(font
-				(size 1.2 1.2)
-				(thickness 0.18)
-			)
-			(justify left bottom)
-		)
-	)
-	(gr_text "PSRAM 2\ngeneric, 8 parts,\n2026-10-28"
-		(at 719.365 69.505 0)
-		(layer "Cmts.User")
-		(effects
-			(font
-				(size 0.7 0.7)
-				(thickness 0.105)
-			)
-			(justify left top)
-		)
-	)
-	(group "island U4"
-		(members
-			"035430b6-38a9-4cc9-8077-50d94f6ccc25"
-			"3908bccd-3a88-4443-aadd-8807410e1a3b"
-			"f891e4e5-095a-4dbb-a7d1-7b45dc7927aa"
-			"62639d28-b422-48f7-bb12-5b05809368df"
-			"3dce851b-c1d7-423a-b9b5-e62e67b2e988"
-			"e4e95a77-c096-4aed-a275-ae91fdd11587"
-			"131d45e5-36a0-4e94-a774-f70f3f74d4b1"
-			"204f0825-35d5-461c-b29e-2f8c95a0da05"
-			"13197684-9de0-44b1-b733-4b802d2df35c"
-			"8b7698c7-8e23-4147-ab0f-02fbad9a4a77"
-			"34755f31-8f10-4ebb-bb2a-000c589898e9"
-			"d9f197ea-1b5a-40fe-8191-f3ad335885b0"
-		)
-	)
-	(gr_rect
 		(start 731.925 97.495)
 		(end 788.075 157.865)
@@
 		)
 	)
+	(gr_rect
+		(start 429.995 234.135)
+		(end 447.335 251.155)
+		(stroke
+			(width 0.15)
+			(type dash)
+		)
+		(fill no)
+		(layer "Cmts.User")
+	)
+	(gr_rect
+		(start 429.995 228.995)
+		(end 447.335 234.135)
+		(stroke
+			(width 0.15)
+			(type solid)
+		)
+		(fill no)
+		(layer "Cmts.User")
+	)
+	(gr_text "island U4"
+		(at 430.395 230.595 0)
+		(layer "Cmts.User")
+		(effects
+			(font
+				(size 1.2 1.2)
+				(thickness 0.18)
+			)
+			(justify left bottom)
+		)
+	)
+	(gr_text "PSRAM 2\ngeneric, 8 parts,\n2026-10-29"
+		(at 430.395 230.895 0)
+		(layer "Cmts.User")
+		(effects
+			(font
+				(size 0.7 0.7)
+				(thickness 0.105)
+			)
+			(justify left top)
+		)
+	)
+	(group "island U4"
+		(members
+			"35b3dc86-fd29-4c1a-bf81-de447bc89598"
+			"b7dd53cd-fa4f-483e-8069-e0ab49f2b5bb"
+			"44b5994b-551a-42bf-a447-bd870b5a6af1"
+			"fb274e93-d1e4-42a8-aa03-4c6a6a5f189f"
+			"3dce851b-c1d7-423a-b9b5-e62e67b2e988"
+			"e4e95a77-c096-4aed-a275-ae91fdd11587"
+			"c07240bd-76b4-40fa-84d6-4a4362e3409d"
+			"79d3b9ac-5d0d-4a95-8f81-52baa8b809a0"
+			"f8e7f2b8-3492-42e5-bdb0-1f5d50af927b"
+			"b5d6c43c-d692-4075-93a2-9cdc6aa9cce1"
+			"e2a3eac6-5993-45f0-b6fe-ba03931e37a5"
+			"646c4cac-24b3-48db-8a79-c432947de4f3"
+		)
+	)

Commit message: Island U5 extended: PSRAM3 power-up resistors
Parts:
- moved C114 327.1 mm to (435.9, 264.0)
- moved U5 327.1 mm to (439.9, 266.6)
- moved R193 307.9 mm to (440.8, 261.1), turned to 90 degrees
- moved R192 305.3 mm to (433.0, 269.2)
- moved R194 305.2 mm to (444.3, 264.0)
- moved R195 293.0 mm to (438.9, 272.1), turned to -90 degrees
- moved R196 288.8 mm to (440.8, 272.1), turned to -90 degrees
- moved R197 282.3 mm to (438.9, 261.1), turned to 90 degrees
Other:
- board text added: "PSRAM 3 generic, 8 parts, 2026-10-29"
- board text removed: "PSRAM 3 generic, 8 parts, 2026-10-28"
Changed lines of the file:
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@@
 	(footprint "Resistor_SMD:R_0603_1608Metric"
 		(layer "F.Cu")
-		(at 153.205 299.001231)
+		(at 440.76 272.14 -90)
 		(descr "10k pull-down on PSRAM3_IO2_MEM, for U5 (PSRAM 3): holds the line low from power-up until the FPGA drives it (APS6404L section 8)")
 		(tags "resistor")
 		(property "Reference" "R196"
-			(at 0 -1.43 0)
+			(at 0 -1.43 270)
 			(layer "F.Fab")
 			(effects
@@
 		)
 		(property "Value" "10k"
-			(at 0 1.43 0)
+			(at 0 1.43 270)
 			(layer "F.Fab")
 			(effects
@@
 		)
 		(property "Datasheet" ""
-			(at 0 0 0)
+			(at 0 0 270)
 			(layer "F.Fab")
 			(hide yes)
@@
 		)
 		(property "Description" "10k pull-down on PSRAM3_IO2_MEM, for U5 (PSRAM 3): holds the line low from power-up until the FPGA drives it (APS6404L section 8)"
-			(at 0 0 0)
+			(at 0 0 270)
 			(layer "F.Fab")
 			(hide yes)
@@
 		)
 		(fp_text user "${REFERENCE}"
-			(at 0 0 0)
+			(at 0 0 270)
 			(layer "F.Fab")
 			(effects
@@
 		)
 		(pad "1" smd roundrect
-			(at -0.825 0)
+			(at -0.825 0 270)
 			(size 0.8 0.95)
 			(layers "F.Cu" "F.Mask" "F.Paste")
@@
 		)
 		(pad "2" smd roundrect
-			(at 0.825 0)
+			(at 0.825 0 270)
 			(size 0.8 0.95)
 			(layers "F.Cu" "F.Mask" "F.Paste")
@@
 	(footprint "Resistor_SMD:R_0603_1608Metric"
 		(layer "F.Cu")
-		(at 129.165 299.001231)
+		(at 433.01 269.24)
 		(descr "10k pull-up of PSRAM3_CE_B_MEM to +1V8_IO, for U5 (PSRAM 3): CE# high and tracking VDD from power-up until the FPGA drives it (APS6404L section 8)")
 		(tags "resistor")
@@
 	(footprint "EasyEDA:SOIC-8_L4.9-W3.9-P1.27-LS6.0-BL"
 		(layer "F.Cu")
-		(at 722.91 102.68)
+		(at 439.86 266.64)
 		(descr "PSRAM 3: AP Memory APS6404L-SQN, 8 MB QSPI RAM, 1.8 V, on bank 13.")
 		(property "Reference" "U5"
@@
 	(footprint "Resistor_SMD:R_0603_1608Metric"
 		(layer "F.Cu")
-		(at 159.215 299.001231)
+		(at 438.95 261.14 90)
 		(descr "10k pull-down on PSRAM3_IO3_MEM, for U5 (PSRAM 3): holds the line low from power-up until the FPGA drives it (APS6404L section 8)")
 		(tags "resistor")
 		(property "Reference" "R197"
-			(at 0 -1.43 0)
+			(at 0 -1.43 90)
 			(layer "F.Fab")
 			(effects
@@
 		)
 		(property "Value" "10k"
-			(at 0 1.43 0)
+			(at 0 1.43 90)
 			(layer "F.Fab")
 			(effects
@@
 		)
 		(property "Datasheet" ""
-			(at 0 0 0)
+			(at 0 0 90)
 			(layer "F.Fab")
 			(hide yes)
@@
 		)
 		(property "Description" "10k pull-down on PSRAM3_IO3_MEM, for U5 (PSRAM 3): holds the line low from power-up until the FPGA drives it (APS6404L section 8)"
-			(at 0 0 0)
+			(at 0 0 90)
 			(layer "F.Fab")
 			(hide yes)
@@
 		)
 		(fp_text user "${REFERENCE}"
-			(at 0 0 0)
+			(at 0 0 90)
 			(layer "F.Fab")
 			(effects
@@
 		)
 		(pad "1" smd roundrect
-			(at -0.825 0)
+			(at -0.825 0 90)
 			(size 0.8 0.95)
 			(layers "F.Cu" "F.Mask" "F.Paste")
@@
 		)
 		(pad "2" smd roundrect
-			(at 0.825 0)
+			(at 0.825 0 90)
 			(size 0.8 0.95)
 			(layers "F.Cu" "F.Mask" "F.Paste")
@@
 	(footprint "Capacitor_SMD:C_0402_1005Metric"
 		(layer "F.Cu")
-		(at 719 100.08 180)
+		(at 435.95 264.04 180)
 		(descr "100nF bypass on +1V8_IO, for U5 (PSRAM 3)")
 		(tags "capacitor")
@@
 	(footprint "Resistor_SMD:R_0603_1608Metric"
 		(layer "F.Cu")
-		(at 135.175 299.001231)
+		(at 440.76 261.14 90)
 		(descr "10k pull-down on PSRAM3_SCK_MEM, for U5 (PSRAM 3): holds the line low from power-up until the FPGA drives it (APS6404L section 8)")
 		(tags "resistor")
 		(property "Reference" "R193"
-			(at 0 -1.43 0)
+			(at 0 -1.43 90)
 			(layer "F.Fab")
 			(effects
@@
 		)
 		(property "Value" "10k"
-			(at 0 1.43 0)
+			(at 0 1.43 90)
 			(layer "F.Fab")
 			(effects
@@
 		)
 		(property "Datasheet" ""
-			(at 0 0 0)
+			(at 0 0 90)
 			(layer "F.Fab")
 			(hide yes)
@@
 		)
 		(property "Description" "10k pull-down on PSRAM3_SCK_MEM, for U5 (PSRAM 3): holds the line low from power-up until the FPGA drives it (APS6404L section 8)"
-			(at 0 0 0)
+			(at 0 0 90)
 			(layer "F.Fab")
 			(hide yes)
@@
 		)
 		(fp_text user "${REFERENCE}"
-			(at 0 0 0)
+			(at 0 0 90)
 			(layer "F.Fab")
 			(effects
@@
 		)
 		(pad "1" smd roundrect
-			(at -0.825 0)
+			(at -0.825 0 90)
 			(size 0.8 0.95)
 			(layers "F.Cu" "F.Mask" "F.Paste")
@@
 		)
 		(pad "2" smd roundrect
-			(at 0.825 0)
+			(at 0.825 0 90)
 			(size 0.8 0.95)
 			(layers "F.Cu" "F.Mask" "F.Paste")
@@
 	(footprint "Resistor_SMD:R_0603_1608Metric"
 		(layer "F.Cu")
-		(at 141.185 299.001231)
+		(at 444.34 264.04)
 		(descr "10k pull-down on PSRAM3_IO0_MEM, for U5 (PSRAM 3): holds the line low from power-up until the FPGA drives it (APS6404L section 8)")
 		(tags "resistor")
@@
 	(footprint "Resistor_SMD:R_0603_1608Metric"
 		(layer "F.Cu")
-		(at 147.195 299.001231)
+		(at 438.95 272.14 -90)
 		(descr "10k pull-down on PSRAM3_IO1_MEM, for U5 (PSRAM 3): holds the line low from power-up until the FPGA drives it (APS6404L section 8)")
 		(tags "resistor")
 		(property "Reference" "R195"
-			(at 0 -1.43 0)
+			(at 0 -1.43 270)
 			(layer "F.Fab")
 			(effects
@@
 		)
 		(property "Value" "10k"
-			(at 0 1.43 0)
+			(at 0 1.43 270)
 			(layer "F.Fab")
 			(effects
@@
 		)
 		(property "Datasheet" ""
-			(at 0 0 0)
+			(at 0 0 270)
 			(layer "F.Fab")
 			(hide yes)
@@
 		)
 		(property "Description" "10k pull-down on PSRAM3_IO1_MEM, for U5 (PSRAM 3): holds the line low from power-up until the FPGA drives it (APS6404L section 8)"
-			(at 0 0 0)
+			(at 0 0 270)
 			(layer "F.Fab")
 			(hide yes)
@@
 		)
 		(fp_text user "${REFERENCE}"
-			(at 0 0 0)
+			(at 0 0 270)
 			(layer "F.Fab")
 			(effects
@@
 		)
 		(pad "1" smd roundrect
-			(at -0.825 0)
+			(at -0.825 0 270)
 			(size 0.8 0.95)
 			(layers "F.Cu" "F.Mask" "F.Paste")
@@
 		)
 		(pad "2" smd roundrect
-			(at 0.825 0)
+			(at 0.825 0 270)
 			(size 0.8 0.95)
 			(layers "F.Cu" "F.Mask" "F.Paste")
@@
 	)
 	(gr_rect
-		(start 716.565 95.265)
-		(end 729.295 110.095)
-		(stroke
-			(width 0.15)
-			(type dash)
-		)
-		(fill no)
-		(layer "Cmts.User")
-	)
-	(gr_rect
-		(start 716.565 90.125)
-		(end 729.295 95.265)
-		(stroke
-			(width 0.15)
-			(type solid)
-		)
-		(fill no)
-		(layer "Cmts.User")
-	)
-	(gr_text "island U5"
-		(at 716.965 91.725 0)
-		(layer "Cmts.User")
-		(effects
-			(font
-				(size 1.2 1.2)
-				(thickness 0.18)
-			)
-			(justify left bottom)
-		)
-	)
-	(gr_text "PSRAM 3\ngeneric, 8 parts,\n2026-10-28"
-		(at 716.965 92.025 0)
-		(layer "Cmts.User")
-		(effects
-			(font
-				(size 0.7 0.7)
-				(thickness 0.105)
-			)
-			(justify left top)
-		)
-	)
-	(group "island U5"
-		(members
-			"7fd655e2-f412-440b-866f-dccaf1754a88"
-			"54402d88-a103-4e48-af03-f2247d6fdd9e"
-			"c645a99d-253a-4610-84e4-af7d83be0d05"
-			"952f90ec-5ea1-4b83-b2db-ac3b38c91897"
-			"5cfe6412-6f61-49e9-b524-839ea70cdf54"
-			"7839cb45-0d13-405c-a442-93ecfdf0e79b"
-			"afebfd83-13f6-4080-b6a7-804e5e65e66c"
-			"9ac38606-231b-49e7-8a32-b731fa0be927"
-			"2d7e9207-deac-4c1e-b226-7409324ec759"
-			"54efd2ac-de25-4800-9290-4d723943f8eb"
-			"862040cd-ee75-4168-81e9-424223b4057d"
-			"983bf86a-7410-43a9-82b8-ade7983e5167"
-		)
-	)
-	(gr_rect
 		(start 731.925 97.495)
 		(end 788.075 157.865)
@@
 		)
 	)
+	(gr_rect
+		(start 430.005 258.135)
+		(end 447.345 275.145)
+		(stroke
+			(width 0.15)
+			(type dash)
+		)
+		(fill no)
+		(layer "Cmts.User")
+	)
+	(gr_rect
+		(start 430.005 252.995)
+		(end 447.345 258.135)
+		(stroke
+			(width 0.15)
+			(type solid)
+		)
+		(fill no)
+		(layer "Cmts.User")
+	)
+	(gr_text "island U5"
+		(at 430.405 254.595 0)
+		(layer "Cmts.User")
+		(effects
+			(font
+				(size 1.2 1.2)
+				(thickness 0.18)
+			)
+			(justify left bottom)
+		)
+	)
+	(gr_text "PSRAM 3\ngeneric, 8 parts,\n2026-10-29"
+		(at 430.405 254.895 0)
+		(layer "Cmts.User")
+		(effects
+			(font
+				(size 0.7 0.7)
+				(thickness 0.105)
+			)
+			(justify left top)
+		)
+	)
+	(group "island U5"
+		(members
+			"2ea553b0-9c3b-45f2-9f63-91b8a1531740"
+			"1b614cfa-f205-4f92-9488-228b239a847e"
+			"68ec764e-246a-4836-924e-e20b0153f5a2"
+			"49a771cf-6116-4844-9c79-44273e90c59f"
+			"5cfe6412-6f61-49e9-b524-839ea70cdf54"
+			"7839cb45-0d13-405c-a442-93ecfdf0e79b"
+			"5aa90a53-7c65-4e89-943c-767a9b268714"
+			"85faee0d-4182-4649-90a8-9bc81bb4c118"
+			"a11d9daf-9ea9-4b4f-a7a7-e4dbc07d32b0"
+			"f883e76b-115e-4199-9276-027a12a11221"
+			"02bbd1f3-4d29-486c-a661-67ebe91248fc"
+			"6307c238-c29f-46f1-aeca-c5015976db58"
+		)
+	)
