File: kicad/odin.kicad_pcb (KiCad board)
At the start: 8 copper layers, 100 x 100 mm, 544 parts, among them J1 USB-C, J19 2.54-2*3P, J2 FPGA JTAG, J20 2.54-2*3P, J3 WingTAT 2044-2X32G00SA, J5 WingTAT 2044-2X32G00SA, J50 9-21V POWER IN, J51 CTRL SWD, J52 PZ254V-11-02P, J53 XFCN PM254V-11-07-H85, J54 XFCN PM254V-11-07-H85, J55 XFCN PM254V-11-07-H85, J56 XFCN PM254V-11-07-H85, J57 XFCN PM254V-11-07-H85, J58 XFCN PM254V-11-07-H85, J62 XFCN PM254V-11-07-H85, J63 XFCN PM254V-11-07-H85, J64 XFCN PM254V-11-07-H85, J65 XFCN PM254V-11-07-H85, J68 AUX IN 9-28V UNREGULATED, J7 PM254-2-08-Z-8.5, J70 ETH, J71 LINK P, J72 LINK Q, J73 HDMI OUT, J74 microSD, J8 PM254-2-08-Z-8.5, Q3 BSS138LT1G, Q4 BSS138LT1G, SW1 CTRL BOOT, U1 XC7A100T-2FGG676I, U10 SN74LXC8T245PWR, U11 AP63300WU-7, U12 AP63300WU-7, U13 TLV62569DRLR, U14 TLV62569DRLR, U15 SY8047QDC, U16 TLV62569DRLR, U17 PCF8574T_3,518, U18 CH224K, U2 APS6404L-SQN-SN, U20 SN74CB3Q3384APWR, U21 TPS22950CDDCR, U22 TPS22950CDDCR, U23 TPS22953DSQR, U24 TPS22953DSQR, U26 TPS259470ARPWR, U3 APS6404L-SQN-SN, U30 RTL8211FD-CG, U31 TPD12S016PWR, U32 W9825G6KH-6, U33 MR25H10CDF, U34 TPS2121RUXR, U4 APS6404L-SQN-SN, U5 APS6404L-SQN-SN, U6 W25Q256JVEIQ, U7 RP2350B, U8 W25Q32JVZP, U9 SN74LXC8T245PWR, X3 25MHz 12pF, X4 50MHz CMOS, Y1 12MHz ABM8-272-T3

Commit message: Island U23 extended: TPS22953 bias, rise-time and output capacitors
Parts:
- moved C271 504.1 mm to (471.6, 25.2)
- moved C273 503.3 mm to (464.3, 28.5), turned to -90 degrees
- moved C272 496.6 mm to (464.1, 18.6), turned to 90 degrees
- moved R72 254.3 mm to (468.6, 24.3)
- moved C220 254.3 mm to (465.2, 21.5)
- moved U23 254.3 mm to (465.2, 25.2)
Other:
- board text added: "slots A-D PIN V switch TPS22953, 6 parts, 2026-10-29"
- board text removed: "slots A-D PIN V switch TPS22950, 4 parts, 2026-10-28"
Changed lines of the file:
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@@
 	(footprint "Package_DFN_QFN:Texas_DSQ0010A_WSON-10-1EP_2x2mm_P0.4mm_EP0.9x1.5mm"
 		(layer "F.Cu")
-		(at 706.54 105.21 180)
+		(at 465.16 25.19 180)
 		(descr "slots A-D PIN V switch: TI TPS22953 load switch, biased from +3V3 so it works at 1.8 V: VCCIO_1 to the PIN V pin of slots A-D. Blocks reverse current while off; the slot fuses limit the current.")
 		(tags "Texas WSON NoLead")
@@
 	(footprint "Capacitor_SMD:C_0603_1608Metric"
 		(layer "F.Cu")
-		(at 706.54 101.52 90)
+		(at 465.16 21.5 90)
 		(descr "1uF bypass on VCCIO_1, for U23 (slots A-D PIN V switch)")
 		(tags "capacitor")
@@
 	(footprint "Capacitor_SMD:C_0402_1005Metric"
 		(layer "F.Cu")
-		(at 37.5 272.746231)
+		(at 464.15 18.56 90)
 		(descr "1nF 50V filter capacitor on U23_CT, for U23 (slots A-D PIN V switch): sets how fast U23 ramps its output, about 1.5 ms (TPS22953 CT)")
 		(tags "capacitor")
 		(property "Reference" "C272"
-			(at 0 -1.16 0)
+			(at 0 -1.16 90)
 			(layer "F.Fab")
 			(effects
@@
 		)
 		(property "Value" "1nF 50V"
-			(at 0 1.16 0)
+			(at 0 1.16 90)
 			(layer "F.Fab")
 			(effects
@@
 		)
 		(property "Datasheet" ""
-			(at 0 0 0)
+			(at 0 0 90)
 			(layer "F.Fab")
 			(hide yes)
@@
 		)
 		(property "Description" "1nF 50V filter capacitor on U23_CT, for U23 (slots A-D PIN V switch): sets how fast U23 ramps its output, about 1.5 ms (TPS22953 CT)"
-			(at 0 0 0)
+			(at 0 0 90)
 			(layer "F.Fab")
 			(hide yes)
@@
 		)
 		(property "LCSC Part" "C1525"
-			(at 0 0 0)
+			(at 0 0 90)
 			(layer "F.SilkS")
 			(hide yes)
@@
 		)
 		(fp_text user "${REFERENCE}"
-			(at 0 0 0)
+			(at 0 0 90)
 			(layer "F.Fab")
 			(effects
@@
 		)
 		(pad "1" smd roundrect
-			(at -0.48 0)
+			(at -0.48 0 90)
 			(size 0.56 0.62)
 			(layers "F.Cu" "F.Mask" "F.Paste")
@@
 		)
 		(pad "2" smd roundrect
-			(at 0.48 0)
+			(at 0.48 0 90)
 			(size 0.56 0.62)
 			(layers "F.Cu" "F.Mask" "F.Paste")
@@
 	(footprint "Capacitor_SMD:C_0402_1005Metric"
 		(layer "F.Cu")
-		(at 32.5 272.746231)
+		(at 471.59 25.19)
 		(descr "100nF bypass on +3V3, for U23 (slots A-D PIN V switch)")
 		(tags "capacitor")
@@
 	(footprint "Capacitor_SMD:C_0603_1608Metric"
 		(layer "F.Cu")
-		(at 33.005 288.001231)
+		(at 464.26 28.47 -90)
 		(descr "1uF bypass on VCCIO_1_EXT, for U23 (slots A-D PIN V switch)")
 		(tags "capacitor")
 		(property "Reference" "C273"
-			(at 0 -1.43 0)
+			(at 0 -1.43 270)
 			(layer "F.Fab")
 			(effects
@@
 		)
 		(property "Value" "1uF"
-			(at 0 1.43 0)
+			(at 0 1.43 270)
 			(layer "F.Fab")
 			(effects
@@
 		)
 		(property "Datasheet" ""
-			(at 0 0 0)
+			(at 0 0 270)
 			(layer "F.Fab")
 			(hide yes)
@@
 		)
 		(property "Description" "1uF bypass on VCCIO_1_EXT, for U23 (slots A-D PIN V switch)"
-			(at 0 0 0)
+			(at 0 0 270)
 			(layer "F.Fab")
 			(hide yes)
@@
 		)
 		(property "LCSC Part" "C29936"
-			(at 0 0 0)
+			(at 0 0 270)
 			(layer "F.SilkS")
 			(hide yes)
@@
 		)
 		(fp_text user "${REFERENCE}"
-			(at 0 0 0)
+			(at 0 0 270)
 			(layer "F.Fab")
 			(effects
@@
 		)
 		(pad "1" smd roundrect
-			(at -0.775 0)
+			(at -0.775 0 270)
 			(size 0.9 0.95)
 			(layers "F.Cu" "F.Mask" "F.Paste")
@@
 		)
 		(pad "2" smd roundrect
-			(at 0.775 0)
+			(at 0.775 0 270)
 			(size 0.9 0.95)
 			(layers "F.Cu" "F.Mask" "F.Paste")
@@
 	(footprint "Resistor_SMD:R_0603_1608Metric"
 		(layer "F.Cu")
-		(at 710.03 104.28)
+		(at 468.65 24.26)
 		(descr "100k pull-down on EXT_EN, for U7 (board controller): from the board controller: turns extension power on; off by default")
 		(tags "resistor")
@@
 	)
 	(gr_rect
-		(start 703.385 98.515)
-		(end 714.385 107.985)
-		(stroke
-			(width 0.15)
-			(type dash)
-		)
-		(fill no)
-		(layer "Cmts.User")
-	)
-	(gr_rect
-		(start 703.385 92.395)
-		(end 714.385 98.515)
-		(stroke
-			(width 0.15)
-			(type solid)
-		)
-		(fill no)
-		(layer "Cmts.User")
-	)
-	(gr_text "island U23"
-		(at 703.785 93.995 0)
-		(layer "Cmts.User")
-		(effects
-			(font
-				(size 1.2 1.2)
-				(thickness 0.18)
-			)
-			(justify left bottom)
-		)
-	)
-	(gr_text "slots A-D PIN V\nswitch\nTPS22950, 4\nparts, 2026-10-28"
-		(at 703.785 94.295 0)
-		(layer "Cmts.User")
-		(effects
-			(font
-				(size 0.7 0.7)
-				(thickness 0.105)
-			)
-			(justify left top)
-		)
-	)
-	(group "island U23"
-		(members
-			"2ec31b6d-3e1a-4f5b-9ee5-697e3d86eea2"
-			"e4f251cd-8192-4adc-9342-8a98a1ade891"
-			"ebe0d239-9355-4ca0-80ad-a26210508172"
-			"35465a74-07d6-45de-9c83-caf430871a5b"
-			"293169d7-f977-4b02-b6c2-c5421c474f29"
-			"327ff684-8b3a-4f57-bb17-c1fb0e7a58aa"
-			"948fad0b-066d-45de-843b-20b2ee57c26d"
-		)
-	)
-	(gr_rect
 		(start 689.475 97.615)
 		(end 700.475 107.496)
@@
 		)
 	)
+	(gr_rect
+		(start 462.005 16.125)
+		(end 474.025 31.475)
+		(stroke
+			(width 0.15)
+			(type dash)
+		)
+		(fill no)
+		(layer "Cmts.User")
+	)
+	(gr_rect
+		(start 462.005 10.005)
+		(end 474.025 16.125)
+		(stroke
+			(width 0.15)
+			(type solid)
+		)
+		(fill no)
+		(layer "Cmts.User")
+	)
+	(gr_text "island U23"
+		(at 462.405 11.605 0)
+		(layer "Cmts.User")
+		(effects
+			(font
+				(size 1.2 1.2)
+				(thickness 0.18)
+			)
+			(justify left bottom)
+		)
+	)
+	(gr_text "slots A-D PIN V\nswitch\nTPS22953, 6 parts,\n2026-10-29"
+		(at 462.405 11.905 0)
+		(layer "Cmts.User")
+		(effects
+			(font
+				(size 0.7 0.7)
+				(thickness 0.105)
+			)
+			(justify left top)
+		)
+	)
+	(group "island U23"
+		(members
+			"f197ebef-c68e-414d-8b35-22419809fae9"
+			"a266e72e-b288-4adc-bd9d-c5ef3cad071a"
+			"4bb4b738-5eb1-416b-9502-571a75ed259e"
+			"fea2c0ce-7ea7-44a9-8819-895278c89e6f"
+			"293169d7-f977-4b02-b6c2-c5421c474f29"
+			"327ff684-8b3a-4f57-bb17-c1fb0e7a58aa"
+			"3a586a72-344b-4692-bd5c-0777e04c0ec0"
+			"362a86d8-645b-4b44-9b83-9f81d91f7ddf"
+			"932acc0c-fef3-4f4c-840a-fb3a374999bd"
+			"948fad0b-066d-45de-843b-20b2ee57c26d"
+		)
+	)

Commit message: Island U24 extended: TPS22953 bias, rise-time and output capacitors
Parts:
- moved C274 495.0 mm to (471.6, 48.2)
- moved C275 487.5 mm to (464.1, 41.6), turned to 90 degrees
- moved C276 477.9 mm to (464.2, 51.5), turned to -90 degrees
- moved C221 365.7 mm to (465.1, 44.5)
- moved R73 365.7 mm to (468.6, 49.1)
- moved U24 365.7 mm to (465.1, 48.2)
Other:
- board text added: "slots E-H PIN V switch TPS22953, 6 parts, 2026-10-29"
- board text removed: "slots E-H PIN V switch TPS22950, 4 parts, 2026-10-28"
Changed lines of the file:
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@@
 	(footprint "Capacitor_SMD:C_0402_1005Metric"
 		(layer "F.Cu")
-		(at 38.51 288.001231)
+		(at 471.58 48.19)
 		(descr "100nF bypass on +3V3, for U24 (slots E-H PIN V switch)")
 		(tags "capacitor")
@@
 	(footprint "Package_DFN_QFN:Texas_DSQ0010A_WSON-10-1EP_2x2mm_P0.4mm_EP0.9x1.5mm"
 		(layer "F.Cu")
-		(at 825.1 112.75 180)
+		(at 465.15 48.19 180)
 		(descr "slots E-H PIN V switch: TI TPS22953 load switch, biased from +3V3 so it works at 1.8 V: VCCIO_2 to the PIN V pin of slots E-H. Blocks reverse current while off; the slot fuses limit the current.")
 		(tags "Texas WSON NoLead")
@@
 	(footprint "Capacitor_SMD:C_0402_1005Metric"
 		(layer "F.Cu")
-		(at 43.51 288.001231)
+		(at 464.14 41.56 90)
 		(descr "1nF 50V filter capacitor on U24_CT, for U24 (slots E-H PIN V switch): sets how fast U24 ramps its output, about 1.5 ms (TPS22953 CT)")
 		(tags "capacitor")
 		(property "Reference" "C275"
-			(at 0 -1.16 0)
+			(at 0 -1.16 90)
 			(layer "F.Fab")
 			(effects
@@
 		)
 		(property "Value" "1nF 50V"
-			(at 0 1.16 0)
+			(at 0 1.16 90)
 			(layer "F.Fab")
 			(effects
@@
 		)
 		(property "Datasheet" ""
-			(at 0 0 0)
+			(at 0 0 90)
 			(layer "F.Fab")
 			(hide yes)
@@
 		)
 		(property "Description" "1nF 50V filter capacitor on U24_CT, for U24 (slots E-H PIN V switch): sets how fast U24 ramps its output, about 1.5 ms (TPS22953 CT)"
-			(at 0 0 0)
+			(at 0 0 90)
 			(layer "F.Fab")
 			(hide yes)
@@
 		)
 		(fp_text user "${REFERENCE}"
-			(at 0 0 0)
+			(at 0 0 90)
 			(layer "F.Fab")
 			(effects
@@
 		)
 		(pad "1" smd roundrect
-			(at -0.48 0)
+			(at -0.48 0 90)
 			(size 0.56 0.62)
 			(layers "F.Cu" "F.Mask" "F.Paste")
@@
 		)
 		(pad "2" smd roundrect
-			(at 0.48 0)
+			(at 0.48 0 90)
 			(size 0.56 0.62)
 			(layers "F.Cu" "F.Mask" "F.Paste")
@@
 	(footprint "Capacitor_SMD:C_0603_1608Metric"
 		(layer "F.Cu")
-		(at 49.015 288.001231)
+		(at 464.25 51.47 -90)
 		(descr "1uF bypass on VCCIO_2_EXT, for U24 (slots E-H PIN V switch)")
 		(tags "capacitor")
 		(property "Reference" "C276"
-			(at 0 -1.43 0)
+			(at 0 -1.43 270)
 			(layer "F.Fab")
 			(effects
@@
 		)
 		(property "Value" "1uF"
-			(at 0 1.43 0)
+			(at 0 1.43 270)
 			(layer "F.Fab")
 			(effects
@@
 		)
 		(property "Datasheet" ""
-			(at 0 0 0)
+			(at 0 0 270)
 			(layer "F.Fab")
 			(hide yes)
@@
 		)
 		(property "Description" "1uF bypass on VCCIO_2_EXT, for U24 (slots E-H PIN V switch)"
-			(at 0 0 0)
+			(at 0 0 270)
 			(layer "F.Fab")
 			(hide yes)
@@
 		)
 		(property "LCSC Part" "C29936"
-			(at 0 0 0)
+			(at 0 0 270)
 			(layer "F.SilkS")
 			(hide yes)
@@
 		)
 		(fp_text user "${REFERENCE}"
-			(at 0 0 0)
+			(at 0 0 270)
 			(layer "F.Fab")
 			(effects
@@
 		)
 		(pad "1" smd roundrect
-			(at -0.775 0)
+			(at -0.775 0 270)
 			(size 0.9 0.95)
 			(layers "F.Cu" "F.Mask" "F.Paste")
@@
 		)
 		(pad "2" smd roundrect
-			(at 0.775 0)
+			(at 0.775 0 270)
 			(size 0.9 0.95)
 			(layers "F.Cu" "F.Mask" "F.Paste")
@@
 	(footprint "Resistor_SMD:R_0603_1608Metric"
 		(layer "F.Cu")
-		(at 828.59 113.68 180)
+		(at 468.64 49.12 180)
 		(descr "10k pull-up of EXT_FAULT to +3V3, for U7 (board controller): shared fault line, low when a protected supply trips")
 		(tags "resistor")
@@
 	(footprint "Capacitor_SMD:C_0603_1608Metric"
 		(layer "F.Cu")
-		(at 825.1 109.06 90)
+		(at 465.15 44.5 90)
 		(descr "1uF bypass on VCCIO_2, for U24 (slots E-H PIN V switch)")
 		(tags "capacitor")
@@
 	)
 	(gr_rect
-		(start 821.945 106.055)
-		(end 832.945 115.935)
-		(stroke
-			(width 0.15)
-			(type dash)
-		)
-		(fill no)
-		(layer "Cmts.User")
-	)
-	(gr_rect
-		(start 821.945 99.935)
-		(end 832.945 106.055)
-		(stroke
-			(width 0.15)
-			(type solid)
-		)
-		(fill no)
-		(layer "Cmts.User")
-	)
-	(gr_text "island U24"
-		(at 822.345 101.535 0)
-		(layer "Cmts.User")
-		(effects
-			(font
-				(size 1.2 1.2)
-				(thickness 0.18)
-			)
-			(justify left bottom)
-		)
-	)
-	(gr_text "slots E-H PIN V\nswitch\nTPS22950, 4\nparts, 2026-10-28"
-		(at 822.345 101.835 0)
-		(layer "Cmts.User")
-		(effects
-			(font
-				(size 0.7 0.7)
-				(thickness 0.105)
-			)
-			(justify left top)
-		)
-	)
-	(group "island U24"
-		(members
-			"ea8755d1-ca73-4f34-8046-a50fead70bba"
-			"1b869dab-1ed3-4ff7-adfe-18fb13bd9b3c"
-			"1c9b0e5c-52b8-4a68-9565-d497a71220cd"
-			"0da6ee37-b628-4b32-a015-a29a06ffa1d5"
-			"7fb7d766-c9dd-4d0b-beb2-e7f69d8e713c"
-			"efd3a221-0645-4cae-b03c-a55a86529f82"
-			"ee05c57d-c8f9-4b8f-b710-f3e493c66c80"
-		)
-	)
-	(gr_rect
 		(start 689.475 97.615)
 		(end 700.475 107.496)
@@
 		)
 	)
+	(gr_rect
+		(start 461.995 39.125)
+		(end 474.015 54.475)
+		(stroke
+			(width 0.15)
+			(type dash)
+		)
+		(fill no)
+		(layer "Cmts.User")
+	)
+	(gr_rect
+		(start 461.995 33.005)
+		(end 474.015 39.125)
+		(stroke
+			(width 0.15)
+			(type solid)
+		)
+		(fill no)
+		(layer "Cmts.User")
+	)
+	(gr_text "island U24"
+		(at 462.395 34.605 0)
+		(layer "Cmts.User")
+		(effects
+			(font
+				(size 1.2 1.2)
+				(thickness 0.18)
+			)
+			(justify left bottom)
+		)
+	)
+	(gr_text "slots E-H PIN V\nswitch\nTPS22953, 6 parts,\n2026-10-29"
+		(at 462.395 34.905 0)
+		(layer "Cmts.User")
+		(effects
+			(font
+				(size 0.7 0.7)
+				(thickness 0.105)
+			)
+			(justify left top)
+		)
+	)
+	(group "island U24"
+		(members
+			"2d6ace83-c610-4a09-914f-e5b95efdd0d2"
+			"c92f0b16-5637-4e3c-932c-f5961d5f19b2"
+			"ee2d2b9c-cec1-4093-a512-ad8846e13fab"
+			"b98db0ef-37f5-4e9f-aca3-9a3562f94d2d"
+			"7fb7d766-c9dd-4d0b-beb2-e7f69d8e713c"
+			"efd3a221-0645-4cae-b03c-a55a86529f82"
+			"3f33f2f7-ef79-4625-a311-c678d7d3d470"
+			"a4356e60-ddf3-4bf6-92a0-43f8e8d04e4b"
+			"be3be9ce-ac88-433f-a459-38e610ef1cd2"
+			"ee05c57d-c8f9-4b8f-b710-f3e493c66c80"
+		)
+	)
