File: kicad/odin.kicad_pcb (KiCad board)
At the start: 8 copper layers, 100 x 100 mm, 553 parts, among them J1 USB-C, J19 2.54-2*3P, J2 FPGA JTAG, J20 2.54-2*3P, J3 WingTAT 2044-2X32G00SA, J5 WingTAT 2044-2X32G00SA, J50 9-21V POWER IN, J51 CTRL SWD, J52 PZ254V-11-02P, J53 XFCN PM254V-11-07-H85, J54 XFCN PM254V-11-07-H85, J55 XFCN PM254V-11-07-H85, J56 XFCN PM254V-11-07-H85, J57 XFCN PM254V-11-07-H85, J58 XFCN PM254V-11-07-H85, J62 XFCN PM254V-11-07-H85, J63 XFCN PM254V-11-07-H85, J64 XFCN PM254V-11-07-H85, J65 XFCN PM254V-11-07-H85, J68 AUX IN 9-28V UNREGULATED, J7 PM254-2-08-Z-8.5, J70 ETH, J71 LINK P, J72 LINK Q, J73 HDMI OUT, J74 microSD, J8 PM254-2-08-Z-8.5, Q3 BSS138LT1G, Q4 BSS138LT1G, Q6 BSS138LT1G, Q7 BSS138LT1G, SW1 CTRL BOOT, U1 XC7A100T-2FGG676I, U10 SN74LXC8T245PWR, U11 AP63300WU-7, U12 AP63300WU-7, U13 TLV62569DRLR, U14 TLV62569DRLR, U15 SY8047QDC, U16 TLV62569DRLR, U17 PCF8574T_3,518, U18 CH224K, U2 APS6404L-SQN-SN, U20 SN74CB3Q3384APWR, U21 TPS22950CDDCR, U22 TPS22950CDDCR, U23 TPS22953DSQR, U24 TPS22953DSQR, U26 TPS259470ARPWR, U3 APS6404L-SQN-SN, U30 RTL8211FD-CG, U31 TPD12S016PWR, U32 W9825G6KH-6, U33 MR25H10CDF, U34 TPS2121RUXR, U4 APS6404L-SQN-SN, U5 APS6404L-SQN-SN, U6 W25Q256JVEIQ, U7 RP2350B, U8 W25Q32JVZP, U9 SN74LXC8T245PWR, X3 25MHz 12pF, X4 50MHz CMOS, Y1 12MHz ABM8-272-T3

Commit message: Island Q6: the mux hold transistor with D24 and its 470k/10 uF timing network
Parts:
- moved C279 470.8 mm to (437.3, 17.6)
- moved D24 464.1 mm to (441.9, 17.4)
- moved Q6 450.7 mm to (433.3, 17.1)
- moved R200 450.0 mm to (446.3, 17.9)
Other:
- board text added: "island Q6"
- board text added: "mux: 9 V request hold generic, 4 parts, 2026-10-29"
Changed lines of the file:
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@@
 	(footprint "EasyEDA:SOT-23-3_L2.9-W1.6-P1.90-LS2.8-BR"
 		(layer "F.Cu")
-		(at 53.5675 259.911231)
+		(at 433.28 17.14)
 		(descr "mux: 9 V request hold: Small N-MOSFET that pulls U34's PR1 to ground while the board controller asks for 9 V and for 2-7 s after it stops (D24, R, C hold), so the +5V rail is on U11 before VBUS moves and until it is back at 5 V.")
 		(property "Reference" "Q6"
@@
 	(footprint "Resistor_SMD:R_0603_1608Metric"
 		(layer "F.Cu")
-		(at 66.51 259.296231)
+		(at 446.26 17.87)
 		(descr "470k resistor from SEL_IN2 to GND, for Q6 (mux: 9 V request hold): Q6's gate: charged from PD_REQ_9V through D24, drains through 470k/10 uF in 2-7 s")
 		(tags "resistor")
@@
 	(footprint "Diode_SMD:D_SOD-123"
 		(layer "F.Cu")
-		(at 46.3575 260.307856)
+		(at 441.88 17.45)
 		(descr "mux hold diode: 1N4148W: charges the Q6 hold capacitor from PD_REQ_9V at once and lets it drain slowly through its own resistor.")
 		(tags "SOD-123")
@@
 	(footprint "Capacitor_SMD:C_0805_2012Metric"
 		(layer "F.Cu")
-		(at 33.225 259.301231)
+		(at 437.28 17.62)
 		(descr "10uF capacitor from SEL_IN2 to GND, for Q6 (mux: 9 V request hold): Q6's gate: charged from PD_REQ_9V through D24, drains through 470k/10 uF in 2-7 s")
 		(tags "capacitor")
@@
 	)
 	(embedded_fonts no)
+	(gr_rect
+		(start 430.0025 14.156231)
+		(end 449.265 20.126231)
+		(stroke
+			(width 0.15)
+			(type dash)
+		)
+		(fill no)
+		(layer "Cmts.User")
+	)
+	(gr_rect
+		(start 430.0025 9.996231)
+		(end 449.265 14.156231)
+		(stroke
+			(width 0.15)
+			(type solid)
+		)
+		(fill no)
+		(layer "Cmts.User")
+	)
+	(gr_text "island Q6"
+		(at 430.4025 11.596231 0)
+		(layer "Cmts.User")
+		(effects
+			(font
+				(size 1.2 1.2)
+				(thickness 0.18)
+			)
+			(justify left bottom)
+		)
+	)
+	(gr_text "mux: 9 V request hold\ngeneric, 4 parts, 2026-10-29"
+		(at 430.4025 11.896231 0)
+		(layer "Cmts.User")
+		(effects
+			(font
+				(size 0.7 0.7)
+				(thickness 0.105)
+			)
+			(justify left top)
+		)
+	)
+	(group "island Q6"
+		(members
+			"6adc36bc-8f1b-4597-9ef3-3faed5d11433"
+			"cf77d17e-6669-4a8f-a7f9-c522a68c76dd"
+			"5e8b5994-9db2-4a9f-8b5f-0755e051bdae"
+			"90db85d2-e7d2-417e-8c1d-1305310d1299"
+			"b39d0a36-a1f0-416f-9de7-8040ef8e85ae"
+			"f3762cb9-3d11-4f36-978f-f82d396e5074"
+			"ef43770b-edc6-466f-96d9-5fc5e1f4624e"
+			"e5ee0c86-b200-4953-a148-ead6b6d00103"
+		)
+	)
 )

Commit message: Island Q7: the screw-input presence transistor with its 100k/33k divider
Parts:
- moved Q7 437.7 mm to (433.3, 31.1)
- moved R201 429.7 mm to (437.1, 31.8), turned to 180 degrees
- moved R202 427.6 mm to (440.6, 31.8)
Other:
- board text added: "island Q7"
- board text added: "mux: screw input present generic, 3 parts, 2026-10-29"
Changed lines of the file:
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@@
 	(footprint "Resistor_SMD:R_0603_1608Metric"
 		(layer "F.Cu")
-		(at 78.53 259.296231)
+		(at 440.56 31.83)
 		(descr "33k pull-down on EXT_PRESENT, for Q7 (mux: screw input present): Q7's gate: 100k/33k from the screw input, on above 3.2-6 V of VIN_EXT")
 		(tags "resistor")
@@
 	(footprint "EasyEDA:SOT-23-3_L2.9-W1.6-P1.90-LS2.8-BR"
 		(layer "F.Cu")
-		(at 60.1925 259.911231)
+		(at 433.27 31.1)
 		(descr "mux: screw input present: Small N-MOSFET that pulls U34's PR1 to ground while the screw input (J50) carries voltage, so the whole board runs from J50 through U11 even with a 5 V USB cable plugged in.")
 		(property "Reference" "Q7"
@@
 	(footprint "Resistor_SMD:R_0603_1608Metric"
 		(layer "F.Cu")
-		(at 72.52 259.296231)
+		(at 437.05 31.83 180)
 		(descr "100k series resistor between EXT_PRESENT and VIN_EXT, for J50 (POWER IN screw terminal): Q7's gate: 100k/33k from the screw input, on above 3.2-6 V of VIN_EXT")
 		(tags "resistor")
 		(property "Reference" "R201"
-			(at 0 -1.43 0)
+			(at 0 -1.43 180)
 			(layer "F.Fab")
 			(effects
@@
 		)
 		(property "Value" "100k"
-			(at 0 1.43 0)
+			(at 0 1.43 180)
 			(layer "F.Fab")
 			(effects
@@
 		)
 		(property "Datasheet" ""
-			(at 0 0 0)
+			(at 0 0 180)
 			(layer "F.Fab")
 			(hide yes)
@@
 		)
 		(property "Description" "100k series resistor between EXT_PRESENT and VIN_EXT, for J50 (POWER IN screw terminal): Q7's gate: 100k/33k from the screw input, on above 3.2-6 V of VIN_EXT"
-			(at 0 0 0)
+			(at 0 0 180)
 			(layer "F.Fab")
 			(hide yes)
@@
 		)
 		(fp_text user "${REFERENCE}"
-			(at 0 0 0)
+			(at 0 0 180)
 			(layer "F.Fab")
 			(effects
@@
 		)
 		(pad "1" smd roundrect
-			(at -0.825 0)
+			(at -0.825 0 180)
 			(size 0.8 0.95)
 			(layers "F.Cu" "F.Mask" "F.Paste")
@@
 		)
 		(pad "2" smd roundrect
-			(at 0.825 0)
+			(at 0.825 0 180)
 			(size 0.8 0.95)
 			(layers "F.Cu" "F.Mask" "F.Paste")
@@
 		)
 	)
+	(gr_rect
+		(start 429.9975 28.116231)
+		(end 443.565 34.086231)
+		(stroke
+			(width 0.15)
+			(type dash)
+		)
+		(fill no)
+		(layer "Cmts.User")
+	)
+	(gr_rect
+		(start 429.9975 21.996231)
+		(end 443.565 28.116231)
+		(stroke
+			(width 0.15)
+			(type solid)
+		)
+		(fill no)
+		(layer "Cmts.User")
+	)
+	(gr_text "island Q7"
+		(at 430.3975 23.596231 0)
+		(layer "Cmts.User")
+		(effects
+			(font
+				(size 1.2 1.2)
+				(thickness 0.18)
+			)
+			(justify left bottom)
+		)
+	)
+	(gr_text "mux: screw input\npresent\ngeneric, 3 parts,\n2026-10-29"
+		(at 430.3975 23.896231 0)
+		(layer "Cmts.User")
+		(effects
+			(font
+				(size 0.7 0.7)
+				(thickness 0.105)
+			)
+			(justify left top)
+		)
+	)
+	(group "island Q7"
+		(members
+			"23997547-c32d-485f-a700-df11380441e5"
+			"10042f2e-45fa-4c02-8a63-10736af6baaf"
+			"fed4d53d-4b97-4bd5-b0c1-f0d97ec3e915"
+			"81094ee5-dc77-4a4d-810e-57a51d286643"
+			"43b7676e-8bbf-4939-9347-47936db614a3"
+			"ca5f2df8-706f-45ff-91b1-4d037de39973"
+			"0495d7cd-18f9-49a5-907b-69c7160c7fda"
+		)
+	)

Commit message: Island U34 re-applied: the IN2 bypass at its pin; the hold transistors now in their own islands
Parts:
- moved C280 446.6 mm to (433.0, 48.2), turned to 180 degrees
- moved C266 404.7 mm to (436.7, 47.5)
- moved C263 404.7 mm to (440.2, 44.7)
- moved R162 404.7 mm to (441.2, 51.6)
- moved R163 404.7 mm to (441.2, 55.1)
- moved R166 404.7 mm to (437.9, 51.6)
- moved R167 404.7 mm to (437.9, 55.1)
- moved R168 404.7 mm to (441.6, 44.1)
- moved U34 404.7 mm to (440.4, 47.9)
- moved C264 404.7 mm to (443.4, 48.2)
- moved C265 404.7 mm to (444.1, 46.6)
- moved R164 404.7 mm to (439.5, 51.6)
- moved R165 404.7 mm to (439.5, 55.1)
- moved R169 404.7 mm to (438.8, 44.1)
Other:
- board text added: "+5V source mux TPS2121, 14 parts, 2026-10-29"
- board text removed: "+5V source mux TPS2121, 13 parts, 2026-10-29"
Changed lines of the file:
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@@
 	(footprint "Resistor_SMD:R_0603_1608Metric"
 		(layer "F.Cu")
-		(at 836.44 138.56 90)
+		(at 441.16 51.6 90)
 		(descr "100k resistor from VBUS5_PR1 to VBUS, for U34 (+5V source mux): U34 priority sense: VBUS wins above 4.44 V (PR1 above CP2) unless Q6 (9 V request) or Q7 (screw input present) holds it at ground")
 		(tags "resistor")
@@
 	(footprint "Package_DFN_QFN:Texas_VQFN-HR-12_2x2.5mm_P0.5mm"
 		(layer "F.Cu")
-		(at 835.72 134.83)
+		(at 440.44 47.87)
 		(descr "+5V source mux: TI TPS2121 power mux: passes plain 5 V USB straight to the +5V rail; hands the rail to U11 while the board controller asks for 9 V (Q6), while the screw input is powered (Q7), or if VBUS goes above about 5.6 V or away. Blocks reverse current both ways, limits to about 2.5 A.")
 		(tags "RUX0012A Texas VQFN-HR NoLead")
@@
 	(footprint "Capacitor_SMD:C_0805_2012Metric"
 		(layer "F.Cu")
-		(at 832.03 134.48 180)
+		(at 436.74 47.52 180)
 		(descr "22uF bypass on +5V, for U34 (+5V source mux)")
 		(tags "capacitor")
@@
 	(footprint "Capacitor_SMD:C_0402_1005Metric"
 		(layer "F.Cu")
-		(at 835.47 131.67 90)
+		(at 440.19 44.71 90)
 		(descr "100nF capacitor from VBUS5_SS to GND, for U34 (+5V source mux): sets how fast U34 ramps the +5V rail, about 780 V/s")
 		(tags "capacitor")
@@
 	(footprint "Resistor_SMD:R_0603_1608Metric"
 		(layer "F.Cu")
-		(at 836.87 131.1 90)
+		(at 441.59 44.14 90)
 		(descr "44.2k resistor from VBUS5_ILIM to GND, for U34 (+5V source mux): sets U34's current limit, about 2.5 A")
 		(tags "resistor")
@@
 	(footprint "Resistor_SMD:R_0603_1608Metric"
 		(layer "F.Cu")
-		(at 834.04 131.1 -90)
+		(at 438.76 44.14 -90)
 		(descr "10k resistor from VBUS5_ST to +3V3, for U7 (board controller): U34 status to the board controller: low when U11 feeds +5V")
 		(tags "resistor")
@@
 	(footprint "Resistor_SMD:R_0603_1608Metric"
 		(layer "F.Cu")
-		(at 836.44 142.07 -90)
+		(at 441.16 55.11 -90)
 		(descr "36.5k resistor from VBUS5_PR1 to GND, for U34 (+5V source mux): U34 priority sense: VBUS wins above 4.44 V (PR1 above CP2) unless Q6 (9 V request) or Q7 (screw input present) holds it at ground")
 		(tags "resistor")
@@
 	(footprint "Capacitor_SMD:C_0805_2012Metric"
 		(layer "F.Cu")
-		(at 839.42 133.58)
+		(at 444.14 46.62)
 		(descr "22uF bypass on +5V, for U34 (+5V source mux)")
 		(tags "capacitor")
@@
 	(footprint "Resistor_SMD:R_0603_1608Metric"
 		(layer "F.Cu")
-		(at 833.2 142.07 -90)
+		(at 437.92 55.11 -90)
 		(descr "56.2k resistor from VBUS5_CP2 to GND, for U34 (+5V source mux): U34 comparison level, 1.19 V from +3V3; enables the 5 us switchover")
 		(tags "resistor")
@@
 	(footprint "Resistor_SMD:R_0603_1608Metric"
 		(layer "F.Cu")
-		(at 834.77 138.56 90)
+		(at 439.49 51.6 90)
 		(descr "100k resistor from VBUS5_OV1 to VBUS, for U34 (+5V source mux): U34 VBUS overvoltage backstop: VBUS is dropped above 5.3-5.9 V (5.63 V typical) if a source raises it unasked")
 		(tags "resistor")
@@
 	(footprint "Resistor_SMD:R_0603_1608Metric"
 		(layer "F.Cu")
-		(at 834.77 142.07 -90)
+		(at 439.49 55.11 -90)
 		(descr "23.2k resistor from VBUS5_OV1 to GND, for U34 (+5V source mux): U34 VBUS overvoltage backstop: VBUS is dropped above 5.3-5.9 V (5.63 V typical) if a source raises it unasked")
 		(tags "resistor")
@@
 	(footprint "Capacitor_SMD:C_0402_1005Metric"
 		(layer "F.Cu")
-		(at 838.63 135.18)
+		(at 443.35 48.22)
 		(descr "100nF 25V bypass on VBUS, for U34 (+5V source mux)")
 		(tags "capacitor")
@@
 	(footprint "Resistor_SMD:R_0603_1608Metric"
 		(layer "F.Cu")
-		(at 833.2 138.56 90)
+		(at 437.92 51.6 90)
 		(descr "100k resistor from VBUS5_CP2 to +3V3, for U34 (+5V source mux): U34 comparison level, 1.19 V from +3V3; enables the 5 us switchover")
 		(tags "resistor")
@@
 	(footprint "Capacitor_SMD:C_0603_1608Metric"
 		(layer "F.Cu")
-		(at 39.455 259.296231)
+		(at 433.01 48.22 180)
 		(descr "1uF bypass on +5V_BUCK, for U34 (+5V source mux)")
 		(tags "capacitor")
 		(property "Reference" "C280"
-			(at 0 -1.43 0)
+			(at 0 -1.43 180)
 			(layer "F.Fab")
 			(effects
@@
 		)
 		(property "Value" "1uF"
-			(at 0 1.43 0)
+			(at 0 1.43 180)
 			(layer "F.Fab")
 			(effects
@@
 		)
 		(property "Datasheet" ""
-			(at 0 0 0)
+			(at 0 0 180)
 			(layer "F.Fab")
 			(hide yes)
@@
 		)
 		(property "Description" "1uF bypass on +5V_BUCK, for U34 (+5V source mux)"
-			(at 0 0 0)
+			(at 0 0 180)
 			(layer "F.Fab")
 			(hide yes)
@@
 		)
 		(property "LCSC Part" "C29936"
-			(at 0 0 0)
+			(at 0 0 180)
 			(layer "F.SilkS")
 			(hide yes)
@@
 		)
 		(fp_text user "${REFERENCE}"
-			(at 0 0 0)
+			(at 0 0 180)
 			(layer "F.Fab")
 			(effects
@@
 		)
 		(pad "1" smd roundrect
-			(at -0.775 0)
+			(at -0.775 0 180)
 			(size 0.9 0.95)
 			(layers "F.Cu" "F.Mask" "F.Paste")
@@
 		)
 		(pad "2" smd roundrect
-			(at 0.775 0)
+			(at 0.775 0 180)
 			(size 0.9 0.95)
 			(layers "F.Cu" "F.Mask" "F.Paste")
@@
 	)
 	(gr_rect
-		(start 828.805 122.955)
-		(end 842.645 128.095)
-		(stroke
-			(width 0.15)
-			(type solid)
-		)
-		(fill no)
-		(layer "Cmts.User")
-	)
-	(gr_rect
-		(start 828.805 128.095)
-		(end 842.645 145.075)
-		(stroke
-			(width 0.15)
-			(type dash)
-		)
-		(fill no)
-		(layer "Cmts.User")
-	)
-	(gr_rect
 		(start 830.915 147.185)
 		(end 842.935 153.305)
@@
 		)
 	)
-	(gr_text "+5V source mux\nTPS2121, 13 parts,\n2026-10-29"
-		(at 829.205 124.855 0)
-		(layer "Cmts.User")
-		(effects
-			(font
-				(size 0.7 0.7)
-				(thickness 0.105)
-			)
-			(justify left top)
-		)
-	)
 	(gr_text "slots E-H PIN V\nswitch\nTPS22953, 6 parts,\n2026-10-29"
 		(at 831.315 149.085 0)
@@
 		)
 	)
-	(gr_text "island U34"
-		(at 829.205 124.555 0)
-		(layer "Cmts.User")
-		(effects
-			(font
-				(size 1.2 1.2)
-				(thickness 0.18)
-			)
-			(justify left bottom)
-		)
-	)
 	(gr_text "island U24"
 		(at 831.315 148.785 0)
@@
 		)
 	)
-	(group "island U34"
-		(members "129e5539-868e-484c-aac2-f123f45fd224" "13ecfdc8-8b61-4334-810e-42b36423c172"
-			"18808443-2533-422d-9f53-e28884f18db6" "193fa7af-0bea-4d12-b820-0e6b36612de6"
-			"1aca21b5-7d8e-4b4f-9384-0ba20e24a880" "24959646-1c6e-4526-a8b3-dd75fda10463"
-			"2700677e-3f29-4dc4-be74-d9767a362100" "295d9c81-1697-4fcf-a433-eb2690991e77"
-			"6ec2506c-4962-4beb-9354-48dd8fbd2ca1" "7f271b8c-c7be-4c58-b658-abb724ac0b66"
-			"840d7df2-00ce-4f2f-a36b-6edcc915a6ae" "963a14c2-712a-4597-af16-da2dece7dc8c"
-			"aa05c60d-190e-4c6f-9700-20619c323da8" "b41f6eba-f5ee-4b08-a599-42a4b7f55e7b"
-			"ca83a37c-a8a4-4131-a2d0-8cae3ce637fe" "ec784f77-1bae-4880-ad6c-2971dc1c967b"
-			"ecc88d94-8cc6-417d-91da-ecd33751adfb"
-		)
-	)
 	(group "island J19"
 		(members "4d068040-ba21-42e4-b03f-9590b70190a1" "51e2cede-3862-4485-a9a1-6affe551c1b3"
@@
 		)
 	)
+	(gr_rect
+		(start 430.005 41.135)
+		(end 447.365 58.115)
+		(stroke
+			(width 0.15)
+			(type dash)
+		)
+		(fill no)
+		(layer "Cmts.User")
+	)
+	(gr_rect
+		(start 430.005 35.995)
+		(end 447.365 41.135)
+		(stroke
+			(width 0.15)
+			(type solid)
+		)
+		(fill no)
+		(layer "Cmts.User")
+	)
+	(gr_text "island U34"
+		(at 430.405 37.595 0)
+		(layer "Cmts.User")
+		(effects
+			(font
+				(size 1.2 1.2)
+				(thickness 0.18)
+			)
+			(justify left bottom)
+		)
+	)
+	(gr_text "+5V source mux\nTPS2121, 14 parts,\n2026-10-29"
+		(at 430.405 37.895 0)
+		(layer "Cmts.User")
+		(effects
+			(font
+				(size 0.7 0.7)
+				(thickness 0.105)
+			)
+			(justify left top)
+		)
+	)
+	(group "island U34"
+		(members
+			"35deaf51-a170-4e1a-9ef6-d068fa9181ed"
+			"8369e237-ea62-4907-a6a0-54b78e98bf71"
+			"0596f1c4-8e6c-4502-afe7-404ebe20fb43"
+			"c245fbf2-7c0c-4847-baaa-8121932f2aab"
+			"13ecfdc8-8b61-4334-810e-42b36423c172"
+			"1aca21b5-7d8e-4b4f-9384-0ba20e24a880"
+			"ca83a37c-a8a4-4131-a2d0-8cae3ce637fe"
+			"840d7df2-00ce-4f2f-a36b-6edcc915a6ae"
+			"18808443-2533-422d-9f53-e28884f18db6"
+			"f8709ad8-ded8-4274-bbbf-2f5360151898"
+			"129e5539-868e-484c-aac2-f123f45fd224"
+			"295d9c81-1697-4fcf-a433-eb2690991e77"
+			"aa05c60d-190e-4c6f-9700-20619c323da8"
+			"b41f6eba-f5ee-4b08-a599-42a4b7f55e7b"
+			"ec784f77-1bae-4880-ad6c-2971dc1c967b"
+			"963a14c2-712a-4597-af16-da2dece7dc8c"
+			"24959646-1c6e-4526-a8b3-dd75fda10463"
+			"2700677e-3f29-4dc4-be74-d9767a362100"
+		)
+	)
