File: kicad/supervisor.kicad_sch (KiCad schematic)
At the start: 74 parts, among them J1 USB-C, J2 FPGA JTAG, J51 CTRL SWD, J52 PZ254V-11-02P, SW1 CTRL BOOT, U17 PCF8574T_3,518, U18 CH224K, U20 SN74CB3Q3384APWR, U7 RP2350B, U8 W25Q32JVZP, Y1 12MHz ABM8-272-T3

Commit message: Power path: U34 mux replaces the Q2 bypass, U11/U14 always on, PD defaults to 5 V, USB series resistors, native controller pins
Parts:
- added C271, C272: 100nF, Capacitor_SMD:C_0402_1005Metric, symbol Device:C
- added Q3: BSS138LT1G, EasyEDA:SOT-23-3_L2.9-W1.6-P1.90-LS2.8-BR, symbol Transistor_FET:Q_NMOS_GSD
- added R170, R171: 27, Resistor_SMD:R_0402_1005Metric, symbol Device:R
- added R172: 10k, Resistor_SMD:R_0402_1005Metric, symbol Device:R
- added R173: 100k, Resistor_SMD:R_0402_1005Metric, symbol Device:R
- added R174, R175: 1k, Resistor_SMD:R_0603_1608Metric, symbol Device:R
Connections:
- net EXT_FAULT: now also U7.43 (GPIO34); no longer U7.58 (GPIO47/ADC7)
- net GND: now also U18.2 (CFG2), U18.3 (CFG3), C271.2, C272.2, Q3.2 (S), R173.2
- net PD_CFG1: now also Q3.3 (D), R172.2; no longer U7.28 (GPIO27)
- net PD_VDD: now also R172.1
- net SUP_CCLK: now also U7.8 (GPIO10); no longer U7.4 (GPIO7)
- net SUP_FD0: now also U7.9 (GPIO11); no longer U7.8 (GPIO10)
- net SUP_FD1: now also U7.11 (GPIO12); no longer U7.9 (GPIO11)
- net SUP_FD2: now also U7.12 (GPIO13); no longer U7.11 (GPIO12)
- net SUP_FD3: now also U7.4 (GPIO7); no longer U7.12 (GPIO13)
- net SUP_SCL: now also U7.39 (GPIO31); no longer U7.13 (GPIO14)
- net SUP_SDA: now also U7.13 (GPIO14); no longer U7.39 (GPIO31)
- net SUP_UART_RX: now also U7.42 (GPIO33); no longer U7.20 (GPIO20)
- net SUP_UART_TX: now also U7.40 (GPIO32); no longer U7.19 (GPIO19)
- net USB_DM: now also R171.1; no longer U7.66 (USB_DM)
- net USB_DP: now also R170.1; no longer U7.67 (USB_DP)
- net MON_VCCIO_1: now reaches U7.57 (GPIO46/ADC6)
- net MON_VCCIO_1: now also C271.1, R174.2
- net EN_1V8: no longer names the net of U7.23 (GPIO23)
- net EN_5V: no longer names the net of U7.27 (GPIO26)
- net EN_VBUS5 renamed VBUS5_ST
- net PD_CFG2: no longer names the net of U7.36 (GPIO28)
- net PD_CFG2: no longer U18.2 (CFG2)
- net PD_CFG3: no longer names the net of U7.37 (GPIO29)
- net PD_CFG3: no longer U18.3 (CFG3)
- new net MON_VCCIO_2: C272.1, R175.2, U7.58 (GPIO47/ADC7)
- new net PD_REQ_9V: Q3.1 (G), R173.1, U7.28 (GPIO27)
- new net USB_DM_MCU: R171.2, U7.66 (USB_DM)
- new net USB_DP_MCU: R170.2, U7.67 (USB_DP)
- new net VCCIO_1: R174.1
- new net VCCIO_2: R175.1
- no-connect marks 31 -> 33
Other:
- note added: "Lets the board controller measure every supply. Each rail goes to one of its eight analog inputs (ADC), which read 0-3.3 V. Rails at or below 3.3 V go through a 1 k resistor that protects the pin; VSYS and +5V are higher, so two resistors divide them down first. A 100 nF capacitor on each input steadies the reading. MON_1V8 reads +1V8 itself, the FPGA's VCCAUX behind the bead, so an open bead sho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"
- note added: "Negotiates the supply voltage with a USB-PD charger. Out of the box it asks for 5 V: CFG1 is pulled up to the chip's own 3.3 V and CFG2/CFG3 are grounded, so the only other request the pins can form is 9 V, which the board controller selects by turning Q3 on (PD_REQ_9V). A dead or resetting controller leaves it at 5 V. PD_PG tells the controller whether the charger agreed."
- note added: "Two 27 ohm resistors in the USB data lines, right at the board controller, as Raspberry Pi's hardware design guide (section 5.1) asks. The ESD clamp D6 stays at the connector."
- note added: "U7 USB series resistors"
- note added: "rail monitors"
- note removed: "Negotiates the supply voltage with a USB-PD charger. The board controller tells it what to ask for (PD_CFG1-3: 5 V or 9 V, never more) and reads PD_PG to know whether the charger agreed."
- moved on the sheet: C137, C138, C182, D10, D11, D9, J2, J51, J52, R11, R12, R128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

Commit message: PSRAM power-up states with PUDC_B high; TPS22953 for the jumpered PIN V exports
Parts:
- removed C271, C272: 100nF, Capacitor_SMD:C_0402_1005Metric, symbol Device:C
- removed R174, R175: 1k, Resistor_SMD:R_0603_1608Metric, symbol Device:R
Other:
- note removed: "Lets the board controller measure every supply. Each rail goes to one of its eight analog inputs (ADC), which read 0-3.3 V. Rails at or below 3.3 V go through a 1 k resistor that protects the pin; VSYS and +5V are higher, so two resistors divide them down first. A 100 nF capacitor on each input steadies the reading. MON_1V8 reads +1V8 itself, the FPGA's VCCAUX behind the bead, so an open bead sho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"
- note removed: "rail monitors"

Commit message: Tools: honest gate verdicts, source-side island ownership, key posts at their rows, J1 pads clear of the holes, budget checks for capacitance, inductors and sources
Parts:
- J1: footprint Connector_USB:USB_C_Receptacle_HCTL_HC-TYPE-C-16P-01A -> odin:USB_C_Receptacle_HCTL_HC-TYPE-C-16P-01A_Odin
Changed lines of the file:
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@@
 		(property "Reference" "J1" (at 271.78 400.05 0) (effects (font (size 1.27 1.27))))
 		(property "Value" "USB-C" (at 271.78 453.39 0) (effects (font (size 1.27 1.27))))
-		(property "Footprint" "Connector_USB:USB_C_Receptacle_HCTL_HC-TYPE-C-16P-01A" (at 271.78 453.39 0) (effects (font (size 1.27 1.27)) (hide yes)))
+		(property "Footprint" "odin:USB_C_Receptacle_HCTL_HC-TYPE-C-16P-01A_Odin" (at 271.78 453.39 0) (effects (font (size 1.27 1.27)) (hide yes)))
 		(property "LCSC" "C2894897" (at 271.78 453.39 0) (effects (font (size 1.27 1.27)) (hide yes)))
 		(property "Description" "USB-C connector: Power in and USB 2.0 data to the board controller." (at 271.78 453.39 0) (effects (font (size 1.27 1.27)) (hide yes)))
